Commit message: create midlevel

File: world_v0/models/building/models/building.model.xacro (robot description, xacro)
@@ -76,5 +76,5 @@
   <xacro:macro name="front_wall_with_door" params="name depth width height">
     <collision name='${name}_front_top_collision' laser_retro='0.000000'>
-      <origin pose='${(wall_thickness/2)} 0.0 ${(height-door_height)/2+door_height} 0.000000 -0.000000 0.000000'/>
+      <origin pose='-${(wall_thickness/2)} 0.0 ${(height-door_height)/2+door_height} 0.000000 -0.000000 0.000000'/>
       <geometry>
         <box size='${wall_thickness} ${width} ${height-door_height}'/>
@@ -91,5 +91,5 @@
     </collision>
     <visual name='${name}_front_top_visual' cast_shadows='1' laser_retro='0.000000' transparency='0.000000'>
-      <origin pose='${(wall_thickness/2)} 0.0 ${(height-door_height)/2+door_height} 0.000000 -0.000000 0.000000'/>
+      <origin pose='-${(wall_thickness/2)} 0.0 ${(height-door_height)/2+door_height} 0.000000 -0.000000 0.000000'/>
       <geometry>
         <box size='${wall_thickness} ${width} ${height-door_height}'/>
@@ -97,5 +97,5 @@
     </visual>
     <collision name='${name}_front_left_collision' laser_retro='0.000000'>
-      <origin pose='${(wall_thickness/2)} ${door_width/2 + (width-door_width)/4} ${door_height/2} 0.000000 -0.000000 0.000000'/>
+      <origin pose='-${(wall_thickness/2)} ${door_width/2 + (width-door_width)/4} ${door_height/2} 0.000000 -0.000000 0.000000'/>
       <geometry>
         <box size='${wall_thickness} ${(width-door_width)/2} ${door_height}'/>
@@ -112,5 +112,5 @@
     </collision>
     <visual name='${name}_front_left_visual' cast_shadows='1' laser_retro='0.000000' transparency='0.000000'>
-      <origin pose='${(wall_thickness/2)} ${door_width/2 + (width-door_width)/4} ${door_height/2} 0.000000 -0.000000 0.000000'/>
+      <origin pose='-${(wall_thickness/2)} ${door_width/2 + (width-door_width)/4} ${door_height/2} 0.000000 -0.000000 0.000000'/>
       <geometry>
         <box size='${wall_thickness} ${(width-door_width)/2} ${door_height}'/>
@@ -118,5 +118,5 @@
     </visual>
     <collision name='${name}_front_right_collision' laser_retro='0.000000'>
-      <origin pose='${(wall_thickness/2)} -${door_width/2 + (width-door_width)/4} ${door_height/2} 0.000000 -0.000000 0.000000'/>
+      <origin pose='-${(wall_thickness/2)} -${door_width/2 + (width-door_width)/4} ${door_height/2} 0.000000 -0.000000 0.000000'/>
       <geometry>
         <box size='${wall_thickness} ${(width-door_width)/2} ${door_height}'/>
@@ -133,5 +133,5 @@
     </collision>
     <visual name='${name}_front_right_visual' cast_shadows='1' laser_retro='0.000000' transparency='0.000000'>
-      <origin pose='${(wall_thickness/2)} -${door_width/2 + (width-door_width)/4} ${door_height/2} 0.000000 -0.000000 0.000000'/>
+      <origin pose='-${(wall_thickness/2)} -${door_width/2 + (width-door_width)/4} ${door_height/2} 0.000000 -0.000000 0.000000'/>
       <geometry>
         <box size='${wall_thickness} ${(width-door_width)/2} ${door_height}'/>
@@ -205,4 +205,5 @@
       </geometry>
     </visual>
+<!--
     <collision name='${name}_top_collision' laser_retro='0.000000'>
       <origin pose='${(depth-wall_thickness)/2} 0.0 ${height-wall_thickness/2} 0.000000 -0.000000 0.000000'/>
@@ -224,4 +225,26 @@
       <geometry>
         <box size='${depth} ${width} ${wall_thickness}'/>
+      </geometry>
+    </visual>
+-->
+    <collision name='${name}_mid_collision' laser_retro='0.000000'>
+      <origin pose='${(depth-wall_thickness)/2} ${width/4} ${height/2} 0.000000 -0.000000 0.000000'/>
+      <geometry>
+        <box size='${depth} ${width/2} ${wall_thickness}'/>
+      </geometry>
+      <surface>
+        <friction>
+          <ode mu='-1.000000' mu2='-1.000000' fdir1='0.000000 0.000000 0.000000' slip1='0.000000' slip2='0.000000'/>
+        </friction>
+        <bounce restitution_coefficient='0.000000' threshold='100000.000000'/>
+        <contact>
+          <ode soft_cfm='0.000000' soft_erp='0.200000' kp='1000000000000.000000' kd='1.000000' max_vel='0.000000' min_depth='0.001000'/>
+        </contact>
+      </surface>
+    </collision>
+    <visual name='${name}_mid_visual' cast_shadows='1' laser_retro='0.000000' transparency='0.000000'>
+      <origin pose='${(depth-wall_thickness)/2} ${width/4} ${height/2} 0.000000 -0.000000 0.000000'/>
+      <geometry>
+        <box size='${depth} ${width/2} ${wall_thickness}'/>
       </geometry>
     </visual>
