Commit message: update test

File: models_v0/camhand/robots/camhand_1.urdf.xacro (robot description, xacro)
@@ -7,8 +7,8 @@
   <link name="world"/>
   <xacro:camhand side="right" parent="world">
-    <origin xyz="0 0 1" rpy="0 1.57079 3.14159"/>
+    <origin xyz="0 0 0" rpy="0 0 0"/>
   </xacro:camhand>
   <xacro:camhand side="left" parent="world">
-    <origin xyz="0 1 1" rpy="0 1.57079 3.14159"/>
+    <origin xyz="0 1 0" rpy="0 0 0"/>
   </xacro:camhand>
 </robot>

File: models_v0/camhand/urdf/camhand.urdf.xacro (robot description, xacro)
@@ -175,7 +175,4 @@
       <insert_block name="origin" />
     </joint>
-<!--
-    <xacro:finger side="${side}" idx="0" x="0.0" y="0.00000" z="0" r="0" p="0" yaw="0.0"/>
--->
     <xacro:finger side="${side}" idx="0" x="0.140" y="0.00000" z="0" r="0" p="0" yaw="0.3"/>
     <xacro:finger side="${side}" idx="1" x="0.115" y="0.03122" z="0" r="0" p="0" yaw="0.3"/>
