Commit message: cleanup

File: models_v0/humanoid/robots/humanoid.urdf.xacro (robot description, xacro)
@@ -8,14 +8,8 @@
   <xacro:ragdoll/>
   <xacro:camhand side="r" parent="r_wrist">
-<!--
-    <origin xyz="0 0 0.0" rpy="0 0 0"/>
--->
     <origin xyz="0 0 -0.03" rpy="0 1.57079 3.14159"/>
   </xacro:camhand>
   <xacro:camhand side="l" parent="l_wrist">
-<!--
-    <origin xyz="0 0 0.0" rpy="0 0 0"/>
--->
-    <origin xyz="0 0 -0.03" rpy="0 1.57079 3.14159"/>
+    <origin xyz="0 0 -0.3" rpy="0 1.57079 3.14159"/>
   </xacro:camhand>
 </robot>

Commit message: added basic join controllers

File: models_v0/humanoid/robots/humanoid.urdf.xacro (robot description, xacro)
@@ -11,5 +11,5 @@
   </xacro:camhand>
   <xacro:camhand side="l" parent="l_wrist">
-    <origin xyz="0 0 -0.3" rpy="0 1.57079 3.14159"/>
+    <origin xyz="0 0 -0.03" rpy="0 1.57079 3.14159"/>
   </xacro:camhand>
 </robot>

File: models_v0/humanoid/urdf/ragdoll.urdf.xacro (robot description, xacro)
@@ -1,3 +1,4 @@
-<robot name="ragdoll" xmlns:xacro="http://ros.org/wiki/xacro">
+<robot name="ragdoll" xmlns:xacro="http://ros.org/wiki/xacro"
+                      xmlns:controller="http://playerstage.sourceforge.net/gazebo/xmlschema/#controller">
   <!-- hip is the root link -->
   <property name="M_PI" value="3.1415926535897931" />
@@ -79,4 +80,9 @@
       <child link="head"/>
     </joint>
+    <transmission type="pr2_mechanism_model/SimpleTransmission" name="head_trans">
+      <actuator name="head_motor" />
+      <joint name="head_joint" />
+      <mechanicalReduction>1</mechanicalReduction>
+    </transmission>
     <link name="neck">
       <inertial>
@@ -111,4 +117,9 @@
       <child link="neck"/>
     </joint>
+    <transmission type="pr2_mechanism_model/SimpleTransmission" name="neck_trans">
+      <actuator name="neck_motor" />
+      <joint name="neck_joint" />
+      <mechanicalReduction>1</mechanicalReduction>
+    </transmission>
     <link name="torso">
       <inertial>
@@ -143,4 +154,9 @@
       <child link="torso"/>
     </joint>
+    <transmission type="pr2_mechanism_model/SimpleTransmission" name="torso_trans">
+      <actuator name="torso_motor" />
+      <joint name="torso_joint" />
+      <mechanicalReduction>1</mechanicalReduction>
+    </transmission>
     <link name="hip">
       <inertial>
@@ -177,4 +193,9 @@
       <child link="hip"/>
     </joint>
+    <transmission type="pr2_mechanism_model/SimpleTransmission" name="hip_trans">
+      <actuator name="hip_motor" />
+      <joint name="hip_joint" />
+      <mechanicalReduction>1</mechanicalReduction>
+    </transmission>
     -->
   </xacro:macro>
@@ -212,4 +233,9 @@
       <child link="${side}_thigh_pan"/>
     </joint>
+    <transmission type="pr2_mechanism_model/SimpleTransmission" name="${side}_thigh_pan_trans">
+      <actuator name="${side}_thigh_pan_motor" />
+      <joint name="${side}_thigh_pan_joint" />
+      <mechanicalReduction>1</mechanicalReduction>
+    </transmission>
     <link name="${side}_thigh_lift">
       <inertial>
@@ -244,4 +270,9 @@
       <child link="${side}_thigh_lift"/>
     </joint>
+    <transmission type="pr2_mechanism_model/SimpleTransmission" name="${side}_thigh_lift_trans">
+      <actuator name="${side}_thigh_lift_motor" />
+      <joint name="${side}_thigh_lift_joint" />
+      <mechanicalReduction>1</mechanicalReduction>
+    </transmission>
     <link name="${side}_calf">
       <inertial>
@@ -276,4 +307,9 @@
       <child link="${side}_calf"/>
     </joint>
+    <transmission type="pr2_mechanism_model/SimpleTransmission" name="${side}_calf_trans">
+      <actuator name="${side}_calf_motor" />
+      <joint name="${side}_calf_joint" />
+      <mechanicalReduction>1</mechanicalReduction>
+    </transmission>
     <link name="${side}_ankle">
       <inertial>
@@ -308,4 +344,9 @@
       <child link="${side}_ankle"/>
     </joint>
+    <transmission type="pr2_mechanism_model/SimpleTransmission" name="${side}_ankle_trans">
+      <actuator name="${side}_ankle_motor" />
+      <joint name="${side}_ankle_joint" />
+      <mechanicalReduction>1</mechanicalReduction>
+    </transmission>
     <link name="${side}_foot">
       <inertial>
@@ -340,4 +381,9 @@
       <child link="${side}_foot"/>
     </joint>
+    <transmission type="pr2_mechanism_model/SimpleTransmission" name="${side}_foot_trans">
+      <actuator name="${side}_foot_motor" />
+      <joint name="${side}_foot_joint" />
+      <mechanicalReduction>1</mechanicalReduction>
+    </transmission>
   </xacro:macro>
   <xacro:macro name="arm" params="side *origin">
@@ -374,4 +420,9 @@
       <child link="${side}_shoulder"/>
     </joint>
+    <transmission type="pr2_mechanism_model/SimpleTransmission" name="${side}_shoulder_trans">
+      <actuator name="${side}_shoulder_motor" />
+      <joint name="${side}_shoulder_joint" />
+      <mechanicalReduction>1</mechanicalReduction>
+    </transmission>
     <link name="${side}_upper_arm">
       <inertial>
@@ -406,4 +457,9 @@
       <child link="${side}_upper_arm"/>
     </joint>
+    <transmission type="pr2_mechanism_model/SimpleTransmission" name="${side}_upper_arm_trans">
+      <actuator name="${side}_upper_arm_motor" />
+      <joint name="${side}_upper_arm_joint" />
+      <mechanicalReduction>1</mechanicalReduction>
+    </transmission>
     <link name="${side}_forearm">
       <inertial>
@@ -438,4 +494,9 @@
       <child link="${side}_forearm"/>
     </joint>
+    <transmission type="pr2_mechanism_model/SimpleTransmission" name="${side}_forearm_trans">
+      <actuator name="${side}_forearm_motor" />
+      <joint name="${side}_forearm_joint" />
+      <mechanicalReduction>1</mechanicalReduction>
+    </transmission>
     <link name="${side}_wrist">
       <inertial>
@@ -470,4 +531,9 @@
       <child link="${side}_wrist"/>
     </joint>
+    <transmission type="pr2_mechanism_model/SimpleTransmission" name="${side}_wrist_trans">
+      <actuator name="${side}_wrist_motor" />
+      <joint name="${side}_wrist_joint" />
+      <mechanicalReduction>1</mechanicalReduction>
+    </transmission>
     <!--
     <link name="${side}_hand">
@@ -503,4 +569,9 @@
       <child link="${side}_hand"/>
     </joint>
+    <transmission type="pr2_mechanism_model/SimpleTransmission" name="${side}_hand_trans">
+      <actuator name="${side}_hand_motor" />
+      <joint name="${side}_hand_joint" />
+      <mechanicalReduction>1</mechanicalReduction>
+    </transmission>
     -->
   </xacro:macro>
@@ -519,4 +590,10 @@
       <origin xyz="0 ${-torso_y/2-shoulder_radius/2} ${torso_z-shoulder_radius/2}" rpy="0 0 0"/>
     </xacro:arm>
+    <gazebo>
+      <controller:gazebo_ros_controller_manager name="gazebo_ros_controller_manager" plugin="libgazebo_ros_controller_manager.so">
+        <alwaysOn>true</alwaysOn>
+        <updateRate>1000.0</updateRate>
+      </controller:gazebo_ros_controller_manager>
+    </gazebo>
   </xacro:macro>
 </robot>
