Commit message: testing

File: models_v0/humanoid/bdi/test.urdf (robot description, URDF)
Before this commit: robot drc, 29 links, 0 joints
Links:
- link head: mass None -> 2.6
- link l_clav: mass None -> 2.369
- link l_farm: mass None -> 0.981
- link l_foot: mass None -> 1.634
- link l_hand: mass None -> 2.263
- link l_larm: mass None -> 2.148
- link l_lglut: mass None -> 0.69
- link l_lleg: mass None -> 4.367
- link l_scap: mass None -> 2.707
- link l_talus: mass None -> 0.1
- link l_uarm: mass None -> 1.881
- link l_uglut: mass None -> 0.5166
- link l_uleg: mass None -> 7.34
- link ltorso: mass None -> 1.92
- link mtorso: mass None -> 0.55
- link pelvis: mass None -> 14.2529
- link r_clav: mass None -> 2.369
- link r_farm: mass None -> 0.981
- link r_foot: mass None -> 1.634
- link r_hand: mass None -> 2.263
- link r_larm: mass None -> 2.148
- link r_lglut: mass None -> 0.69
- link r_lleg: mass None -> 4.367
- link r_scap: mass None -> 2.707
- link r_talus: mass None -> 0.1
- link r_uarm: mass None -> 1.881
- link r_uglut: mass None -> 0.5166
- link r_uleg: mass None -> 7.34
- link utorso: mass None -> 18.484

Commit message: fix bdi_parser

File: models_v0/humanoid/bdi/test.urdf (robot description, URDF)
Before this commit: robot drc_skeleton, 29 links, 0 joints
Links:
- link head: geometry collision sphere radius=0.03; visual sphere radius=0.03
- link l_clav: geometry collision sphere radius=0.03; visual sphere radius=0.03
- link l_farm: geometry collision sphere radius=0.03; visual sphere radius=0.03
- link l_foot: geometry collision sphere radius=0.03; visual sphere radius=0.03
- link l_hand: geometry collision sphere radius=0.03; visual sphere radius=0.03
- link l_larm: geometry collision sphere radius=0.03; visual sphere radius=0.03
- link l_lglut: geometry collision sphere radius=0.03; visual sphere radius=0.03
- link l_lleg: geometry collision sphere radius=0.03; visual sphere radius=0.03
- link l_scap: geometry collision sphere radius=0.03; visual sphere radius=0.03
- link l_talus: geometry collision sphere radius=0.03; visual sphere radius=0.03
- link l_uarm: geometry collision sphere radius=0.03; visual sphere radius=0.03
- link l_uglut: geometry collision sphere radius=0.03; visual sphere radius=0.03
- link l_uleg: geometry collision sphere radius=0.03; visual sphere radius=0.03
- link ltorso: geometry collision sphere radius=0.03; visual sphere radius=0.03
- link mtorso: geometry collision sphere radius=0.03; visual sphere radius=0.03
- link pelvis: geometry collision sphere radius=0.03; visual sphere radius=0.03
- link r_clav: geometry collision sphere radius=0.03; visual sphere radius=0.03
- link r_farm: geometry collision sphere radius=0.03; visual sphere radius=0.03
- link r_foot: geometry collision sphere radius=0.03; visual sphere radius=0.03
- link r_hand: geometry collision sphere radius=0.03; visual sphere radius=0.03
- link r_larm: geometry collision sphere radius=0.03; visual sphere radius=0.03
- link r_lglut: geometry collision sphere radius=0.03; visual sphere radius=0.03
- link r_lleg: geometry collision sphere radius=0.03; visual sphere radius=0.03
- link r_scap: geometry collision sphere radius=0.03; visual sphere radius=0.03
- link r_talus: geometry collision sphere radius=0.03; visual sphere radius=0.03
- link r_uarm: geometry collision sphere radius=0.03; visual sphere radius=0.03
- link r_uglut: geometry collision sphere radius=0.03; visual sphere radius=0.03
- link r_uleg: geometry collision sphere radius=0.03; visual sphere radius=0.03
- link utorso: geometry collision sphere radius=0.03; visual sphere radius=0.03
Joints:
- added joint back.lbz: type revolute, parent pelvis, child ltorso, origin xyz=-0.0125 0 4.94066e-324 rpy=0 -0 0, axis 0 0 1.39804e-76
- added joint back.mby: type revolute, parent ltorso, child mtorso, origin xyz=0 0 1.39804e-76 rpy=0 -0 0, axis 0 1 1.39804e-76
- added joint back.ubx: type revolute, parent mtorso, child utorso, origin xyz=0 0 1.39804e-76 rpy=0 -0 0, axis 1 0 1.39804e-76
- added joint l.arm.elx: type revolute, parent l_uarm, child l_larm, origin xyz=0 0.121 3.87688e-265 rpy=0 -0 0, axis 1 0 1.38185e-76
- added joint l.arm.ely: type revolute, parent l_scap, child l_uarm, origin xyz=0 0.185 3.87688e-265 rpy=0 -0 0, axis 0 1 1.38186e-76
- added joint l.arm.mwx: type revolute, parent l_farm, child l_hand, origin xyz=0 0.095 3.87688e-265 rpy=0 -0 0, axis 1 0 1.39804e-76
- added joint l.arm.shx: type revolute, parent l_clav, child l_scap, origin xyz=0 0.075 1.96839e+161 rpy=0 -0 0, axis 1 0 1.38186e-76
- added joint l.arm.usy: type revolute, parent utorso, child l_clav, origin xyz=0.024 0.221 3.87688e-265 rpy=0 -0 0, axis 0 -0.5 1.38186e-76
- added joint l.arm.uwy: type revolute, parent l_larm, child l_farm, origin xyz=0 0.183 3.87688e-265 rpy=0 -0 0, axis 0 1 1.74882e-77
- added joint l.leg.kny: type revolute, parent l_uleg, child l_lleg, origin xyz=-0.05 0 3.87687e-265 rpy=0 -0 0, axis 0 1 1.3994e-76
- added joint l.leg.lax: type revolute, parent l_talus, child l_foot, origin xyz=0 0 3.87687e-265 rpy=0 -0 0, axis 1 0 1.39804e-76
- added joint l.leg.lhy: type revolute, parent l_lglut, child l_uleg, origin xyz=0.05 0 3.87687e-265 rpy=0 -0 0, axis 0 1 1.39805e-76
- added joint l.leg.mhx: type revolute, parent l_uglut, child l_lglut, origin xyz=0 0 7.60811e+271 rpy=0 -0 0, axis 1 0 1.39804e-76
- added joint l.leg.uay: type revolute, parent l_lleg, child l_talus, origin xyz=0 0 3.87687e-265 rpy=0 -0 0, axis 0 1 1.39872e-76
- added joint l.leg.uhz: type revolute, parent pelvis, child l_uglut, origin xyz=0 0.089 3.87687e-265 rpy=0 -0 0, axis 0 0 1.39804e-76
- added joint neck.ay: type revolute, parent utorso, child head, origin xyz=0.011 0 1.39804e-76 rpy=0 -0 0, axis 0 1 1.20271e-153
- added joint r.arm.elx: type revolute, parent r_uarm, child r_larm, origin xyz=0 -0.121 3.87688e-265 rpy=0 -0 0, axis 1 0 1.72732e-77
- added joint r.arm.ely: type revolute, parent r_scap, child r_uarm, origin xyz=0 -0.185 3.87688e-265 rpy=0 -0 0, axis 0 1 1.74967e-77
- added joint r.arm.mwx: type revolute, parent r_farm, child r_hand, origin xyz=0 -0.095 3.87688e-265 rpy=0 -0 0, axis 1 0 1.39804e-76
- added joint r.arm.shx: type revolute, parent r_clav, child r_scap, origin xyz=0 -0.075 1.96839e+161 rpy=0 -0 0, axis 1 0 1.72732e-77
- added joint r.arm.usy: type revolute, parent utorso, child r_clav, origin xyz=0.024 -0.221 3.87688e-265 rpy=0 -0 0, axis 0 0.5 1.38186e-76
- added joint r.arm.uwy: type revolute, parent r_larm, child r_farm, origin xyz=0 -0.183 3.87688e-265 rpy=0 -0 0, axis 0 1 1.74882e-77
- added joint r.leg.aky: type None, parent r_talus, child r_foot, origin xyz=0 0 0 rpy=0 -0 0, axis 0 0 0
- added joint r.leg.kny: type revolute, parent r_uleg, child r_lleg, origin xyz=-0.05 0 3.87687e-265 rpy=0 -0 0, axis 0 1 1.3994e-76
- added joint r.leg.lhy: type revolute, parent r_lglut, child r_uleg, origin xyz=0.05 0 3.87687e-265 rpy=0 -0 0, axis 0 1 1.39805e-76
- added joint r.leg.mhx: type revolute, parent r_uglut, child r_lglut, origin xyz=0 0 3.87687e-265 rpy=0 -0 0, axis 1 0 1.39804e-76
- added joint r.leg.uay: type revolute, parent r_lleg, child r_talus, origin xyz=0 0 3.87687e-265 rpy=0 -0 0, axis 0 1 1.39872e-76
- added joint r.leg.uhz: type revolute, parent pelvis, child r_uglut, origin xyz=0 -0.089 3.87687e-265 rpy=0 -0 0, axis 0 0 1.39804e-76

Commit message: finally, a version that passes check_urdf

File: models_v0/humanoid/bdi/test.urdf (robot description, URDF)
Before this commit: robot drc_skeleton, 29 links, 28 joints
Joints:
- removed joint r.leg.aky
- added joint r.leg.lax: type revolute, parent r_talus, child r_foot, origin xyz=0 0 3.87687e-265 rpy=0 -0 0, axis 1 0 1.39804e-76, limit lower=-0.436 upper=0.436 effort=90 velocity=12
- joint back.lbz: limit (none) -> lower=-0.610865 upper=0.610865 effort=124.016 velocity=12
- joint back.mby: limit (none) -> lower=-1.2 upper=1.28 effort=206.843 velocity=12
- joint back.ubx: limit (none) -> lower=-0.790809 upper=0 effort=94.91 velocity=12
- joint l.arm.elx: limit (none) -> lower=0 upper=2.35619 effort=114 velocity=12
- joint l.arm.ely: limit (none) -> lower=0 upper=3.14159 effort=114 velocity=12
- joint l.arm.mwx: limit (none) -> lower=-0.436 upper=1.571 effort=60 velocity=12
- joint l.arm.shx: limit (none) -> lower=-1.39626 upper=1.74533 effort=170 velocity=12
- joint l.arm.usy: limit (none) -> lower=-1.9635 upper=1.9635 effort=212 velocity=12
- joint l.arm.uwy: limit (none) -> lower=-1.571 upper=1.571 effort=114 velocity=12
- joint l.leg.kny: limit (none) -> lower=0 upper=2.45 effort=220 velocity=12
- joint l.leg.lax: limit (none) -> lower=-0.436 upper=0.436 effort=90 velocity=12
- joint l.leg.lhy: limit (none) -> lower=-1.75 upper=0.524 effort=260 velocity=12
- joint l.leg.mhx: limit (none) -> lower=-0.47 upper=0.495 effort=180 velocity=12
- joint l.leg.uay: limit (none) -> lower=-0.698 upper=0.698 effort=220 velocity=12
- joint l.leg.uhz: limit (none) -> lower=-0.32 upper=1.14 effort=110 velocity=12
- joint neck.ay: limit (none) -> lower=0.785398 upper=0.785398 effort=5 velocity=12
- joint r.arm.elx: limit (none) -> lower=-2.35619 upper=0 effort=114 velocity=12
- joint r.arm.ely: limit (none) -> lower=0 upper=3.14159 effort=114 velocity=12
- joint r.arm.mwx: limit (none) -> lower=-1.571 upper=0.436 effort=60 velocity=12
- joint r.arm.shx: limit (none) -> lower=-1.74533 upper=1.39626 effort=170 velocity=12
- joint r.arm.usy: limit (none) -> lower=-1.9635 upper=1.9635 effort=212 velocity=12
- joint r.arm.uwy: limit (none) -> lower=-1.571 upper=1.571 effort=114 velocity=12
- joint r.leg.kny: limit (none) -> lower=0 upper=2.45 effort=220 velocity=12
- joint r.leg.lhy: limit (none) -> lower=-1.745 upper=0.524 effort=260 velocity=12
- joint r.leg.mhx: limit (none) -> lower=-0.495 upper=0.47 effort=180 velocity=12
- joint r.leg.uay: limit (none) -> lower=-0.698 upper=0.698 effort=220 velocity=12
- joint r.leg.uhz: limit (none) -> lower=-1.14 upper=0.32 effort=260 velocity=12

Commit message: fix major parser bug, update test.urdf

File: models_v0/humanoid/bdi/test.urdf (robot description, URDF)
Before this commit: robot drc_skeleton, 29 links, 28 joints
Joints:
- joint back.lbz: axis 0 0 1.39804e-76 -> 0 0 1; origin xyz=-0.0125 0 4.94066e-324 rpy=0 -0 0 -> xyz=-0.0125 0 0 rpy=0 -0 0
- joint back.mby: axis 0 1 1.39804e-76 -> 0 1 0; origin xyz=0 0 1.39804e-76 rpy=0 -0 0 -> xyz=0 0 0.14 rpy=0 -0 0
- joint back.ubx: axis 1 0 1.39804e-76 -> 1 0 0; origin xyz=0 0 1.39804e-76 rpy=0 -0 0 -> xyz=0 0 0.05 rpy=0 -0 0
- joint l.arm.elx: axis 1 0 1.38185e-76 -> 1 0 0; origin xyz=0 0.121 3.87688e-265 rpy=0 -0 0 -> xyz=0 0.121 0.013 rpy=0 -0 0
- joint l.arm.ely: axis 0 1 1.38186e-76 -> 0 1 0; origin xyz=0 0.185 3.87688e-265 rpy=0 -0 0 -> xyz=0 0.185 0 rpy=0 -0 0
- joint l.arm.mwx: axis 1 0 1.39804e-76 -> 1 0 0; origin xyz=0 0.095 3.87688e-265 rpy=0 -0 0 -> xyz=0 0.095 0 rpy=0 -0 0
- joint l.arm.shx: axis 1 0 1.38186e-76 -> 1 0 0; origin xyz=0 0.075 1.96839e+161 rpy=0 -0 0 -> xyz=0 0.075 0.036 rpy=0 -0 0
- joint l.arm.usy: axis 0 -0.5 1.38186e-76 -> 0 -0.5 0.866025; origin xyz=0.024 0.221 3.87688e-265 rpy=0 -0 0 -> xyz=0.024 0.221 0.289 rpy=0 -0 0
- joint l.arm.uwy: axis 0 1 1.74882e-77 -> 0 1 0; origin xyz=0 0.183 3.87688e-265 rpy=0 -0 0 -> xyz=0 0.183 -0.013 rpy=0 -0 0
- joint l.leg.kny: axis 0 1 1.3994e-76 -> 0 1 0; origin xyz=-0.05 0 3.87687e-265 rpy=0 -0 0 -> xyz=-0.05 0 -0.374 rpy=0 -0 0
- joint l.leg.lax: axis 1 0 1.39804e-76 -> 1 0 0; origin xyz=0 0 3.87687e-265 rpy=0 -0 0 -> xyz=0 0 0 rpy=0 -0 0
- joint l.leg.lhy: axis 0 1 1.39805e-76 -> 0 1 0; origin xyz=0.05 0 3.87687e-265 rpy=0 -0 0 -> xyz=0.05 0 -0.05 rpy=0 -0 0
- joint l.leg.mhx: axis 1 0 1.39804e-76 -> 1 0 0; origin xyz=0 0 7.60811e+271 rpy=0 -0 0 -> xyz=0 0 0 rpy=0 -0 0
- joint l.leg.uay: axis 0 1 1.39872e-76 -> 0 1 0; origin xyz=0 0 3.87687e-265 rpy=0 -0 0 -> xyz=0 0 -0.422 rpy=0 -0 0
- joint l.leg.uhz: axis 0 0 1.39804e-76 -> 0 0 1; origin xyz=0 0.089 3.87687e-265 rpy=0 -0 0 -> xyz=0 0.089 0 rpy=0 -0 0
- joint neck.ay: axis 0 1 1.20271e-153 -> 0 1 0; origin xyz=0.011 0 1.39804e-76 rpy=0 -0 0 -> xyz=0.011 0 0.49 rpy=0 -0 0
- joint r.arm.elx: axis 1 0 1.72732e-77 -> 1 0 0; origin xyz=0 -0.121 3.87688e-265 rpy=0 -0 0 -> xyz=0 -0.121 0.013 rpy=0 -0 0
- joint r.arm.ely: axis 0 1 1.74967e-77 -> 0 1 0; origin xyz=0 -0.185 3.87688e-265 rpy=0 -0 0 -> xyz=0 -0.185 0 rpy=0 -0 0
- joint r.arm.mwx: axis 1 0 1.39804e-76 -> 1 0 0; origin xyz=0 -0.095 3.87688e-265 rpy=0 -0 0 -> xyz=0 -0.095 0 rpy=0 -0 0
- joint r.arm.shx: axis 1 0 1.72732e-77 -> 1 0 0; origin xyz=0 -0.075 1.96839e+161 rpy=0 -0 0 -> xyz=0 -0.075 0.036 rpy=0 -0 0
- joint r.arm.usy: axis 0 0.5 1.38186e-76 -> 0 0.5 0.866025; origin xyz=0.024 -0.221 3.87688e-265 rpy=0 -0 0 -> xyz=0.024 -0.221 0.289 rpy=0 -0 0
- joint r.arm.uwy: axis 0 1 1.74882e-77 -> 0 1 0; origin xyz=0 -0.183 3.87688e-265 rpy=0 -0 0 -> xyz=0 -0.183 -0.013 rpy=0 -0 0
- joint r.leg.kny: axis 0 1 1.3994e-76 -> 0 1 0; origin xyz=-0.05 0 3.87687e-265 rpy=0 -0 0 -> xyz=-0.05 0 -0.374 rpy=0 -0 0
- joint r.leg.lax: axis 1 0 1.39804e-76 -> 1 0 0; origin xyz=0 0 3.87687e-265 rpy=0 -0 0 -> xyz=0 0 0 rpy=0 -0 0
- joint r.leg.lhy: axis 0 1 1.39805e-76 -> 0 1 0; origin xyz=0.05 0 3.87687e-265 rpy=0 -0 0 -> xyz=0.05 0 -0.05 rpy=0 -0 0
- joint r.leg.mhx: axis 1 0 1.39804e-76 -> 1 0 0; origin xyz=0 0 3.87687e-265 rpy=0 -0 0 -> xyz=0 0 0 rpy=0 -0 0
- joint r.leg.uay: axis 0 1 1.39872e-76 -> 0 1 0; origin xyz=0 0 3.87687e-265 rpy=0 -0 0 -> xyz=0 0 -0.422 rpy=0 -0 0
- joint r.leg.uhz: axis 0 0 1.39804e-76 -> 0 0 1; origin xyz=0 -0.089 3.87687e-265 rpy=0 -0 0 -> xyz=0 -0.089 0 rpy=0 -0 0
