Commit message: remove package:// prefix

File: models_v0/camhand/urdf/camhand.urdf.xacro (robot description, xacro)
@@ -29,5 +29,5 @@
         <origin xyz="0 0 0" rpy="0 0 0"/>
         <geometry>
-          <mesh filename="package://camhand/urdf/camhand/f0.stl"/>
+          <mesh filename="camhand/f0.stl"/>
         </geometry>
       </collision>
@@ -35,5 +35,5 @@
         <origin xyz="0 0 0" rpy="0 0 0"/>
         <geometry>
-          <mesh filename="package://camhand/urdf/camhand/f0.stl"/>
+          <mesh filename="camhand/f0.stl"/>
         </geometry>
         <material name="${side}_camhand_skin_suntan">
@@ -52,5 +52,5 @@
         <origin xyz="0 0 0" rpy="0 0 0"/>
         <geometry>
-          <mesh filename="package://camhand/urdf/camhand/f1.stl"/>
+          <mesh filename="camhand/f1.stl"/>
         </geometry>
       </collision>
@@ -58,5 +58,5 @@
         <origin xyz="0 0 0" rpy="0 0 0"/>
         <geometry>
-          <mesh filename="package://camhand/urdf/camhand/f1.stl"/>
+          <mesh filename="camhand/f1.stl"/>
         </geometry>
         <material name="${side}_camhand_skin">
@@ -83,5 +83,5 @@
         <origin xyz="0 0 0" rpy="0 0 0"/>
         <geometry>
-          <mesh filename="package://camhand/urdf/camhand/f2.stl"/>
+          <mesh filename="camhand/f2.stl"/>
         </geometry>
       </collision>
@@ -89,5 +89,5 @@
         <origin xyz="0 0 0" rpy="0 0 0"/>
         <geometry>
-          <mesh filename="package://camhand/urdf/camhand/f2.stl"/>
+          <mesh filename="camhand/f2.stl"/>
         </geometry>
         <material name="${side}_camhand_skin_suntan">
@@ -157,5 +157,5 @@
         <origin xyz="0 0 0" rpy="0 0 0"/>
         <geometry>
-          <mesh filename="package://camhand/urdf/camhand/palm.stl"/>
+          <mesh filename="camhand/palm.stl"/>
         </geometry>
       </collision>
@@ -163,5 +163,5 @@
         <origin xyz="0 0 0" rpy="0 0 0"/>
         <geometry>
-          <mesh filename="package://camhand/urdf/camhand/palm.stl"/>
+          <mesh filename="camhand/palm.stl"/>
         </geometry>
         <material name="${side}_camhand_skin">

File: models_v0/humanoid/robots/humanoid.urdf.xacro (robot description, xacro)
@@ -7,4 +7,5 @@
   <include filename="$(find camhand)/urdf/camhand.urdf.xacro" />
   <xacro:ragdoll/>
+<!--
   <xacro:camhand side="r" parent="r_wrist">
     <origin xyz="0 0 -0.03" rpy="0 1.57079 3.14159"/>
@@ -13,3 +14,4 @@
     <origin xyz="0 0 -0.03" rpy="0 1.57079 3.14159"/>
   </xacro:camhand>
+-->
 </robot>
