Commit message: moving things around

File: prototyping/drc_robot/urdf/drc_robot.urdf (robot description, URDF)
Before this commit: robot drc_skeleton, 29 links, 28 joints
Links:
- link head: geometry collision mesh filename=drc_robot/meshes/head.dae scale=1 1 1; visual mesh filename=drc_robot/meshes/head.dae scale=1 1 1
- link l_clav: geometry collision mesh filename=drc_robot/meshes/l_clav.dae scale=1 1 1; visual mesh filename=drc_robot/meshes/l_clav.dae scale=1 1 1
- link l_farm: geometry collision mesh filename=drc_robot/meshes/l_farm.dae scale=1 1 1; visual mesh filename=drc_robot/meshes/l_farm.dae scale=1 1 1
- link l_foot: geometry collision mesh filename=drc_robot/meshes/l_foot.dae scale=1 1 1; visual mesh filename=drc_robot/meshes/l_foot.dae scale=1 1 1
- link l_hand: geometry collision mesh filename=drc_robot/meshes/l_hand.dae scale=1 1 1; visual mesh filename=drc_robot/meshes/l_hand.dae scale=1 1 1
- link l_larm: geometry collision mesh filename=drc_robot/meshes/l_larm.dae scale=1 1 1; visual mesh filename=drc_robot/meshes/l_larm.dae scale=1 1 1
- link l_lglut: geometry collision mesh filename=drc_robot/meshes/l_lglut.dae scale=1 1 1; visual mesh filename=drc_robot/meshes/l_lglut.dae scale=1 1 1
- link l_lleg: geometry collision mesh filename=drc_robot/meshes/l_lleg.dae scale=1 1 1; visual mesh filename=drc_robot/meshes/l_lleg.dae scale=1 1 1
- link l_scap: geometry collision mesh filename=drc_robot/meshes/l_scap.dae scale=1 1 1; visual mesh filename=drc_robot/meshes/l_scap.dae scale=1 1 1
- link l_talus: geometry collision mesh filename=drc_robot/meshes/l_talus.dae scale=1 1 1; visual mesh filename=drc_robot/meshes/l_talus.dae scale=1 1 1
- link l_uarm: geometry collision mesh filename=drc_robot/meshes/l_uarm.dae scale=1 1 1; visual mesh filename=drc_robot/meshes/l_uarm.dae scale=1 1 1
- link l_uglut: geometry collision mesh filename=drc_robot/meshes/l_uglut.dae scale=1 1 1; visual mesh filename=drc_robot/meshes/l_uglut.dae scale=1 1 1
- link l_uleg: geometry collision mesh filename=drc_robot/meshes/l_uleg.dae scale=1 1 1; visual mesh filename=drc_robot/meshes/l_uleg.dae scale=1 1 1
- link ltorso: geometry collision mesh filename=drc_robot/meshes/ltorso.dae scale=1 1 1; visual mesh filename=drc_robot/meshes/ltorso.dae scale=1 1 1
- link mtorso: geometry collision mesh filename=drc_robot/meshes/mtorso.dae scale=1 1 1; visual mesh filename=drc_robot/meshes/mtorso.dae scale=1 1 1
- link pelvis: geometry collision mesh filename=drc_robot/meshes/pelvis.dae scale=1 1 1; visual mesh filename=drc_robot/meshes/pelvis.dae scale=1 1 1
- link r_clav: geometry collision mesh filename=drc_robot/meshes/r_clav.dae scale=1 1 1; visual mesh filename=drc_robot/meshes/r_clav.dae scale=1 1 1
- link r_farm: geometry collision mesh filename=drc_robot/meshes/r_farm.dae scale=1 1 1; visual mesh filename=drc_robot/meshes/r_farm.dae scale=1 1 1
- link r_foot: geometry collision mesh filename=drc_robot/meshes/r_foot.dae scale=1 1 1; visual mesh filename=drc_robot/meshes/r_foot.dae scale=1 1 1
- link r_hand: geometry collision mesh filename=drc_robot/meshes/r_hand.dae scale=1 1 1; visual mesh filename=drc_robot/meshes/r_hand.dae scale=1 1 1
- link r_larm: geometry collision mesh filename=drc_robot/meshes/r_larm.dae scale=1 1 1; visual mesh filename=drc_robot/meshes/r_larm.dae scale=1 1 1
- link r_lglut: geometry collision mesh filename=drc_robot/meshes/r_lglut.dae scale=1 1 1; visual mesh filename=drc_robot/meshes/r_lglut.dae scale=1 1 1
- link r_lleg: geometry collision mesh filename=drc_robot/meshes/r_lleg.dae scale=1 1 1; visual mesh filename=drc_robot/meshes/r_lleg.dae scale=1 1 1
- link r_scap: geometry collision mesh filename=drc_robot/meshes/r_scap.dae scale=1 1 1; visual mesh filename=drc_robot/meshes/r_scap.dae scale=1 1 1
- link r_talus: geometry collision mesh filename=drc_robot/meshes/r_talus.dae scale=1 1 1; visual mesh filename=drc_robot/meshes/r_talus.dae scale=1 1 1
- link r_uarm: geometry collision mesh filename=drc_robot/meshes/r_uarm.dae scale=1 1 1; visual mesh filename=drc_robot/meshes/r_uarm.dae scale=1 1 1
- link r_uglut: geometry collision mesh filename=drc_robot/meshes/r_uglut.dae scale=1 1 1; visual mesh filename=drc_robot/meshes/r_uglut.dae scale=1 1 1
- link r_uleg: geometry collision mesh filename=drc_robot/meshes/r_uleg.dae scale=1 1 1; visual mesh filename=drc_robot/meshes/r_uleg.dae scale=1 1 1
- link utorso: geometry collision mesh filename=drc_robot/meshes/utorso.dae scale=1 1 1; visual mesh filename=drc_robot/meshes/utorso.dae scale=1 1 1

Commit message: bug fix, drc inertia

File: prototyping/drc_robot/urdf/drc_robot.urdf (robot description, URDF)
Before this commit: robot drc_skeleton, 29 links, 28 joints
Links:
- link head: geometry collision mesh filename=drc_robot/meshes/head.stl scale=1 1 1; visual mesh filename=drc_robot/meshes/head.dae scale=1 1 1
- link l_clav: geometry collision mesh filename=drc_robot/meshes/l_clav.stl scale=1 1 1; visual mesh filename=drc_robot/meshes/l_clav.dae scale=1 1 1
- link l_farm: geometry collision mesh filename=drc_robot/meshes/l_farm.stl scale=1 1 1; visual mesh filename=drc_robot/meshes/l_farm.dae scale=1 1 1
- link l_foot: geometry collision mesh filename=drc_robot/meshes/l_foot.stl scale=1 1 1; visual mesh filename=drc_robot/meshes/l_foot.dae scale=1 1 1
- link l_hand: geometry collision mesh filename=drc_robot/meshes/l_hand.stl scale=1 1 1; visual mesh filename=drc_robot/meshes/l_hand.dae scale=1 1 1
- link l_larm: geometry collision mesh filename=drc_robot/meshes/l_larm.stl scale=1 1 1; visual mesh filename=drc_robot/meshes/l_larm.dae scale=1 1 1
- link l_lglut: geometry collision mesh filename=drc_robot/meshes/l_lglut.stl scale=1 1 1; visual mesh filename=drc_robot/meshes/l_lglut.dae scale=1 1 1
- link l_lleg: geometry collision mesh filename=drc_robot/meshes/l_lleg.stl scale=1 1 1; visual mesh filename=drc_robot/meshes/l_lleg.dae scale=1 1 1
- link l_scap: geometry collision mesh filename=drc_robot/meshes/l_scap.stl scale=1 1 1; visual mesh filename=drc_robot/meshes/l_scap.dae scale=1 1 1
- link l_talus: geometry collision mesh filename=drc_robot/meshes/l_talus.stl scale=1 1 1; visual mesh filename=drc_robot/meshes/l_talus.dae scale=1 1 1
- link l_uarm: geometry collision mesh filename=drc_robot/meshes/l_uarm.stl scale=1 1 1; visual mesh filename=drc_robot/meshes/l_uarm.dae scale=1 1 1
- link l_uglut: geometry collision mesh filename=drc_robot/meshes/l_uglut.stl scale=1 1 1; visual mesh filename=drc_robot/meshes/l_uglut.dae scale=1 1 1
- link l_uleg: geometry collision mesh filename=drc_robot/meshes/l_uleg.stl scale=1 1 1; visual mesh filename=drc_robot/meshes/l_uleg.dae scale=1 1 1
- link ltorso: geometry collision mesh filename=drc_robot/meshes/ltorso.stl scale=1 1 1; visual mesh filename=drc_robot/meshes/ltorso.dae scale=1 1 1
- link mtorso: geometry collision mesh filename=drc_robot/meshes/mtorso.stl scale=1 1 1; visual mesh filename=drc_robot/meshes/mtorso.dae scale=1 1 1
- link pelvis: geometry collision mesh filename=drc_robot/meshes/pelvis.stl scale=1 1 1; visual mesh filename=drc_robot/meshes/pelvis.dae scale=1 1 1
- link r_clav: geometry collision mesh filename=drc_robot/meshes/r_clav.stl scale=1 1 1; visual mesh filename=drc_robot/meshes/r_clav.dae scale=1 1 1
- link r_farm: geometry collision mesh filename=drc_robot/meshes/r_farm.stl scale=1 1 1; visual mesh filename=drc_robot/meshes/r_farm.dae scale=1 1 1
- link r_foot: geometry collision mesh filename=drc_robot/meshes/r_foot.stl scale=1 1 1; visual mesh filename=drc_robot/meshes/r_foot.dae scale=1 1 1
- link r_hand: geometry collision mesh filename=drc_robot/meshes/r_hand.stl scale=1 1 1; visual mesh filename=drc_robot/meshes/r_hand.dae scale=1 1 1
- link r_larm: geometry collision mesh filename=drc_robot/meshes/r_larm.stl scale=1 1 1; visual mesh filename=drc_robot/meshes/r_larm.dae scale=1 1 1
- link r_lglut: geometry collision mesh filename=drc_robot/meshes/r_lglut.stl scale=1 1 1; visual mesh filename=drc_robot/meshes/r_lglut.dae scale=1 1 1
- link r_lleg: geometry collision mesh filename=drc_robot/meshes/r_lleg.stl scale=1 1 1; visual mesh filename=drc_robot/meshes/r_lleg.dae scale=1 1 1
- link r_scap: geometry collision mesh filename=drc_robot/meshes/r_scap.stl scale=1 1 1; visual mesh filename=drc_robot/meshes/r_scap.dae scale=1 1 1
- link r_talus: geometry collision mesh filename=drc_robot/meshes/r_talus.stl scale=1 1 1; visual mesh filename=drc_robot/meshes/r_talus.dae scale=1 1 1
- link r_uarm: geometry collision mesh filename=drc_robot/meshes/r_uarm.stl scale=1 1 1; visual mesh filename=drc_robot/meshes/r_uarm.dae scale=1 1 1
- link r_uglut: geometry collision mesh filename=drc_robot/meshes/r_uglut.stl scale=1 1 1; visual mesh filename=drc_robot/meshes/r_uglut.dae scale=1 1 1
- link r_uleg: geometry collision mesh filename=drc_robot/meshes/r_uleg.stl scale=1 1 1; visual mesh filename=drc_robot/meshes/r_uleg.dae scale=1 1 1
- link utorso: geometry collision mesh filename=drc_robot/meshes/utorso.stl scale=1 1 1; visual mesh filename=drc_robot/meshes/utorso.dae scale=1 1 1
