Commit message: update camhand mesh location

File: prototyping/camhand/urdf/camhand.urdf.xacro (robot description, xacro)
@@ -29,5 +29,5 @@
         <origin xyz="0 0 0" rpy="0 0 0"/>
         <geometry>
-          <mesh filename="camhand/f0.stl"/>
+          <mesh filename="model://camhand/meshes/f0.stl"/>
         </geometry>
       </collision>
@@ -35,5 +35,5 @@
         <origin xyz="0 0 0" rpy="0 0 0"/>
         <geometry>
-          <mesh filename="camhand/f0.stl"/>
+          <mesh filename="model://camhand/meshes/f0.stl"/>
         </geometry>
         <material name="${side}_camhand_skin_suntan">
@@ -52,5 +52,5 @@
         <origin xyz="0 0 0" rpy="0 0 0"/>
         <geometry>
-          <mesh filename="camhand/f1.stl"/>
+          <mesh filename="model://camhand/meshes/f1.stl"/>
         </geometry>
       </collision>
@@ -58,5 +58,5 @@
         <origin xyz="0 0 0" rpy="0 0 0"/>
         <geometry>
-          <mesh filename="camhand/f1.stl"/>
+          <mesh filename="model://camhand/meshes/f1.stl"/>
         </geometry>
         <material name="${side}_camhand_skin">
@@ -83,5 +83,5 @@
         <origin xyz="0 0 0" rpy="0 0 0"/>
         <geometry>
-          <mesh filename="camhand/f2.stl"/>
+          <mesh filename="model://camhand/meshes/f2.stl"/>
         </geometry>
       </collision>
@@ -89,5 +89,5 @@
         <origin xyz="0 0 0" rpy="0 0 0"/>
         <geometry>
-          <mesh filename="camhand/f2.stl"/>
+          <mesh filename="model://camhand/meshes/f2.stl"/>
         </geometry>
         <material name="${side}_camhand_skin_suntan">
@@ -157,5 +157,5 @@
         <origin xyz="0 0 0" rpy="0 0 0"/>
         <geometry>
-          <mesh filename="camhand/palm.stl"/>
+          <mesh filename="model://camhand/meshes/palm.stl"/>
         </geometry>
       </collision>
@@ -163,5 +163,5 @@
         <origin xyz="0 0 0" rpy="0 0 0"/>
         <geometry>
-          <mesh filename="camhand/palm.stl"/>
+          <mesh filename="model://camhand/meshes/palm.stl"/>
         </geometry>
         <material name="${side}_camhand_skin">
