Commit message: renaming joints: replace . with _ so it satisfies ROS Graph Resource name convention.  install bdi_parser.  rearrange urdf xacro locations.

File: ros/camhand_utils/urdf/camhand.urdf.xacro (robot description, xacro)
@@ -31,5 +31,5 @@
         <origin xyz="0 0 0" rpy="0 0 0"/>
         <geometry>
-          <mesh filename="model://camhand/meshes/f0.stl"/>
+          <mesh filename="package://camhand/meshes/f0.stl"/>
         </geometry>
       </collision>
@@ -37,5 +37,5 @@
         <origin xyz="0 0 0" rpy="0 0 0"/>
         <geometry>
-          <mesh filename="model://camhand/meshes/f0.stl"/>
+          <mesh filename="package://camhand/meshes/f0.stl"/>
         </geometry>
         <material name="${side}_camhand_skin_suntan">
@@ -54,5 +54,5 @@
         <origin xyz="0 0 0" rpy="0 0 0"/>
         <geometry>
-          <mesh filename="model://camhand/meshes/f1.stl"/>
+          <mesh filename="package://camhand/meshes/f1.stl"/>
         </geometry>
       </collision>
@@ -60,5 +60,5 @@
         <origin xyz="0 0 0" rpy="0 0 0"/>
         <geometry>
-          <mesh filename="model://camhand/meshes/f1.stl"/>
+          <mesh filename="package://camhand/meshes/f1.stl"/>
         </geometry>
         <material name="${side}_camhand_skin">
@@ -85,5 +85,5 @@
         <origin xyz="0 0 0" rpy="0 0 0"/>
         <geometry>
-          <mesh filename="model://camhand/meshes/f2.stl"/>
+          <mesh filename="package://camhand/meshes/f2.stl"/>
         </geometry>
       </collision>
@@ -91,5 +91,5 @@
         <origin xyz="0 0 0" rpy="0 0 0"/>
         <geometry>
-          <mesh filename="model://camhand/meshes/f2.stl"/>
+          <mesh filename="package://camhand/meshes/f2.stl"/>
         </geometry>
         <material name="${side}_camhand_skin_suntan">
@@ -166,5 +166,5 @@
         <origin xyz="0 0 0" rpy="0 0 0"/>
         <geometry>
-          <mesh filename="model://camhand/meshes/palm.stl"/>
+          <mesh filename="package://camhand/meshes/palm.stl"/>
         </geometry>
       </collision>
@@ -172,5 +172,5 @@
         <origin xyz="0 0 0" rpy="0 0 0"/>
         <geometry>
-          <mesh filename="model://camhand/meshes/palm.stl"/>
+          <mesh filename="package://camhand/meshes/palm.stl"/>
         </geometry>
         <material name="${side}_camhand_skin">

File: ros/drc_robot_utils/robots/drc_robot.model.xacro (robot description, xacro)
@@ -12,6 +12,6 @@
     <origin xyz="0  0.1 -0.03" rpy="0 3.1416 -1.57079"/>
   </xacro:camhand>
-  <include filename="$(find drc_robot_utils)/drc_robot.gazebo" />
-  <include filename="$(find drc_robot_utils)/drc_robot.transmission" />
-  <include filename="$(find drc_robot_utils)/drc_robot.sensors" />
+  <include filename="$(find drc_robot_utils)/urdf/drc_robot.gazebo" />
+  <include filename="$(find drc_robot_utils)/urdf/drc_robot.transmission" />
+  <include filename="$(find drc_robot_utils)/urdf/drc_robot.sensors" />
 </robot>

File: ros/drc_robot_utils/urdf/drc_robot.urdf (robot description, URDF)
Before this commit: robot drc_skeleton, 29 links, 28 joints
Joints:
- removed joint back.lbz
- removed joint back.mby
- removed joint back.ubx
- removed joint l.arm.elx
- removed joint l.arm.ely
- removed joint l.arm.mwx
- removed joint l.arm.shx
- removed joint l.arm.usy
- removed joint l.arm.uwy
- removed joint l.leg.kny
- removed joint l.leg.lax
- removed joint l.leg.lhy
- removed joint l.leg.mhx
- removed joint l.leg.uay
- removed joint l.leg.uhz
- removed joint neck.ay
- removed joint r.arm.elx
- removed joint r.arm.ely
- removed joint r.arm.mwx
- removed joint r.arm.shx
- removed joint r.arm.usy
- removed joint r.arm.uwy
- removed joint r.leg.kny
- removed joint r.leg.lax
- removed joint r.leg.lhy
- removed joint r.leg.mhx
- removed joint r.leg.uay
- removed joint r.leg.uhz
- added joint back_lbz: type revolute, parent pelvis, child ltorso, origin xyz=-0.0125 0 0 rpy=0 -0 0, axis 0 0 1, limit lower=-0.610865 upper=0.610865 effort=124.016 velocity=12
- added joint back_mby: type revolute, parent ltorso, child mtorso, origin xyz=0 0 0.14 rpy=0 -0 0, axis 0 1 0, limit lower=-1.2 upper=1.28 effort=206.843 velocity=12
- added joint back_ubx: type revolute, parent mtorso, child utorso, origin xyz=0 0 0.05 rpy=0 -0 0, axis 1 0 0, limit lower=-0.790809 upper=0 effort=94.91 velocity=12
- added joint l_arm_elx: type revolute, parent l_uarm, child l_larm, origin xyz=0 0.121 0.013 rpy=0 -0 0, axis 1 0 0, limit lower=0 upper=2.35619 effort=114 velocity=12
- added joint l_arm_ely: type revolute, parent l_scap, child l_uarm, origin xyz=0 0.185 0 rpy=0 -0 0, axis 0 1 0, limit lower=0 upper=3.14159 effort=114 velocity=12
- added joint l_arm_mwx: type revolute, parent l_farm, child l_hand, origin xyz=0 0.095 0 rpy=0 -0 0, axis 1 0 0, limit lower=-0.436 upper=1.571 effort=60 velocity=12
- added joint l_arm_shx: type revolute, parent l_clav, child l_scap, origin xyz=0 0.075 0.036 rpy=0 -0 0, axis 1 0 0, limit lower=-1.39626 upper=1.74533 effort=170 velocity=12
- added joint l_arm_usy: type revolute, parent utorso, child l_clav, origin xyz=0.024 0.221 0.289 rpy=0 -0 0, axis 0 -0.5 0.866025, limit lower=-1.9635 upper=1.9635 effort=212 velocity=12
- added joint l_arm_uwy: type revolute, parent l_larm, child l_farm, origin xyz=0 0.183 -0.013 rpy=0 -0 0, axis 0 1 0, limit lower=-1.571 upper=1.571 effort=114 velocity=12
- added joint l_leg_kny: type revolute, parent l_uleg, child l_lleg, origin xyz=-0.05 0 -0.374 rpy=0 -0 0, axis 0 1 0, limit lower=0 upper=2.45 effort=220 velocity=12
- added joint l_leg_lax: type revolute, parent l_talus, child l_foot, origin xyz=0 0 0 rpy=0 -0 0, axis 1 0 0, limit lower=-0.436 upper=0.436 effort=90 velocity=12
- added joint l_leg_lhy: type revolute, parent l_lglut, child l_uleg, origin xyz=0.05 0 -0.05 rpy=0 -0 0, axis 0 1 0, limit lower=-1.75 upper=0.524 effort=260 velocity=12
- added joint l_leg_mhx: type revolute, parent l_uglut, child l_lglut, origin xyz=0 0 0 rpy=0 -0 0, axis 1 0 0, limit lower=-0.47 upper=0.495 effort=180 velocity=12
- added joint l_leg_uay: type revolute, parent l_lleg, child l_talus, origin xyz=0 0 -0.422 rpy=0 -0 0, axis 0 1 0, limit lower=-0.698 upper=0.698 effort=220 velocity=12
- added joint l_leg_uhz: type revolute, parent pelvis, child l_uglut, origin xyz=0 0.089 0 rpy=0 -0 0, axis 0 0 1, limit lower=-0.32 upper=1.14 effort=110 velocity=12
- added joint neck_ay: type revolute, parent utorso, child head, origin xyz=0.011 0 0.49 rpy=0 -0 0, axis 0 1 0, limit lower=0.785398 upper=0.785398 effort=5 velocity=12
- added joint r_arm_elx: type revolute, parent r_uarm, child r_larm, origin xyz=0 -0.121 0.013 rpy=0 -0 0, axis 1 0 0, limit lower=-2.35619 upper=0 effort=114 velocity=12
- added joint r_arm_ely: type revolute, parent r_scap, child r_uarm, origin xyz=0 -0.185 0 rpy=0 -0 0, axis 0 1 0, limit lower=0 upper=3.14159 effort=114 velocity=12
- added joint r_arm_mwx: type revolute, parent r_farm, child r_hand, origin xyz=0 -0.095 0 rpy=0 -0 0, axis 1 0 0, limit lower=-1.571 upper=0.436 effort=60 velocity=12
- added joint r_arm_shx: type revolute, parent r_clav, child r_scap, origin xyz=0 -0.075 0.036 rpy=0 -0 0, axis 1 0 0, limit lower=-1.74533 upper=1.39626 effort=170 velocity=12
- added joint r_arm_usy: type revolute, parent utorso, child r_clav, origin xyz=0.024 -0.221 0.289 rpy=0 -0 0, axis 0 0.5 0.866025, limit lower=-1.9635 upper=1.9635 effort=212 velocity=12
- added joint r_arm_uwy: type revolute, parent r_larm, child r_farm, origin xyz=0 -0.183 -0.013 rpy=0 -0 0, axis 0 1 0, limit lower=-1.571 upper=1.571 effort=114 velocity=12
- added joint r_leg_kny: type revolute, parent r_uleg, child r_lleg, origin xyz=-0.05 0 -0.374 rpy=0 -0 0, axis 0 1 0, limit lower=0 upper=2.45 effort=220 velocity=12
- added joint r_leg_lax: type revolute, parent r_talus, child r_foot, origin xyz=0 0 0 rpy=0 -0 0, axis 1 0 0, limit lower=-0.436 upper=0.436 effort=90 velocity=12
- added joint r_leg_lhy: type revolute, parent r_lglut, child r_uleg, origin xyz=0.05 0 -0.05 rpy=0 -0 0, axis 0 1 0, limit lower=-1.745 upper=0.524 effort=260 velocity=12
- added joint r_leg_mhx: type revolute, parent r_uglut, child r_lglut, origin xyz=0 0 0 rpy=0 -0 0, axis 1 0 0, limit lower=-0.495 upper=0.47 effort=180 velocity=12
- added joint r_leg_uay: type revolute, parent r_lleg, child r_talus, origin xyz=0 0 -0.422 rpy=0 -0 0, axis 0 1 0, limit lower=-0.698 upper=0.698 effort=220 velocity=12
- added joint r_leg_uhz: type revolute, parent pelvis, child r_uglut, origin xyz=0 -0.089 0 rpy=0 -0 0, axis 0 0 1, limit lower=-1.14 upper=0.32 effort=260 velocity=12
