Commit message: update irobot hand

File: prototyping/irobot_hand/handle/handle_description/meshes/handle.urdf (robot description, URDF)
Before this commit: robot armh_handle, 66 links, 65 joints
Links:
- link base_link: mass None -> 0.1
- link finger[0]/base_rotation_link: mass None -> 0.1
- link finger[0]/distal_link: mass None -> 0.1
- link finger[0]/flexible_link_1: mass None -> 0.1
- link finger[0]/flexible_link_2: mass None -> 0.1
- link finger[0]/flexible_link_3: mass None -> 0.1
- link finger[0]/flexible_link_4: mass None -> 0.1
- link finger[0]/flexible_link_5: mass None -> 0.1
- link finger[0]/flexible_link_6: mass None -> 0.1
- link finger[0]/flexible_link_7: mass None -> 0.1
- link finger[0]/flexible_link_8: mass None -> 0.1
- link finger[0]/flexible_link_9: mass None -> 0.1
- link finger[0]/flexible_link_hidden_between_1_and_2: mass None -> 0.1
- link finger[0]/flexible_link_hidden_between_2_and_3: mass None -> 0.1
- link finger[0]/flexible_link_hidden_between_3_and_4: mass None -> 0.1
- link finger[0]/flexible_link_hidden_between_4_and_5: mass None -> 0.1
- link finger[0]/flexible_link_hidden_between_5_and_6: mass None -> 0.1
- link finger[0]/flexible_link_hidden_between_6_and_7: mass None -> 0.1
- link finger[0]/flexible_link_hidden_between_7_and_8: mass None -> 0.1
- link finger[0]/flexible_link_hidden_between_8_and_9: mass None -> 0.1
- link finger[0]/flexible_link_hidden_between_9_and_distal_link: mass None -> 0.1
- link finger[0]/flexible_link_hidden_between_proximal_link_and_1: mass None -> 0.1
- link finger[0]/proximal_link: mass None -> 0.1
- link finger[1]/base_rotation_link: mass None -> 0.1
- link finger[1]/distal_link: mass None -> 0.1
- link finger[1]/flexible_link_1: mass None -> 0.1
- link finger[1]/flexible_link_2: mass None -> 0.1
- link finger[1]/flexible_link_3: mass None -> 0.1
- link finger[1]/flexible_link_4: mass None -> 0.1
- link finger[1]/flexible_link_5: mass None -> 0.1
- link finger[1]/flexible_link_6: mass None -> 0.1
- link finger[1]/flexible_link_7: mass None -> 0.1
- link finger[1]/flexible_link_8: mass None -> 0.1
- link finger[1]/flexible_link_9: mass None -> 0.1
- link finger[1]/flexible_link_hidden_between_1_and_2: mass None -> 0.1
- link finger[1]/flexible_link_hidden_between_2_and_3: mass None -> 0.1
- link finger[1]/flexible_link_hidden_between_3_and_4: mass None -> 0.1
- link finger[1]/flexible_link_hidden_between_4_and_5: mass None -> 0.1
- link finger[1]/flexible_link_hidden_between_5_and_6: mass None -> 0.1
- link finger[1]/flexible_link_hidden_between_6_and_7: mass None -> 0.1
- link finger[1]/flexible_link_hidden_between_7_and_8: mass None -> 0.1
- link finger[1]/flexible_link_hidden_between_8_and_9: mass None -> 0.1
- link finger[1]/flexible_link_hidden_between_9_and_distal_link: mass None -> 0.1
- link finger[1]/flexible_link_hidden_between_proximal_link_and_1: mass None -> 0.1
- link finger[1]/proximal_link: mass None -> 0.1
- link finger[2]/distal_link: mass None -> 0.1
- link finger[2]/flexible_link_1: mass None -> 0.1
- link finger[2]/flexible_link_2: mass None -> 0.1
- link finger[2]/flexible_link_3: mass None -> 0.1
- link finger[2]/flexible_link_4: mass None -> 0.1
- link finger[2]/flexible_link_5: mass None -> 0.1
- link finger[2]/flexible_link_6: mass None -> 0.1
- link finger[2]/flexible_link_7: mass None -> 0.1
- link finger[2]/flexible_link_8: mass None -> 0.1
- link finger[2]/flexible_link_9: mass None -> 0.1
- link finger[2]/flexible_link_hidden_between_1_and_2: mass None -> 0.1
- link finger[2]/flexible_link_hidden_between_2_and_3: mass None -> 0.1
- link finger[2]/flexible_link_hidden_between_3_and_4: mass None -> 0.1
- link finger[2]/flexible_link_hidden_between_4_and_5: mass None -> 0.1
- link finger[2]/flexible_link_hidden_between_5_and_6: mass None -> 0.1
- link finger[2]/flexible_link_hidden_between_6_and_7: mass None -> 0.1
- link finger[2]/flexible_link_hidden_between_7_and_8: mass None -> 0.1
- link finger[2]/flexible_link_hidden_between_8_and_9: mass None -> 0.1
- link finger[2]/flexible_link_hidden_between_9_and_distal_link: mass None -> 0.1
- link finger[2]/flexible_link_hidden_between_proximal_link_and_1: mass None -> 0.1
- link finger[2]/proximal_link: mass None -> 0.1

File: prototyping/irobot_hand/handle/handle_description/meshes/handle.urdf.xacro (robot description, xacro)
@@ -11,13 +11,7 @@
   <link name="finger[${finger_id}]/flexible_link_${link_id}">
     <inertial>
-      <mass>0.1</mass>
-      <inertia>
-        <ixx>0.1</ixx>
-        <ixy>0.0</ixy>
-        <ixz>0.0</ixz>
-        <iyy>0.1</iyy>
-        <iyz>0.0</iyz>
-        <izz>0.1</izz>
-      </inertia>
+      <mass value="0.1"/>
+      <origin xyz="0 0 0"/>
+      <inertia ixx="0.001" ixy="0.0" ixz="0.0" iyy="0.001" iyz="0.0" izz="0.001"/>
     </inertial>
     <visual>
@@ -42,13 +36,7 @@
   <link name="finger[${finger_id}]/flexible_link_hidden_between_${link_from}_and_${link_to}">
     <inertial>
-      <mass>0.1</mass>
-      <inertia>
-        <ixx>0.1</ixx>
-        <ixy>0.0</ixy>
-        <ixz>0.0</ixz>
-        <iyy>0.1</iyy>
-        <iyz>0.0</iyz>
-        <izz>0.1</izz>
-      </inertia>
+      <mass value="0.1"/>
+      <origin xyz="0 0 0"/>
+      <inertia ixx="0.001" ixy="0.0" ixz="0.0" iyy="0.001" iyz="0.0" izz="0.001"/>
     </inertial>
     <visual>
@@ -78,13 +66,7 @@
   <link name="finger[${finger_id}]/flexible_link_hidden_between_proximal_link_and_1">
     <inertial>
-      <mass>0.1</mass>
-      <inertia>
-        <ixx>0.1</ixx>
-        <ixy>0.0</ixy>
-        <ixz>0.0</ixz>
-        <iyy>0.1</iyy>
-        <iyz>0.0</iyz>
-        <izz>0.1</izz>
-      </inertia>
+      <mass value="0.1"/>
+      <origin xyz="0 0 0"/>
+      <inertia ixx="0.001" ixy="0.0" ixz="0.0" iyy="0.001" iyz="0.0" izz="0.001"/>
     </inertial>
     <visual>
@@ -112,13 +94,7 @@
   <link name="finger[${finger_id}]/flexible_link_hidden_between_9_and_distal_link">
     <inertial>
-      <mass>0.1</mass>
-      <inertia>
-        <ixx>0.1</ixx>
-        <ixy>0.0</ixy>
-        <ixz>0.0</ixz>
-        <iyy>0.1</iyy>
-        <iyz>0.0</iyz>
-        <izz>0.1</izz>
-      </inertia>
+      <mass value="0.1"/>
+      <origin xyz="0 0 0"/>
+      <inertia ixx="0.001" ixy="0.0" ixz="0.0" iyy="0.001" iyz="0.0" izz="0.001"/>
     </inertial>
     <visual>
@@ -192,15 +168,9 @@
 <xacro:flex_joint_connector finger_id="2"/>
 <link name="base_link">
-  <inertial>
-    <mass>0.1</mass>
-    <inertia>
-      <ixx>0.1</ixx>
-      <ixy>0.0</ixy>
-      <ixz>0.0</ixz>
-      <iyy>0.1</iyy>
-      <iyz>0.0</iyz>
-      <izz>0.1</izz>
-    </inertia>
-  </inertial>
+    <inertial>
+      <mass value="0.1"/>
+      <origin xyz="0 0 0"/>
+      <inertia ixx="0.001" ixy="0.0" ixz="0.0" iyy="0.001" iyz="0.0" izz="0.001"/>
+    </inertial>
   <visual>
     <geometry>
@@ -214,15 +184,9 @@
 </link>
 <link name="finger[0]/base_rotation_link">
-  <inertial>
-    <mass>0.1</mass>
-    <inertia>
-      <ixx>0.1</ixx>
-      <ixy>0.0</ixy>
-      <ixz>0.0</ixz>
-      <iyy>0.1</iyy>
-      <iyz>0.0</iyz>
-      <izz>0.1</izz>
-    </inertia>
-  </inertial>
+    <inertial>
+      <mass value="0.1"/>
+      <origin xyz="0 0 0"/>
+      <inertia ixx="0.001" ixy="0.0" ixz="0.0" iyy="0.001" iyz="0.0" izz="0.001"/>
+    </inertial>
   <visual>
     <geometry>
@@ -236,15 +200,9 @@
 </link>
 <link name="finger[0]/proximal_link">
-  <inertial>
-    <mass>0.1</mass>
-    <inertia>
-      <ixx>0.1</ixx>
-      <ixy>0.0</ixy>
-      <ixz>0.0</ixz>
-      <iyy>0.1</iyy>
-      <iyz>0.0</iyz>
-      <izz>0.1</izz>
-    </inertia>
-  </inertial>
+    <inertial>
+      <mass value="0.1"/>
+      <origin xyz="0 0 0"/>
+      <inertia ixx="0.001" ixy="0.0" ixz="0.0" iyy="0.001" iyz="0.0" izz="0.001"/>
+    </inertial>
   <visual>
     <geometry>
@@ -258,15 +216,9 @@
 </link>
 <link name="finger[0]/distal_link">
-  <inertial>
-    <mass>0.1</mass>
-    <inertia>
-      <ixx>0.1</ixx>
-      <ixy>0.0</ixy>
-      <ixz>0.0</ixz>
-      <iyy>0.1</iyy>
-      <iyz>0.0</iyz>
-      <izz>0.1</izz>
-    </inertia>
-  </inertial>
+    <inertial>
+      <mass value="0.1"/>
+      <origin xyz="0 0 0"/>
+      <inertia ixx="0.001" ixy="0.0" ixz="0.0" iyy="0.001" iyz="0.0" izz="0.001"/>
+    </inertial>
   <visual>
     <geometry>
@@ -280,15 +232,9 @@
 </link>
 <link name="finger[1]/base_rotation_link">
-  <inertial>
-    <mass>0.1</mass>
-    <inertia>
-      <ixx>0.1</ixx>
-      <ixy>0.0</ixy>
-      <ixz>0.0</ixz>
-      <iyy>0.1</iyy>
-      <iyz>0.0</iyz>
-      <izz>0.1</izz>
-    </inertia>
-  </inertial>
+    <inertial>
+      <mass value="0.1"/>
+      <origin xyz="0 0 0"/>
+      <inertia ixx="0.001" ixy="0.0" ixz="0.0" iyy="0.001" iyz="0.0" izz="0.001"/>
+    </inertial>
   <visual>
     <geometry>
@@ -302,15 +248,9 @@
 </link>
 <link name="finger[1]/proximal_link">
-  <inertial>
-    <mass>0.1</mass>
-    <inertia>
-      <ixx>0.1</ixx>
-      <ixy>0.0</ixy>
-      <ixz>0.0</ixz>
-      <iyy>0.1</iyy>
-      <iyz>0.0</iyz>
-      <izz>0.1</izz>
-    </inertia>
-  </inertial>
+    <inertial>
+      <mass value="0.1"/>
+      <origin xyz="0 0 0"/>
+      <inertia ixx="0.001" ixy="0.0" ixz="0.0" iyy="0.001" iyz="0.0" izz="0.001"/>
+    </inertial>
   <visual>
     <geometry>
@@ -324,15 +264,9 @@
 </link>
 <link name="finger[1]/distal_link">
-  <inertial>
-    <mass>0.1</mass>
-    <inertia>
-      <ixx>0.1</ixx>
-      <ixy>0.0</ixy>
-      <ixz>0.0</ixz>
-      <iyy>0.1</iyy>
-      <iyz>0.0</iyz>
-      <izz>0.1</izz>
-    </inertia>
-  </inertial>
+    <inertial>
+      <mass value="0.1"/>
+      <origin xyz="0 0 0"/>
+      <inertia ixx="0.001" ixy="0.0" ixz="0.0" iyy="0.001" iyz="0.0" izz="0.001"/>
+    </inertial>
   <visual>
     <geometry>
@@ -346,15 +280,9 @@
 </link>
 <link name="finger[2]/proximal_link">
-  <inertial>
-    <mass>0.1</mass>
-    <inertia>
-      <ixx>0.1</ixx>
-      <ixy>0.0</ixy>
-      <ixz>0.0</ixz>
-      <iyy>0.1</iyy>
-      <iyz>0.0</iyz>
-      <izz>0.1</izz>
-    </inertia>
-  </inertial>
+    <inertial>
+      <mass value="0.1"/>
+      <origin xyz="0 0 0"/>
+      <inertia ixx="0.001" ixy="0.0" ixz="0.0" iyy="0.001" iyz="0.0" izz="0.001"/>
+    </inertial>
   <visual>
     <geometry>
@@ -368,15 +296,9 @@
 </link>
 <link name="finger[2]/distal_link">
-  <inertial>
-    <mass>0.1</mass>
-    <inertia>
-      <ixx>0.1</ixx>
-      <ixy>0.0</ixy>
-      <ixz>0.0</ixz>
-      <iyy>0.1</iyy>
-      <iyz>0.0</iyz>
-      <izz>0.1</izz>
-    </inertia>
-  </inertial>
+    <inertial>
+      <mass value="0.1"/>
+      <origin xyz="0 0 0"/>
+      <inertia ixx="0.001" ixy="0.0" ixz="0.0" iyy="0.001" iyz="0.0" izz="0.001"/>
+    </inertial>
   <visual>
     <geometry>
