Commit message: consequences of renaming camhand files, but drc_robot.launch works again.

File: ros/sandia_hand_utils/robots/sandia_hand_both.urdf.xacro (robot description, xacro)
@@ -25,8 +25,8 @@
   </link>
   <xacro:sandia_hand side="right" parent="base">
-    <origin xyz="0 0.2 0.5" rpy="0 0 0"/>
+    <origin xyz="0 0.2 0.5" rpy="0 -1.57079 0"/>
   </xacro:sandia_hand>
   <xacro:sandia_hand side="left" parent="base">
-    <origin xyz="0 -0.2 0.5" rpy="0 0 0"/>
+    <origin xyz="0 -0.2 0.5" rpy="0 -1.57079 0"/>
   </xacro:sandia_hand>
 </robot>

File: ros/sandia_hand_utils/robots/sandia_hand_left.urdf.xacro (robot description, xacro)
@@ -25,5 +25,5 @@
   </link>
   <xacro:sandia_hand side="left" parent="base">
-    <origin xyz="0 0 0.5" rpy="0 0 0"/>
+    <origin xyz="0 0 0.5" rpy="0 -1.57079 0"/>
   </xacro:sandia_hand>
 </robot>

File: ros/sandia_hand_utils/robots/sandia_hand_right.urdf.xacro (robot description, xacro)
@@ -25,5 +25,5 @@
   </link>
   <xacro:sandia_hand side="right" parent="base">
-    <origin xyz="0 0 0.5" rpy="0 0 0"/>
+    <origin xyz="0 0 0.5" rpy="0 -1.57079 0"/>
   </xacro:sandia_hand>
 </robot>
