Commit message: reorganize irobot hand utils package

File: ros/irobot_hand_utils/urdf/sandia_hand.urdf (robot description, URDF)
Before this commit: robot armh_handle, 66 links, 65 joints
Links:
- link base_link: geometry collision mesh filename=package://irobot_hand/meshes/palm.stl
- link finger[0]/base_rotation_link: geometry collision mesh filename=package://irobot_hand/meshes/finger_base.stl; visual mesh filename=package://irobot_hand/meshes/finger_base.stl
- link finger[0]/distal_link: geometry collision mesh filename=package://irobot_hand/meshes/finger_distal.stl; visual mesh filename=package://irobot_hand/meshes/finger_distal.stl
- link finger[0]/flexible_link_1: geometry collision box size=.014 0.00176 .006; visual box size=.014 0.00176 .006
- link finger[0]/flexible_link_2: geometry collision box size=.014 0.00176 .006; visual box size=.014 0.00176 .006
- link finger[0]/flexible_link_3: geometry collision box size=.014 0.00176 .006; visual box size=.014 0.00176 .006
- link finger[0]/flexible_link_4: geometry collision box size=.014 0.00176 .006; visual box size=.014 0.00176 .006
- link finger[0]/flexible_link_5: geometry collision box size=.014 0.00176 .006; visual box size=.014 0.00176 .006
- link finger[0]/flexible_link_6: geometry collision box size=.014 0.00176 .006; visual box size=.014 0.00176 .006
- link finger[0]/flexible_link_7: geometry collision box size=.014 0.00176 .006; visual box size=.014 0.00176 .006
- link finger[0]/flexible_link_8: geometry collision box size=.014 0.00176 .006; visual box size=.014 0.00176 .006
- link finger[0]/flexible_link_9: geometry collision box size=.014 0.00176 .006; visual box size=.014 0.00176 .006
- link finger[0]/flexible_link_hidden_between_1_and_2: geometry collision box size=0 0 0; visual box size=0 0 0
- link finger[0]/flexible_link_hidden_between_2_and_3: geometry collision box size=0 0 0; visual box size=0 0 0
- link finger[0]/flexible_link_hidden_between_3_and_4: geometry collision box size=0 0 0; visual box size=0 0 0
- link finger[0]/flexible_link_hidden_between_4_and_5: geometry collision box size=0 0 0; visual box size=0 0 0
- link finger[0]/flexible_link_hidden_between_5_and_6: geometry collision box size=0 0 0; visual box size=0 0 0
- link finger[0]/flexible_link_hidden_between_6_and_7: geometry collision box size=0 0 0; visual box size=0 0 0
- link finger[0]/flexible_link_hidden_between_7_and_8: geometry collision box size=0 0 0; visual box size=0 0 0
- link finger[0]/flexible_link_hidden_between_8_and_9: geometry collision box size=0 0 0; visual box size=0 0 0
- link finger[0]/flexible_link_hidden_between_9_and_distal_link: geometry collision box size=0 0 0; visual box size=0 0 0
- link finger[0]/flexible_link_hidden_between_proximal_link_and_1: geometry collision box size=0 0 0; visual box size=0 0 0
- link finger[0]/proximal_link: geometry collision mesh filename=package://irobot_hand/meshes/finger_proximal.stl; visual mesh filename=package://irobot_hand/meshes/finger_proximal.stl
- link finger[1]/base_rotation_link: geometry collision mesh filename=package://irobot_hand/meshes/finger_base.stl; visual mesh filename=package://irobot_hand/meshes/finger_base.stl
- link finger[1]/distal_link: geometry collision mesh filename=package://irobot_hand/meshes/finger_distal.stl; visual mesh filename=package://irobot_hand/meshes/finger_distal.stl
- link finger[1]/flexible_link_1: geometry collision box size=.014 0.00176 .006; visual box size=.014 0.00176 .006
- link finger[1]/flexible_link_2: geometry collision box size=.014 0.00176 .006; visual box size=.014 0.00176 .006
- link finger[1]/flexible_link_3: geometry collision box size=.014 0.00176 .006; visual box size=.014 0.00176 .006
- link finger[1]/flexible_link_4: geometry collision box size=.014 0.00176 .006; visual box size=.014 0.00176 .006
- link finger[1]/flexible_link_5: geometry collision box size=.014 0.00176 .006; visual box size=.014 0.00176 .006
- link finger[1]/flexible_link_6: geometry collision box size=.014 0.00176 .006; visual box size=.014 0.00176 .006
- link finger[1]/flexible_link_7: geometry collision box size=.014 0.00176 .006; visual box size=.014 0.00176 .006
- link finger[1]/flexible_link_8: geometry collision box size=.014 0.00176 .006; visual box size=.014 0.00176 .006
- link finger[1]/flexible_link_9: geometry collision box size=.014 0.00176 .006; visual box size=.014 0.00176 .006
- link finger[1]/flexible_link_hidden_between_1_and_2: geometry collision box size=0 0 0; visual box size=0 0 0
- link finger[1]/flexible_link_hidden_between_2_and_3: geometry collision box size=0 0 0; visual box size=0 0 0
- link finger[1]/flexible_link_hidden_between_3_and_4: geometry collision box size=0 0 0; visual box size=0 0 0
- link finger[1]/flexible_link_hidden_between_4_and_5: geometry collision box size=0 0 0; visual box size=0 0 0
- link finger[1]/flexible_link_hidden_between_5_and_6: geometry collision box size=0 0 0; visual box size=0 0 0
- link finger[1]/flexible_link_hidden_between_6_and_7: geometry collision box size=0 0 0; visual box size=0 0 0
- link finger[1]/flexible_link_hidden_between_7_and_8: geometry collision box size=0 0 0; visual box size=0 0 0
- link finger[1]/flexible_link_hidden_between_8_and_9: geometry collision box size=0 0 0; visual box size=0 0 0
- link finger[1]/flexible_link_hidden_between_9_and_distal_link: geometry collision box size=0 0 0; visual box size=0 0 0
- link finger[1]/flexible_link_hidden_between_proximal_link_and_1: geometry collision box size=0 0 0; visual box size=0 0 0
- link finger[1]/proximal_link: geometry collision mesh filename=package://irobot_hand/meshes/finger_proximal.stl; visual mesh filename=package://irobot_hand/meshes/finger_proximal.stl
- link finger[2]/distal_link: geometry collision mesh filename=package://irobot_hand/meshes/finger_distal.stl; visual mesh filename=package://irobot_hand/meshes/finger_distal.stl
- link finger[2]/flexible_link_1: geometry collision box size=.014 0.00176 .006; visual box size=.014 0.00176 .006
- link finger[2]/flexible_link_2: geometry collision box size=.014 0.00176 .006; visual box size=.014 0.00176 .006
- link finger[2]/flexible_link_3: geometry collision box size=.014 0.00176 .006; visual box size=.014 0.00176 .006
- link finger[2]/flexible_link_4: geometry collision box size=.014 0.00176 .006; visual box size=.014 0.00176 .006
- link finger[2]/flexible_link_5: geometry collision box size=.014 0.00176 .006; visual box size=.014 0.00176 .006
- link finger[2]/flexible_link_6: geometry collision box size=.014 0.00176 .006; visual box size=.014 0.00176 .006
- link finger[2]/flexible_link_7: geometry collision box size=.014 0.00176 .006; visual box size=.014 0.00176 .006
- link finger[2]/flexible_link_8: geometry collision box size=.014 0.00176 .006; visual box size=.014 0.00176 .006
- link finger[2]/flexible_link_9: geometry collision box size=.014 0.00176 .006; visual box size=.014 0.00176 .006
- link finger[2]/flexible_link_hidden_between_1_and_2: geometry collision box size=0 0 0; visual box size=0 0 0
- link finger[2]/flexible_link_hidden_between_2_and_3: geometry collision box size=0 0 0; visual box size=0 0 0
- link finger[2]/flexible_link_hidden_between_3_and_4: geometry collision box size=0 0 0; visual box size=0 0 0
- link finger[2]/flexible_link_hidden_between_4_and_5: geometry collision box size=0 0 0; visual box size=0 0 0
- link finger[2]/flexible_link_hidden_between_5_and_6: geometry collision box size=0 0 0; visual box size=0 0 0
- link finger[2]/flexible_link_hidden_between_6_and_7: geometry collision box size=0 0 0; visual box size=0 0 0
- link finger[2]/flexible_link_hidden_between_7_and_8: geometry collision box size=0 0 0; visual box size=0 0 0
- link finger[2]/flexible_link_hidden_between_8_and_9: geometry collision box size=0 0 0; visual box size=0 0 0
- link finger[2]/flexible_link_hidden_between_9_and_distal_link: geometry collision box size=0 0 0; visual box size=0 0 0
- link finger[2]/flexible_link_hidden_between_proximal_link_and_1: geometry collision box size=0 0 0; visual box size=0 0 0
- link finger[2]/proximal_link: geometry collision mesh filename=package://irobot_hand/meshes/finger_proximal.stl; visual mesh filename=package://irobot_hand/meshes/finger_proximal.stl
