Commit message: add collisions to hand model

File: ros/irobot_hand_utils/robots/sandia_hand.urdf.xacro (robot description, xacro)
@@ -203,4 +203,13 @@
     <origin rpy="0 0 0" xyz="0 -0.038 -0.023"/>
   </collision>
+  <visual>
+    <geometry>
+      <mesh filename="package://irobot_hand/meshes/palm.stl"/>
+    </geometry>
+    <material name="darkgray">
+      <color rgba="0.2 0.2 0.2 1"/>
+    </material>
+    <origin rpy="0 0 0" xyz="0 -0.038 -0.023"/>
+  </visual>
 </link>
 <link name="finger[0]/base_rotation_link">

File: ros/irobot_hand_utils/urdf/sandia_hand.urdf (robot description, URDF)
Before this commit: robot armh_handle, 66 links, 65 joints
Links:
- link base_link: geometry collision mesh filename=package://irobot_hand/meshes/palm.stl; visual mesh filename=package://irobot_hand/meshes/palm.stl
