Commit message: update recover masses

File: ros/drc_robot_utils/robots/drc_robot_sandia_hands.model.xacro (robot description, xacro)
@@ -5,4 +5,11 @@
        name="drc_robot" >
   <include filename="$(find drc_robot_utils)/urdf/drc_robot.urdf" />
+  <include filename="$(find sandia_hand_utils)/urdf/sandia_hand.urdf.xacro" />
+  <xacro:sandia_hand side="r" parent="r_hand">
+    <origin xyz="0 -0.1 -0.03" rpy="0 3.1416  1.57079"/>
+  </xacro:sandia_hand>
+  <xacro:sandia_hand side="l" parent="l_hand">
+    <origin xyz="0  0.1 -0.03" rpy="0 3.1416 -1.57079"/>
+  </xacro:sandia_hand>
   <include filename="$(find drc_robot_utils)/urdf/drc_robot.gazebo" />
   <include filename="$(find drc_robot_utils)/urdf/drc_robot.transmission" />
