Commit message: renamed camhand to sandia_hand, and change references

File: ros/drc_robot_utils/robots/drc_robot.model.xacro (robot description, xacro)
@@ -5,11 +5,11 @@
        name="drc_robot" >
   <include filename="$(find drc_robot_utils)/urdf/drc_robot.urdf" />
-  <include filename="$(find camhand_utils)/urdf/camhand.urdf.xacro" />
-  <xacro:camhand side="r" parent="r_hand">
+  <include filename="$(find sandia_hand_utils)/urdf/sandia_hand.urdf.xacro" />
+  <xacro:sandia_hand side="r" parent="r_hand">
     <origin xyz="0 -0.1 -0.03" rpy="0 3.1416  1.57079"/>
-  </xacro:camhand>
-  <xacro:camhand side="l" parent="l_hand">
+  </xacro:sandia_hand>
+  <xacro:sandia_hand side="l" parent="l_hand">
     <origin xyz="0  0.1 -0.03" rpy="0 3.1416 -1.57079"/>
-  </xacro:camhand>
+  </xacro:sandia_hand>
   <include filename="$(find drc_robot_utils)/urdf/drc_robot.gazebo" />
   <include filename="$(find drc_robot_utils)/urdf/drc_robot.transmission" />

File: ros/drc_robot_utils/urdf/drc_robot.urdf (robot description, URDF)
Before this commit: robot drc_skeleton, 29 links, 28 joints
Joints:
- joint back_mby: origin xyz=0 0 0.14 rpy=0 -0 0 -> xyz=0 0 0.09 rpy=0 -0 0
- joint neck_ay: origin xyz=0.011 0 0.49 rpy=0 -0 0 -> xyz=0.011 0 0.44 rpy=0 -0 0

File: ros/sandia_hand_utils/robots/sandia_hand.urdf.xacro (robot description, xacro)
@@ -4,11 +4,11 @@
        xmlns:xacro="http://playerstage.sourceforge.net/gazebo/xmlschema/#interface"
        name="humanoid" >
-  <include filename="$(find camhand_utils)/urdf/camhand.urdf.xacro" />
+  <include filename="$(find sandia_hand_utils)/urdf/sandia_hand.urdf.xacro" />
   <link name="world"/>
-  <xacro:camhand side="right" parent="world">
+  <xacro:sandia_hand side="right" parent="world">
     <origin xyz="0 0 0" rpy="0 0 0"/>
-  </xacro:camhand>
-  <xacro:camhand side="left" parent="world">
+  </xacro:sandia_hand>
+  <xacro:sandia_hand side="left" parent="world">
     <origin xyz="0 1 0" rpy="0 0 0"/>
-  </xacro:camhand>
+  </xacro:sandia_hand>
 </robot>

File: ros/sandia_hand_utils/urdf/sandia_hand.gazebo.xacro (robot description, xacro)
@@ -1,6 +1,6 @@
 <?xml version="1.0"?>
-<robot name="camhand"
+<robot name="sandia_hand"
        xmlns:xacro="http://www.ros.org/wiki/xacro">
-  <xacro:macro name="camhand_gazebo" params="side">
+  <xacro:macro name="sandia_hand_gazebo" params="side">
     <gazebo>
       <plugin filename="libgazebo_ros_controller_manager.so" name="gazebo_ros_controller_manager">

File: ros/sandia_hand_utils/urdf/sandia_hand.transmission.xacro (robot description, xacro)
@@ -1,4 +1,4 @@
 <?xml version="1.0"?>
-<robot name="camhand"
+<robot name="sandia_hand"
        xmlns:xacro="http://www.ros.org/wiki/xacro">
   <xacro:macro name="finger_transmission" params="idx x y z r p yaw side">

File: ros/sandia_hand_utils/urdf/sandia_hand.urdf.xacro (robot description, xacro)
@@ -1,7 +1,7 @@
 <?xml version="1.0"?>
-<robot name="camhand"
+<robot name="sandia_hand"
        xmlns:xacro="http://www.ros.org/wiki/xacro">
-  <include filename="$(find camhand_utils)/urdf/camhand.gazebo.xacro" />
-  <include filename="$(find camhand_utils)/urdf/camhand.transmission.xacro" />
+  <include filename="$(find sandia_hand_utils)/urdf/sandia_hand.gazebo.xacro" />
+  <include filename="$(find sandia_hand_utils)/urdf/sandia_hand.transmission.xacro" />
   <xacro:macro name="finger" params="idx x y z r p yaw side">
     <link name="${side}_f${idx}_base">
@@ -31,5 +31,5 @@
         <origin xyz="0 0 0" rpy="0 0 0"/>
         <geometry>
-          <mesh filename="package://camhand/meshes/f0.stl"/>
+          <mesh filename="package://sandia_hand/meshes/f0.stl"/>
         </geometry>
       </collision>
@@ -37,7 +37,7 @@
         <origin xyz="0 0 0" rpy="0 0 0"/>
         <geometry>
-          <mesh filename="package://camhand/meshes/f0.stl"/>
+          <mesh filename="package://sandia_hand/meshes/f0.stl"/>
         </geometry>
-        <material name="${side}_camhand_skin_suntan">
+        <material name="${side}_sandia_hand_skin_suntan">
           <color rgba="0.7 0.4 0.2 1.0"/>
         </material>
@@ -54,5 +54,5 @@
         <origin xyz="0 0 0" rpy="0 0 0"/>
         <geometry>
-          <mesh filename="package://camhand/meshes/f1.stl"/>
+          <mesh filename="package://sandia_hand/meshes/f1.stl"/>
         </geometry>
       </collision>
@@ -60,7 +60,7 @@
         <origin xyz="0 0 0" rpy="0 0 0"/>
         <geometry>
-          <mesh filename="package://camhand/meshes/f1.stl"/>
+          <mesh filename="package://sandia_hand/meshes/f1.stl"/>
         </geometry>
-        <material name="${side}_camhand_skin">
+        <material name="${side}_sandia_hand_skin">
           <color rgba="0.835 0.655 0.345 1.0"/>
         </material>
@@ -85,5 +85,5 @@
         <origin xyz="0 0 0" rpy="0 0 0"/>
         <geometry>
-          <mesh filename="package://camhand/meshes/f2.stl"/>
+          <mesh filename="package://sandia_hand/meshes/f2.stl"/>
         </geometry>
       </collision>
@@ -91,7 +91,7 @@
         <origin xyz="0 0 0" rpy="0 0 0"/>
         <geometry>
-          <mesh filename="package://camhand/meshes/f2.stl"/>
+          <mesh filename="package://sandia_hand/meshes/f2.stl"/>
         </geometry>
-        <material name="${side}_camhand_skin_suntan">
+        <material name="${side}_sandia_hand_skin_suntan">
           <color rgba="0.8 0.6 0.3 1.0"/>
         </material>
@@ -155,5 +155,5 @@
     <xacro:finger_transmission side="${side}" idx="${idx}" x="${x}" y="${y}" z="${z}" r="${r}" p="${p}" yaw="${yaw}"/>
   </xacro:macro>
-  <xacro:macro name="camhand" params="side parent *origin">
+  <xacro:macro name="sandia_hand" params="side parent *origin">
     <link name="${side}_palm">
       <origin xyz="0 0 0" rpy="0 0 0"/>
@@ -166,5 +166,5 @@
         <origin xyz="0 0 0" rpy="0 0 0"/>
         <geometry>
-          <mesh filename="package://camhand/meshes/palm.stl"/>
+          <mesh filename="package://sandia_hand/meshes/palm.stl"/>
         </geometry>
       </collision>
@@ -172,12 +172,12 @@
         <origin xyz="0 0 0" rpy="0 0 0"/>
         <geometry>
-          <mesh filename="package://camhand/meshes/palm.stl"/>
+          <mesh filename="package://sandia_hand/meshes/palm.stl"/>
         </geometry>
-        <material name="${side}_camhand_skin">
+        <material name="${side}_sandia_hand_skin">
           <color rgba="0.835 0.655 0.345 1.0"/>
         </material>
       </visual>
     </link>
-    <joint name="${side}_camhand_joint" type="fixed">
+    <joint name="${side}_sandia_hand_joint" type="fixed">
       <parent link="${parent}"/>
       <child link="${side}_palm"/>
@@ -189,5 +189,5 @@
     <xacro:finger side="${side}" idx="3" x="0.03995" y="-0.04383" z="0.014" r="0" p="-1.57079" yaw="-2.3562"/>
     <!-- not needed unless simulating the hand by itself
-    <xacro:camhand_gazebo side="${side}" />
+    <xacro:sandia_hand_gazebo side="${side}" />
     -->
   </xacro:macro>

Commit message: Merge with default

File: ros/drc_robot_utils/robots/drc_robot.model.xacro (robot description, xacro)
@@ -5,11 +5,4 @@
        name="drc_robot" >
   <include filename="$(find drc_robot_utils)/urdf/drc_robot.urdf" />
-  <include filename="$(find sandia_hand_utils)/urdf/sandia_hand.urdf.xacro" />
-  <xacro:sandia_hand side="r" parent="r_hand">
-    <origin xyz="0 -0.1 -0.03" rpy="0 3.1416  1.57079"/>
-  </xacro:sandia_hand>
-  <xacro:sandia_hand side="l" parent="l_hand">
-    <origin xyz="0  0.1 -0.03" rpy="0 3.1416 -1.57079"/>
-  </xacro:sandia_hand>
   <include filename="$(find drc_robot_utils)/urdf/drc_robot.gazebo" />
   <include filename="$(find drc_robot_utils)/urdf/drc_robot.transmission" />

File: ros/drc_robot_utils/urdf/drc_robot.urdf (robot description, URDF)
Before this commit: robot drc_skeleton, 29 links, 28 joints
Joints:
- joint back_ubx: limit lower=-0.790809 upper=0 effort=94.91 velocity=12 -> lower=-0.790809 upper=0.790809 effort=94.91 velocity=12
- joint l_arm_mwx: origin xyz=0 0.095 0 rpy=0 -0 0 -> xyz=0 0.058 0 rpy=0 -0 0
- joint l_arm_usy: axis 0 -0.5 0.866025 -> 0 0.5 0.866025
- joint l_arm_uwy: origin xyz=0 0.183 -0.013 rpy=0 -0 0 -> xyz=0 0.188 -0.013 rpy=0 -0 0
- joint r_arm_mwx: origin xyz=0 -0.095 0 rpy=0 -0 0 -> xyz=0 -0.058 0 rpy=0 -0 0
- joint r_arm_usy: axis 0 0.5 0.866025 -> 0 -0.5 0.866025
- joint r_arm_uwy: origin xyz=0 -0.183 -0.013 rpy=0 -0 0 -> xyz=0 -0.188 -0.013 rpy=0 -0 0
