Commit message: update offsets based on newest specs

File: models/drc_robot/model.urdf (robot description, URDF)
Before this commit: robot drc_robot, 40 links, 39 joints
Joints:
- joint center_bottom_led_frame_joint: origin xyz=0.00585 0.0 -0.016 -> xyz=0.01125 0.0 -0.0155
- joint center_top_led_frame_joint: origin xyz=0.00585 0.0 0.01 -> xyz=0.01125 0.0 0.0105
- joint hokuyo_joint: origin xyz=-0.050 0 0.0875 rpy=0 0 0 -> xyz=-0.0446 0 0.0880 rpy=0 0 0
- joint left_camera_frame_joint: origin xyz=0.00585 0.035 -0.0025 -> xyz=0.01125 0.035 -0.002
- joint left_led_frame_joint: origin xyz=-0.01983 0.07452 0.049846 rpy=0 -0.15 0.53 -> xyz=-0.01443 0.07452 0.050346 rpy=0 -0.15 0.53
- joint neck_ay: origin xyz=0.011 0 0.48 rpy=0 0 0 -> xyz=0.16555 0 0.50823 rpy=0 0 0
- joint right_camera_frame_joint: origin xyz=0.00585 -0.035 -0.0025 -> xyz=0.01125 -0.035 -0.002
- joint right_led_frame_joint: origin xyz=-0.01983 -0.07452 0.049846 rpy=0 -0.15 -0.53 -> xyz=-0.01443 -0.07452 0.050346 rpy=0 -0.15 -0.53

Commit message: update head nodding range of motion (joint limits) based on new slides

File: models/drc_robot/model.urdf (robot description, URDF)
Before this commit: robot drc_robot, 40 links, 39 joints
Joints:
- joint neck_ay: limit lower=-0.436332313 upper=1.13446401 effort=5 velocity=12 -> lower=-0.610865238 upper=1.13446401 effort=5 velocity=12

Commit message: update camera optical frame location to collocate with head tilt dof

File: models/drc_robot/model.urdf (robot description, URDF)
Before this commit: robot drc_robot, 40 links, 39 joints
Joints:
- joint left_camera_frame_joint: origin xyz=0.01125 0.035 -0.002 -> xyz=0.0 0.035 -0.002
- joint right_camera_frame_joint: origin xyz=0.01125 -0.035 -0.002 -> xyz=0.0 -0.035 -0.002

Commit message: merging from default

File: models/drc_robot/model.urdf (robot description, URDF)
Before this commit: robot drc_robot, 35 links, 34 joints
Links:
- added link center_bottom_led_frame, mass 0.1
- added link center_top_led_frame, mass 0.1
- added link hokuyo_link, mass 0.057664; collision mesh filename=package://multisense_sl/meshes/hokuyo_link.STL; visual mesh filename=package://multisense_sl/meshes/hokuyo_link.STL
- added link left_led_frame, mass 0.1
- added link right_led_frame, mass 0.1
- link head: mass 2.6 -> 1.4199; geometry collision mesh filename=package://multisense_sl/meshes/base_link.STL; visual mesh filename=package://multisense_sl/meshes/base_link.STL
- link head_hokuyo: mass 0.1 -> 0.01
Joints:
- added joint center_bottom_led_frame_joint: type fixed, parent head, child center_bottom_led_frame, origin xyz=0.01125 0.0 -0.0155
- added joint center_top_led_frame_joint: type fixed, parent head, child center_top_led_frame, origin xyz=0.01125 0.0 0.0105
- added joint hokuyo_joint: type continuous, parent head, child hokuyo_link, origin xyz=-0.0446 0 0.0880 rpy=0 0 0, axis 1 0 0
- added joint left_led_frame_joint: type fixed, parent head, child left_led_frame, origin xyz=-0.01443 0.07452 0.050346 rpy=0 -0.15 0.53
- added joint right_led_frame_joint: type fixed, parent head, child right_led_frame, origin xyz=-0.01443 -0.07452 0.050346 rpy=0 -0.15 -0.53
- joint head_hokuyo_joint: origin xyz=0.03 0 0.13 rpy=0 0 0 -> xyz=0.03 0 0.015 rpy=0 0 0; parent head -> hokuyo_link
- joint imu_joint: origin xyz=0 0 0 rpy=0 0 0 -> xyz=0 0 0 rpy=0.05991527603 0 -0.01415; parent ltorso -> pelvis
- joint left_camera_frame_joint: origin xyz=0.03 0.1 0.1 -> xyz=0.0 0.035 -0.002
- joint neck_ay: limit lower=-0.785398 upper=0.785398 effort=5 velocity=12 -> lower=-0.610865238 upper=1.13446401 effort=5 velocity=12; origin xyz=0.011 0 0.44 rpy=0 -0 0 -> xyz=0.16555 0 0.50823 rpy=0 0 0
- joint right_camera_frame_joint: origin xyz=0.03 -0.1 0.1 -> xyz=0.0 -0.035 -0.002

File: models/drc_robot_irobot_hand/model.urdf (robot description, URDF)
Before this commit: robot drc_robot, 101 links, 100 joints
Joints:
- joint imu_joint: origin xyz=0 0 0 rpy=0 0 0 -> xyz=0 0 0 rpy=0.05991527603 0 -0.01415; parent ltorso -> pelvis

File: models/drc_robot_sandia_hand/model.urdf (robot description, URDF)
Before this commit: robot drc_robot, 93 links, 92 joints
Joints:
- joint imu_joint: origin xyz=0 0 0 rpy=0 0 0 -> xyz=0 0 0 rpy=0.05991527603 0 -0.01415; parent ltorso -> pelvis

Commit message: make imu_joint non-fixed to prevent lumping by fixed joint reduction.  added provideFeedback tags for arm_mwx

File: models/drc_robot/model.urdf (robot description, URDF)
Before this commit: robot drc_robot, 40 links, 39 joints
Joints:
- joint imu_joint: axis (none) -> 0 0 1; limit (none) -> lower=0 upper=0 effort=0 velocity=0; type fixed -> revolute

Commit message: merging from vrc

File: models/drc_robot/model.urdf (robot description, URDF)
Before this commit: robot drc_robot, 35 links, 34 joints
Links:
- added link center_bottom_led_frame, mass 0.1
- added link center_top_led_frame, mass 0.1
- added link hokuyo_link, mass 0.057664; collision mesh filename=package://multisense_sl/meshes/hokuyo_link.STL; visual mesh filename=package://multisense_sl/meshes/hokuyo_link.STL
- added link left_led_frame, mass 0.1
- added link right_led_frame, mass 0.1
- link head: mass 2.6 -> 1.4199; geometry collision mesh filename=package://multisense_sl/meshes/base_link.STL; visual mesh filename=package://multisense_sl/meshes/base_link.STL
- link head_hokuyo: mass 0.1 -> 0.01
Joints:
- added joint center_bottom_led_frame_joint: type fixed, parent head, child center_bottom_led_frame, origin xyz=0.01125 0.0 -0.0155
- added joint center_top_led_frame_joint: type fixed, parent head, child center_top_led_frame, origin xyz=0.01125 0.0 0.0105
- added joint hokuyo_joint: type continuous, parent head, child hokuyo_link, origin xyz=-0.0446 0 0.0880 rpy=0 0 0, axis 1 0 0
- added joint left_led_frame_joint: type fixed, parent head, child left_led_frame, origin xyz=-0.01443 0.07452 0.050346 rpy=0 -0.15 0.53
- added joint right_led_frame_joint: type fixed, parent head, child right_led_frame, origin xyz=-0.01443 -0.07452 0.050346 rpy=0 -0.15 -0.53
- joint head_hokuyo_joint: origin xyz=0.03 0 0.13 rpy=0 0 0 -> xyz=0.03 0 0.015 rpy=0 0 0; parent head -> hokuyo_link
- joint imu_joint: axis (none) -> 0 0 1; limit (none) -> lower=0 upper=0 effort=0 velocity=0; origin xyz=0 0 0 rpy=0 0 0 -> xyz=0 0 0 rpy=0.05991527603 0 -0.01415; parent ltorso -> pelvis; type fixed -> revolute
- joint left_camera_frame_joint: origin xyz=0.03 0.1 0.1 -> xyz=0.0 0.035 -0.002
- joint neck_ay: limit lower=-0.785398 upper=0.785398 effort=5 velocity=12 -> lower=-0.610865238 upper=1.13446401 effort=5 velocity=12; origin xyz=0.011 0 0.44 rpy=0 -0 0 -> xyz=0.16555 0 0.50823 rpy=0 0 0
- joint right_camera_frame_joint: origin xyz=0.03 -0.1 0.1 -> xyz=0.0 -0.035 -0.002

Commit message: fix for issue #68

File: models/drc_robot/model.urdf (robot description, URDF)
Before this commit: robot drc_robot, 40 links, 39 joints
Joints:
- joint r_arm_usy: axis 0 -0.5 0.866025 -> 0 0.5 -0.866025

File: models/drc_robot_irobot_hand/model.urdf (robot description, URDF)
Before this commit: robot drc_robot, 101 links, 100 joints
Joints:
- joint r_arm_usy: axis 0 -0.5 0.866025 -> 0 0.5 -0.866025

File: models/drc_robot_sandia_hand/model.urdf (robot description, URDF)
Before this commit: robot drc_robot, 93 links, 92 joints
Joints:
- joint r_arm_usy: axis 0 -0.5 0.866025 -> 0 0.5 -0.866025

File: ros/drc_robot_utils/urdf/drc_robot.urdf (robot description, URDF)
Before this commit: robot drc_skeleton, 29 links, 28 joints
Joints:
- joint r_arm_usy: axis 0 -0.5 0.866025 -> 0 0.5 -0.866025
