Commit message: merging and changing launch files to reflect model.sdf to model.urdf name change

File: models/drc_robot_irobot_hand/model.urdf (robot description, URDF)
Before this commit: robot drc_robot, 101 links, 100 joints
Joints:
- joint imu_joint: origin xyz=0 0 0 rpy=0 0 0 -> xyz=0 0 0 rpy=0.05991527603 0 -0.01415; parent ltorso -> pelvis

File: models/drc_robot_sandia_hand/model.urdf (robot description, URDF)
Before this commit: robot drc_robot, 93 links, 92 joints
Joints:
- joint imu_joint: origin xyz=0 0 0 rpy=0 0 0 -> xyz=0 0 0 rpy=0.05991527603 0 -0.01415; parent ltorso -> pelvis

Commit message: Pushed changes to other models and upstream sources

File: models/drc_robot_irobot_hand/model.urdf (robot description, URDF)
Before this commit: robot drc_robot, 101 links, 100 joints
Joints:
- joint imu_joint: origin xyz=0 0 0 rpy=0.05991527603 0 -0.01415 -> xyz=0.05991527603 0 -0.01415 rpy=0 0 0

File: models/drc_robot_sandia_hand/model.urdf (robot description, URDF)
Before this commit: robot drc_robot, 93 links, 92 joints
Joints:
- joint imu_joint: origin xyz=0 0 0 rpy=0.05991527603 0 -0.01415 -> xyz=0.05991527603 0 -0.01415 rpy=0 0 0

Commit message: Partial propagation of drc_robot model changes

File: models/drc_robot_irobot_hand/model.urdf (robot description, URDF)
Before this commit: robot drc_robot, 101 links, 100 joints
Joints:
- joint imu_joint: axis (none) -> 0 0 1; limit (none) -> lower=0 upper=0 effort=0 velocity=0; type fixed -> revolute

File: models/drc_robot_sandia_hand/model.urdf (robot description, URDF)
Before this commit: robot drc_robot, 93 links, 92 joints
Joints:
- joint imu_joint: axis (none) -> 0 0 1; limit (none) -> lower=0 upper=0 effort=0 velocity=0; type fixed -> revolute
