Commit message: atlas simple collision corrections

File: models/atlas/model_simple_collision.urdf (robot description, URDF)
Before this commit: robot atlas, 40 links, 39 joints
Links:
- link l_foot: geometry collision box size=0.26 0.124887 0.01; visual mesh filename=package://atlas/meshes/l_foot.dae scale=1 1 1
- link r_foot: geometry collision box size=0.26 0.124887 0.01; visual mesh filename=package://atlas/meshes/r_foot.dae scale=1 1 1

Commit message: hide some internal parts.  fix head collision.

File: models/atlas/model_simple_collision.urdf (robot description, URDF)
Before this commit: robot atlas, 40 links, 39 joints
Links:
- link head: geometry collision box size=0.0468 0.12 0.1184; collision box size=0.1311 0.12 0.0591
- link hokuyo_link: geometry collision box size=0.08 0.06 0.04238; collision cylinder length=0.047 radius=0.024425
- link ltorso: geometry visual mesh filename=package://atlas/meshes/ltorso.dae scale=1 1 1
- link utorso: geometry collision box size=0.3188 0.24 0.3662; collision cylinder length=0.22375 radius=0.0363
