Commit message: clean up

File: models/atlas/model.urdf (robot description, URDF)
Before this commit: robot atlas, 40 links, 39 joints
Links:
- link head: geometry collision box size=0.0468 0.12 0.1184; collision box size=0.1311 0.12 0.0591
- link hokuyo_link: geometry collision box size=0.08 0.06 0.04238; collision cylinder length=0.047 radius=0.024425
- link l_clav: geometry collision cylinder length=0.027 radius=0.04; collision cylinder length=0.1525 radius=0.045
- link l_farm: geometry collision cylinder length=0.035181 radius=0.0458825; collision cylinder length=0.050472 radius=0.0279
- link l_foot: geometry collision box size=0.26 0.124887 0.01; visual mesh filename=package://atlas/meshes/l_foot.dae scale=1 1 1
- link l_hand: geometry collision cylinder length=0.019 radius=0.035939; collision cylinder length=0.019 radius=0.035939
- link l_larm: geometry collision cylinder length=0.0161 radius=0.045; collision cylinder length=0.0161 radius=0.045
- link l_lglut: geometry collision cylinder length=0.060306 radius=0.02009687; collision cylinder length=0.12 radius=0.02
- link l_lleg: geometry collision box size=0.1465 0.1205 0.476; visual mesh filename=package://atlas/meshes/l_lleg.dae scale=1 1 1
- link l_scap: geometry collision cylinder length=0.013737 radius=0.048709; collision cylinder length=0.013937 radius=0.048709
- link l_talus: geometry collision cylinder length=0.010059 radius=0.010348; collision cylinder length=0.029542 radius=0.010181
- link l_uarm: geometry collision cylinder length=0.088934 radius=0.04504847; collision cylinder length=0.116677 radius=0.0449
- link l_uglut: geometry collision cylinder length=0.078396 radius=0.019096; collision cylinder length=0.080842 radius=0.019841
- link l_uleg: geometry collision box size=0.2 0.1865 0.26; visual mesh filename=package://atlas/meshes/l_uleg.dae scale=1 1 1
- link ltorso: geometry visual mesh filename=package://atlas/meshes/ltorso.dae scale=1 1 1
- link mtorso: geometry collision cylinder length=0.02 radius=0.015; collision cylinder length=0.02 radius=0.015
- link pelvis: geometry collision cylinder length=0.07 radius=0.130; collision cylinder length=0.07 radius=0.130
- link r_clav: geometry collision cylinder length=0.027 radius=0.04; collision cylinder length=0.1525 radius=0.045
- link r_farm: geometry collision cylinder length=0.035181 radius=0.0458825; collision cylinder length=0.050472 radius=0.0279
- link r_foot: geometry collision box size=0.26 0.124887 0.01; visual mesh filename=package://atlas/meshes/r_foot.dae scale=1 1 1
- link r_hand: geometry collision cylinder length=0.019 radius=0.035939; collision cylinder length=0.019 radius=0.035939
- link r_larm: geometry collision cylinder length=0.0161 radius=0.045; collision cylinder length=0.0161 radius=0.045
- link r_lglut: geometry collision cylinder length=0.060306 radius=0.02009687; collision cylinder length=0.12 radius=0.02
- link r_lleg: geometry collision box size=0.1465 0.1205 0.476; visual mesh filename=package://atlas/meshes/r_lleg.dae scale=1 1 1
- link r_scap: geometry collision cylinder length=0.013737 radius=0.048709; collision cylinder length=0.013937 radius=0.048709
- link r_talus: geometry collision cylinder length=0.010059 radius=0.010348; collision cylinder length=0.029542 radius=0.010181
- link r_uarm: geometry collision cylinder length=0.088934 radius=0.04504847; collision cylinder length=0.116677 radius=0.0449
- link r_uglut: geometry collision cylinder length=0.078396 radius=0.019096; collision cylinder length=0.080842 radius=0.019841
- link r_uleg: geometry collision box size=0.2 0.1865 0.26; visual mesh filename=package://atlas/meshes/r_uleg.dae scale=1 1 1
- link utorso: geometry collision box size=0.3188 0.24 0.3662; collision cylinder length=0.22375 radius=0.0363
