Commit message: Manually synchronize atlas xacro files with downstream model.urdf

File: ros/atlas_utils/urdf/atlas.urdf (robot description, URDF)
Before this commit: robot drc_skeleton, 29 links, 28 joints
Links:
- added link center_bottom_led_frame, mass 0.1
- added link center_top_led_frame, mass 0.1
- added link hokuyo_link, mass 0.057664; collision mesh filename=package://multisense_sl/meshes/hokuyo_link.STL; visual mesh filename=package://multisense_sl/meshes/hokuyo_link.STL
- added link left_led_frame, mass 0.1
- added link right_led_frame, mass 0.1
- link head: mass 2.6 -> 1.4199; geometry collision mesh filename=package://multisense_sl/meshes/base_link.STL; visual mesh filename=package://multisense_sl/meshes/base_link.STL
Joints:
- added joint center_bottom_led_frame_joint: type fixed, parent head, child center_bottom_led_frame, origin xyz=0.01125 0.0 -0.0155
- added joint center_top_led_frame_joint: type fixed, parent head, child center_top_led_frame, origin xyz=0.01125 0.0 0.0105
- added joint hokuyo_joint: type continuous, parent head, child hokuyo_link, origin xyz=-0.0446 0 0.0880 rpy=0 0 0, axis 1 0 0
- added joint left_led_frame_joint: type fixed, parent head, child left_led_frame, origin xyz=-0.01443 0.07452 0.050346 rpy=0 -0.15 0.53
- added joint right_led_frame_joint: type fixed, parent head, child right_led_frame, origin xyz=-0.01443 -0.07452 0.050346 rpy=0 -0.15 -0.53
- joint neck_ay: limit lower=-0.785398 upper=0.785398 effort=5 velocity=12 -> lower=-0.610865238 upper=1.13446401 effort=5 velocity=12; origin xyz=0.011 0 0.44 rpy=0 -0 0 -> xyz=0.16555 0 0.50823 rpy=0 0 0

Commit message: propagate model.urdf upstream into xacro files

File: ros/atlas_utils/urdf/atlas.urdf (robot description, URDF)
Before this commit: robot drc_skeleton, 29 links, 28 joints
Links:
- added link hokuyo_link, mass 0.057664; collision mesh filename=package://multisense_sl/meshes/hokuyo_link.STL; visual mesh filename=package://multisense_sl/meshes/hokuyo_link.STL
- link head: mass 2.6 -> 1.4199; geometry collision mesh filename=package://multisense_sl/meshes/base_link.STL; visual mesh filename=package://multisense_sl/meshes/base_link.STL
Joints:
- added joint hokuyo_joint: type continuous, parent head, child hokuyo_link, origin xyz=-0.0446 0 0.0880 rpy=0 0 0, axis 1 0 0
- joint neck_ay: limit lower=-0.785398 upper=0.785398 effort=5 velocity=12 -> lower=-0.610865238 upper=1.13446401 effort=5 velocity=12; origin xyz=0.011 0 0.44 rpy=0 -0 0 -> xyz=0.16555 0 0.50823 rpy=0 -0 0
