Commit message: Changed pose offsets for entering drc_vehicle

File: ros/atlas_description/robots/atlas_sandia_hands.urdf.xacro (robot description, xacro)
@@ -3,8 +3,8 @@
   <include filename="$(find sandia_hand_description)/urdf/sandia_hand_simple_shapes.urdf.xacro" />
   <xacro:sandia_hand side="right" parent="r_hand" reflect="1">
-    <origin xyz="0 -0.1 -0.03" rpy="0 3.1416  1.57079"/>
+    <origin xyz="0 -0.1 -0.03" rpy="-1.57079 0 -1.57079"/>
   </xacro:sandia_hand>
   <xacro:sandia_hand side="left" parent="l_hand" reflect="-1">
-    <origin xyz="0  0.1 -0.03" rpy="0 3.1416 -1.57079"/>
+    <origin xyz="0  0.1 -0.03" rpy=" 1.57079 0  1.57079"/>
   </xacro:sandia_hand>
   <include filename="$(find atlas_description)/urdf/atlas.gazebo" />

Commit message: Fixed wrist offset for sandia hands

File: ros/atlas_description/robots/atlas_sandia_hands.urdf.xacro (robot description, xacro)
@@ -3,8 +3,8 @@
   <include filename="$(find sandia_hand_description)/urdf/sandia_hand_simple_shapes.urdf.xacro" />
   <xacro:sandia_hand side="right" parent="r_hand" reflect="1">
-    <origin xyz="0 -0.1 -0.03" rpy="-1.57079 0 -1.57079"/>
+    <origin xyz="0 -0.1 0" rpy="-1.57079 0 -1.57079"/>
   </xacro:sandia_hand>
   <xacro:sandia_hand side="left" parent="l_hand" reflect="-1">
-    <origin xyz="0  0.1 -0.03" rpy=" 1.57079 0  1.57079"/>
+    <origin xyz="0  0.1 0" rpy=" 1.57079 0  1.57079"/>
   </xacro:sandia_hand>
   <include filename="$(find atlas_description)/urdf/atlas.gazebo" />
