Commit message: propagate bug fixes in atlas_simple_shapes.urdf to atlas.urdf.  test with atlas.urdf.

File: ros/atlas_description/robots/atlas.urdf.xacro (robot description, xacro)
@@ -1,4 +1,4 @@
 <robot name="atlas" >
-  <include filename="$(find atlas_description)/urdf/atlas_simple_shapes.urdf" />
+  <include filename="$(find atlas_description)/urdf/atlas.urdf" />
   <include filename="$(find atlas_description)/urdf/atlas.gazebo" />
   <include filename="$(find atlas_description)/urdf/atlas.transmission" />

File: ros/atlas_description/robots/atlas_sandia_hands.urdf.xacro (robot description, xacro)
@@ -1,4 +1,4 @@
 <robot xmlns:xacro="http://playerstage.sourceforge.net/gazebo/xmlschema/#interface" name="atlas" >
-  <include filename="$(find atlas_description)/urdf/atlas_simple_shapes.urdf" />
+  <include filename="$(find atlas_description)/urdf/atlas.urdf" />
   <include filename="$(find sandia_hand_description)/urdf/sandia_hand_simple_shapes.urdf.xacro" />
   <xacro:sandia_hand side="right" parent="r_hand" reflect="1" joint_type="revolute" thumb_angle="0">

File: ros/atlas_description/urdf/atlas.urdf (robot description, URDF)
Before this commit: robot drc_skeleton, 28 links, 28 joints
Links:
- link l_lleg: geometry collision mesh filename=package://atlas/meshes/l_lleg.stl scale=1 1 1; visual mesh filename=package://atlas/meshes/l_lleg.dae scale=1.0 1.0 1.0
- link pelvis: geometry collision mesh filename=package://atlas/meshes/pelvis.stl scale=1 1 1; visual mesh filename=package://atlas/meshes/pelvis.dae scale=1.0 1.0 1.0
- link r_larm: geometry collision mesh filename=package://atlas/meshes/r_larm.stl scale=1 1 1; visual mesh filename=package://atlas/meshes/r_larm.dae scale=1.0 1.0 1.0
- link r_lglut: geometry collision mesh filename=package://atlas/meshes/r_lglut.stl scale=1 1 1; visual mesh filename=package://atlas/meshes/r_lglut.dae scale=1.0 1.0 1.0
- link r_lleg: geometry collision mesh filename=package://atlas/meshes/r_lleg.stl scale=1 1 1; visual mesh filename=package://atlas/meshes/r_lleg.dae scale=1.0 1.0 1.0
- link r_uarm: geometry collision mesh filename=package://atlas/meshes/r_uarm.stl scale=1 1 1; visual mesh filename=package://atlas/meshes/r_uarm.dae scale=1.0 1.0 1.0
- link r_uglut: geometry collision mesh filename=package://atlas/meshes/r_uglut.stl scale=1 1 1; visual mesh filename=package://atlas/meshes/r_uglut.dae scale=1.0 1.0 1.0
- link r_uleg: geometry collision mesh filename=package://atlas/meshes/r_uleg.stl scale=1 1 1; visual mesh filename=package://atlas/meshes/r_uleg.dae scale=1.0 1.0 1.0
Joints:
- joint l_leg_kny: limit lower=0 upper=2.45 effort=220 velocity=12 -> lower=0 upper=2.45 effort=400 velocity=12
- joint l_leg_uay: limit lower=-0.698 upper=0.698 effort=220 velocity=12 -> lower=-0.9 upper=0.698 effort=220 velocity=12
- joint neck_ay: origin xyz=0.16555 0 0.50823 rpy=0 -0 0 -> xyz=0.21672 0 0.53796 rpy=0 -0 0
- joint r_leg_kny: limit lower=0 upper=2.45 effort=220 velocity=12 -> lower=0 upper=2.45 effort=400 velocity=12
- joint r_leg_uay: limit lower=-0.698 upper=0.698 effort=220 velocity=12 -> lower=-0.9 upper=0.698 effort=220 velocity=12

Commit message: revert inertia from original urdf.  revert to simple shape collision geometries.

File: ros/atlas_description/robots/atlas.urdf.xacro (robot description, xacro)
@@ -1,4 +1,4 @@
 <robot name="atlas" >
-  <include filename="$(find atlas_description)/urdf/atlas.urdf" />
+  <include filename="$(find atlas_description)/urdf/atlas_simple_shapes.urdf" />
   <include filename="$(find atlas_description)/urdf/atlas.gazebo" />
   <include filename="$(find atlas_description)/urdf/atlas.transmission" />

File: ros/atlas_description/robots/atlas_sandia_hands.urdf.xacro (robot description, xacro)
@@ -1,4 +1,4 @@
 <robot xmlns:xacro="http://playerstage.sourceforge.net/gazebo/xmlschema/#interface" name="atlas" >
-  <include filename="$(find atlas_description)/urdf/atlas.urdf" />
+  <include filename="$(find atlas_description)/urdf/atlas_simple_shapes.urdf" />
   <include filename="$(find sandia_hand_description)/urdf/sandia_hand_simple_shapes.urdf.xacro" />
   <xacro:sandia_hand side="right" parent="r_hand" reflect="1" joint_type="revolute" thumb_angle="0">

File: ros/atlas_description/urdf/atlas.urdf (robot description, URDF)
Before this commit: robot drc_skeleton, 28 links, 28 joints
Links:
- link l_uleg: geometry collision mesh filename=package://atlas/meshes/l_uleg.stl scale=1 1 1; visual mesh filename=package://atlas/meshes/l_uleg.dae scale=1.0 1.0 1.0

File: ros/atlas_description/urdf/atlas_simple_shapes.urdf (robot description, URDF)
Before this commit: robot drc_skeleton, 28 links, 28 joints
Links:
- link l_foot: mass 0.867 -> 1.634
- link l_lglut: mass 0.803 -> 0.69
- link l_talus: mass 0.867 -> 0.1
- link l_uglut: mass 1.51622 -> 0.5166
- link l_uleg: mass 7.227 -> 7.34
- link ltorso: mass 1.62729 -> 1.92
- link mtorso: mass 3.8068 -> 0.55
- link pelvis: mass 12.54638 -> 14.2529
- link r_foot: mass 0.867 -> 1.634
- link r_lglut: mass 0.803 -> 0.69
- link r_talus: mass 0.867 -> 0.1
- link r_uglut: mass 1.51622 -> 0.5166
- link r_uleg: mass 7.227 -> 7.34
- link utorso: mass 15.2272 -> 18.484
