Commit message: align hand to end of atlas arms by flipping x and z.

File: ros/atlas_description/robots/atlas_v3_sandia_hands.urdf.xacro (robot description, xacro)
@@ -3,8 +3,8 @@
   <xacro:include filename="$(find sandia_hand_description)/urdf/sandia_hand_simple_shapes.urdf.xacro" />
   <xacro:sandia_hand side="right" parent="r_hand" reflect="1" joint_type="revolute" thumb_angle="0">
-    <origin xyz="0.00179 -0.13516 -0.01176" rpy="0 0 -1.57079"/>
+    <origin xyz="-0.00179 -0.13516 0.01176" rpy="0 0 -1.57079"/>
   </xacro:sandia_hand>
   <xacro:sandia_hand side="left" parent="l_hand" reflect="-1" joint_type="revolute" thumb_angle="0">
-    <origin xyz="-0.00179  0.13516 -0.01176" rpy="3.14159 0  1.57079"/>
+    <origin xyz="0.00179  0.13516 0.01176" rpy="3.14159 0  1.57079"/>
   </xacro:sandia_hand>
   <xacro:include filename="$(find atlas_description)/urdf/atlas_v3.gazebo" />

File: ros/atlas_description/robots/atlas_v3_with_v1_inertia_sandia_hands.urdf.xacro (robot description, xacro)
@@ -3,8 +3,8 @@
   <xacro:include filename="$(find sandia_hand_description)/urdf/sandia_hand_simple_shapes.urdf.xacro" />
   <xacro:sandia_hand side="right" parent="r_hand" reflect="1" joint_type="revolute" thumb_angle="0">
-    <origin xyz="0.00179 -0.13516 -0.01176" rpy="0 0 -1.57079"/>
+    <origin xyz="-0.00179 -0.13516 0.01176" rpy="0 0 -1.57079"/>
   </xacro:sandia_hand>
   <xacro:sandia_hand side="left" parent="l_hand" reflect="-1" joint_type="revolute" thumb_angle="0">
-    <origin xyz="-0.00179  0.13516 -0.01176" rpy="3.14159 0  1.57079"/>
+    <origin xyz="0.00179  0.13516 0.01176" rpy="3.14159 0  1.57079"/>
   </xacro:sandia_hand>
   <xacro:include filename="$(find atlas_description)/urdf/atlas_v3.gazebo" />

Commit message: correction: both palms should face upwards.

File: ros/atlas_description/robots/atlas_v3_sandia_hands.urdf.xacro (robot description, xacro)
@@ -6,5 +6,5 @@
   </xacro:sandia_hand>
   <xacro:sandia_hand side="left" parent="l_hand" reflect="-1" joint_type="revolute" thumb_angle="0">
-    <origin xyz="0.00179  0.13516 0.01176" rpy="3.14159 0  1.57079"/>
+    <origin xyz="0.00179  0.13516 0.01176" rpy="0 0  1.57079"/>
   </xacro:sandia_hand>
   <xacro:include filename="$(find atlas_description)/urdf/atlas_v3.gazebo" />

File: ros/atlas_description/robots/atlas_v3_with_v1_inertia_sandia_hands.urdf.xacro (robot description, xacro)
@@ -6,5 +6,5 @@
   </xacro:sandia_hand>
   <xacro:sandia_hand side="left" parent="l_hand" reflect="-1" joint_type="revolute" thumb_angle="0">
-    <origin xyz="0.00179  0.13516 0.01176" rpy="3.14159 0  1.57079"/>
+    <origin xyz="0.00179  0.13516 0.01176" rpy="0 0  1.57079"/>
   </xacro:sandia_hand>
   <xacro:include filename="$(find atlas_description)/urdf/atlas_v3.gazebo" />
