Commit message: update mesh references for irobot_hand

File: ros/irobot_hand_description/urdf/irobot_hand.urdf.xacro (robot description, xacro)
@@ -206,5 +206,5 @@
     <collision>
       <geometry>
-        <mesh filename="package://irobot_hand/meshes/palm.stl"/>
+        <mesh filename="package://irobot_hand_description/meshes/palm.stl"/>
       </geometry>
       <origin rpy="0 0 0" xyz="0 -0.038 -0.023"/>
@@ -212,5 +212,5 @@
     <visual>
       <geometry>
-        <mesh filename="package://irobot_hand/meshes/palm.stl"/>
+        <mesh filename="package://irobot_hand_description/meshes/palm.stl"/>
       </geometry>
       <material name="darkgray">
@@ -228,5 +228,5 @@
     <collision>
       <geometry>
-        <mesh filename="package://irobot_hand/meshes/finger_base.stl"/>
+        <mesh filename="package://irobot_hand_description/meshes/finger_base.stl"/>
       </geometry>
       <origin rpy="${pi/2} 0 0" xyz="0 0 0"/>
@@ -234,5 +234,5 @@
     <visual>
       <geometry>
-        <mesh filename="package://irobot_hand/meshes/finger_base.stl"/>
+        <mesh filename="package://irobot_hand_description/meshes/finger_base.stl"/>
       </geometry>
       <material name="darkgray">
@@ -250,11 +250,11 @@
     <collision>
       <geometry>
-        <mesh filename="package://irobot_hand/meshes/finger_proximal.stl"/>
-      </geometry>
-      <origin rpy="${pi/2} -${pi/2} 0" xyz="0 0 0"/>
-    </collision>
-    <visual>
-      <geometry>
-        <mesh filename="package://irobot_hand/meshes/finger_proximal.stl"/>
+        <mesh filename="package://irobot_hand_description/meshes/finger_proximal.stl"/>
+      </geometry>
+      <origin rpy="${pi/2} -${pi/2} 0" xyz="0 0 0"/>
+    </collision>
+    <visual>
+      <geometry>
+        <mesh filename="package://irobot_hand_description/meshes/finger_proximal.stl"/>
       </geometry>
       <material name="green">
@@ -272,11 +272,11 @@
     <collision>
       <geometry>
-        <mesh filename="package://irobot_hand/meshes/finger_distal.stl"/>
-      </geometry>
-      <origin rpy="0 ${pi} 0" xyz="0 0 0"/>
-    </collision>
-    <visual>
-      <geometry>
-        <mesh filename="package://irobot_hand/meshes/finger_distal.stl"/>
+        <mesh filename="package://irobot_hand_description/meshes/finger_distal.stl"/>
+      </geometry>
+      <origin rpy="0 ${pi} 0" xyz="0 0 0"/>
+    </collision>
+    <visual>
+      <geometry>
+        <mesh filename="package://irobot_hand_description/meshes/finger_distal.stl"/>
       </geometry>
       <material name="green">
@@ -294,5 +294,5 @@
     <collision>
       <geometry>
-        <mesh filename="package://irobot_hand/meshes/finger_base.stl"/>
+        <mesh filename="package://irobot_hand_description/meshes/finger_base.stl"/>
       </geometry>
       <origin rpy="${pi/2} 0 0" xyz="0 0 0"/>
@@ -300,5 +300,5 @@
     <visual>
       <geometry>
-        <mesh filename="package://irobot_hand/meshes/finger_base.stl"/>
+        <mesh filename="package://irobot_hand_description/meshes/finger_base.stl"/>
       </geometry>
       <material name="darkgray">
@@ -316,11 +316,11 @@
     <collision>
       <geometry>
-        <mesh filename="package://irobot_hand/meshes/finger_proximal.stl"/>
-      </geometry>
-      <origin rpy="${pi/2} -${pi/2} 0" xyz="0 0 0"/>
-    </collision>
-    <visual>
-      <geometry>
-        <mesh filename="package://irobot_hand/meshes/finger_proximal.stl"/>
+        <mesh filename="package://irobot_hand_description/meshes/finger_proximal.stl"/>
+      </geometry>
+      <origin rpy="${pi/2} -${pi/2} 0" xyz="0 0 0"/>
+    </collision>
+    <visual>
+      <geometry>
+        <mesh filename="package://irobot_hand_description/meshes/finger_proximal.stl"/>
       </geometry>
       <material name="green">
@@ -338,11 +338,11 @@
     <collision>
       <geometry>
-        <mesh filename="package://irobot_hand/meshes/finger_distal.stl"/>
-      </geometry>
-      <origin rpy="0 ${pi} 0" xyz="0 0 0"/>
-    </collision>
-    <visual>
-      <geometry>
-        <mesh filename="package://irobot_hand/meshes/finger_distal.stl"/>
+        <mesh filename="package://irobot_hand_description/meshes/finger_distal.stl"/>
+      </geometry>
+      <origin rpy="0 ${pi} 0" xyz="0 0 0"/>
+    </collision>
+    <visual>
+      <geometry>
+        <mesh filename="package://irobot_hand_description/meshes/finger_distal.stl"/>
       </geometry>
       <material name="green">
@@ -360,11 +360,11 @@
     <collision>
       <geometry>
-        <mesh filename="package://irobot_hand/meshes/finger_proximal.stl"/>
-      </geometry>
-      <origin rpy="${pi/2} -${pi/2} 0" xyz="0 0 0"/>
-    </collision>
-    <visual>
-      <geometry>
-        <mesh filename="package://irobot_hand/meshes/finger_proximal.stl"/>
+        <mesh filename="package://irobot_hand_description/meshes/finger_proximal.stl"/>
+      </geometry>
+      <origin rpy="${pi/2} -${pi/2} 0" xyz="0 0 0"/>
+    </collision>
+    <visual>
+      <geometry>
+        <mesh filename="package://irobot_hand_description/meshes/finger_proximal.stl"/>
       </geometry>
       <material name="green">
@@ -382,11 +382,11 @@
     <collision>
       <geometry>
-        <mesh filename="package://irobot_hand/meshes/finger_distal.stl"/>
-      </geometry>
-      <origin rpy="0 ${pi} 0" xyz="0 0 0"/>
-    </collision>
-    <visual>
-      <geometry>
-        <mesh filename="package://irobot_hand/meshes/finger_distal.stl"/>
+        <mesh filename="package://irobot_hand_description/meshes/finger_distal.stl"/>
+      </geometry>
+      <origin rpy="0 ${pi} 0" xyz="0 0 0"/>
+    </collision>
+    <visual>
+      <geometry>
+        <mesh filename="package://irobot_hand_description/meshes/finger_distal.stl"/>
       </geometry>
       <material name="green">
