Commit message: moving the meshes to make proper multisense_sl_description ros style package

File: ros/multisense_sl_description/urdf/multisense_sl.urdf (robot description, URDF)
Before this commit: robot multisense_sl, 11 links, 10 joints
Links:
- link head: geometry collision box size=0.0468 0.12 0.1184; collision box size=0.1311 0.12 0.0591
- link hokuyo_link: geometry collision box size=0.08 0.06 0.04238; collision cylinder length=0.047 radius=0.024425

Commit message: update imu location per drawing.

File: ros/multisense_sl_description/urdf/multisense_sl.urdf (robot description, URDF)
Before this commit: robot multisense_sl, 12 links, 11 joints
Links:
- removed link imu_link
- added link head_imu_link, mass 0.1; collision box size=0.01 0.01 0.01; visual box size=0.01 0.01 0.01
Joints:
- removed joint imu_joint
- added joint head_imu_joint: type fixed, parent head, child head_imu_link, origin xyz=-0.0475 0.035 0.0 rpy=0 0 0

Commit message: remove collision geom of imu link per pull request comment

File: ros/multisense_sl_description/urdf/multisense_sl.urdf (robot description, URDF)
Before this commit: robot multisense_sl, 12 links, 11 joints
Links:
- link head_imu_link: geometry visual box size=0.01 0.01 0.01

Commit message: update inertia of fixed attached frames at the end of kinematic chain in multisense_sl head model (to be lumped to parent link) such that
  * overall mass is conserved (move CG to parent link location, subtract mass from parent link)
  * MOI added is 1e-6 kg*m^2 for each frame so it's insignificant.

ref:  http://answers.gazebosim.org/question/2150/drcsim-fat-head-random-head-parts-have-too-large/
ref:  issue #157

File: ros/multisense_sl_description/urdf/multisense_sl.urdf (robot description, URDF)
Before this commit: robot multisense_sl, 12 links, 11 joints
Links:
- link center_bottom_led_frame: mass 0.1 -> 1e-5
- link center_top_led_frame: mass 0.1 -> 1e-5
- link head: mass 1.4199 -> 1.41984
- link head_hokuyo_frame: mass 0.01 -> 1e-5
- link head_imu_link: mass 0.1 -> 1e-5
- link hokuyo_link: mass 0.057664 -> 0.057654
- link left_camera_frame: mass 0.1 -> 1e-5
- link left_led_frame: mass 0.1 -> 1e-5
- link right_camera_frame: mass 0.1 -> 1e-5
- link right_led_frame: mass 0.1 -> 1e-5
