Commit message: changes from issue #68 and pull request #67

File: ros/atlas_description/urdf/atlas.urdf (robot description, URDF)
Before this commit: robot drc_skeleton, 30 links, 29 joints
Joints:
- joint r_arm_usy: axis 0 -0.5 0.866025 -> 0 0.5 -0.866025

Commit message: move head urdf into atlas.sensors

File: ros/atlas_description/urdf/atlas.urdf (robot description, URDF)
Before this commit: robot drc_skeleton, 30 links, 29 joints
Links:
- added link head_hokuyo_frame, mass 0.01
Joints:
- added joint head_hokuyo_joint: type fixed, parent hokuyo_link, child head_hokuyo_frame, origin xyz=0.03 0 0.015 rpy=0 0 0, axis 0 1 0

Commit message: move head into atlas.sensorrs

File: ros/atlas_description/urdf/atlas.urdf (robot description, URDF)
Before this commit: robot drc_skeleton, 31 links, 30 joints
Links:
- removed link head
- removed link head_hokuyo_frame
- removed link hokuyo_link
Joints:
- removed joint head_hokuyo_joint
- removed joint hokuyo_joint

Commit message: revert changes per issue #68, making a separate pull reuqest

File: ros/atlas_description/urdf/atlas.urdf (robot description, URDF)
Before this commit: robot drc_skeleton, 28 links, 28 joints
Joints:
- joint r_arm_usy: axis 0 0.5 -0.866025 -> 0 -0.5 0.866025

Commit message: merging from default

File: ros/atlas_description/urdf/atlas.urdf (robot description, URDF)
Before this commit: robot drc_skeleton, 28 links, 28 joints
Links:
- link l_clav: geometry collision mesh filename=package://atlas_description/meshes/l_clav.stl scale=1 1 1; visual mesh filename=package://atlas_description/meshes/l_clav.dae scale=1 1 1
- link l_farm: geometry collision mesh filename=package://atlas_description/meshes/l_farm.stl scale=1 1 1; visual mesh filename=package://atlas_description/meshes/l_farm.dae scale=1 1 1
- link l_foot: geometry collision mesh filename=package://atlas_description/meshes/l_foot.stl scale=1 1 1; visual mesh filename=package://atlas_description/meshes/l_foot.dae scale=1 1 1
- link l_hand: geometry collision mesh filename=package://atlas_description/meshes/l_hand.stl scale=1 1 1; visual mesh filename=package://atlas_description/meshes/l_hand.dae scale=1 1 1
- link l_larm: geometry collision mesh filename=package://atlas_description/meshes/l_larm.stl scale=1 1 1; visual mesh filename=package://atlas_description/meshes/l_larm.dae scale=1 1 1
- link l_lglut: geometry collision mesh filename=package://atlas_description/meshes/l_lglut.stl scale=1 1 1; visual mesh filename=package://atlas_description/meshes/l_lglut.dae scale=1 1 1
- link l_lleg: geometry collision mesh filename=package://atlas_description/meshes/l_lleg.stl scale=1 1 1; visual mesh filename=package://atlas_description/meshes/l_lleg.dae scale=1 1 1
- link l_scap: geometry collision mesh filename=package://atlas_description/meshes/l_scap.stl scale=1 1 1; visual mesh filename=package://atlas_description/meshes/l_scap.dae scale=1 1 1
- link l_talus: geometry collision mesh filename=package://atlas_description/meshes/l_talus.stl scale=1 1 1; visual mesh filename=package://atlas_description/meshes/l_talus.dae scale=1 1 1
- link l_uarm: geometry collision mesh filename=package://atlas_description/meshes/l_uarm.stl scale=1 1 1; visual mesh filename=package://atlas_description/meshes/l_uarm.dae scale=1 1 1
- link l_uglut: geometry collision mesh filename=package://atlas_description/meshes/l_uglut.stl scale=1 1 1; visual mesh filename=package://atlas_description/meshes/l_uglut.dae scale=1 1 1
- link l_uleg: geometry collision mesh filename=package://atlas_description/meshes/l_uleg.stl scale=1 1 1; visual mesh filename=package://atlas_description/meshes/l_uleg.dae scale=1 1 1
- link ltorso: geometry collision mesh filename=package://atlas_description/meshes/ltorso.stl scale=1 1 1; visual mesh filename=package://atlas_description/meshes/ltorso.dae scale=1 1 1
- link mtorso: geometry collision mesh filename=package://atlas_description/meshes/mtorso.stl scale=1 1 1; visual mesh filename=package://atlas_description/meshes/mtorso.dae scale=1 1 1
- link pelvis: geometry collision mesh filename=package://atlas_description/meshes/pelvis.stl scale=1 1 1; visual mesh filename=package://atlas_description/meshes/pelvis.dae scale=1 1 1
- link r_clav: geometry collision mesh filename=package://atlas_description/meshes/r_clav.stl scale=1 1 1; visual mesh filename=package://atlas_description/meshes/r_clav.dae scale=1 1 1
- link r_farm: geometry collision mesh filename=package://atlas_description/meshes/r_farm.stl scale=1 1 1; visual mesh filename=package://atlas_description/meshes/r_farm.dae scale=1 1 1
- link r_foot: geometry collision mesh filename=package://atlas_description/meshes/r_foot.stl scale=1 1 1; visual mesh filename=package://atlas_description/meshes/r_foot.dae scale=1 1 1
- link r_hand: geometry collision mesh filename=package://atlas_description/meshes/r_hand.stl scale=1 1 1; visual mesh filename=package://atlas_description/meshes/r_hand.dae scale=1 1 1
- link r_larm: geometry collision mesh filename=package://atlas_description/meshes/r_larm.stl scale=1 1 1; visual mesh filename=package://atlas_description/meshes/r_larm.dae scale=1 1 1
- link r_lglut: geometry collision mesh filename=package://atlas_description/meshes/r_lglut.stl scale=1 1 1; visual mesh filename=package://atlas_description/meshes/r_lglut.dae scale=1 1 1
- link r_lleg: geometry collision mesh filename=package://atlas_description/meshes/r_lleg.stl scale=1 1 1; visual mesh filename=package://atlas_description/meshes/r_lleg.dae scale=1 1 1
- link r_scap: geometry collision mesh filename=package://atlas_description/meshes/r_scap.stl scale=1 1 1; visual mesh filename=package://atlas_description/meshes/r_scap.dae scale=1 1 1
- link r_talus: geometry collision mesh filename=package://atlas_description/meshes/r_talus.stl scale=1 1 1; visual mesh filename=package://atlas_description/meshes/r_talus.dae scale=1 1 1
- link r_uarm: geometry collision mesh filename=package://atlas_description/meshes/r_uarm.stl scale=1 1 1; visual mesh filename=package://atlas_description/meshes/r_uarm.dae scale=1 1 1
- link r_uglut: geometry collision mesh filename=package://atlas_description/meshes/r_uglut.stl scale=1 1 1; visual mesh filename=package://atlas_description/meshes/r_uglut.dae scale=1 1 1
- link r_uleg: geometry collision mesh filename=package://atlas_description/meshes/r_uleg.stl scale=1 1 1; visual mesh filename=package://atlas_description/meshes/r_uleg.dae scale=1 1 1
- link utorso: geometry collision mesh filename=package://atlas_description/meshes/utorso.stl scale=1 1 1; visual mesh filename=package://atlas_description/meshes/utorso.dae scale=1 1 1

File: ros/atlas_description/urdf/atlas_simple_shapes.urdf (robot description, URDF)
Before this commit: robot drc_skeleton, 28 links, 28 joints
Links:
- link l_clav: geometry collision cylinder length=0.027 radius=0.04; collision cylinder length=0.1525 radius=0.045
- link l_farm: geometry collision cylinder length=0.035181 radius=0.0458825; collision cylinder length=0.050472 radius=0.0279
- link l_foot: geometry collision box size=0.26 0.124887 0.01; visual mesh filename=package://atlas_description/meshes/l_foot.dae scale=1 1 1
- link l_hand: geometry collision cylinder length=0.019 radius=0.035939; collision cylinder length=0.019 radius=0.035939
- link l_larm: geometry collision cylinder length=0.0161 radius=0.045; collision cylinder length=0.0161 radius=0.045
- link l_lglut: geometry collision cylinder length=0.060306 radius=0.02009687; collision cylinder length=0.12 radius=0.02
- link l_lleg: geometry collision box size=0.1465 0.1205 0.476; visual mesh filename=package://atlas_description/meshes/l_lleg.dae scale=1 1 1
- link l_scap: geometry collision cylinder length=0.013737 radius=0.048709; collision cylinder length=0.013937 radius=0.048709
- link l_talus: geometry collision cylinder length=0.010059 radius=0.010348; collision cylinder length=0.029542 radius=0.010181
- link l_uarm: geometry collision cylinder length=0.088934 radius=0.04504847; collision cylinder length=0.116677 radius=0.0449
- link l_uglut: geometry collision cylinder length=0.078396 radius=0.019096; collision cylinder length=0.080842 radius=0.019841
- link l_uleg: geometry collision cylinder length=0.10 radius=0.1; collision cylinder length=0.15 radius=0.07
- link ltorso: geometry visual mesh filename=package://atlas_description/meshes/ltorso.dae scale=1 1 1
- link mtorso: geometry collision cylinder length=0.02 radius=0.015; collision cylinder length=0.02 radius=0.015
- link pelvis: geometry collision cylinder length=0.022 radius=0.130; collision cylinder length=0.022 radius=0.130
- link r_clav: geometry collision cylinder length=0.027 radius=0.04; collision cylinder length=0.1525 radius=0.045
- link r_farm: geometry collision cylinder length=0.035181 radius=0.0458825; collision cylinder length=0.050472 radius=0.0279
- link r_foot: geometry collision box size=0.26 0.124887 0.01; visual mesh filename=package://atlas_description/meshes/r_foot.dae scale=1 1 1
- link r_hand: geometry collision cylinder length=0.019 radius=0.035939; collision cylinder length=0.019 radius=0.035939
- link r_larm: geometry collision cylinder length=0.0161 radius=0.045; collision cylinder length=0.0161 radius=0.045
- link r_lglut: geometry collision cylinder length=0.060306 radius=0.02009687; collision cylinder length=0.12 radius=0.02
- link r_lleg: geometry collision box size=0.1465 0.1205 0.476; visual mesh filename=package://atlas_description/meshes/r_lleg.dae scale=1 1 1
- link r_scap: geometry collision cylinder length=0.013737 radius=0.048709; collision cylinder length=0.013937 radius=0.048709
- link r_talus: geometry collision cylinder length=0.010059 radius=0.010348; collision cylinder length=0.029542 radius=0.010181
- link r_uarm: geometry collision cylinder length=0.088934 radius=0.04504847; collision cylinder length=0.116677 radius=0.0449
- link r_uglut: geometry collision cylinder length=0.078396 radius=0.019096; collision cylinder length=0.080842 radius=0.019841
- link r_uleg: geometry collision cylinder length=0.10 radius=0.1; collision cylinder length=0.15 radius=0.07
- link utorso: geometry collision box size=0.3188 0.24 0.3162; collision cylinder length=0.22375 radius=0.0363

Commit message: merging from default

File: ros/atlas_description/urdf/atlas.urdf (robot description, URDF)
Before this commit: robot drc_skeleton, 28 links, 28 joints
Links:
- link l_clav: geometry collision mesh filename=package://atlas/meshes/l_clav.stl scale=1 1 1; visual mesh filename=package://atlas/meshes/l_clav.dae scale=1 1 1
- link l_farm: geometry collision mesh filename=package://atlas/meshes/l_farm.stl scale=1 1 1; visual mesh filename=package://atlas/meshes/l_farm.dae scale=1 1 1
- link l_foot: geometry collision mesh filename=package://atlas/meshes/l_foot.stl scale=1 1 1; visual mesh filename=package://atlas/meshes/l_foot.dae scale=1 1 1
- link l_hand: geometry collision mesh filename=package://atlas/meshes/l_hand.stl scale=1 1 1; visual mesh filename=package://atlas/meshes/l_hand.dae scale=1 1 1
- link l_larm: geometry collision mesh filename=package://atlas/meshes/l_larm.stl scale=1 1 1; visual mesh filename=package://atlas/meshes/l_larm.dae scale=1 1 1
- link l_lglut: geometry collision mesh filename=package://atlas/meshes/l_lglut.stl scale=1 1 1; visual mesh filename=package://atlas/meshes/l_lglut.dae scale=1 1 1
- link l_lleg: geometry collision mesh filename=package://atlas/meshes/l_lleg.stl scale=1 1 1; visual mesh filename=package://atlas/meshes/l_lleg.dae scale=1 1 1
- link l_scap: geometry collision mesh filename=package://atlas/meshes/l_scap.stl scale=1 1 1; visual mesh filename=package://atlas/meshes/l_scap.dae scale=1 1 1
- link l_talus: geometry collision mesh filename=package://atlas/meshes/l_talus.stl scale=1 1 1; visual mesh filename=package://atlas/meshes/l_talus.dae scale=1 1 1
- link l_uarm: geometry collision mesh filename=package://atlas/meshes/l_uarm.stl scale=1 1 1; visual mesh filename=package://atlas/meshes/l_uarm.dae scale=1 1 1
- link l_uglut: geometry collision mesh filename=package://atlas/meshes/l_uglut.stl scale=1 1 1; visual mesh filename=package://atlas/meshes/l_uglut.dae scale=1 1 1
- link l_uleg: geometry collision mesh filename=package://atlas/meshes/l_uleg.stl scale=1 1 1; visual mesh filename=package://atlas/meshes/l_uleg.dae scale=1 1 1
- link ltorso: geometry collision mesh filename=package://atlas/meshes/ltorso.stl scale=1 1 1; visual mesh filename=package://atlas/meshes/ltorso.dae scale=1 1 1
- link mtorso: geometry collision mesh filename=package://atlas/meshes/mtorso.stl scale=1 1 1; visual mesh filename=package://atlas/meshes/mtorso.dae scale=1 1 1
- link pelvis: geometry collision mesh filename=package://atlas/meshes/pelvis.stl scale=1 1 1; visual mesh filename=package://atlas/meshes/pelvis.dae scale=1 1 1
- link r_clav: geometry collision mesh filename=package://atlas/meshes/r_clav.stl scale=1 1 1; visual mesh filename=package://atlas/meshes/r_clav.dae scale=1 1 1
- link r_farm: geometry collision mesh filename=package://atlas/meshes/r_farm.stl scale=1 1 1; visual mesh filename=package://atlas/meshes/r_farm.dae scale=1 1 1
- link r_foot: geometry collision mesh filename=package://atlas/meshes/r_foot.stl scale=1 1 1; visual mesh filename=package://atlas/meshes/r_foot.dae scale=1 1 1
- link r_hand: geometry collision mesh filename=package://atlas/meshes/r_hand.stl scale=1 1 1; visual mesh filename=package://atlas/meshes/r_hand.dae scale=1 1 1
- link r_larm: geometry collision mesh filename=package://atlas/meshes/r_larm.stl scale=1 1 1; visual mesh filename=package://atlas/meshes/r_larm.dae scale=1 1 1
- link r_lglut: geometry collision mesh filename=package://atlas/meshes/r_lglut.stl scale=1 1 1; visual mesh filename=package://atlas/meshes/r_lglut.dae scale=1 1 1
- link r_lleg: geometry collision mesh filename=package://atlas/meshes/r_lleg.stl scale=1 1 1; visual mesh filename=package://atlas/meshes/r_lleg.dae scale=1 1 1
- link r_scap: geometry collision mesh filename=package://atlas/meshes/r_scap.stl scale=1 1 1; visual mesh filename=package://atlas/meshes/r_scap.dae scale=1 1 1
- link r_talus: geometry collision mesh filename=package://atlas/meshes/r_talus.stl scale=1 1 1; visual mesh filename=package://atlas/meshes/r_talus.dae scale=1 1 1
- link r_uarm: geometry collision mesh filename=package://atlas/meshes/r_uarm.stl scale=1 1 1; visual mesh filename=package://atlas/meshes/r_uarm.dae scale=1 1 1
- link r_uglut: geometry collision mesh filename=package://atlas/meshes/r_uglut.stl scale=1 1 1; visual mesh filename=package://atlas/meshes/r_uglut.dae scale=1 1 1
- link r_uleg: geometry collision mesh filename=package://atlas/meshes/r_uleg.stl scale=1 1 1; visual mesh filename=package://atlas/meshes/r_uleg.dae scale=1 1 1
- link utorso: geometry collision mesh filename=package://atlas/meshes/utorso.stl scale=1 1 1; visual mesh filename=package://atlas/meshes/utorso.dae scale=1 1 1

File: ros/atlas_description/urdf/atlas_simple_shapes.urdf (robot description, URDF)
Before this commit: robot drc_skeleton, 28 links, 28 joints
Links:
- link l_clav: geometry collision cylinder length=0.027 radius=0.04; collision cylinder length=0.1525 radius=0.045
- link l_farm: geometry collision cylinder length=0.035181 radius=0.0458825; collision cylinder length=0.050472 radius=0.0279
- link l_foot: geometry collision box size=0.26 0.124887 0.01; visual mesh filename=package://atlas/meshes/l_foot.dae scale=1 1 1
- link l_hand: geometry collision cylinder length=0.019 radius=0.035939; collision cylinder length=0.019 radius=0.035939
- link l_larm: geometry collision cylinder length=0.0161 radius=0.045; collision cylinder length=0.0161 radius=0.045
- link l_lglut: geometry collision cylinder length=0.060306 radius=0.02009687; collision cylinder length=0.12 radius=0.02
- link l_lleg: geometry collision box size=0.1465 0.1205 0.476; visual mesh filename=package://atlas/meshes/l_lleg.dae scale=1 1 1
- link l_scap: geometry collision cylinder length=0.013737 radius=0.048709; collision cylinder length=0.013937 radius=0.048709
- link l_talus: geometry collision cylinder length=0.010059 radius=0.010348; collision cylinder length=0.029542 radius=0.010181
- link l_uarm: geometry collision cylinder length=0.088934 radius=0.04504847; collision cylinder length=0.116677 radius=0.0449
- link l_uglut: geometry collision cylinder length=0.078396 radius=0.019096; collision cylinder length=0.080842 radius=0.019841
- link l_uleg: geometry collision cylinder length=0.10 radius=0.1; collision cylinder length=0.15 radius=0.07
- link ltorso: geometry visual mesh filename=package://atlas/meshes/ltorso.dae scale=1 1 1
- link mtorso: geometry collision cylinder length=0.02 radius=0.015; collision cylinder length=0.02 radius=0.015
- link pelvis: geometry collision cylinder length=0.022 radius=0.130; collision cylinder length=0.022 radius=0.130
- link r_clav: geometry collision cylinder length=0.027 radius=0.04; collision cylinder length=0.1525 radius=0.045
- link r_farm: geometry collision cylinder length=0.035181 radius=0.0458825; collision cylinder length=0.050472 radius=0.0279
- link r_foot: geometry collision box size=0.26 0.124887 0.01; visual mesh filename=package://atlas/meshes/r_foot.dae scale=1 1 1
- link r_hand: geometry collision cylinder length=0.019 radius=0.035939; collision cylinder length=0.019 radius=0.035939
- link r_larm: geometry collision cylinder length=0.0161 radius=0.045; collision cylinder length=0.0161 radius=0.045
- link r_lglut: geometry collision cylinder length=0.060306 radius=0.02009687; collision cylinder length=0.12 radius=0.02
- link r_lleg: geometry collision box size=0.1465 0.1205 0.476; visual mesh filename=package://atlas/meshes/r_lleg.dae scale=1 1 1
- link r_scap: geometry collision cylinder length=0.013737 radius=0.048709; collision cylinder length=0.013937 radius=0.048709
- link r_talus: geometry collision cylinder length=0.010059 radius=0.010348; collision cylinder length=0.029542 radius=0.010181
- link r_uarm: geometry collision cylinder length=0.088934 radius=0.04504847; collision cylinder length=0.116677 radius=0.0449
- link r_uglut: geometry collision cylinder length=0.078396 radius=0.019096; collision cylinder length=0.080842 radius=0.019841
- link r_uleg: geometry collision cylinder length=0.10 radius=0.1; collision cylinder length=0.15 radius=0.07
- link utorso: geometry collision box size=0.3188 0.24 0.3162; collision cylinder length=0.22375 radius=0.0363

Commit message: fixed my bad guesses, with John's help

File: ros/atlas_description/urdf/atlas.urdf (robot description, URDF)
Before this commit: robot drc_skeleton, 28 links, 28 joints
Joints:
- joint l_leg_uhz: limit lower=-0.32 upper=1.14 effort=260 velocity=12 -> lower=-0.32 upper=1.14 effort=110 velocity=12
- joint r_leg_uhz: limit lower=-1.14 upper=0.32 effort=260 velocity=12 -> lower=-1.14 upper=0.32 effort=110 velocity=12

Commit message: merging from default

File: ros/atlas_description/urdf/atlas.urdf (robot description, URDF)
Before this commit: robot drc_skeleton, 28 links, 28 joints
Joints:
- joint r_leg_uhz: limit lower=-1.14 upper=0.32 effort=260 velocity=12 -> lower=-1.14 upper=0.32 effort=110 velocity=12

File: ros/atlas_description/urdf/atlas_simple_shapes.urdf (robot description, URDF)
Before this commit: robot drc_skeleton, 28 links, 28 joints
Links:
- link l_clav: geometry collision box size=0.13 0.15 0.05; collision cylinder length=0.1525 radius=0.045
- link l_farm: geometry collision box size=0.135 0.1 0.045; collision cylinder length=0.125 radius=0.045
- link l_foot: mass 0.817 -> 0.867; geometry collision box size=0.26 0.124887 0.05; visual mesh filename=package://atlas/meshes/l_foot.dae scale=1 1 1
- link l_hand: geometry collision box size=0.13 0.09 0.07; collision cylinder length=0.05 radius=0.03
- link l_larm: geometry collision box size=0.135 0.15 0.06; collision cylinder length=0.125 radius=0.045
- link l_lglut: mass 0.69 -> 0.803
- link l_lleg: geometry collision cylinder length=0.40 radius=0.07; visual mesh filename=package://atlas/meshes/l_lleg.dae scale=100. 100. 100.
- link l_scap: geometry collision box size=0.15 0.15 0.06; collision cylinder length=0.125 radius=0.045
- link l_talus: mass 0.817 -> 0.867
- link l_uarm: geometry collision box size=0.04 0.07 0.13; collision cylinder length=0.125 radius=0.045
- link l_uglut: mass 0.5166 -> 1.51622
- link l_uleg: mass 7.34 -> 7.227; geometry collision cylinder length=0.10 radius=0.1; collision cylinder length=0.15 radius=0.07
- link ltorso: mass 1.92 -> 1.62729
- link mtorso: mass 0.55 -> 3.8068
- link pelvis: mass 14.2529 -> 12.54638; geometry collision box size=0.1 0.15 0.2; collision cylinder length=0.05 radius=0.16
- link r_clav: geometry collision box size=0.13 0.15 0.05; collision cylinder length=0.1525 radius=0.045
- link r_farm: geometry collision box size=0.135 0.1 0.045; collision cylinder length=0.125 radius=0.045
- link r_foot: mass 0.817 -> 0.867; geometry collision box size=0.26 0.124887 0.05; visual mesh filename=package://atlas/meshes/r_foot.dae scale=1 1 1
- link r_hand: geometry collision box size=0.13 0.09 0.07; collision cylinder length=0.05 radius=0.03
- link r_larm: geometry collision box size=0.135 0.15 0.06; collision cylinder length=0.125 radius=0.045
- link r_lglut: mass 0.69 -> 0.803; geometry collision cylinder length=0.060306 radius=0.02009687; collision cylinder length=0.12 radius=0.02
- link r_lleg: geometry collision cylinder length=0.40 radius=0.07; visual mesh filename=package://atlas/meshes/r_lleg.dae scale=100. 100. 100.
- link r_scap: geometry collision box size=0.15 0.15 0.06; collision cylinder length=0.125 radius=0.045
- link r_talus: mass 0.817 -> 0.867
- link r_uarm: geometry collision box size=0.04 0.07 0.13; collision cylinder length=0.125 radius=0.045
- link r_uglut: mass 0.5166 -> 1.51622; geometry collision cylinder length=0.078396 radius=0.019096; collision cylinder length=0.080842 radius=0.019841
- link r_uleg: mass 7.34 -> 7.227; geometry collision cylinder length=0.10 radius=0.1; collision cylinder length=0.15 radius=0.07
- link utorso: mass 18.484 -> 15.2272
Joints:
- joint neck_ay: origin xyz=0.16555 0 0.50823 rpy=0 -0 0 -> xyz=0.21672 0 0.53796 rpy=0 -0 0

File: ros/multisense_sl_description/urdf/multisense_sl.urdf (robot description, URDF)
Before this commit: robot multisense_sl, 12 links, 11 joints
Links:
- link center_bottom_led_frame: mass 0.1 -> 1e-5
- link center_top_led_frame: mass 0.1 -> 1e-5
- link head: mass 1.4199 -> 1.41984; geometry collision box size=0.0468 0.12 0.1184; collision box size=0.1311 0.12 0.0591
- link head_hokuyo_frame: mass 0.01 -> 1e-5
- link head_imu_link: mass 0.1 -> 1e-5
- link hokuyo_link: mass 0.057664 -> 0.057654; geometry collision box size=0.08 0.06 0.04238; collision cylinder length=0.047 radius=0.024425
- link left_camera_frame: mass 0.1 -> 1e-5
- link left_led_frame: mass 0.1 -> 1e-5
- link right_camera_frame: mass 0.1 -> 1e-5
- link right_led_frame: mass 0.1 -> 1e-5
