Commit message: getting things to compile, except DRCVehicleROSPlugin

File: ros/atlas_description/urdf/atlas_simple_shapes.urdf (robot description, URDF)
Before this commit: robot drc_skeleton, 30 links, 29 joints
Links:
- removed link head
- removed link hokuyo_link
Joints:
- removed joint hokuyo_joint

Commit message: reorganize atlas_description so it is a consistent ros package

File: ros/atlas_description/urdf/atlas_simple_shapes.urdf (robot description, URDF)
Before this commit: robot drc_skeleton, 28 links, 28 joints
Links:
- link l_clav: geometry collision cylinder length=0.027 radius=0.04; collision cylinder length=0.1525 radius=0.045
- link l_farm: geometry collision cylinder length=0.035181 radius=0.0458825; collision cylinder length=0.050472 radius=0.0279
- link l_foot: geometry collision box size=0.26 0.124887 0.01; visual mesh filename=package://atlas_description/meshes/l_foot.dae scale=1 1 1
- link l_hand: geometry collision cylinder length=0.019 radius=0.035939; collision cylinder length=0.019 radius=0.035939
- link l_larm: geometry collision cylinder length=0.0161 radius=0.045; collision cylinder length=0.0161 radius=0.045
- link l_lglut: geometry collision cylinder length=0.060306 radius=0.02009687; collision cylinder length=0.12 radius=0.02
- link l_lleg: geometry collision box size=0.1465 0.1205 0.476; visual mesh filename=package://atlas_description/meshes/l_lleg.dae scale=1 1 1
- link l_scap: geometry collision cylinder length=0.013737 radius=0.048709; collision cylinder length=0.013937 radius=0.048709
- link l_talus: geometry collision cylinder length=0.010059 radius=0.010348; collision cylinder length=0.029542 radius=0.010181
- link l_uarm: geometry collision cylinder length=0.088934 radius=0.04504847; collision cylinder length=0.116677 radius=0.0449
- link l_uglut: geometry collision cylinder length=0.078396 radius=0.019096; collision cylinder length=0.080842 radius=0.019841
- link l_uleg: geometry collision box size=0.2 0.1865 0.26; visual mesh filename=package://atlas_description/meshes/l_uleg.dae scale=1 1 1
- link ltorso: geometry visual mesh filename=package://atlas_description/meshes/ltorso.dae scale=1 1 1
- link mtorso: geometry collision cylinder length=0.02 radius=0.015; collision cylinder length=0.02 radius=0.015
- link pelvis: geometry collision cylinder length=0.07 radius=0.130; collision cylinder length=0.07 radius=0.130
- link r_clav: geometry collision cylinder length=0.027 radius=0.04; collision cylinder length=0.1525 radius=0.045
- link r_farm: geometry collision cylinder length=0.035181 radius=0.0458825; collision cylinder length=0.050472 radius=0.0279
- link r_foot: geometry collision box size=0.26 0.124887 0.01; visual mesh filename=package://atlas_description/meshes/r_foot.dae scale=1 1 1
- link r_hand: geometry collision cylinder length=0.019 radius=0.035939; collision cylinder length=0.019 radius=0.035939
- link r_larm: geometry collision cylinder length=0.0161 radius=0.045; collision cylinder length=0.0161 radius=0.045
- link r_lglut: geometry collision cylinder length=0.060306 radius=0.02009687; collision cylinder length=0.12 radius=0.02
- link r_lleg: geometry collision box size=0.1465 0.1205 0.476; visual mesh filename=package://atlas_description/meshes/r_lleg.dae scale=1 1 1
- link r_scap: geometry collision cylinder length=0.013737 radius=0.048709; collision cylinder length=0.013937 radius=0.048709
- link r_talus: geometry collision cylinder length=0.010059 radius=0.010348; collision cylinder length=0.029542 radius=0.010181
- link r_uarm: geometry collision cylinder length=0.088934 radius=0.04504847; collision cylinder length=0.116677 radius=0.0449
- link r_uglut: geometry collision cylinder length=0.078396 radius=0.019096; collision cylinder length=0.080842 radius=0.019841
- link r_uleg: geometry collision box size=0.2 0.1865 0.26; visual mesh filename=package://atlas_description/meshes/r_uleg.dae scale=1 1 1
- link utorso: geometry collision box size=0.3188 0.24 0.3662; collision cylinder length=0.22375 radius=0.0363

Commit message: split talus and foot inertia equally between the two links.

File: ros/atlas_description/urdf/atlas_simple_shapes.urdf (robot description, URDF)
Before this commit: robot drc_skeleton, 28 links, 28 joints
Links:
- link l_foot: mass 1.634 -> 0.817
- link l_talus: mass 0.1 -> 0.817
- link r_foot: mass 1.634 -> 0.817
- link r_talus: mass 0.1 -> 0.817

Commit message: Remove/resize collisions around pelvis

File: ros/atlas_description/urdf/atlas_simple_shapes.urdf (robot description, URDF)
Before this commit: robot drc_skeleton, 28 links, 28 joints
Links:
- link pelvis: geometry collision cylinder length=0.03 radius=0.130; collision cylinder length=0.03 radius=0.130
- link utorso: geometry collision box size=0.3188 0.24 0.3162; collision cylinder length=0.22375 radius=0.0363

Commit message: Add cylinders collisions to pelvis

File: ros/atlas_description/urdf/atlas_simple_shapes.urdf (robot description, URDF)
Before this commit: robot drc_skeleton, 28 links, 28 joints
Links:
- link pelvis: geometry collision cylinder length=0.03 radius=0.10; collision cylinder length=0.03 radius=0.10

Commit message: More changes to atlas model

File: ros/atlas_description/urdf/atlas_simple_shapes.urdf (robot description, URDF)
Before this commit: robot drc_skeleton, 28 links, 28 joints
Links:
- link pelvis: geometry collision cylinder length=0.022 radius=0.130; collision cylinder length=0.022 radius=0.130

Commit message: merging from default

File: ros/atlas_description/urdf/atlas_simple_shapes.urdf (robot description, URDF)
Before this commit: robot drc_skeleton, 28 links, 28 joints
Links:
- link l_uleg: geometry collision cylinder length=0.10 radius=0.1; collision cylinder length=0.15 radius=0.07
- link pelvis: geometry collision cylinder length=0.022 radius=0.130; collision cylinder length=0.022 radius=0.130
- link r_uleg: geometry collision cylinder length=0.10 radius=0.1; collision cylinder length=0.15 radius=0.07
- link utorso: geometry collision box size=0.3188 0.24 0.3162; collision cylinder length=0.22375 radius=0.0363

Commit message: merge with default

File: ros/atlas_description/urdf/atlas_simple_shapes.urdf (robot description, URDF)
Before this commit: robot drc_skeleton, 28 links, 28 joints
Links:
- link l_clav: geometry collision cylinder length=0.027 radius=0.04; collision cylinder length=0.1525 radius=0.045
- link l_farm: geometry collision cylinder length=0.035181 radius=0.0458825; collision cylinder length=0.050472 radius=0.0279
- link l_foot: geometry collision box size=0.26 0.124887 0.01; visual mesh filename=package://atlas_description/meshes/l_foot.dae scale=1 1 1
- link l_hand: geometry collision cylinder length=0.019 radius=0.035939; collision cylinder length=0.019 radius=0.035939
- link l_larm: geometry collision cylinder length=0.0161 radius=0.045; collision cylinder length=0.0161 radius=0.045
- link l_lglut: geometry collision cylinder length=0.060306 radius=0.02009687; collision cylinder length=0.12 radius=0.02
- link l_lleg: geometry collision box size=0.1465 0.1205 0.476; visual mesh filename=package://atlas_description/meshes/l_lleg.dae scale=1 1 1
- link l_scap: geometry collision cylinder length=0.013737 radius=0.048709; collision cylinder length=0.013937 radius=0.048709
- link l_talus: geometry collision cylinder length=0.010059 radius=0.010348; collision cylinder length=0.029542 radius=0.010181
- link l_uarm: geometry collision cylinder length=0.088934 radius=0.04504847; collision cylinder length=0.116677 radius=0.0449
- link l_uglut: geometry collision cylinder length=0.078396 radius=0.019096; collision cylinder length=0.080842 radius=0.019841
- link l_uleg: geometry collision cylinder length=0.10 radius=0.1; collision cylinder length=0.15 radius=0.07
- link ltorso: geometry visual mesh filename=package://atlas_description/meshes/ltorso.dae scale=1 1 1
- link mtorso: geometry collision cylinder length=0.02 radius=0.015; collision cylinder length=0.02 radius=0.015
- link pelvis: geometry collision cylinder length=0.022 radius=0.130; collision cylinder length=0.022 radius=0.130
- link r_clav: geometry collision cylinder length=0.027 radius=0.04; collision cylinder length=0.1525 radius=0.045
- link r_farm: geometry collision cylinder length=0.035181 radius=0.0458825; collision cylinder length=0.050472 radius=0.0279
- link r_foot: geometry collision box size=0.26 0.124887 0.01; visual mesh filename=package://atlas_description/meshes/r_foot.dae scale=1 1 1
- link r_hand: geometry collision cylinder length=0.019 radius=0.035939; collision cylinder length=0.019 radius=0.035939
- link r_larm: geometry collision cylinder length=0.0161 radius=0.045; collision cylinder length=0.0161 radius=0.045
- link r_lglut: geometry collision cylinder length=0.060306 radius=0.02009687; collision cylinder length=0.12 radius=0.02
- link r_lleg: geometry collision box size=0.1465 0.1205 0.476; visual mesh filename=package://atlas_description/meshes/r_lleg.dae scale=1 1 1
- link r_scap: geometry collision cylinder length=0.013737 radius=0.048709; collision cylinder length=0.013937 radius=0.048709
- link r_talus: geometry collision cylinder length=0.010059 radius=0.010348; collision cylinder length=0.029542 radius=0.010181
- link r_uarm: geometry collision cylinder length=0.088934 radius=0.04504847; collision cylinder length=0.116677 radius=0.0449
- link r_uglut: geometry collision cylinder length=0.078396 radius=0.019096; collision cylinder length=0.080842 radius=0.019841
- link r_uleg: geometry collision cylinder length=0.10 radius=0.1; collision cylinder length=0.15 radius=0.07
- link utorso: geometry collision box size=0.3188 0.24 0.3162; collision cylinder length=0.22375 radius=0.0363

Commit message: merge with default

File: ros/atlas_description/urdf/atlas_simple_shapes.urdf (robot description, URDF)
Before this commit: robot drc_skeleton, 28 links, 28 joints
Links:
- link l_clav: geometry collision cylinder length=0.027 radius=0.04; collision cylinder length=0.1525 radius=0.045
- link l_farm: geometry collision cylinder length=0.035181 radius=0.0458825; collision cylinder length=0.050472 radius=0.0279
- link l_foot: mass 1.634 -> 0.817; geometry collision box size=0.26 0.124887 0.01; visual mesh filename=package://atlas/meshes/l_foot.dae scale=1 1 1
- link l_hand: geometry collision cylinder length=0.019 radius=0.035939; collision cylinder length=0.019 radius=0.035939
- link l_larm: geometry collision cylinder length=0.0161 radius=0.045; collision cylinder length=0.0161 radius=0.045
- link l_lglut: geometry collision cylinder length=0.060306 radius=0.02009687; collision cylinder length=0.12 radius=0.02
- link l_lleg: geometry collision box size=0.1465 0.1205 0.476; visual mesh filename=package://atlas/meshes/l_lleg.dae scale=1 1 1
- link l_scap: geometry collision cylinder length=0.013737 radius=0.048709; collision cylinder length=0.013937 radius=0.048709
- link l_talus: mass 0.1 -> 0.817; geometry collision cylinder length=0.010059 radius=0.010348; collision cylinder length=0.029542 radius=0.010181
- link l_uarm: geometry collision cylinder length=0.088934 radius=0.04504847; collision cylinder length=0.116677 radius=0.0449
- link l_uglut: geometry collision cylinder length=0.078396 radius=0.019096; collision cylinder length=0.080842 radius=0.019841
- link l_uleg: geometry collision cylinder length=0.10 radius=0.1; collision cylinder length=0.15 radius=0.07
- link ltorso: geometry visual mesh filename=package://atlas/meshes/ltorso.dae scale=1 1 1
- link mtorso: geometry collision cylinder length=0.02 radius=0.015; collision cylinder length=0.02 radius=0.015
- link pelvis: geometry collision cylinder length=0.022 radius=0.130; collision cylinder length=0.022 radius=0.130
- link r_clav: geometry collision cylinder length=0.027 radius=0.04; collision cylinder length=0.1525 radius=0.045
- link r_farm: geometry collision cylinder length=0.035181 radius=0.0458825; collision cylinder length=0.050472 radius=0.0279
- link r_foot: mass 1.634 -> 0.817; geometry collision box size=0.26 0.124887 0.01; visual mesh filename=package://atlas/meshes/r_foot.dae scale=1 1 1
- link r_hand: geometry collision cylinder length=0.019 radius=0.035939; collision cylinder length=0.019 radius=0.035939
- link r_larm: geometry collision cylinder length=0.0161 radius=0.045; collision cylinder length=0.0161 radius=0.045
- link r_lglut: geometry collision cylinder length=0.060306 radius=0.02009687; collision cylinder length=0.12 radius=0.02
- link r_lleg: geometry collision box size=0.1465 0.1205 0.476; visual mesh filename=package://atlas/meshes/r_lleg.dae scale=1 1 1
- link r_scap: geometry collision cylinder length=0.013737 radius=0.048709; collision cylinder length=0.013937 radius=0.048709
- link r_talus: mass 0.1 -> 0.817; geometry collision cylinder length=0.010059 radius=0.010348; collision cylinder length=0.029542 radius=0.010181
- link r_uarm: geometry collision cylinder length=0.088934 radius=0.04504847; collision cylinder length=0.116677 radius=0.0449
- link r_uglut: geometry collision cylinder length=0.078396 radius=0.019096; collision cylinder length=0.080842 radius=0.019841
- link r_uleg: geometry collision cylinder length=0.10 radius=0.1; collision cylinder length=0.15 radius=0.07
- link utorso: geometry collision box size=0.3188 0.24 0.3162; collision cylinder length=0.22375 radius=0.0363

Commit message: fixed simple collision shapes for lleg

File: ros/atlas_description/urdf/atlas_simple_shapes.urdf (robot description, URDF)
Before this commit: robot drc_skeleton, 28 links, 28 joints
Links:
- link l_lleg: geometry collision cylinder length=0.20 radius=0.06; collision cylinder length=0.22 radius=0.06
- link r_lleg: geometry collision cylinder length=0.20 radius=0.06; collision cylinder length=0.22 radius=0.06

Commit message: fix larm shapes as well (issue #133)

File: ros/atlas_description/urdf/atlas_simple_shapes.urdf (robot description, URDF)
Before this commit: robot drc_skeleton, 28 links, 28 joints
Links:
- link l_larm: geometry collision cylinder length=0.0161 radius=0.045; collision cylinder length=0.0161 radius=0.045
- link r_larm: geometry collision cylinder length=0.0161 radius=0.045; collision cylinder length=0.0161 radius=0.045

Commit message: mass tweak analysis

File: ros/atlas_description/urdf/atlas_simple_shapes.urdf (robot description, URDF)
Before this commit: robot drc_skeleton, 28 links, 28 joints
Links:
- link l_foot: mass 0.817 -> 1.634
- link l_talus: mass 0.817 -> 0.1
- link r_foot: mass 0.817 -> 1.634
- link r_talus: mass 0.817 -> 0.1

Commit message: tweaked inertia

File: ros/atlas_description/urdf/atlas_simple_shapes.urdf (robot description, URDF)
Before this commit: robot drc_skeleton, 28 links, 28 joints
Links:
- link l_foot: mass 1.634 -> 0.867
- link l_lglut: mass 0.69 -> 0.803
- link l_talus: mass 0.1 -> 0.867
- link l_uglut: mass 0.5166 -> 1.51622
- link l_uleg: mass 7.34 -> 7.227
- link mtorso: mass 0.55 -> 3.8068
- link pelvis: mass 14.2529 -> 13.646
- link r_foot: mass 1.634 -> 0.867
- link r_lglut: mass 0.69 -> 0.803
- link r_talus: mass 0.1 -> 0.867
- link r_uglut: mass 0.5166 -> 1.51622
- link r_uleg: mass 7.34 -> 7.227
- link utorso: mass 18.484 -> 15.2272

Commit message: merged from default and resolved conflicts

File: ros/atlas_description/urdf/atlas_simple_shapes.urdf (robot description, URDF)
Before this commit: robot drc_skeleton, 28 links, 28 joints
Links:
- link l_foot: mass 1.634 -> 0.817
- link l_larm: geometry collision cylinder length=0.0161 radius=0.045; collision cylinder length=0.0161 radius=0.045
- link l_lleg: geometry collision cylinder length=0.20 radius=0.06; collision cylinder length=0.22 radius=0.06
- link l_talus: mass 0.1 -> 0.817
- link l_uleg: geometry collision cylinder length=0.10 radius=0.1; collision cylinder length=0.15 radius=0.07
- link pelvis: geometry collision cylinder length=0.022 radius=0.130; collision cylinder length=0.022 radius=0.130
- link r_foot: mass 1.634 -> 0.817
- link r_larm: geometry collision cylinder length=0.0161 radius=0.045; collision cylinder length=0.0161 radius=0.045
- link r_lleg: geometry collision cylinder length=0.20 radius=0.06; collision cylinder length=0.22 radius=0.06
- link r_talus: mass 0.1 -> 0.817
- link r_uleg: geometry collision cylinder length=0.10 radius=0.1; collision cylinder length=0.15 radius=0.07
- link utorso: geometry collision box size=0.3188 0.24 0.3162; collision cylinder length=0.22375 radius=0.0363

File: ros/multisense_sl_description/urdf/multisense_sl.urdf (robot description, URDF)
Before this commit: robot multisense_sl, 11 links, 10 joints
Links:
- added link head_imu_link, mass 0.1; visual box size=0.01 0.01 0.01
Joints:
- added joint head_imu_joint: type fixed, parent head, child head_imu_link, origin xyz=-0.0475 0.035 0.0 rpy=0 0 0

Commit message: merging from atlas_inertial_tweaks.  fix one deprecated function call on ConnectWorldUpdateStart.

File: ros/atlas_description/urdf/atlas_simple_shapes.urdf (robot description, URDF)
Before this commit: robot drc_skeleton, 28 links, 28 joints
Links:
- link l_foot: mass 0.817 -> 0.867
- link l_lglut: mass 0.69 -> 0.803
- link l_talus: mass 0.817 -> 0.867
- link l_uglut: mass 0.5166 -> 1.51622
- link l_uleg: mass 7.34 -> 7.227
- link mtorso: mass 0.55 -> 3.8068
- link pelvis: mass 14.2529 -> 13.646
- link r_foot: mass 0.817 -> 0.867
- link r_lglut: mass 0.69 -> 0.803
- link r_talus: mass 0.817 -> 0.867
- link r_uglut: mass 0.5166 -> 1.51622
- link r_uleg: mass 7.34 -> 7.227
- link utorso: mass 18.484 -> 15.2272

File: ros/multisense_sl_description/urdf/multisense_sl.urdf (robot description, URDF)
Before this commit: robot multisense_sl, 12 links, 11 joints
Links:
- link center_bottom_led_frame: mass 0.1 -> 1e-5
- link center_top_led_frame: mass 0.1 -> 1e-5
- link head: mass 1.4199 -> 1.41984
- link head_hokuyo_frame: mass 0.01 -> 1e-5
- link head_imu_link: mass 0.1 -> 1e-5
- link hokuyo_link: mass 0.057664 -> 0.057654
- link left_camera_frame: mass 0.1 -> 1e-5
- link left_led_frame: mass 0.1 -> 1e-5
- link right_camera_frame: mass 0.1 -> 1e-5
- link right_led_frame: mass 0.1 -> 1e-5

Commit message: merging from default

File: ros/atlas_description/urdf/atlas_simple_shapes.urdf (robot description, URDF)
Before this commit: robot drc_skeleton, 28 links, 28 joints
Links:
- link ltorso: mass 1.92 -> 1.62729
- link pelvis: mass 13.646 -> 12.54638

Commit message: Merged from default

File: ros/atlas_description/urdf/atlas_simple_shapes.urdf (robot description, URDF)
Before this commit: robot drc_skeleton, 28 links, 28 joints
Links:
- link l_foot: mass 0.817 -> 0.867
- link l_lglut: mass 0.69 -> 0.803
- link l_talus: mass 0.817 -> 0.867
- link l_uglut: mass 0.5166 -> 1.51622
- link l_uleg: mass 7.34 -> 7.227
- link ltorso: mass 1.92 -> 1.62729
- link mtorso: mass 0.55 -> 3.8068
- link pelvis: mass 14.2529 -> 12.54638
- link r_foot: mass 0.817 -> 0.867
- link r_lglut: mass 0.69 -> 0.803
- link r_talus: mass 0.817 -> 0.867
- link r_uglut: mass 0.5166 -> 1.51622
- link r_uleg: mass 7.34 -> 7.227
- link utorso: mass 18.484 -> 15.2272

File: ros/multisense_sl_description/urdf/multisense_sl.urdf (robot description, URDF)
Before this commit: robot multisense_sl, 12 links, 11 joints
Links:
- link center_bottom_led_frame: mass 0.1 -> 1e-5
- link center_top_led_frame: mass 0.1 -> 1e-5
- link head: mass 1.4199 -> 1.41984
- link head_hokuyo_frame: mass 0.01 -> 1e-5
- link head_imu_link: mass 0.1 -> 1e-5
- link hokuyo_link: mass 0.057664 -> 0.057654
- link left_camera_frame: mass 0.1 -> 1e-5
- link left_led_frame: mass 0.1 -> 1e-5
- link right_camera_frame: mass 0.1 -> 1e-5
- link right_led_frame: mass 0.1 -> 1e-5

Commit message: adjust l_lleg, r_lleg, l_foot and r_foot collision to match new visuals.

File: ros/atlas_description/urdf/atlas_simple_shapes.urdf (robot description, URDF)
Before this commit: robot drc_skeleton, 28 links, 28 joints
Links:
- link l_foot: geometry collision box size=0.26 0.124887 0.05; visual mesh filename=package://atlas/meshes/l_foot.dae scale=1 1 1
- link l_lleg: geometry collision cylinder length=0.40 radius=0.07; visual mesh filename=package://atlas/meshes/l_lleg.dae scale=1 1 1
- link r_foot: geometry collision box size=0.26 0.124887 0.05; visual mesh filename=package://atlas/meshes/r_foot.dae scale=1 1 1
- link r_lleg: geometry collision cylinder length=0.40 radius=0.07; visual mesh filename=package://atlas/meshes/r_lleg.dae scale=1 1 1

Commit message: adjust collision shapes for pelvis and r_lleg, l_lleg

File: ros/atlas_description/urdf/atlas_simple_shapes.urdf (robot description, URDF)
Before this commit: robot drc_skeleton, 28 links, 28 joints
Links:
- link pelvis: geometry collision cylinder length=0.05 radius=0.16; collision cylinder length=0.05 radius=0.16

Commit message: rear tripod

File: ros/atlas_description/urdf/atlas_simple_shapes.urdf (robot description, URDF)
Before this commit: robot drc_skeleton, 28 links, 28 joints
Links:
- link pelvis: geometry collision box size=0.1 0.15 0.2; collision cylinder length=0.05 radius=0.16

Commit message: new head kinematics, neck pivot point shifted forward 5.117cm and upward 2.973cm.

File: ros/atlas_description/urdf/atlas_simple_shapes.urdf (robot description, URDF)
Before this commit: robot drc_skeleton, 28 links, 28 joints
Joints:
- joint neck_ay: origin xyz=0.16555 0 0.50823 rpy=0 -0 0 -> xyz=0.21672 0 0.53796 rpy=0 -0 0

Commit message: testing changing visual to match collision

File: ros/atlas_description/urdf/atlas_simple_shapes.urdf (robot description, URDF)
Before this commit: robot drc_skeleton, 28 links, 28 joints
Links:
- link l_foot: geometry collision box size=0.26 0.124887 0.01; visual mesh filename=package://atlas/meshes/l_foot.dae scale=1 1 1
- link l_lleg: geometry collision cylinder length=0.20 radius=0.06; collision cylinder length=0.22 radius=0.06
- link pelvis: geometry collision box size=0.1 0.15 0.2; collision cylinder length=0.022 radius=0.130
- link r_foot: geometry collision box size=0.26 0.124887 0.01; visual mesh filename=package://atlas/meshes/r_foot.dae scale=1 1 1
- link r_lleg: geometry collision cylinder length=0.20 radius=0.06; collision cylinder length=0.22 radius=0.06

Commit message: revert neck kinematics change, hold for after VRC.

File: ros/atlas_description/urdf/atlas_simple_shapes.urdf (robot description, URDF)
Before this commit: robot drc_skeleton, 28 links, 28 joints
Joints:
- joint neck_ay: origin xyz=0.21672 0 0.53796 rpy=0 -0 0 -> xyz=0.16555 0 0.50823 rpy=0 -0 0
