Commit message: adjust collada unit, name and urdf scale

File: ros/atlas_description/urdf/atlas_simple_shapes.urdf (robot description, URDF)
Before this commit: robot drc_skeleton, 28 links, 28 joints
Links:
- link l_lleg: geometry collision cylinder length=0.40 radius=0.07; visual mesh filename=package://atlas/meshes/l_lleg.dae scale=100. 100. 100.
- link l_uleg: geometry collision cylinder length=0.10 radius=0.1; collision cylinder length=0.15 radius=0.07
- link pelvis: geometry collision box size=0.1 0.15 0.2; collision cylinder length=0.05 radius=0.16
- link r_larm: geometry collision cylinder length=0.0161 radius=0.045; collision cylinder length=0.0161 radius=0.045
- link r_lglut: geometry collision cylinder length=0.060306 radius=0.02009687; collision cylinder length=0.12 radius=0.02
- link r_lleg: geometry collision cylinder length=0.40 radius=0.07; visual mesh filename=package://atlas/meshes/r_lleg.dae scale=100. 100. 100.
- link r_uarm: geometry collision cylinder length=0.088934 radius=0.04504847; collision cylinder length=0.116677 radius=0.0449
- link r_uglut: geometry collision cylinder length=0.078396 radius=0.019096; collision cylinder length=0.080842 radius=0.019841
- link r_uleg: geometry collision cylinder length=0.10 radius=0.1; collision cylinder length=0.15 radius=0.07

Commit message: updated collision geometries to new mesh visuals

File: ros/atlas_description/urdf/atlas_simple_shapes.urdf (robot description, URDF)
Before this commit: robot drc_skeleton, 28 links, 28 joints
Links:
- link l_clav: geometry collision box size=0.13 0.15 0.05; collision cylinder length=0.1525 radius=0.045
- link l_farm: geometry collision box size=0.135 0.1 0.045; collision cylinder length=0.125 radius=0.045
- link l_hand: geometry collision box size=0.13 0.09 0.07; collision cylinder length=0.05 radius=0.03
- link l_larm: geometry collision box size=0.135 0.15 0.06; collision cylinder length=0.125 radius=0.045
- link l_scap: geometry collision box size=0.15 0.15 0.06; collision cylinder length=0.125 radius=0.045
- link l_uarm: geometry collision box size=0.04 0.07 0.13; collision cylinder length=0.125 radius=0.045
- link r_clav: geometry collision box size=0.13 0.15 0.05; collision cylinder length=0.1525 radius=0.045
- link r_farm: geometry collision box size=0.135 0.1 0.045; collision cylinder length=0.125 radius=0.045
- link r_hand: geometry collision box size=0.13 0.09 0.07; collision cylinder length=0.05 radius=0.03
- link r_larm: geometry collision box size=0.135 0.15 0.06; collision cylinder length=0.125 radius=0.045
- link r_scap: geometry collision box size=0.15 0.15 0.06; collision cylinder length=0.125 radius=0.045
- link r_uarm: geometry collision box size=0.04 0.07 0.13; collision cylinder length=0.125 radius=0.045
Joints:
- joint neck_ay: origin xyz=0.16555 0 0.50823 rpy=0 -0 0 -> xyz=0.21672 0 0.53796 rpy=0 -0 0

Commit message: hacking

File: ros/atlas_description/urdf/atlas_simple_shapes.urdf (robot description, URDF)
Before this commit: robot drc_skeleton, 28 links, 28 joints
Links:
- link l_foot: geometry collision box size=0.13 0.124887 0.05; collision box size=0.13 0.124887 0.05
- link r_foot: geometry collision box size=0.13 0.124887 0.05; collision box size=0.13 0.124887 0.05

Commit message: make foot friction coefficient 1.5

File: ros/atlas_description/urdf/atlas_simple_shapes.urdf (robot description, URDF)
Before this commit: robot drc_skeleton, 28 links, 28 joints
Links:
- link l_foot: geometry collision box size=0.26 0.124887 0.05; visual mesh filename=package://atlas/meshes/l_foot.dae scale=1 1 1
- link r_foot: geometry collision box size=0.26 0.124887 0.05; visual mesh filename=package://atlas/meshes/r_foot.dae scale=1 1 1

Commit message: increasing upper limit of uay from 0.698 to 0.9 radians

File: ros/atlas_description/urdf/atlas_simple_shapes.urdf (robot description, URDF)
Before this commit: robot drc_skeleton, 28 links, 28 joints
Joints:
- joint l_leg_uay: limit lower=-0.698 upper=0.698 effort=220 velocity=12 -> lower=-0.698 upper=0.9 effort=220 velocity=12
- joint r_leg_uay: limit lower=-0.698 upper=0.698 effort=220 velocity=12 -> lower=-0.698 upper=0.9 effort=220 velocity=12

Commit message: flip bounds.

File: ros/atlas_description/urdf/atlas_simple_shapes.urdf (robot description, URDF)
Before this commit: robot drc_skeleton, 28 links, 28 joints
Joints:
- joint l_leg_uay: limit lower=-0.698 upper=0.9 effort=220 velocity=12 -> lower=-0.9 upper=0.698 effort=220 velocity=12
- joint r_leg_uay: limit lower=-0.698 upper=0.9 effort=220 velocity=12 -> lower=-0.9 upper=0.698 effort=220 velocity=12

Commit message: Merged in drcsim_2.6 (pull request #334)
merge 2.6 to default

File: ros/atlas_description/urdf/atlas_simple_shapes.urdf (robot description, URDF)
Before this commit: robot drc_skeleton, 28 links, 28 joints
Joints:
- joint l_leg_kny: limit lower=0 upper=2.45 effort=220 velocity=12 -> lower=0 upper=2.45 effort=400 velocity=12
- joint l_leg_uay: limit lower=-0.698 upper=0.698 effort=220 velocity=12 -> lower=-0.9 upper=0.698 effort=220 velocity=12
- joint r_leg_kny: limit lower=0 upper=2.45 effort=220 velocity=12 -> lower=0 upper=2.45 effort=400 velocity=12
- joint r_leg_uay: limit lower=-0.698 upper=0.698 effort=220 velocity=12 -> lower=-0.9 upper=0.698 effort=220 velocity=12
