Commit message: fix link name

File: ros/atlas_description/urdf/atlas_v3_with_v1_inertia.urdf (robot description, URDF)
Before this commit: robot drc_skeleton, 32 links, 32 joints
Joints:
- joint l_situational_awareness_camera_optical_frame_joint: parent l_situational_awareness_camera_frame -> l_situational_awareness_camera_link
- joint r_situational_awareness_camera_optical_frame_joint: parent r_situational_awareness_camera_frame -> r_situational_awareness_camera_link

Commit message: fix atlas_v3_with_v1_inertia.urdf to refer to the right mesh resources.

File: ros/atlas_description/urdf/atlas_v3_with_v1_inertia.urdf (robot description, URDF)
Before this commit: robot drc_skeleton, 32 links, 32 joints
Links:
- link l_clav: geometry collision mesh filename=package://atlas_description/meshes_v3/l_clav.DAE scale=1 1 1; visual mesh filename=package://atlas_description/meshes_v3/l_clav.DAE scale=1 1 1
- link l_farm: geometry collision mesh filename=package://atlas_description/meshes_v3/l_farm.DAE scale=1 1 1; visual mesh filename=package://atlas_description/meshes_v3/l_farm.DAE scale=1 1 1
- link l_foot: geometry collision mesh filename=package://atlas_description/meshes_v3/l_foot.DAE scale=1 1 1; visual mesh filename=package://atlas_description/meshes_v3/l_foot.DAE scale=1 1 1
- link l_hand: geometry collision mesh filename=package://atlas_description/meshes_v3/l_hand.DAE scale=1 1 1; visual mesh filename=package://atlas_description/meshes_v3/l_hand.DAE scale=1 1 1
- link l_larm: geometry collision mesh filename=package://atlas_description/meshes_v3/l_elbow_rx.DAE scale=1 1 1; visual mesh filename=package://atlas_description/meshes_v3/l_elbow_rx.DAE scale=1 1 1
- link l_lglut: geometry collision mesh filename=package://atlas_description/meshes_v3/l_lglut.DAE scale=1 1 1; visual mesh filename=package://atlas_description/meshes_v3/l_lglut.DAE scale=1 1 1
- link l_lleg: geometry collision mesh filename=package://atlas_description/meshes_v3/l_lleg.DAE scale=1 1 1; visual mesh filename=package://atlas_description/meshes_v3/l_lleg.DAE scale=1 1 1
- link l_scap: geometry collision mesh filename=package://atlas_description/meshes_v3/l_sh_rx.DAE scale=1 1 1; visual mesh filename=package://atlas_description/meshes_v3/l_sh_rx.DAE scale=1 1 1
- link l_talus: geometry collision mesh filename=package://atlas_description/meshes_v3/l_talus.DAE scale=1 1 1; visual mesh filename=package://atlas_description/meshes_v3/l_talus.DAE scale=1 1 1
- link l_uarm: geometry collision mesh filename=package://atlas_description/meshes_v3/l_elbow_ry.DAE scale=1 1 1; visual mesh filename=package://atlas_description/meshes_v3/l_elbow_ry.DAE scale=1 1 1
- link l_uglut: geometry collision mesh filename=package://atlas_description/meshes_v3/l_uglut.DAE scale=1 1 1; visual mesh filename=package://atlas_description/meshes_v3/l_uglut.DAE scale=1 1 1
- link l_uleg: geometry collision mesh filename=package://atlas_description/meshes_v3/l_uleg.DAE scale=1 1 1; visual mesh filename=package://atlas_description/meshes_v3/l_uleg.DAE scale=1 1 1
- link ltorso: geometry collision mesh filename=package://atlas_description/meshes_v3/ltorso.DAE scale=1 1 1; visual mesh filename=package://atlas_description/meshes_v3/ltorso.DAE scale=1 1 1
- link mtorso: geometry collision mesh filename=package://atlas_description/meshes_v3/mtorso.DAE scale=1 1 1; visual mesh filename=package://atlas_description/meshes_v3/mtorso.DAE scale=1 1 1
- link pelvis: geometry collision mesh filename=package://atlas_description/meshes_v3/pelvis.DAE scale=1 1 1; visual mesh filename=package://atlas_description/meshes_v3/pelvis.DAE scale=1 1 1
- link r_clav: geometry collision mesh filename=package://atlas_description/meshes_v3/r_clav.DAE scale=1 1 1; visual mesh filename=package://atlas_description/meshes_v3/r_clav.DAE scale=1 1 1
- link r_farm: geometry collision mesh filename=package://atlas_description/meshes_v3/r_farm.DAE scale=1 1 1; visual mesh filename=package://atlas_description/meshes_v3/r_farm.DAE scale=1 1 1
- link r_foot: geometry collision mesh filename=package://atlas_description/meshes_v3/r_foot.DAE scale=1 1 1; visual mesh filename=package://atlas_description/meshes_v3/r_foot.DAE scale=1 1 1
- link r_hand: geometry collision mesh filename=package://atlas_description/meshes_v3/r_hand.DAE scale=1 1 1; visual mesh filename=package://atlas_description/meshes_v3/r_hand.DAE scale=1 1 1
- link r_larm: geometry collision mesh filename=package://atlas_description/meshes_v3/r_elbow_rx.DAE scale=1 1 1; visual mesh filename=package://atlas_description/meshes_v3/r_elbow_rx.DAE scale=1 1 1
- link r_lglut: geometry collision mesh filename=package://atlas_description/meshes_v3/r_lglut.DAE scale=1 1 1; visual mesh filename=package://atlas_description/meshes_v3/r_lglut.DAE scale=1 1 1
- link r_lleg: geometry collision mesh filename=package://atlas_description/meshes_v3/r_lleg.DAE scale=1 1 1; visual mesh filename=package://atlas_description/meshes_v3/r_lleg.DAE scale=1 1 1
- link r_scap: geometry collision mesh filename=package://atlas_description/meshes_v3/r_sh_rx.DAE scale=1 1 1; visual mesh filename=package://atlas_description/meshes_v3/r_sh_rx.DAE scale=1 1 1
- link r_talus: geometry collision mesh filename=package://atlas_description/meshes_v3/r_talus.DAE scale=1 1 1; visual mesh filename=package://atlas_description/meshes_v3/r_talus.DAE scale=1 1 1
- link r_uarm: geometry collision mesh filename=package://atlas_description/meshes_v3/r_elbow_ry.DAE scale=1 1 1; visual mesh filename=package://atlas_description/meshes_v3/r_elbow_ry.DAE scale=1 1 1
- link r_uglut: geometry collision mesh filename=package://atlas_description/meshes_v3/r_uglut.DAE scale=1 1 1; visual mesh filename=package://atlas_description/meshes_v3/r_uglut.DAE scale=1 1 1
- link r_uleg: geometry collision mesh filename=package://atlas_description/meshes_v3/r_uleg.DAE scale=1 1 1; visual mesh filename=package://atlas_description/meshes_v3/r_uleg.DAE scale=1 1 1
- link utorso: geometry collision mesh filename=package://atlas_description/meshes_v3/utorso.DAE scale=1 1 1; collision mesh filename=package://atlas_description/meshes_v3/utorso_pack.DAE scale=1 1 1

Commit message: fix atlas_v3_with_v1_inertia.urdf to refer to the right mesh resources.

File: ros/atlas_description/urdf/atlas_v3_with_v1_inertia.urdf (robot description, URDF)
Before this commit: robot drc_skeleton, 32 links, 32 joints
Links:
- link l_clav: geometry collision mesh filename=package://atlas/meshes_v3/l_clav.DAE scale=1 1 1; visual mesh filename=package://atlas/meshes_v3/l_clav.DAE scale=1 1 1
- link l_farm: geometry collision mesh filename=package://atlas/meshes_v3/l_farm.DAE scale=1 1 1; visual mesh filename=package://atlas/meshes_v3/l_farm.DAE scale=1 1 1
- link l_foot: geometry collision mesh filename=package://atlas/meshes_v3/l_foot.DAE scale=1 1 1; visual mesh filename=package://atlas/meshes_v3/l_foot.DAE scale=1 1 1
- link l_hand: geometry collision mesh filename=package://atlas/meshes_v3/l_hand.DAE scale=1 1 1; visual mesh filename=package://atlas/meshes_v3/l_hand.DAE scale=1 1 1
- link l_larm: geometry collision mesh filename=package://atlas/meshes_v3/l_elbow_rx.DAE scale=1 1 1; visual mesh filename=package://atlas/meshes_v3/l_elbow_rx.DAE scale=1 1 1
- link l_lglut: geometry collision mesh filename=package://atlas/meshes_v3/l_lglut.DAE scale=1 1 1; visual mesh filename=package://atlas/meshes_v3/l_lglut.DAE scale=1 1 1
- link l_lleg: geometry collision mesh filename=package://atlas/meshes_v3/l_lleg.DAE scale=1 1 1; visual mesh filename=package://atlas/meshes_v3/l_lleg.DAE scale=1 1 1
- link l_scap: geometry collision mesh filename=package://atlas/meshes_v3/l_sh_rx.DAE scale=1 1 1; visual mesh filename=package://atlas/meshes_v3/l_sh_rx.DAE scale=1 1 1
- link l_talus: geometry collision mesh filename=package://atlas/meshes_v3/l_talus.DAE scale=1 1 1; visual mesh filename=package://atlas/meshes_v3/l_talus.DAE scale=1 1 1
- link l_uarm: geometry collision mesh filename=package://atlas/meshes_v3/l_elbow_ry.DAE scale=1 1 1; visual mesh filename=package://atlas/meshes_v3/l_elbow_ry.DAE scale=1 1 1
- link l_uglut: geometry collision mesh filename=package://atlas/meshes_v3/l_uglut.DAE scale=1 1 1; visual mesh filename=package://atlas/meshes_v3/l_uglut.DAE scale=1 1 1
- link l_uleg: geometry collision mesh filename=package://atlas/meshes_v3/l_uleg.DAE scale=1 1 1; visual mesh filename=package://atlas/meshes_v3/l_uleg.DAE scale=1 1 1
- link ltorso: geometry collision mesh filename=package://atlas/meshes_v3/ltorso.DAE scale=1 1 1; visual mesh filename=package://atlas/meshes_v3/ltorso.DAE scale=1 1 1
- link mtorso: geometry collision mesh filename=package://atlas/meshes_v3/mtorso.DAE scale=1 1 1; visual mesh filename=package://atlas/meshes_v3/mtorso.DAE scale=1 1 1
- link pelvis: geometry collision mesh filename=package://atlas/meshes_v3/pelvis.DAE scale=1 1 1; visual mesh filename=package://atlas/meshes_v3/pelvis.DAE scale=1 1 1
- link r_clav: geometry collision mesh filename=package://atlas/meshes_v3/r_clav.DAE scale=1 1 1; visual mesh filename=package://atlas/meshes_v3/r_clav.DAE scale=1 1 1
- link r_farm: geometry collision mesh filename=package://atlas/meshes_v3/r_farm.DAE scale=1 1 1; visual mesh filename=package://atlas/meshes_v3/r_farm.DAE scale=1 1 1
- link r_foot: geometry collision mesh filename=package://atlas/meshes_v3/r_foot.DAE scale=1 1 1; visual mesh filename=package://atlas/meshes_v3/r_foot.DAE scale=1 1 1
- link r_hand: geometry collision mesh filename=package://atlas/meshes_v3/r_hand.DAE scale=1 1 1; visual mesh filename=package://atlas/meshes_v3/r_hand.DAE scale=1 1 1
- link r_larm: geometry collision mesh filename=package://atlas/meshes_v3/r_elbow_rx.DAE scale=1 1 1; visual mesh filename=package://atlas/meshes_v3/r_elbow_rx.DAE scale=1 1 1
- link r_lglut: geometry collision mesh filename=package://atlas/meshes_v3/r_lglut.DAE scale=1 1 1; visual mesh filename=package://atlas/meshes_v3/r_lglut.DAE scale=1 1 1
- link r_lleg: geometry collision mesh filename=package://atlas/meshes_v3/r_lleg.DAE scale=1 1 1; visual mesh filename=package://atlas/meshes_v3/r_lleg.DAE scale=1 1 1
- link r_scap: geometry collision mesh filename=package://atlas/meshes_v3/r_sh_rx.DAE scale=1 1 1; visual mesh filename=package://atlas/meshes_v3/r_sh_rx.DAE scale=1 1 1
- link r_talus: geometry collision mesh filename=package://atlas/meshes_v3/r_talus.DAE scale=1 1 1; visual mesh filename=package://atlas/meshes_v3/r_talus.DAE scale=1 1 1
- link r_uarm: geometry collision mesh filename=package://atlas/meshes_v3/r_elbow_ry.DAE scale=1 1 1; visual mesh filename=package://atlas/meshes_v3/r_elbow_ry.DAE scale=1 1 1
- link r_uglut: geometry collision mesh filename=package://atlas/meshes_v3/r_uglut.DAE scale=1 1 1; visual mesh filename=package://atlas/meshes_v3/r_uglut.DAE scale=1 1 1
- link r_uleg: geometry collision mesh filename=package://atlas/meshes_v3/r_uleg.DAE scale=1 1 1; visual mesh filename=package://atlas/meshes_v3/r_uleg.DAE scale=1 1 1
- link utorso: geometry collision mesh filename=package://atlas/meshes_v3/utorso.DAE scale=1 1 1; collision mesh filename=package://atlas/meshes_v3/utorso_pack.DAE scale=1 1 1
