Commit message: change r_leg_hpz effort limit to 110 (previously 110(l) and 260(r))

File: ros/atlas_description/urdf/atlas_v3.urdf (robot description, URDF)
Before this commit: robot drc_skeleton, 28 links, 28 joints
Joints:
- joint r_leg_hpz: limit lower=-1.22173 upper=0.174533 effort=260 velocity=12 -> lower=-1.22173 upper=0.174533 effort=110 velocity=12

File: ros/atlas_description/urdf/atlas_v3_with_v1_inertia.urdf (robot description, URDF)
Before this commit: robot drc_skeleton, 28 links, 28 joints
Joints:
- joint r_leg_hpz: limit lower=-1.22173 upper=0.174533 effort=260 velocity=12 -> lower=-1.22173 upper=0.174533 effort=110 velocity=12

Commit message: add situaltional awareness camera

File: ros/atlas_description/urdf/atlas_v3.urdf (robot description, URDF)
Before this commit: robot drc_skeleton, 28 links, 28 joints
Links:
- added link l_situational_awareness_camera_link, mass 0.1; visual box size=0.01 0.01 0.01
- added link l_situational_awareness_camera_optical_frame
- added link r_situational_awareness_camera_link, mass 0.1; visual box size=0.01 0.01 0.01
- added link r_situational_awareness_camera_optical_frame
Joints:
- added joint l_situational_awareness_camera_joint: type fixed, parent utorso, child l_situational_awareness_camera_link, origin xyz=0.216409 0.121799 0.406759 rpy=-1.57079633 0 2.87979327
- added joint l_situational_awareness_camera_optical_frame_joint: type fixed, parent l_situational_awareness_camera_link, child l_situational_awareness_camera_optical_frame, origin xyz=0 0 0 rpy=-1.5708 0.0 -1.5708
- added joint r_situational_awareness_camera_joint: type fixed, parent utorso, child r_situational_awareness_camera_link, origin xyz=0.216409 -0.121799 0.406759 rpy=1.57079633 0 -2.87979327
- added joint r_situational_awareness_camera_optical_frame_joint: type fixed, parent r_situational_awareness_camera_link, child r_situational_awareness_camera_optical_frame, origin xyz=0 0 0 rpy=-1.5708 0.0 -1.5708

File: ros/atlas_description/urdf/atlas_v3_with_v1_inertia.urdf (robot description, URDF)
Before this commit: robot drc_skeleton, 28 links, 28 joints
Links:
- added link l_situational_awareness_camera_link, mass 0.1; visual box size=0.01 0.01 0.01
- added link l_situational_awareness_camera_optical_frame
- added link r_situational_awareness_camera_link, mass 0.1; visual box size=0.01 0.01 0.01
- added link r_situational_awareness_camera_optical_frame
Joints:
- added joint l_situational_awareness_camera_joint: type fixed, parent utorso, child l_situational_awareness_camera_link, origin xyz=0.216409 0.121799 0.406759 rpy=-1.57079633 0 2.87979327
- added joint l_situational_awareness_camera_optical_frame_joint: type fixed, parent l_situational_awareness_camera_frame, child l_situational_awareness_camera_optical_frame, origin xyz=0 0 0 rpy=-1.5708 0.0 -1.5708
- added joint r_situational_awareness_camera_joint: type fixed, parent utorso, child r_situational_awareness_camera_link, origin xyz=0.216409 -0.121799 0.406759 rpy=1.57079633 0 -2.87979327
- added joint r_situational_awareness_camera_optical_frame_joint: type fixed, parent r_situational_awareness_camera_frame, child r_situational_awareness_camera_optical_frame, origin xyz=0 0 0 rpy=-1.5708 0.0 -1.5708

Commit message: move <gazebo> blocks into atlas_v3.gazebo.  lower hfov for situational awareness cameras until the fisheye implementation is done.

File: ros/atlas_description/urdf/atlas_v3.urdf (robot description, URDF)
Before this commit: robot drc_skeleton, 32 links, 32 joints
Joints:
- joint l_situational_awareness_camera_joint: origin xyz=0.216409 0.121799 0.406759 rpy=-1.57079633 0 2.87979327 -> xyz=0.216409 0.121799 0.406759 rpy=-1.57079633 0 1.30899694
- joint r_situational_awareness_camera_joint: origin xyz=0.216409 -0.121799 0.406759 rpy=1.57079633 0 -2.87979327 -> xyz=0.216409 -0.121799 0.406759 rpy=1.57079633 0 -1.30899694

File: ros/atlas_description/urdf/atlas_v3_with_v1_inertia.urdf (robot description, URDF)
Before this commit: robot drc_skeleton, 32 links, 32 joints
Joints:
- joint l_situational_awareness_camera_joint: origin xyz=0.216409 0.121799 0.406759 rpy=-1.57079633 0 2.87979327 -> xyz=0.216409 0.121799 0.406759 rpy=-1.57079633 0 1.30899694
- joint r_situational_awareness_camera_joint: origin xyz=0.216409 -0.121799 0.406759 rpy=1.57079633 0 -2.87979327 -> xyz=0.216409 -0.121799 0.406759 rpy=1.57079633 0 -1.30899694

Commit message: switch collisions to use stl.

File: ros/atlas_description/urdf/atlas_v3.urdf (robot description, URDF)
Before this commit: robot drc_skeleton, 32 links, 32 joints
Links:
- link l_clav: geometry collision mesh filename=package://atlas/meshes_v3/l_clav.stl scale=1 1 1; visual mesh filename=package://atlas/meshes_v3/l_clav.DAE scale=1 1 1
- link l_farm: geometry collision mesh filename=package://atlas/meshes_v3/l_farm.stl scale=1 1 1; visual mesh filename=package://atlas/meshes_v3/l_farm.DAE scale=1 1 1
- link l_foot: geometry collision mesh filename=package://atlas/meshes_v3/l_foot.stl scale=1 1 1; visual mesh filename=package://atlas/meshes_v3/l_foot.DAE scale=1 1 1
- link l_hand: geometry collision mesh filename=package://atlas/meshes_v3/l_hand.stl scale=1 1 1; visual mesh filename=package://atlas/meshes_v3/l_hand.DAE scale=1 1 1
- link l_larm: geometry collision mesh filename=package://atlas/meshes_v3/l_elbow_rx.stl scale=1 1 1; visual mesh filename=package://atlas/meshes_v3/l_elbow_rx.DAE scale=1 1 1
- link l_lglut: geometry collision mesh filename=package://atlas/meshes_v3/l_lglut.stl scale=1 1 1; visual mesh filename=package://atlas/meshes_v3/l_lglut.DAE scale=1 1 1
- link l_lleg: geometry collision mesh filename=package://atlas/meshes_v3/l_lleg.stl scale=1 1 1; visual mesh filename=package://atlas/meshes_v3/l_lleg.DAE scale=1 1 1
- link l_scap: geometry collision mesh filename=package://atlas/meshes_v3/l_sh_rx.stl scale=1 1 1; visual mesh filename=package://atlas/meshes_v3/l_sh_rx.DAE scale=1 1 1
- link l_talus: geometry collision mesh filename=package://atlas/meshes_v3/l_talus.stl scale=1 1 1; visual mesh filename=package://atlas/meshes_v3/l_talus.DAE scale=1 1 1
- link l_uarm: geometry collision mesh filename=package://atlas/meshes_v3/l_elbow_ry.stl scale=1 1 1; visual mesh filename=package://atlas/meshes_v3/l_elbow_ry.DAE scale=1 1 1
- link l_uglut: geometry collision mesh filename=package://atlas/meshes_v3/l_uglut.stl scale=1 1 1; visual mesh filename=package://atlas/meshes_v3/l_uglut.DAE scale=1 1 1
- link l_uleg: geometry collision mesh filename=package://atlas/meshes_v3/l_uleg.stl scale=1 1 1; visual mesh filename=package://atlas/meshes_v3/l_uleg.DAE scale=1 1 1
- link ltorso: geometry collision mesh filename=package://atlas/meshes_v3/ltorso.stl scale=1 1 1; visual mesh filename=package://atlas/meshes_v3/ltorso.DAE scale=1 1 1
- link mtorso: geometry collision mesh filename=package://atlas/meshes_v3/mtorso.stl scale=1 1 1; visual mesh filename=package://atlas/meshes_v3/mtorso.DAE scale=1 1 1
- link pelvis: geometry collision mesh filename=package://atlas/meshes_v3/pelvis.stl scale=1 1 1; visual mesh filename=package://atlas/meshes_v3/pelvis.DAE scale=1 1 1
- link r_clav: geometry collision mesh filename=package://atlas/meshes_v3/r_clav.stl scale=1 1 1; visual mesh filename=package://atlas/meshes_v3/r_clav.DAE scale=1 1 1
- link r_farm: geometry collision mesh filename=package://atlas/meshes_v3/r_farm.stl scale=1 1 1; visual mesh filename=package://atlas/meshes_v3/r_farm.DAE scale=1 1 1
- link r_foot: geometry collision mesh filename=package://atlas/meshes_v3/r_foot.stl scale=1 1 1; visual mesh filename=package://atlas/meshes_v3/r_foot.DAE scale=1 1 1
- link r_hand: geometry collision mesh filename=package://atlas/meshes_v3/r_hand.stl scale=1 1 1; visual mesh filename=package://atlas/meshes_v3/r_hand.DAE scale=1 1 1
- link r_larm: geometry collision mesh filename=package://atlas/meshes_v3/r_elbow_rx.stl scale=1 1 1; visual mesh filename=package://atlas/meshes_v3/r_elbow_rx.DAE scale=1 1 1
- link r_lglut: geometry collision mesh filename=package://atlas/meshes_v3/r_lglut.stl scale=1 1 1; visual mesh filename=package://atlas/meshes_v3/r_lglut.DAE scale=1 1 1
- link r_lleg: geometry collision mesh filename=package://atlas/meshes_v3/r_lleg.stl scale=1 1 1; visual mesh filename=package://atlas/meshes_v3/r_lleg.DAE scale=1 1 1
- link r_scap: geometry collision mesh filename=package://atlas/meshes_v3/r_sh_rx.stl scale=1 1 1; visual mesh filename=package://atlas/meshes_v3/r_sh_rx.DAE scale=1 1 1
- link r_talus: geometry collision mesh filename=package://atlas/meshes_v3/r_talus.stl scale=1 1 1; visual mesh filename=package://atlas/meshes_v3/r_talus.DAE scale=1 1 1
- link r_uarm: geometry collision mesh filename=package://atlas/meshes_v3/r_elbow_ry.stl scale=1 1 1; visual mesh filename=package://atlas/meshes_v3/r_elbow_ry.DAE scale=1 1 1
- link r_uglut: geometry collision mesh filename=package://atlas/meshes_v3/r_uglut.stl scale=1 1 1; visual mesh filename=package://atlas/meshes_v3/r_uglut.DAE scale=1 1 1
- link r_uleg: geometry collision mesh filename=package://atlas/meshes_v3/r_uleg.stl scale=1 1 1; visual mesh filename=package://atlas/meshes_v3/r_uleg.DAE scale=1 1 1
- link utorso: geometry collision mesh filename=package://atlas/meshes_v3/utorso.stl scale=1 1 1; collision mesh filename=package://atlas/meshes_v3/utorso_pack.stl scale=1 1 1

File: ros/atlas_description/urdf/atlas_v3_with_v1_inertia.urdf (robot description, URDF)
Before this commit: robot drc_skeleton, 32 links, 32 joints
Links:
- link l_clav: geometry collision mesh filename=package://atlas/meshes_v3/l_clav.stl scale=1 1 1; visual mesh filename=package://atlas/meshes_v3/l_clav.DAE scale=1 1 1
- link l_farm: geometry collision mesh filename=package://atlas/meshes_v3/l_farm.stl scale=1 1 1; visual mesh filename=package://atlas/meshes_v3/l_farm.DAE scale=1 1 1
- link l_foot: geometry collision mesh filename=package://atlas/meshes_v3/l_foot.stl scale=1 1 1; visual mesh filename=package://atlas/meshes_v3/l_foot.DAE scale=1 1 1
- link l_hand: geometry collision mesh filename=package://atlas/meshes_v3/l_hand.stl scale=1 1 1; visual mesh filename=package://atlas/meshes_v3/l_hand.DAE scale=1 1 1
- link l_larm: geometry collision mesh filename=package://atlas/meshes_v3/l_elbow_rx.stl scale=1 1 1; visual mesh filename=package://atlas/meshes_v3/l_elbow_rx.DAE scale=1 1 1
- link l_lglut: geometry collision mesh filename=package://atlas/meshes_v3/l_lglut.stl scale=1 1 1; visual mesh filename=package://atlas/meshes_v3/l_lglut.DAE scale=1 1 1
- link l_lleg: geometry collision mesh filename=package://atlas/meshes_v3/l_lleg.stl scale=1 1 1; visual mesh filename=package://atlas/meshes_v3/l_lleg.DAE scale=1 1 1
- link l_scap: geometry collision mesh filename=package://atlas/meshes_v3/l_sh_rx.stl scale=1 1 1; visual mesh filename=package://atlas/meshes_v3/l_sh_rx.DAE scale=1 1 1
- link l_talus: geometry collision mesh filename=package://atlas/meshes_v3/l_talus.stl scale=1 1 1; visual mesh filename=package://atlas/meshes_v3/l_talus.DAE scale=1 1 1
- link l_uarm: geometry collision mesh filename=package://atlas/meshes_v3/l_elbow_ry.stl scale=1 1 1; visual mesh filename=package://atlas/meshes_v3/l_elbow_ry.DAE scale=1 1 1
- link l_uglut: geometry collision mesh filename=package://atlas/meshes_v3/l_uglut.stl scale=1 1 1; visual mesh filename=package://atlas/meshes_v3/l_uglut.DAE scale=1 1 1
- link l_uleg: geometry collision mesh filename=package://atlas/meshes_v3/l_uleg.stl scale=1 1 1; visual mesh filename=package://atlas/meshes_v3/l_uleg.DAE scale=1 1 1
- link ltorso: geometry collision mesh filename=package://atlas/meshes_v3/ltorso.stl scale=1 1 1; visual mesh filename=package://atlas/meshes_v3/ltorso.DAE scale=1 1 1
- link mtorso: geometry collision mesh filename=package://atlas/meshes_v3/mtorso.stl scale=1 1 1; visual mesh filename=package://atlas/meshes_v3/mtorso.DAE scale=1 1 1
- link pelvis: geometry collision mesh filename=package://atlas/meshes_v3/pelvis.stl scale=1 1 1; visual mesh filename=package://atlas/meshes_v3/pelvis.DAE scale=1 1 1
- link r_clav: geometry collision mesh filename=package://atlas/meshes_v3/r_clav.stl scale=1 1 1; visual mesh filename=package://atlas/meshes_v3/r_clav.DAE scale=1 1 1
- link r_farm: geometry collision mesh filename=package://atlas/meshes_v3/r_farm.stl scale=1 1 1; visual mesh filename=package://atlas/meshes_v3/r_farm.DAE scale=1 1 1
- link r_foot: geometry collision mesh filename=package://atlas/meshes_v3/r_foot.stl scale=1 1 1; visual mesh filename=package://atlas/meshes_v3/r_foot.DAE scale=1 1 1
- link r_hand: geometry collision mesh filename=package://atlas/meshes_v3/r_hand.stl scale=1 1 1; visual mesh filename=package://atlas/meshes_v3/r_hand.DAE scale=1 1 1
- link r_larm: geometry collision mesh filename=package://atlas/meshes_v3/r_elbow_rx.stl scale=1 1 1; visual mesh filename=package://atlas/meshes_v3/r_elbow_rx.DAE scale=1 1 1
- link r_lglut: geometry collision mesh filename=package://atlas/meshes_v3/r_lglut.stl scale=1 1 1; visual mesh filename=package://atlas/meshes_v3/r_lglut.DAE scale=1 1 1
- link r_lleg: geometry collision mesh filename=package://atlas/meshes_v3/r_lleg.stl scale=1 1 1; visual mesh filename=package://atlas/meshes_v3/r_lleg.DAE scale=1 1 1
- link r_scap: geometry collision mesh filename=package://atlas/meshes_v3/r_sh_rx.stl scale=1 1 1; visual mesh filename=package://atlas/meshes_v3/r_sh_rx.DAE scale=1 1 1
- link r_talus: geometry collision mesh filename=package://atlas/meshes_v3/r_talus.stl scale=1 1 1; visual mesh filename=package://atlas/meshes_v3/r_talus.DAE scale=1 1 1
- link r_uarm: geometry collision mesh filename=package://atlas/meshes_v3/r_elbow_ry.stl scale=1 1 1; visual mesh filename=package://atlas/meshes_v3/r_elbow_ry.DAE scale=1 1 1
- link r_uglut: geometry collision mesh filename=package://atlas/meshes_v3/r_uglut.stl scale=1 1 1; visual mesh filename=package://atlas/meshes_v3/r_uglut.DAE scale=1 1 1
- link r_uleg: geometry collision mesh filename=package://atlas/meshes_v3/r_uleg.stl scale=1 1 1; visual mesh filename=package://atlas/meshes_v3/r_uleg.DAE scale=1 1 1
- link utorso: geometry collision mesh filename=package://atlas/meshes_v3/utorso.stl scale=1 1 1; collision mesh filename=package://atlas/meshes_v3/utorso_pack.stl scale=1 1 1
