Commit message: add atlas_v3

File: atlas_description/robots/atlas_original_inertia.urdf.xacro (robot description, xacro)
@@ -1,3 +1,6 @@
 <robot name="atlas" >
+<!--
+  <include filename="$(find atlas_description)/urdf/atlas_original_inertia.urdf" />
+-->
   <include filename="$(find atlas_description)/urdf/atlas_simple_shapes_original_inertia.urdf" />
   <include filename="$(find atlas_description)/urdf/atlas.gazebo" />

File: atlas_description/urdf/atlas_original_inertia.urdf (robot description, URDF)
Before this commit: robot drc_skeleton, 28 links, 28 joints
Links:
- link l_clav: geometry collision mesh filename=package://atlas_description/meshes/l_clav.stl scale=1 1 1; visual mesh filename=package://atlas_description/meshes/l_clav.dae scale=1 1 1
- link l_farm: geometry collision mesh filename=package://atlas_description/meshes/l_farm.stl scale=1 1 1; visual mesh filename=package://atlas_description/meshes/l_farm.dae scale=1 1 1
- link l_foot: geometry collision mesh filename=package://atlas_description/meshes/l_foot.stl scale=1 1 1; visual mesh filename=package://atlas_description/meshes/l_foot.dae scale=1 1 1
- link l_hand: geometry collision mesh filename=package://atlas_description/meshes/l_hand.stl scale=1 1 1; visual mesh filename=package://atlas_description/meshes/l_hand.dae scale=1 1 1
- link l_larm: geometry collision mesh filename=package://atlas_description/meshes/l_larm.stl scale=1 1 1; visual mesh filename=package://atlas_description/meshes/l_larm.dae scale=1 1 1
- link l_lglut: geometry collision mesh filename=package://atlas_description/meshes/l_lglut.stl scale=1 1 1; visual mesh filename=package://atlas_description/meshes/l_lglut.dae scale=1 1 1
- link l_lleg: geometry collision mesh filename=package://atlas_description/meshes/l_lleg.stl scale=1 1 1; visual mesh filename=package://atlas_description/meshes/l_lleg.dae scale=1.0 1.0 1.0
- link l_scap: geometry collision mesh filename=package://atlas_description/meshes/l_scap.stl scale=1 1 1; visual mesh filename=package://atlas_description/meshes/l_scap.dae scale=1 1 1
- link l_talus: geometry collision mesh filename=package://atlas_description/meshes/l_talus.stl scale=1 1 1; visual mesh filename=package://atlas_description/meshes/l_talus.dae scale=1 1 1
- link l_uarm: geometry collision mesh filename=package://atlas_description/meshes/l_uarm.stl scale=1 1 1; visual mesh filename=package://atlas_description/meshes/l_uarm.dae scale=1 1 1
- link l_uglut: geometry collision mesh filename=package://atlas_description/meshes/l_uglut.stl scale=1 1 1; visual mesh filename=package://atlas_description/meshes/l_uglut.dae scale=1 1 1
- link l_uleg: geometry collision mesh filename=package://atlas_description/meshes/l_uleg.stl scale=1 1 1; visual mesh filename=package://atlas_description/meshes/l_uleg.dae scale=1.0 1.0 1.0
- link ltorso: geometry collision mesh filename=package://atlas_description/meshes/ltorso.stl scale=1 1 1; visual mesh filename=package://atlas_description/meshes/ltorso.dae scale=1 1 1
- link mtorso: geometry collision mesh filename=package://atlas_description/meshes/mtorso.stl scale=1 1 1; visual mesh filename=package://atlas_description/meshes/mtorso.dae scale=1 1 1
- link pelvis: geometry collision mesh filename=package://atlas_description/meshes/pelvis.stl scale=1 1 1; visual mesh filename=package://atlas_description/meshes/pelvis.dae scale=1.0 1.0 1.0
- link r_clav: geometry collision mesh filename=package://atlas_description/meshes/r_clav.stl scale=1 1 1; visual mesh filename=package://atlas_description/meshes/r_clav.dae scale=1 1 1
- link r_farm: geometry collision mesh filename=package://atlas_description/meshes/r_farm.stl scale=1 1 1; visual mesh filename=package://atlas_description/meshes/r_farm.dae scale=1 1 1
- link r_foot: geometry collision mesh filename=package://atlas_description/meshes/r_foot.stl scale=1 1 1; visual mesh filename=package://atlas_description/meshes/r_foot.dae scale=1 1 1
- link r_hand: geometry collision mesh filename=package://atlas_description/meshes/r_hand.stl scale=1 1 1; visual mesh filename=package://atlas_description/meshes/r_hand.dae scale=1 1 1
- link r_larm: geometry collision mesh filename=package://atlas_description/meshes/r_larm.stl scale=1 1 1; visual mesh filename=package://atlas_description/meshes/r_larm.dae scale=1.0 1.0 1.0
- link r_lglut: geometry collision mesh filename=package://atlas_description/meshes/r_lglut.stl scale=1 1 1; visual mesh filename=package://atlas_description/meshes/r_lglut.dae scale=1.0 1.0 1.0
- link r_lleg: geometry collision mesh filename=package://atlas_description/meshes/r_lleg.stl scale=1 1 1; visual mesh filename=package://atlas_description/meshes/r_lleg.dae scale=1.0 1.0 1.0
- link r_scap: geometry collision mesh filename=package://atlas_description/meshes/r_scap.stl scale=1 1 1; visual mesh filename=package://atlas_description/meshes/r_scap.dae scale=1 1 1
- link r_talus: geometry collision mesh filename=package://atlas_description/meshes/r_talus.stl scale=1 1 1; visual mesh filename=package://atlas_description/meshes/r_talus.dae scale=1 1 1
- link r_uarm: geometry collision mesh filename=package://atlas_description/meshes/r_uarm.stl scale=1 1 1; visual mesh filename=package://atlas_description/meshes/r_uarm.dae scale=1.0 1.0 1.0
- link r_uglut: geometry collision mesh filename=package://atlas_description/meshes/r_uglut.stl scale=1 1 1; visual mesh filename=package://atlas_description/meshes/r_uglut.dae scale=1.0 1.0 1.0
- link r_uleg: geometry collision mesh filename=package://atlas_description/meshes/r_uleg.stl scale=1 1 1; visual mesh filename=package://atlas_description/meshes/r_uleg.dae scale=1.0 1.0 1.0
- link utorso: geometry collision mesh filename=package://atlas_description/meshes/utorso.stl scale=1 1 1; visual mesh filename=package://atlas_description/meshes/utorso.dae scale=1 1 1

File: atlas_description/urdf/atlas_simple_shapes_original_inertia.urdf (robot description, URDF)
Before this commit: robot drc_skeleton, 28 links, 28 joints
Links:
- link l_clav: geometry collision cylinder length=0.027 radius=0.04; collision cylinder length=0.1525 radius=0.045
- link l_farm: geometry collision cylinder length=0.035181 radius=0.0458825; collision cylinder length=0.050472 radius=0.0279
- link l_foot: mass 0.867 -> 1.634; geometry collision box size=0.26 0.124887 0.01; visual mesh filename=package://atlas_description/meshes/l_foot.dae scale=1 1 1
- link l_hand: geometry collision cylinder length=0.019 radius=0.035939; collision cylinder length=0.019 radius=0.035939
- link l_larm: geometry collision cylinder length=0.0161 radius=0.045; collision cylinder length=0.0161 radius=0.045
- link l_lglut: mass 0.803 -> 0.69; geometry collision cylinder length=0.060306 radius=0.02009687; collision cylinder length=0.12 radius=0.02
- link l_lleg: geometry collision cylinder length=0.20 radius=0.06; collision cylinder length=0.22 radius=0.06
- link l_scap: geometry collision cylinder length=0.013737 radius=0.048709; collision cylinder length=0.013937 radius=0.048709
- link l_talus: mass 0.867 -> 0.1; geometry collision cylinder length=0.010059 radius=0.010348; collision cylinder length=0.029542 radius=0.010181
- link l_uarm: geometry collision cylinder length=0.088934 radius=0.04504847; collision cylinder length=0.116677 radius=0.0449
- link l_uglut: mass 1.51622 -> 0.5166; geometry collision cylinder length=0.078396 radius=0.019096; collision cylinder length=0.080842 radius=0.019841
- link l_uleg: mass 7.227 -> 7.34; geometry collision cylinder length=0.10 radius=0.1; collision cylinder length=0.15 radius=0.07
- link ltorso: geometry visual mesh filename=package://atlas_description/meshes/ltorso.dae scale=1 1 1
- link mtorso: mass 3.8068 -> 0.55; geometry collision cylinder length=0.02 radius=0.015; collision cylinder length=0.02 radius=0.015
- link pelvis: mass 13.646 -> 14.2529; geometry collision cylinder length=0.022 radius=0.130; collision cylinder length=0.022 radius=0.130
- link r_clav: geometry collision cylinder length=0.027 radius=0.04; collision cylinder length=0.1525 radius=0.045
- link r_farm: geometry collision cylinder length=0.035181 radius=0.0458825; collision cylinder length=0.050472 radius=0.0279
- link r_foot: mass 0.867 -> 1.634; geometry collision box size=0.26 0.124887 0.01; visual mesh filename=package://atlas_description/meshes/r_foot.dae scale=1 1 1
- link r_hand: geometry collision cylinder length=0.019 radius=0.035939; collision cylinder length=0.019 radius=0.035939
- link r_larm: geometry collision cylinder length=0.0161 radius=0.045; collision cylinder length=0.0161 radius=0.045
- link r_lglut: mass 0.803 -> 0.69; geometry collision cylinder length=0.060306 radius=0.02009687; collision cylinder length=0.12 radius=0.02
- link r_lleg: geometry collision cylinder length=0.20 radius=0.06; collision cylinder length=0.22 radius=0.06
- link r_scap: geometry collision cylinder length=0.013737 radius=0.048709; collision cylinder length=0.013937 radius=0.048709
- link r_talus: mass 0.867 -> 0.1; geometry collision cylinder length=0.010059 radius=0.010348; collision cylinder length=0.029542 radius=0.010181
- link r_uarm: geometry collision cylinder length=0.088934 radius=0.04504847; collision cylinder length=0.116677 radius=0.0449
- link r_uglut: mass 1.51622 -> 0.5166; geometry collision cylinder length=0.078396 radius=0.019096; collision cylinder length=0.080842 radius=0.019841
- link r_uleg: mass 7.227 -> 7.34; geometry collision cylinder length=0.10 radius=0.1; collision cylinder length=0.15 radius=0.07
- link utorso: mass 15.2272 -> 18.484; geometry collision box size=0.3188 0.24 0.3162; collision cylinder length=0.22375 radius=0.0363
Joints:
- joint l_leg_kny: limit lower=0 upper=2.45 effort=220 velocity=12 -> lower=0 upper=2.45 effort=400 velocity=12
- joint l_leg_uay: limit lower=-0.698 upper=0.698 effort=220 velocity=12 -> lower=-0.9 upper=0.698 effort=220 velocity=12
- joint neck_ay: origin xyz=0.16555 0 0.50823 rpy=0 -0 0 -> xyz=0.21672 0 0.53796 rpy=0 -0 0
- joint r_leg_kny: limit lower=0 upper=2.45 effort=220 velocity=12 -> lower=0 upper=2.45 effort=400 velocity=12
- joint r_leg_uay: limit lower=-0.698 upper=0.698 effort=220 velocity=12 -> lower=-0.9 upper=0.698 effort=220 velocity=12
- joint r_leg_uhz: limit lower=-1.14 upper=0.32 effort=260 velocity=12 -> lower=-1.14 upper=0.32 effort=110 velocity=12
