Commit message: merging from default

File: atlas_description/robots/atlas_v3_with_v1_inertia.urdf.xacro (robot description, xacro)
@@ -1,4 +1,4 @@
 <robot name="atlas" >
-  <include filename="$(find atlas_description)/urdf/atlas_v3.urdf" />
+  <include filename="$(find atlas_description)/urdf/atlas_v3_with_v1_inertia.urdf" />
   <include filename="$(find atlas_description)/urdf/atlas_v3.gazebo" />
   <include filename="$(find atlas_description)/urdf/atlas_v3.transmission" />

File: atlas_description/urdf/atlas_v3_with_v1_inertia.urdf (robot description, URDF)
Before this commit: robot drc_skeleton, 32 links, 32 joints
Links:
- link l_clav: mass 3.45 -> 2.369
- link l_farm: mass 3.388 -> 0.981
- link l_foot: mass 2.05 -> 1.634
- link l_hand: mass 2.509 -> 2.263
- link l_larm: mass 2.509 -> 2.148
- link l_lglut: mass 0.866 -> 0.69
- link l_lleg: mass 5.479 -> 4.367
- link l_scap: mass 3.012 -> 2.707
- link l_talus: mass 0.125 -> 0.1
- link l_uarm: mass 3.388 -> 1.881
- link l_uglut: mass 0.648 -> 0.5166
- link l_uleg: mass 9.209 -> 7.34
- link ltorso: mass 2.409 -> 1.92
- link mtorso: mass 0.69 -> 0.55
- link pelvis: mass 17.882 -> 14.2529
- link r_clav: mass 3.45 -> 2.369
- link r_farm: mass 3.388 -> 0.981
- link r_foot: mass 2.05 -> 1.634
- link r_hand: mass 2.509 -> 2.263
- link r_larm: mass 2.509 -> 2.148
- link r_lglut: mass 0.866 -> 0.69
- link r_lleg: mass 5.479 -> 4.367
- link r_scap: mass 3.012 -> 2.707
- link r_talus: mass 0.125 -> 0.1
- link r_uarm: mass 3.388 -> 1.881
- link r_uglut: mass 0.648 -> 0.5166
- link r_uleg: mass 9.209 -> 7.34
- link utorso: mass 52.007 -> 18.484
