Commit message: update launch files for atlas with irobot hands

File: atlas_description/robots/atlas_v3_with_v1_inertia_irobot_hands.urdf.xacro (robot description, xacro)
@@ -1,10 +1,10 @@
 <robot xmlns:xacro="http://www.ros.org/wiki/xacro" name="atlas" >
-  <xacro:include filename="$(find atlas_description)/urdf/atlas_simple_shapes.urdf" />
+  <xacro:include filename="$(find atlas_description)/urdf/atlas_v3.urdf" />
   <xacro:include filename="$(find irobot_hand_description)/urdf/irobot_hand.urdf.xacro" />
   <xacro:irobot_hand side="right" parent="r_hand" reflect="1">
-    <origin rpy="1.57079 0 0" xyz="0 -0.09 0"/>
+    <origin xyz="-0.00179 -0.09516 0.01176" rpy="1.57079 0 0"/>
   </xacro:irobot_hand>
   <xacro:irobot_hand side="left" parent="l_hand" reflect="-1">
-    <origin rpy="1.57079 0 3.14159" xyz="0 0.09 0"/>
+    <origin xyz="0.00179  0.09516 0.01176" rpy="1.57079 0 3.14159"/>
   </xacro:irobot_hand>
   <gazebo>
