Commit message: merge from default

File: atlas_description/robots/atlas_v3_irobot_hands.urdf.xacro (robot description, xacro)
@@ -1,10 +1,10 @@
 <robot xmlns:xacro="http://www.ros.org/wiki/xacro" name="atlas" >
-  <xacro:include filename="$(find atlas_description)/urdf/atlas_simple_shapes.urdf" />
+  <xacro:include filename="$(find atlas_description)/urdf/atlas_v3.urdf" />
   <xacro:include filename="$(find irobot_hand_description)/urdf/irobot_hand.urdf.xacro" />
   <xacro:irobot_hand side="right" parent="r_hand" reflect="1">
-    <origin rpy="1.57079 0 0" xyz="0 -0.09 0"/>
+    <origin xyz="-0.00179 -0.09516 0.01176" rpy="1.57079 0 0"/>
   </xacro:irobot_hand>
   <xacro:irobot_hand side="left" parent="l_hand" reflect="-1">
-    <origin rpy="1.57079 0 3.14159" xyz="0 0.09 0"/>
+    <origin xyz="0.00179  0.09516 0.01176" rpy="1.57079 0 3.14159"/>
   </xacro:irobot_hand>
   <gazebo>
@@ -18,6 +18,6 @@
     </plugin>
   </gazebo>
-  <xacro:include filename="$(find atlas_description)/urdf/atlas.gazebo" />
-  <xacro:include filename="$(find atlas_description)/urdf/atlas.transmission" />
+  <xacro:include filename="$(find atlas_description)/urdf/atlas_v3.gazebo" />
+  <xacro:include filename="$(find atlas_description)/urdf/atlas_v3.transmission" />
   <xacro:include filename="$(find multisense_sl_description)/urdf/multisense_sl.urdf" />
 </robot>

File: irobot_hand_description/urdf/irobot_hand.urdf.xacro (robot description, xacro)
@@ -5,13 +5,21 @@
 <!-- tip: use measurements from solid to find the origins and length -->
 <xacro:property name="flex_joint_length" value=".016" />
-<xacro:property name="flex_joint_steps" value="9" />
+<xacro:property name="flex_joint_steps" value="2" />
 <xacro:property name="proximal_link_length" value=".062" />
 <xacro:property name="pi" value="3.14" />
+<xacro:property name="flex_offset" value="0.003"/> <!--${0.5*flex_joint_length/flex_joint_steps}-->
 <xacro:macro name="flex_link" params="side finger_id link_id">
   <link name="${side}_finger[${finger_id}]/flexible_link_${link_id}">
     <inertial>
-      <mass value="0.1"/>
-      <origin xyz="0 0 0"/>
-      <inertia ixx="0.001" ixy="0.0" ixz="0.0" iyy="0.001" iyz="0.0" izz="0.001"/>
+      <mass value="${0.0029 / (2 * flex_joint_steps + 1)}"/>
+      <!-- gazebo -> cad mapping
+           x -> y
+           y -> z
+           z -> x
+      -->
+      <origin xyz="0 0 0" rpy="${-pi/2} ${-pi/2} 0"/>
+      <inertia ixx="8.8101e-8" ixy="0" ixz="0.0"
+               iyy="${2.04906e-7 / (2 * flex_joint_steps + 1)}" iyz="0.0"
+               izz="${2.65921e-7 / (2 * flex_joint_steps + 1)}"/>
     </inertial>
     <collision>
@@ -33,4 +41,7 @@
 </xacro:macro>
 <xacro:macro name="flex_joint" params="side finger_id link_from link_to">
+  <gazebo reference="${side}_finger[${finger_id}]/flexible_joint_flex_from_${link_from}_to_${link_to}">
+    <implicitSpringDamper>1</implicitSpringDamper>
+  </gazebo>
   <joint name="${side}_finger[${finger_id}]/flexible_joint_flex_from_${link_from}_to_${link_to}" type="revolute">
     <parent link="${side}_finger[${finger_id}]/flexible_link_${link_from}"/>
@@ -42,7 +53,14 @@
   <link name="${side}_finger[${finger_id}]/flexible_link_hidden_between_${link_from}_and_${link_to}">
     <inertial>
-      <mass value="0.1"/>
-      <origin xyz="0 0 0"/>
-      <inertia ixx="0.001" ixy="0.0" ixz="0.0" iyy="0.001" iyz="0.0" izz="0.001"/>
+      <mass value="${0.0029 / (2 * flex_joint_steps + 1)}"/>
+      <!-- gazebo -> cad mapping
+           x -> y
+           y -> z
+           z -> x
+      -->
+      <origin xyz="0 0 0" rpy="${-pi/2} ${-pi/2} 0"/>
+      <inertia ixx="8.8101e-8" ixy="0" ixz="0.0"
+               iyy="${2.04906e-7 / (2 * flex_joint_steps + 1)}" iyz="0.0"
+               izz="${2.65921e-7 / (2 * flex_joint_steps + 1)}"/>
     </inertial>
     <collision>
@@ -59,4 +77,7 @@
     </visual>
   </link>
+  <gazebo reference="${side}_finger[${finger_id}]/flexible_joint_twist_from_${link_from}_to_${link_to}">
+    <implicitSpringDamper>1</implicitSpringDamper>
+  </gazebo>
   <joint name="${side}_finger[${finger_id}]/flexible_joint_twist_from_${link_from}_to_${link_to}" type="revolute">
     <parent link="${side}_finger[${finger_id}]/flexible_link_hidden_between_${link_from}_and_${link_to}"/>
@@ -69,8 +90,11 @@
 <xacro:macro name="flex_joint_connector" params="side finger_id">
   <!-- make a connection between proximal to flexible-->
+  <gazebo reference="${side}_finger[${finger_id}]/flexible_joint_flex_from_proximal_to_1">
+    <implicitSpringDamper>1</implicitSpringDamper>
+  </gazebo>
   <joint name="${side}_finger[${finger_id}]/flexible_joint_flex_from_proximal_to_1" type="revolute">
     <parent link="${side}_finger[${finger_id}]/proximal_link"/>
     <child link="${side}_finger[${finger_id}]/flexible_link_hidden_between_proximal_link_and_1"/>
-    <origin xyz="0 0 ${proximal_link_length}" />
+    <origin xyz="0 0 ${proximal_link_length + flex_offset}" />
     <axis xyz="-1 0 0"/>
     <limit effort="1000.0" lower="0.0" upper="${pi/2}" velocity="0.5"/>
@@ -78,7 +102,15 @@
   <link name="${side}_finger[${finger_id}]/flexible_link_hidden_between_proximal_link_and_1">
     <inertial>
-      <mass value="0.1"/>
-      <origin xyz="0 0 0"/>
-      <inertia ixx="0.001" ixy="0.0" ixz="0.0" iyy="0.001" iyz="0.0" izz="0.001"/>
+      <!-- <mass value="${0.0029 / 19}"/> -->
+      <mass value="${0.0029 / (2 * flex_joint_steps + 1)}"/>
+      <!-- gazebo -> cad mapping
+           x -> y
+           y -> z
+           z -> x
+      -->
+      <origin xyz="0 0 0" rpy="${-pi/2} ${-pi/2} 0"/>
+      <inertia ixx="8.8101e-8" ixy="0" ixz="0.0"
+               iyy="${2.04906e-7 / (2 * flex_joint_steps + 1)}" iyz="0.0"
+               izz="${2.65921e-7 / (2 * flex_joint_steps + 1)}"/>
     </inertial>
     <collision>
@@ -95,4 +127,7 @@
     </visual>
   </link>
+  <gazebo reference="${side}_finger[${finger_id}]/flexible_joint_twist_from_proximal_to_1">
+    <implicitSpringDamper>1</implicitSpringDamper>
+  </gazebo>
   <joint name="${side}_finger[${finger_id}]/flexible_joint_twist_from_proximal_to_1" type="revolute">
     <parent link="${side}_finger[${finger_id}]/flexible_link_hidden_between_proximal_link_and_1"/>
@@ -103,16 +138,26 @@
   </joint>
   <!-- make a connection between flexible to distal-->
-  <joint name="${side}_finger[${finger_id}]/flexible_joint_flex_from_9_to_distal" type="revolute">
-    <parent link="${side}_finger[${finger_id}]/flexible_link_9"/>
-    <child link="${side}_finger[${finger_id}]/flexible_link_hidden_between_9_and_distal_link"/>
-    <origin xyz="0 0 ${flex_joint_length/flex_joint_steps}" />
+  <gazebo reference="${side}_finger[${finger_id}]/flexible_joint_flex_from_${flex_joint_steps}_to_distal">
+    <implicitSpringDamper>1</implicitSpringDamper>
+  </gazebo>
+  <joint name="${side}_finger[${finger_id}]/flexible_joint_flex_from_${flex_joint_steps}_to_distal" type="revolute">
+    <parent link="${side}_finger[${finger_id}]/flexible_link_${flex_joint_steps}"/>
+    <child link="${side}_finger[${finger_id}]/flexible_link_hidden_between_${flex_joint_steps}_and_distal_link"/>
+    <origin xyz="0 0 ${flex_joint_length/flex_joint_steps - flex_offset}" />
     <axis xyz="-1 0 0"/>
     <limit effort="1000.0" lower="0.0" upper="${pi/2}" velocity="0.5"/>
   </joint>
-  <link name="${side}_finger[${finger_id}]/flexible_link_hidden_between_9_and_distal_link">
+  <link name="${side}_finger[${finger_id}]/flexible_link_hidden_between_${flex_joint_steps}_and_distal_link">
     <inertial>
-      <mass value="0.1"/>
-      <origin xyz="0 0 0"/>
-      <inertia ixx="0.001" ixy="0.0" ixz="0.0" iyy="0.001" iyz="0.0" izz="0.001"/>
+      <mass value="${0.0029 / (2 * flex_joint_steps + 1)}"/>
+      <!-- gazebo -> cad mapping
+           x -> y
+           y -> z
+           z -> x
+      -->
+      <origin xyz="0 0 0" rpy="${-pi/2} ${-pi/2} 0"/>
+      <inertia ixx="8.8101e-8" ixy="0" ixz="0.0"
+               iyy="${2.04906e-7 / (2 * flex_joint_steps + 1)}" iyz="0.0"
+               izz="${2.65921e-7 / (2 * flex_joint_steps + 1)}"/>
     </inertial>
     <collision>
@@ -129,6 +174,9 @@
     </visual>
   </link>
-  <joint name="${side}_finger[${finger_id}]/flexible_joint_twist_from_9_to_distal" type="revolute">
-    <parent link="${side}_finger[${finger_id}]/flexible_link_hidden_between_9_and_distal_link"/>
+  <gazebo reference="${side}_finger[${finger_id}]/flexible_joint_twist_from_${flex_joint_steps}_to_distal">
+    <implicitSpringDamper>1</implicitSpringDamper>
+  </gazebo>
+  <joint name="${side}_finger[${finger_id}]/flexible_joint_twist_from_${flex_joint_steps}_to_distal" type="revolute">
+    <parent link="${side}_finger[${finger_id}]/flexible_link_hidden_between_${flex_joint_steps}_and_distal_link"/>
     <child link="${side}_finger[${finger_id}]/distal_link"/>
     <origin xyz="0 0 0" />
@@ -136,8 +184,79 @@
     <limit effort="1000.0" lower="0.0" upper="${pi/2}" velocity="0.5"/>
   </joint>
+</xacro:macro>
+<!-- Simplified collisions for the base_rotation_links on fingers 0 and 1 -->
+<xacro:macro name="base_rotation_link_collisions">
+      <collision name='collision_1'>
+        <origin xyz="0 0 -.0025" rpy="0 0 0"/>
+        <geometry>
+          <cylinder length="0.0145" radius="0.025"/>
+        </geometry>
+      </collision>
+      <collision name='collision_2'>
+        <origin xyz="0 0 -.0104" rpy="0 0 0"/>
+        <geometry>
+          <cylinder length="0.0145" radius="0.0165"/>
+        </geometry>
+      </collision>
+      <collision name='collision_3'>
+        <origin xyz="0 0 .0135" rpy="1.5707 0 1.5707"/>
+        <geometry>
+          <cylinder length="0.02" radius="0.002"/>
+        </geometry>
+      </collision>
+      <collision name='collision_4'>
+        <origin xyz="0.013 0 .0135" rpy="1.5707 0 1.5707"/>
+        <geometry>
+          <cylinder length="0.008" radius="0.009"/>
+        </geometry>
+      </collision>
+      <collision name='collision_5'>
+        <origin xyz="-0.013 0 .0135" rpy="1.5707 0 1.5707"/>
+        <geometry>
+          <cylinder length="0.008" radius="0.009"/>
+        </geometry>
+      </collision>
+</xacro:macro>
+<!-- Simplified collisions for the proximal_link on all fingers -->
+<xacro:macro name="proximal_link_collisions">
+      <collision name='collision1'>
+        <origin xyz="0 0.0028 0.033" rpy="0 0 0"/>
+        <geometry>
+          <box size="0.018 0.019 0.055"/>
+        </geometry>
+      </collision>
+      <collision name='collision2'>
+        <origin xyz="0 0 0" rpy="0 1.5707 0"/>
+        <geometry>
+          <cylinder radius="0.009" length="0.018"/>
+        </geometry>
+      </collision>
+</xacro:macro>
+<!-- Simplified collisions for the distal_link on all fingers -->
+<xacro:macro name="distal_link_collisions">
+      <collision name='collision'>
+        <origin xyz="0 0.0024 0.01476" rpy="3.141590 0.001593
+             3.141590"/>
+        <geometry>
+          <box size="0.0175 0.02011 0.03195"/>
+        </geometry>
+      </collision>
+      <collision name='collision_tip'>
+        <origin xyz="0 0.004 0.03" rpy="1.57078 0.001593 1.57078"/>
+        <geometry>
+          <cylinder radius="0.00848" length="0.0175"/>
+        </geometry>
+      </collision>
+      <collision name='collision_nail'>
+        <origin xyz="0 -0.00529 0.032" rpy="1.57078 0.001593 0"/>
+        <geometry>
+          <cylinder radius="0.00750" length="0.00159"/>
+        </geometry>
+      </collision>
 </xacro:macro>
 <xacro:macro name="irobot_hand" params="side parent reflect *origin">
   <xacro:flex_link side="${side}" finger_id="0" link_id="1"/>
   <xacro:flex_link side="${side}" finger_id="0" link_id="2"/>
+  <!-- only up to flex_joint_steps
   <xacro:flex_link side="${side}" finger_id="0" link_id="3"/>
   <xacro:flex_link side="${side}" finger_id="0" link_id="4"/>
@@ -147,5 +266,7 @@
   <xacro:flex_link side="${side}" finger_id="0" link_id="8"/>
   <xacro:flex_link side="${side}" finger_id="0" link_id="9"/>
+  -->
   <xacro:flex_joint side="${side}" finger_id="0" link_from="1" link_to="2"/>
+  <!-- only up to flex_joint_steps
   <xacro:flex_joint side="${side}" finger_id="0" link_from="2" link_to="3"/>
   <xacro:flex_joint side="${side}" finger_id="0" link_from="3" link_to="4"/>
@@ -155,7 +276,9 @@
   <xacro:flex_joint side="${side}" finger_id="0" link_from="7" link_to="8"/>
   <xacro:flex_joint side="${side}" finger_id="0" link_from="8" link_to="9"/>
-  <xacro:flex_joint_connector side="${side}" finger_id="0"/>
+  -->
+  <xacro:flex_joint_connector side="${side}" finger_id="0" />
   <xacro:flex_link side="${side}" finger_id="1" link_id="1"/>
   <xacro:flex_link side="${side}" finger_id="1" link_id="2"/>
+  <!-- only up to flex_joint_steps
   <xacro:flex_link side="${side}" finger_id="1" link_id="3"/>
   <xacro:flex_link side="${side}" finger_id="1" link_id="4"/>
@@ -165,5 +288,7 @@
   <xacro:flex_link side="${side}" finger_id="1" link_id="8"/>
   <xacro:flex_link side="${side}" finger_id="1" link_id="9"/>
+  -->
   <xacro:flex_joint side="${side}" finger_id="1" link_from="1" link_to="2"/>
+  <!-- only up to flex_joint_steps
   <xacro:flex_joint side="${side}" finger_id="1" link_from="2" link_to="3"/>
   <xacro:flex_joint side="${side}" finger_id="1" link_from="3" link_to="4"/>
@@ -173,7 +298,9 @@
   <xacro:flex_joint side="${side}" finger_id="1" link_from="7" link_to="8"/>
   <xacro:flex_joint side="${side}" finger_id="1" link_from="8" link_to="9"/>
-  <xacro:flex_joint_connector side="${side}" finger_id="1"/>
+  -->
+  <xacro:flex_joint_connector side="${side}" finger_id="1" />
   <xacro:flex_link side="${side}" finger_id="2" link_id="1"/>
   <xacro:flex_link side="${side}" finger_id="2" link_id="2"/>
+  <!-- only up to flex_joint_steps
   <xacro:flex_link side="${side}" finger_id="2" link_id="3"/>
   <xacro:flex_link side="${side}" finger_id="2" link_id="4"/>
@@ -183,5 +310,7 @@
   <xacro:flex_link side="${side}" finger_id="2" link_id="8"/>
   <xacro:flex_link side="${side}" finger_id="2" link_id="9"/>
+  -->
   <xacro:flex_joint side="${side}" finger_id="2" link_from="1" link_to="2"/>
+  <!-- only up to flex_joint_steps
   <xacro:flex_joint side="${side}" finger_id="2" link_from="2" link_to="3"/>
   <xacro:flex_joint side="${side}" finger_id="2" link_from="3" link_to="4"/>
@@ -191,5 +320,6 @@
   <xacro:flex_joint side="${side}" finger_id="2" link_from="7" link_to="8"/>
   <xacro:flex_joint side="${side}" finger_id="2" link_from="8" link_to="9"/>
-  <xacro:flex_joint_connector side="${side}" finger_id="2"/>
+  -->
+  <xacro:flex_joint_connector side="${side}" finger_id="2" />
   <!-- joint to irobot hand -->
   <joint name="${side}_irobot_hand_joint" type="fixed">
@@ -200,13 +330,20 @@
   <link name="${side}_base_link">
       <inertial>
-        <mass value="0.1"/>
+        <!-- needs update -->
+        <mass value="1.305"/>
         <origin xyz="0 0 0"/>
-        <inertia ixx="0.001" ixy="0.0" ixz="0.0" iyy="0.001" iyz="0.0" izz="0.001"/>
-      </inertial>
-    <collision>
-      <geometry>
-        <mesh filename="package://irobot_hand_description/meshes/palm.stl"/>
-      </geometry>
-      <origin rpy="0 0 0" xyz="0 -0.038 -0.023"/>
+        <inertia ixx="0.00125" ixy="0.0" ixz="0.0" iyy="0.00125" iyz="0.0" izz="0.0002"/>
+      </inertial>
+    <collision name='collision1'>
+      <origin xyz="0 0.02 0.045" rpy="0 0 0"/>
+      <geometry>
+        <box size="0.114 0.1 0.075"/>
+      </geometry>
+    </collision>
+    <collision name='collision2'>
+      <origin xyz="0 -0.02 0.045" rpy="0 0 0"/>
+      <geometry>
+        <cylinder radius="0.0448" length="0.075"/>
+      </geometry>
     </collision>
     <visual>
@@ -222,14 +359,10 @@
   <link name="${side}_finger[0]/base_rotation_link">
       <inertial>
-        <mass value="0.1"/>
+        <!-- needs update -->
+        <mass value="0.05"/>
         <origin xyz="0 0 0"/>
-        <inertia ixx="0.001" ixy="0.0" ixz="0.0" iyy="0.001" iyz="0.0" izz="0.001"/>
-      </inertial>
-    <collision>
-      <geometry>
-        <mesh filename="package://irobot_hand_description/meshes/finger_base.stl"/>
-      </geometry>
-      <origin rpy="${pi/2} 0 0" xyz="0 0 0"/>
-    </collision>
+        <inertia ixx="0.0000125" ixy="0.0" ixz="0.0" iyy="0.0000125" iyz="0.0" izz="0.000002"/>
+      </inertial>
+    <xacro:base_rotation_link_collisions/>
     <visual>
       <geometry>
@@ -244,14 +377,14 @@
   <link name="${side}_finger[0]/proximal_link">
       <inertial>
-        <mass value="0.1"/>
-        <origin xyz="0 0 0"/>
-        <inertia ixx="0.001" ixy="0.0" ixz="0.0" iyy="0.001" iyz="0.0" izz="0.001"/>
-      </inertial>
-    <collision>
-      <geometry>
-        <mesh filename="package://irobot_hand_description/meshes/finger_proximal.stl"/>
-      </geometry>
-      <origin rpy="${pi/2} -${pi/2} 0" xyz="0 0 0"/>
-    </collision>
+        <mass value="0.0288"/>
+        <!-- gazebo -> cad coordinate mapping
+             x -> -y
+             y -> -z
+             z -> x
+        -->
+        <origin xyz="-0.002630 0.002396 0.021770" rpy="${pi/2} -${pi/2} 0"/>
+        <inertia ixx="2.420689e-6" ixy="-1.449042e-6" ixz="-7.74579e-7" iyy="1.196202e-6" iyz="1.90704e-7" izz="1.2736461e-6"/>
+      </inertial>
+    <xacro:proximal_link_collisions/>
     <visual>
       <geometry>
@@ -264,16 +397,22 @@
     </visual>
   </link>
+  <link name="${side}_finger[0]/proximal_accelerometer" />
+  <joint name="${side}_finger[0]/proximal_link_to_accelerometer" type="fixed">
+    <parent link="${side}_finger[0]/proximal_link"/>
+    <child link="${side}_finger[0]/proximal_accelerometer"/>
+    <origin rpy="${pi/2} 0 0" xyz="0 0 0.05" />
+  </joint>
   <link name="${side}_finger[0]/distal_link">
       <inertial>
-        <mass value="0.1"/>
-        <origin xyz="0 0 0"/>
-        <inertia ixx="0.001" ixy="0.0" ixz="0.0" iyy="0.001" iyz="0.0" izz="0.001"/>
-      </inertial>
-    <collision>
-      <geometry>
-        <mesh filename="package://irobot_hand_description/meshes/finger_distal.stl"/>
-      </geometry>
-      <origin rpy="0 ${pi} 0" xyz="0 0 0"/>
-    </collision>
+        <mass value="0.0133"/>
+        <!-- gazebo -> cad mapping
+             x -> -x
+             y -> y
+             z -> -z
+        -->
+        <origin xyz="-0.000066 -0.003142 0.016633" rpy="0 ${pi} 0" />
+        <inertia ixx="1.624140e-6" ixy="5.60e-10" ixz="1.33e-10" iyy="1.717885e-6" iyz="-1.19970e-7" izz="5.60221e-7"/>
+      </inertial>
+    <xacro:distal_link_collisions/>
     <visual>
       <geometry>
@@ -286,16 +425,17 @@
     </visual>
   </link>
+  <link name="${side}_finger[0]/distal_accelerometer" />
+  <joint name="${side}_finger[0]/distal_link_to_accelerometer" type="fixed">
+    <parent link="${side}_finger[0]/distal_link"/>
+    <child link="${side}_finger[0]/distal_accelerometer"/>
+    <origin rpy="${pi/2} 0 0" xyz="0 0 0.02" />
+  </joint>
   <link name="${side}_finger[1]/base_rotation_link">
       <inertial>
-        <mass value="0.1"/>
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
Commit message: merge default

File: atlas_description/robots/atlas_v3_irobot_hands.urdf.xacro (robot description, xacro)
@@ -1,4 +1,4 @@
 <robot xmlns:xacro="http://www.ros.org/wiki/xacro" name="atlas" >
-  <xacro:include filename="$(find atlas_description)/urdf/atlas_v3.urdf" />
+  <xacro:include filename="$(find atlas_description)/urdf/atlas_v3_simple_shapes.urdf" />
   <xacro:include filename="$(find irobot_hand_description)/urdf/irobot_hand.urdf.xacro" />
   <xacro:irobot_hand side="right" parent="r_hand" reflect="1">
@@ -6,5 +6,5 @@
   </xacro:irobot_hand>
   <xacro:irobot_hand side="left" parent="l_hand" reflect="-1">
-    <origin xyz="0.00179  0.09516 0.01176" rpy="1.57079 0 3.14159"/>
+    <origin xyz="0.00179  0.09516 0.01176" rpy="-1.57079 0 0"/>
   </xacro:irobot_hand>
   <gazebo>

File: atlas_description/robots/atlas_v3_sandia_hands.urdf.xacro (robot description, xacro)
@@ -1,4 +1,4 @@
 <robot xmlns:xacro="http://www.ros.org/wiki/xacro" name="atlas" >
-  <xacro:include filename="$(find atlas_description)/urdf/atlas_v3.urdf" />
+  <xacro:include filename="$(find atlas_description)/urdf/atlas_v3_simple_shapes.urdf" />
   <xacro:include filename="$(find sandia_hand_description)/urdf/sandia_hand_simple_shapes.urdf.xacro" />
   <xacro:sandia_hand side="right" parent="r_hand" reflect="1" joint_type="revolute" thumb_angle="0">
