Commit message: Tweaking xacro.

File: atlas_description/robots/atlas_robotiq_hands.urdf.xacro (robot description, xacro)
@@ -2,9 +2,12 @@
   <xacro:include filename="$(find atlas_description)/urdf/atlas_simple_shapes.urdf" />
   <xacro:include filename="$(find robotiq_hand_description)/urdf/robotiq_hand.urdf.xacro" />
-  <xacro:robotiq_hand side="right" parent="r_hand" reflect="1">
+  <!--<xacro:robotiq_hand side="right" parent="r_hand" reflect="1">
     <origin rpy="1.57079 0 0" xyz="0 -0.09 0"/>
   </xacro:robotiq_hand>
   <xacro:robotiq_hand side="left" parent="l_hand" reflect="-1">
     <origin rpy="1.57079 0 3.14159" xyz="0 0.09 0"/>
+  </xacro:robotiq_hand>-->
+  <xacro:robotiq_hand prefix="left">
+    <origin rpy="1.57079 0 0" xyz="0 -0.09 0"/>
   </xacro:robotiq_hand>
   <!--<gazebo>-->

File: robotiq_hand_description/urdf/robotiq_hand.urdf.xacro (robot description, xacro)
@@ -1,9 +1,10 @@
+<?xml version="1.0"?>
 <!--
-s-model_articulated_macro(prefix)
+robotiq_hand_macro(prefix)
 Creates an articulated s-model hand with the passed in prefix.  If there
 is only one hand in the urdf then an empty prefix can be used "".  If
 there are multiple hands then a prefix followed by an "_" is needed.
 -->
-<robot xmlns:xacro="http://ros.org/wiki/xacro">
+<robot xmlns:xacro="http://ros.org/wiki/xacro" name="robotiq">
 	<xacro:macro name="robotiq_finger" params="prefix">
 	  <gazebo reference="${prefix}link_0">
@@ -149,5 +150,5 @@
 		<!-- end of joint list -->
 	</xacro:macro>
-	<xacro:macro name="s-model_articulated" params="prefix">
+	<xacro:macro name="robotiq_hand" params="prefix">
 	  <xacro:robotiq_finger prefix="${prefix}finger_1_"/>
 	  <xacro:robotiq_finger prefix="${prefix}finger_2_"/>

Commit message: Tweaking xacro.

File: atlas_description/robots/atlas_robotiq_hands.urdf.xacro (robot description, xacro)
@@ -8,7 +8,7 @@
     <origin rpy="1.57079 0 3.14159" xyz="0 0.09 0"/>
   </xacro:robotiq_hand>-->
-  <xacro:robotiq_hand prefix="left">
-    <origin rpy="1.57079 0 0" xyz="0 -0.09 0"/>
-  </xacro:robotiq_hand>
+  <xacro:robotiq_hand prefix="left_"/>
+  <!--  <origin rpy="1.57079 0 0" xyz="0 -0.09 0"/>
+  </xacro:robotiq_hand> -->
   <!--<gazebo>-->
     <!-- plugin for right robotiq hand -->

File: robotiq_hand_description/urdf/robotiq_hand.urdf.xacro (robot description, xacro)
@@ -6,5 +6,5 @@
 there are multiple hands then a prefix followed by an "_" is needed.
 -->
-<robot xmlns:xacro="http://ros.org/wiki/xacro" name="robotiq">
+<robot xmlns:xacro="http://www.ros.org/wiki/xacro" name="robotiq">
 	<xacro:macro name="robotiq_finger" params="prefix">
 	  <gazebo reference="${prefix}link_0">
@@ -162,5 +162,5 @@
 		  	<visual>
 		  		<geometry>
-		  			<mesh filename="package://robotiq_hand_description/meshes/s-  model_articulated/visual/palm.STL" />
+		  			<mesh filename="package://robotiq_hand_description/meshes/s-model_articulated/visual/palm.STL" />
 		  		</geometry>
 		  		<material name="green">
@@ -217,3 +217,5 @@
 		<!-- end of joint list -->
 	</xacro:macro>
+	<!-- Just for testing the xacro -->
+	<xacro:robotiq_hand prefix="left_"/>
 </robot>

Commit message: clean up cmake install of gazebo models. simplify duplicate gazebo models installs

File: atlas_description/robots/atlas_robotiq_hands.urdf.xacro (robot description, xacro)
@@ -2,13 +2,10 @@
   <xacro:include filename="$(find atlas_description)/urdf/atlas_simple_shapes.urdf" />
   <xacro:include filename="$(find robotiq_hand_description)/urdf/robotiq_hand.urdf.xacro" />
-  <!--<xacro:robotiq_hand side="right" parent="r_hand" reflect="1">
+  <xacro:robotiq_hand prefix="right_" parent="r_hand" reflect="1">
     <origin rpy="1.57079 0 0" xyz="0 -0.09 0"/>
   </xacro:robotiq_hand>
-  <xacro:robotiq_hand side="left" parent="l_hand" reflect="-1">
+  <xacro:robotiq_hand prefix="left_" parent="l_hand" reflect="-1">
     <origin rpy="1.57079 0 3.14159" xyz="0 0.09 0"/>
-  </xacro:robotiq_hand>-->
-  <xacro:robotiq_hand prefix="left_"/>
-  <!--  <origin rpy="1.57079 0 0" xyz="0 -0.09 0"/>
-  </xacro:robotiq_hand> -->
+  </xacro:robotiq_hand>
   <!--<gazebo>-->
     <!-- plugin for right robotiq hand -->

File: irobot_hand_description/urdf/irobot_hand.urdf.xacro (robot description, xacro)
@@ -322,5 +322,5 @@
   -->
   <xacro:flex_joint_connector side="${side}" finger_id="2" />
-  <!-- joint to irobot hand -->
+  <!-- joint attaching parent link to irobot hand -->
   <joint name="${side}_irobot_hand_joint" type="fixed">
     <insert_block name="origin"/>

File: robotiq_hand_description/robots/robotiq_hand_on_box.urdf.xacro (robot description, xacro)
@@ -21,5 +21,5 @@
     </collision>
   </link>
-  <xacro:robotiq_hand side="left" parent="base" reflect="-1">
+  <xacro:robotiq_hand prefix="box_" parent="base" reflect="-1">
     <origin rpy="0 0 0" xyz="0 0 1.0"/>
   </xacro:robotiq_hand>

File: robotiq_hand_description/urdf/robotiq_hand.urdf.xacro (robot description, xacro)
@@ -150,5 +150,11 @@
 		<!-- end of joint list -->
 	</xacro:macro>
-	<xacro:macro name="robotiq_hand" params="prefix">
+	<xacro:macro name="robotiq_hand" params="prefix *origin reflect parent">
+    <!-- joint attaching parent link to robotiq hand -->
+    <joint name="${prefix}robotiq_hand_joint" type="fixed">
+      <insert_block name="origin"/>
+      <parent link="${parent}"/>
+      <child link="${prefix}palm"/>
+    </joint>
 	  <xacro:robotiq_finger prefix="${prefix}finger_1_"/>
 	  <xacro:robotiq_finger prefix="${prefix}finger_2_"/>
@@ -217,5 +223,6 @@
 		<!-- end of joint list -->
 	</xacro:macro>
-	<!-- Just for testing the xacro -->
+	<!-- Just for testing the xacro
 	<xacro:robotiq_hand prefix="left_"/>
+  -->
 </robot>

Commit message: fix robotiq hand offset

File: atlas_description/robots/atlas_robotiq_hands.urdf.xacro (robot description, xacro)
@@ -3,8 +3,8 @@
   <xacro:include filename="$(find robotiq_hand_description)/urdf/robotiq_hand.urdf.xacro" />
   <xacro:robotiq_hand prefix="right_" parent="r_hand" reflect="1">
-    <origin rpy="1.57079 0 0" xyz="0 -0.09 0"/>
+    <origin rpy="3.14159 0 0" xyz="-0.00125 -0.17 0.01"/>
   </xacro:robotiq_hand>
   <xacro:robotiq_hand prefix="left_" parent="l_hand" reflect="-1">
-    <origin rpy="1.57079 0 3.14159" xyz="0 0.09 0"/>
+    <origin rpy="3.14159 0 3.14159" xyz="-0.00125 0.17 0.01"/>
   </xacro:robotiq_hand>
   <!--<gazebo>-->

Commit message: First version of the robotiq plugin that open/close hands.

File: atlas_description/robots/atlas_robotiq_hands.urdf.xacro (robot description, xacro)
@@ -2,20 +2,20 @@
   <xacro:include filename="$(find atlas_description)/urdf/atlas_simple_shapes.urdf" />
   <xacro:include filename="$(find robotiq_hand_description)/urdf/robotiq_hand.urdf.xacro" />
-  <xacro:robotiq_hand prefix="right_" parent="r_hand" reflect="1">
+  <xacro:robotiq_hand prefix="r_" parent="r_hand" reflect="1">
     <origin rpy="3.14159 0 0" xyz="-0.00125 -0.17 0.01"/>
   </xacro:robotiq_hand>
-  <xacro:robotiq_hand prefix="left_" parent="l_hand" reflect="-1">
+  <xacro:robotiq_hand prefix="l_" parent="l_hand" reflect="-1">
     <origin rpy="3.14159 0 3.14159" xyz="-0.00125 0.17 0.01"/>
   </xacro:robotiq_hand>
-  <!--<gazebo>-->
+  <gazebo>
     <!-- plugin for right robotiq hand -->
-    <!--<plugin name="right_robotiq_hand_plugin" filename="libRobotiqHandPlugin.so">
-      <side>right</side>
-    </plugin>-->
+    <plugin name="right_robotiq_hand_plugin" filename="libRobotiqHandPlugin.so">
+      <side>r_</side>
+    </plugin>
     <!-- plugin for left robotiq hand -->
-    <!--<plugin name="left_robotiq_hand_plugin" filename="libRobotiqHandPlugin.so">
-      <side>left</side>
+    <plugin name="left_robotiq_hand_plugin" filename="libRobotiqHandPlugin.so">
+      <side>l_</side>
     </plugin>
-  </gazebo>-->
+  </gazebo>
   <xacro:include filename="$(find atlas_description)/urdf/atlas.gazebo" />
   <xacro:include filename="$(find atlas_description)/urdf/atlas.transmission" />

File: robotiq_hand_description/urdf/robotiq_hand.urdf.xacro (robot description, xacro)
@@ -128,7 +128,7 @@
 			<parent link="${prefix}link_0"/>
 			<child link="${prefix}link_1"/>
-        <dynamics damping="0.1" friction="0" />
-        <limit effort="20" velocity="2" lower="-1.5" upper="1.5" />
-        <safety_controller k_position="100" k_velocity="100" soft_lower_limit="-10.6981" soft_upper_limit="10.6981" />
+      <dynamics damping="1" friction="0" />
+      <limit effort="20" velocity="2" lower="-1.5" upper="1.5" />
+      <safety_controller k_position="100" k_velocity="100" soft_lower_limit="-10.6981" soft_upper_limit="10.6981" />
 		</joint>
 		<gazebo reference="${prefix}joint_1">
@@ -139,5 +139,5 @@
 			<parent link="${prefix}link_1"/>
 			<child link="${prefix}link_2"/>
-			<dynamics damping="0.1" friction="0" />
+			<dynamics damping="1" friction="0" />
 			<axis xyz="0 0 1"/>
 			<origin rpy="0 0 -0.52" xyz="0.050 -.028 0"/>
@@ -151,5 +151,5 @@
 			<parent link="${prefix}link_2"/>
 			<child link="${prefix}link_3"/>
-			<dynamics damping="0.1" friction="0" />
+			<dynamics damping="1" friction="0" />
 			<axis xyz="0 0 1"/>
 			<origin rpy="0 0 0.52" xyz="0.039 0 0"/>
@@ -214,23 +214,35 @@
 			<parent link="${prefix}palm"/>
 			<child link="${prefix}finger_1_link_0"/>
+			<dynamics damping="1" friction="0" />
 			<axis xyz="0 1 0"/>
 			<origin rpy="0 3.1416 -1.57" xyz="-0.0455 0.0214 0.036"/>
 			<limit lower="-0.16" upper="0.25" effort="100" velocity="100"/>
 		</joint>
+		<gazebo reference="${prefix}palm_finger_1_joint">
+		  <implicitSpringDamper>1</implicitSpringDamper>
+		</gazebo>
 		<!-- WARNING: LIMITS NOT CORRECT -->
 		<joint name="${prefix}palm_finger_2_joint" type="revolute">
 			<parent link="${prefix}palm"/>
 			<child link="${prefix}finger_2_link_0"/>
+			<dynamics damping="1" friction="0" />
 			<axis xyz="0 1 0"/>
 			<origin rpy="0 3.1416 -1.57" xyz="-0.0455 0.0214 -0.036"/>
 			<limit lower="-0.25" upper="0.16" effort="100" velocity="100"/>
 		</joint>
+		<gazebo reference="${prefix}palm_finger_2_joint">
+		  <implicitSpringDamper>1</implicitSpringDamper>
+		</gazebo>
 		<joint name="${prefix}palm_finger_middle_joint" type="revolute">
 			<parent link="${prefix}palm"/>
 			<child link="${prefix}finger_middle_link_0"/>
+			<dynamics damping="1" friction="0" />
 			<axis xyz="0 1 0"/>
 			<origin rpy="0 0 1.57" xyz="0.0455 0.0214 0"/>
 			<limit lower="-0.25" upper="0.16" effort="100" velocity="100"/>
 		</joint>
+		<gazebo reference="${prefix}palm_finger_middle_joint">
+		  <implicitSpringDamper>1</implicitSpringDamper>
+		</gazebo>
 		<!-- end of joint list -->
 	</xacro:macro>

Commit message: Using Gazebo PIDs and more cleaning.

File: atlas_description/robots/atlas_robotiq_hands.urdf.xacro (robot description, xacro)
@@ -2,18 +2,18 @@
   <xacro:include filename="$(find atlas_description)/urdf/atlas_simple_shapes.urdf" />
   <xacro:include filename="$(find robotiq_hand_description)/urdf/robotiq_hand.urdf.xacro" />
+  <xacro:robotiq_hand prefix="l_" parent="l_hand" reflect="-1">
+    <origin rpy="3.14159 0 3.14159" xyz="-0.00125 0.17 0.01"/>
+  </xacro:robotiq_hand>
   <xacro:robotiq_hand prefix="r_" parent="r_hand" reflect="1">
     <origin rpy="3.14159 0 0" xyz="-0.00125 -0.17 0.01"/>
   </xacro:robotiq_hand>
-  <xacro:robotiq_hand prefix="l_" parent="l_hand" reflect="-1">
-    <origin rpy="3.14159 0 3.14159" xyz="-0.00125 0.17 0.01"/>
-  </xacro:robotiq_hand>
   <gazebo>
+    <!-- plugin for left robotiq hand -->
+    <plugin name="left_robotiq_hand_plugin" filename="libRobotiqHandPlugin.so">
+      <side>left</side>
+    </plugin>
     <!-- plugin for right robotiq hand -->
     <plugin name="right_robotiq_hand_plugin" filename="libRobotiqHandPlugin.so">
       <side>right</side>
-    </plugin>
-    <!-- plugin for left robotiq hand -->
-    <plugin name="left_robotiq_hand_plugin" filename="libRobotiqHandPlugin.so">
-      <side>left</side>
     </plugin>
   </gazebo>
