Commit message: Fixing the orientation of the left hand in Atlas.

File: atlas_description/robots/atlas_robotiq_hands.urdf.xacro (robot description, xacro)
@@ -3,5 +3,5 @@
   <xacro:include filename="$(find robotiq_hand_description)/urdf/robotiq_hand.urdf.xacro" />
   <xacro:robotiq_hand prefix="l_" parent="l_hand" reflect="-1">
-    <origin rpy="3.14159 0 3.14159" xyz="-0.00125 0.17 0.01"/>
+    <origin rpy="3.14159 3.14159 3.14159" xyz="-0.00125 0.17 0.01"/>
   </xacro:robotiq_hand>
   <xacro:robotiq_hand prefix="r_" parent="r_hand" reflect="1">

File: robotiq_hand_description/urdf/robotiq_hand.urdf.xacro (robot description, xacro)
@@ -7,159 +7,160 @@
 -->
 <robot xmlns:xacro="http://www.ros.org/wiki/xacro" name="robotiq">
-	<xacro:macro name="robotiq_finger" params="prefix">
-	  <gazebo reference="${prefix}link_0">
-	    <mu1>1.1</mu1>
-		  <mu2>1.1</mu2>
-	  </gazebo>
-	  <gazebo reference="${prefix}link_1">
-	    <mu1>1.1</mu1>
-		  <mu2>1.1</mu2>
-	  </gazebo>
-	  <gazebo reference="${prefix}link_2">
-	    <mu1>1.1</mu1>
-		  <mu2>1.1</mu2>
-	  </gazebo>
-	  <gazebo reference="${prefix}link_3">
-	    <mu1>1.1</mu1>
-		  <mu2>1.1</mu2>
-	  </gazebo>
-		<!-- link list -->
-		<link name="${prefix}link_0">
-			<visual>
-				<origin xyz="0 0 0" rpy="0 0 0"/>
-				<geometry>
-					<mesh filename="package://robotiq_hand_description/meshes/s-model_articulated/visual/link_0.STL" />
-				</geometry>
-				<material name="green">
-					<color rgba="0 1 0 1"/>
-				</material>
-			</visual>
-			<collision>
-				<origin rpy="0 0 0" xyz="0 0 0"/>
+  <xacro:macro name="robotiq_finger" params="prefix">
+    <!-- Link list -->
+    <!-- Link 0 -->
+    <link name="${prefix}link_0">
+      <visual>
+        <origin xyz="0 0 0" rpy="0 0 0"/>
+        <geometry>
+          <mesh filename="package://robotiq_hand_description/meshes/s-model_articulated/visual/link_0.STL" />
+        </geometry>
+        <material name="green">
+          <color rgba="0 1 0 1"/>
+        </material>
+      </visual>
+      <collision>
+        <origin rpy="0 0 0" xyz="0 0 0"/>
         <geometry>
           <mesh filename="package://robotiq_hand_description/meshes/s-model_articulated/collision/link_0.STL" />
         </geometry>
-				<material name="yellow">
-					<color rgba="0 1 1 1"/>
-				</material>
-			</collision>
-			<inertial>
+        <material name="yellow">
+          <color rgba="0 1 1 1"/>
+        </material>
+      </collision>
+      <inertial>
         <mass value="0.1"/>
-      	<origin xyz="-0.01 0 0"/>
-      	<inertia ixx="0.000018" ixy="0" ixz="0" iyy="0.000025" iyz="0" izz="0.000025"/>
+        <origin xyz="-0.01 0 0"/>
+        <inertia ixx="0.000018" ixy="0" ixz="0" iyy="0.000025" iyz="0" izz="0.000025"/>
       </inertial>
-		</link>
-		<link name="${prefix}link_1">
-			<visual>
-				<origin rpy="0 0 -0.52" xyz="0.050 -.028 0"/>
-				<geometry>
-					<mesh filename="package://robotiq_hand_description/meshes/s-model_articulated/visual/link_1.STL" />
-				</geometry>
-				<material name="green"/>
-			</visual>
-			<collision>
-			  <origin rpy="0 0 -0.52" xyz="0.050 -.028 0"/>
+    </link>
+    <gazebo reference="${prefix}link_0">
+      <mu1>1.1</mu1>
+      <mu2>1.1</mu2>
+    </gazebo>
+    <!-- Link 1 -->
+    <link name="${prefix}link_1">
+      <visual>
+        <origin rpy="0 0 -0.52" xyz="0.050 -.028 0"/>
+        <geometry>
+          <mesh filename="package://robotiq_hand_description/meshes/s-model_articulated/visual/link_1.STL" />
+        </geometry>
+        <material name="green"/>
+      </visual>
+      <collision>
+        <origin rpy="0 0 -0.52" xyz="0.050 -.028 0"/>
         <geometry>
           <mesh filename="package://robotiq_hand_description/meshes/s-model_articulated/collision/link_1.STL"/>
         </geometry>
-				<material name="yellow">
-					<color rgba="0 1 1 1"/>
-				</material>
-			</collision>
-			<inertial>
+        <material name="yellow">
+          <color rgba="0 1 1 1"/>
+        </material>
+      </collision>
+      <inertial>
         <origin rpy="0 0 -0.52" xyz="0.0282 -0.0155 0"/>
         <mass value="0.047"/>
         <inertia ixx="0.00000499332" ixy="0.00000091312" ixz="-0.00000000120" iyy="0.00006434531" iyz="-0.00000000007" izz="0.00006061917"/>
       </inertial>
-		</link>
-		<link name="${prefix}link_2">
-			<!--
-			NOTE: This link has an offset in the z-direction based on the models that were
-			used to generate grap-it poses.  With the offset below the model appears visually
-			correct, but it is suspect.
-			-->
-			<visual>
-				<origin xyz="0.039 0 0.0075" rpy="0 0 0"/>
-				<geometry>
-					<mesh filename="package://robotiq_hand_description/meshes/s-model_articulated/visual/link_2.STL" />
-				</geometry>
-				<material name="green"/>
-			</visual>
-			<collision>
-			  <origin rpy="0 0 0" xyz="0.039 0 0.0075"/>
-			    <geometry>
-			      <mesh filename="package://robotiq_hand_description/meshes/s-model_articulated/collision/link_2.STL"/>
-			    </geometry>
-				<material name="yellow"/>
-			</collision>
-			<inertial>
+    </link>
+    <gazebo reference="${prefix}link_1">
+      <mu1>1.1</mu1>
+      <mu2>1.1</mu2>
+    </gazebo>
+    <!-- Link 2 -->
+    <link name="${prefix}link_2">
+      <visual>
+        <origin xyz="0.039 0 0.0075" rpy="0 0 0"/>
+        <geometry>
+          <mesh filename="package://robotiq_hand_description/meshes/s-model_articulated/visual/link_2.STL" />
+        </geometry>
+        <material name="green"/>
+      </visual>
+      <collision>
+        <origin rpy="0 0 0" xyz="0.039 0 0.0075"/>
+          <geometry>
+            <mesh filename="package://robotiq_hand_description/meshes/s-model_articulated/collision/link_2.STL"/>
+          </geometry>
+        <material name="yellow"/>
+      </collision>
+      <inertial>
         <origin rpy="0 0 0" xyz="0.02167 0.00048 0.00018"/>
         <mass value="0.03284"/>
         <inertia ixx="0.00000348008" ixy="0.00000031940" ixz="0.00000013041" iyy="0.00002248123" iyz="0.00000000291" izz="0.00001986346"/>
       </inertial>
-		</link>
-		<link name="${prefix}link_3">
-			<visual>
-				<origin xyz="0 0 0" rpy="0 0 0"/>
-				<geometry>
-					<mesh filename="package://robotiq_hand_description/meshes/s-model_articulated/visual/link_3.STL" />
-				</geometry>
-				<material name="green"/>
-			</visual>
-			<collision>
-				<origin rpy="0 0 0" xyz="0 0 0"/>
-				<geometry>
-					<mesh filename="package://robotiq_hand_description/meshes/s-model_articulated/collision/link_3.STL"/>
-				</geometry>
-				<material name="yellow"/>
-			</collision>
-			<inertial>
+    </link>
+    <gazebo reference="${prefix}link_2">
+      <mu1>1.1</mu1>
+      <mu2>1.1</mu2>
+    </gazebo>
+    <!-- Link 3 -->
+    <link name="${prefix}link_3">
+      <visual>
+        <origin xyz="0 0 0" rpy="0 0 0"/>
+        <geometry>
+          <mesh filename="package://robotiq_hand_description/meshes/s-model_articulated/visual/link_3.STL" />
+        </geometry>
+        <material name="green"/>
+      </visual>
+      <collision>
+        <origin rpy="0 0 0" xyz="0 0 0"/>
+        <geometry>
+          <mesh filename="package://robotiq_hand_description/meshes/s-model_articulated/collision/link_3.STL"/>
+        </geometry>
+        <material name="yellow"/>
+      </collision>
+      <inertial>
         <origin rpy="0 0 0" xyz="0.01626 0.00049 0.0002"/>
         <mass value="0.03354"/>
         <inertia ixx="0.00000305151" ixy="0.00000089792" ixz="0.00000000249" iyy="0.00001427978" iyz="-0.00000001191" izz="0.00001264126"/>
     </inertial>
-		</link>
-		<!-- end of link list -->
-		<!-- joint list -->
-		<joint name="${prefix}joint_1" type="revolute">
-			<origin rpy="0 0 0" xyz="0 0 0"/>
-			<axis xyz="0 0 1" />
-			<parent link="${prefix}link_0"/>
-			<child link="${prefix}link_1"/>
+    </link>
+    <gazebo reference="${prefix}link_3">
+      <mu1>1.1</mu1>
+      <mu2>1.1</mu2>
+    </gazebo>
+    <!-- End of link list -->
+    <!-- Joint list -->
+    <!-- Joint 1 -->
+    <joint name="${prefix}joint_1" type="revolute">
+      <origin rpy="0 0 0" xyz="0 0 0"/>
+      <axis xyz="0 0 1" />
+      <parent link="${prefix}link_0"/>
+      <child link="${prefix}link_1"/>
       <dynamics damping="1" friction="0" />
       <!-- Limits: [0deg.,70deg.] -->
       <limit effort="20" velocity="-1" lower="0" upper="1.2217" />
-      <!--<safety_controller k_position="100" k_velocity="100" soft_lower_limit="-10.6981" soft_upper_limit="10.6981" />-->
-		</joint>
-		<gazebo reference="${prefix}joint_1">
-		  <implicitSpringDamper>1</implicitSpringDamper>
-		</gazebo>
-		<joint name="${prefix}joint_2" type="revolute">
-			<parent link="${prefix}link_1"/>
-			<child link="${prefix}link_2"/>
-			<dynamics damping="1" friction="0" />
-			<axis xyz="0 0 1"/>
-			<origin rpy="0 0 -0.52" xyz="0.050 -.028 0"/>
-			<!-- Limits: [0deg.,90deg.] -->
-			<limit lower="0" upper="1.5708" effort="20" velocity="-1"/>
-		</joint>
-		<gazebo reference="${prefix}joint_2">
-		  <implicitSpringDamper>1</implicitSpringDamper>
-		</gazebo>
-		<joint name="${prefix}joint_3" type="revolute">
-			<parent link="${prefix}link_2"/>
-			<child link="${prefix}link_3"/>
-			<dynamics damping="1" friction="0" />
-			<axis xyz="0 0 1"/>
-  		<origin rpy="0 0 0.52" xyz="0.039 0 0"/>
-	  	<!-- Limits: [-38deg.,60deg.] -->
-			<limit lower="-0.6632" upper="1.0471" effort="20" velocity="-1"/>
-		</joint>
-		<gazebo reference="${prefix}joint_3">
-		  <implicitSpringDamper>1</implicitSpringDamper>
-		</gazebo>
-		<!-- end of joint list -->
-	</xacro:macro>
-	<xacro:macro name="robotiq_hand" params="prefix *origin reflect parent">
+    </joint>
+    <gazebo reference="${prefix}joint_1">
+      <implicitSpringDamper>1</implicitSpringDamper>
+    </gazebo>
+    <!-- Joint 2 -->
+    <joint name="${prefix}joint_2" type="revolute">
+      <parent link="${prefix}link_1"/>
+      <child link="${prefix}link_2"/>
+      <dynamics damping="1" friction="0" />
+      <axis xyz="0 0 1"/>
+      <origin rpy="0 0 -0.52" xyz="0.050 -.028 0"/>
+      <!-- Limits: [0deg.,90deg.] -->
+      <limit lower="0" upper="1.5708" effort="20" velocity="-1"/>
+    </joint>
+    <gazebo reference="${prefix}joint_2">
+      <implicitSpringDamper>1</implicitSpringDamper>
+    </gazebo>
+    <!-- Joint 3 -->
+    <joint name="${prefix}joint_3" type="revolute">
+      <parent link="${prefix}link_2"/>
+      <child link="${prefix}link_3"/>
+      <dynamics damping="1" friction="0" />
+      <axis xyz="0 0 1"/>
+      <origin rpy="0 0 0.52" xyz="0.039 0 0"/>
+      <!-- Limits: [-38deg.,60deg.] -->
+      <limit lower="-0.6632" upper="1.0471" effort="20" velocity="-1"/>
+    </joint>
+    <gazebo reference="${prefix}joint_3">
+      <implicitSpringDamper>1</implicitSpringDamper>
+    </gazebo>
+    <!-- end of joint list -->
+  </xacro:macro>
+  <xacro:macro name="robotiq_hand" params="prefix *origin reflect parent">
     <!-- joint attaching parent link to robotiq hand -->
     <joint name="${prefix}robotiq_hand_joint" type="fixed">
@@ -168,85 +169,89 @@
       <child link="${prefix}palm"/>
     </joint>
-	  <xacro:robotiq_finger prefix="${prefix}finger_1_"/>
-	  <xacro:robotiq_finger prefix="${prefix}finger_2_"/>
-	  <xacro:robotiq_finger prefix="${prefix}finger_middle_"/>
-		  <!-- link list -->
-	    <gazebo reference="${prefix}palm">
-		    <mu1>1.1</mu1>
-		    <mu2>1.1</mu2>
-		  </gazebo>
-		  <link name="${prefix}palm">
-		  	<visual>
-		  		<geometry>
-		  			<mesh filename="package://robotiq_hand_description/meshes/s-model_articulated/visual/palm.STL" />
-		  		</geometry>
-		  		<material name="green">
-		  			<color rgba="0 1 0 1"/>
-		  		</material>
-		  	</visual>
-		  	<collision>
+    <!-- Insert the fingers -->
+    <xacro:robotiq_finger prefix="${prefix}finger_1_"/>
+    <xacro:robotiq_finger prefix="${prefix}finger_2_"/>
+    <xacro:robotiq_finger prefix="${prefix}finger_middle_"/>
+      <!-- link list -->
+      <!-- Link palm -->
+      <link name="${prefix}palm">
+        <visual>
+          <geometry>
+            <mesh filename="package://robotiq_hand_description/meshes/s-model_articulated/visual/palm.STL" />
+          </geometry>
+          <material name="green">
+            <color rgba="0 1 0 1"/>
+          </material>
+        </visual>
+        <!-- Mesh collision -->
+        <!-- <collision>
           <geometry>
             <mesh filename="package://robotiq_hand_description/meshes/s-model_articulated/collision/palm.STL"/>
           </geometry>
-		  		<material name="yellow">
-		  			<color rgba="0 1 1 1"/>
-		  		</material>
-		  	</collision>
-		  	<collision>
-		  	  <origin rpy="0 0 0" xyz="-0.085 -0.02 0"/>
-          <geometry>
-            <box size="0.08 0.08 0.07"/>
-          </geometry>
-		  		<material name="yellow">
-		  			<color rgba="0 1 1 1"/>
-		  		</material>
-		  	</collision>
-		  	<inertial>
+          <material name="yellow">
+            <color rgba="0 1 1 1"/>
+          </material>
+        </collision> -->
+        <!-- Simple shape collision -->
+        <collision>
+          <origin rpy="0 0 0" xyz="0 0 0"/>
+          <geometry>
+            <box size="0.1 0.1 0.08"/>
+          </geometry>
+          <material name="yellow">
+            <color rgba="0 1 1 1"/>
+          </material>
+        </collision>
+        <inertial>
           <origin rpy="0 0 0" xyz="0 0 0"/>
           <mass value="1.3"/>
           <inertia ixx="0.0035" ixy="0" ixz="-0" iyy="0.0035" iyz="0" izz="0.0035"/>
         </inertial>
-		  </link>
-		<!-- end of link list -->
-		<!-- joint list -->
-		<joint name="${prefix}palm_finger_1_joint" type="revolute">
-			<parent link="${prefix}palm"/>
-			<child link="${prefix}finger_1_link_0"/>
-			<dynamics damping="1" friction="0" />
-			<axis xyz="0 1 0"/>
-			<origin rpy="0 3.1416 -1.57" xyz="-0.0455 0.0214 0.036"/>
-			<!-- Limits: [-17deg.,17deg.] -->
-			<limit lower="-0.2967" upper="0.2967" effort="100" velocity="-1"/>
-		</joint>
-		<gazebo reference="${prefix}palm_finger_1_joint">
-		  <implicitSpringDamper>1</implicitSpringDamper>
-		</gazebo>
-		<joint name="${prefix}palm_finger_2_joint" type="revolute">
-			<parent link="${prefix}palm"/>
-			<child link="${prefix}finger_2_link_0"/>
-			<dynamics damping="1" friction="0" />
-			<axis xyz="0 1 0"/>
-			<origin rpy="0 3.1416 -1.57" xyz="-0.0455 0.0214 -0.036"/>
-			<!-- Limits: [-17deg.,17deg.] -->
-			<limit lower="-0.2967" upper="0.2967" effort="100" velocity="-1"/>
-		</joint>
-		<gazebo reference="${prefix}palm_finger_2_joint">
-		  <implicitSpringDamper>1</implicitSpringDamper>
-		</gazebo>
-		<joint name="${prefix}palm_finger_middle_joint" type="revolute">
-			<parent link="${prefix}palm"/>
-			<child link="${prefix}finger_middle_link_0"/>
-			<dynamics damping="1" friction="0" />
-			<axis xyz="0 1 0"/>
-			<origin rpy="0 0 1.57" xyz="0.0455 0.0214 0"/>
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