Commit message: Tweaking urdf.

File: atlas_description/robots/atlas_v3_robotiq_hands.urdf.xacro (robot description, xacro)
@@ -2,20 +2,24 @@
   <xacro:include filename="$(find atlas_description)/urdf/atlas_v3_simple_shapes.urdf" />
   <xacro:include filename="$(find robotiq_hand_description)/urdf/robotiq_hand.urdf.xacro" />
-  <xacro:robotiq_hand prefix="right_" parent="r_hand" reflect="1">
+  <xacro:robotiq_hand prefix="l_" parent="l_hand" reflect="-1">
+    <origin rpy="3.14159 3.14159 3.14159" xyz="-0.00125 0.17 0.01"/>
+  </xacro:robotiq_hand>
+  <xacro:robotiq_hand prefix="r_" parent="r_hand" reflect="1">
     <origin rpy="3.14159 0 0" xyz="-0.00125 -0.17 0.01"/>
   </xacro:robotiq_hand>
-  <xacro:robotiq_hand prefix="left_" parent="l_hand" reflect="-1">
-    <origin rpy="3.14159 0 3.14159" xyz="-0.00125 0.17 0.01"/>
-  </xacro:robotiq_hand>
-  <!--<gazebo>-->
+  <gazebo>
+    <!-- plugin for left robotiq hand -->
+    <plugin name="left_robotiq_hand_plugin" filename="libRobotiqHandPlugin.so">
+      <side>left</side>
+      <kp_position>1.0</kp_position>
+      <kd_position>0.5</kd_position>
+    </plugin>
     <!-- plugin for right robotiq hand -->
-    <!--<plugin name="right_robotiq_hand_plugin" filename="libRobotiqHandPlugin.so">
+    <plugin name="right_robotiq_hand_plugin" filename="libRobotiqHandPlugin.so">
       <side>right</side>
-    </plugin>-->
-    <!-- plugin for left robotiq hand -->
-    <!--<plugin name="left_robotiq_hand_plugin" filename="libRobotiqHandPlugin.so">
-      <side>left</side>
+      <kp_position>1.0</kp_position>
+      <kd_position>0.5</kd_position>
     </plugin>
-  </gazebo>-->
+  </gazebo>
   <xacro:include filename="$(find atlas_description)/urdf/atlas_v3.gazebo" />
   <xacro:include filename="$(find atlas_description)/urdf/atlas_v3.transmission" />

File: atlas_description/robots/atlas_v4_robotiq_hands.urdf.xacro (robot description, xacro)
@@ -2,20 +2,24 @@
   <xacro:include filename="$(find atlas_description)/urdf/atlas_v4_simple_shapes.urdf" />
   <xacro:include filename="$(find robotiq_hand_description)/urdf/robotiq_hand.urdf.xacro" />
-  <xacro:robotiq_hand prefix="right_" parent="r_hand" reflect="1">
+  <xacro:robotiq_hand prefix="l_" parent="l_hand" reflect="-1">
+    <origin rpy="3.14159 3.14159 3.14159" xyz="-0.00125 0.17 0.01"/>
+  </xacro:robotiq_hand>
+  <xacro:robotiq_hand prefix="r_" parent="r_hand" reflect="1">
     <origin rpy="3.14159 0 0" xyz="-0.00125 -0.17 0.01"/>
   </xacro:robotiq_hand>
-  <xacro:robotiq_hand prefix="left_" parent="l_hand" reflect="-1">
-    <origin rpy="3.14159 0 3.14159" xyz="-0.00125 0.17 0.01"/>
-  </xacro:robotiq_hand>
-  <!--<gazebo>-->
+  <gazebo>
+    <!-- plugin for left robotiq hand -->
+    <plugin name="left_robotiq_hand_plugin" filename="libRobotiqHandPlugin.so">
+      <side>left</side>
+      <kp_position>1.0</kp_position>
+      <kd_position>0.5</kd_position>
+    </plugin>
     <!-- plugin for right robotiq hand -->
-    <!--<plugin name="right_robotiq_hand_plugin" filename="libRobotiqHandPlugin.so">
+    <plugin name="right_robotiq_hand_plugin" filename="libRobotiqHandPlugin.so">
       <side>right</side>
-    </plugin>-->
-    <!-- plugin for left robotiq hand -->
-    <!--<plugin name="left_robotiq_hand_plugin" filename="libRobotiqHandPlugin.so">
-      <side>left</side>
+      <kp_position>1.0</kp_position>
+      <kd_position>0.5</kd_position>
     </plugin>
-  </gazebo>-->
+  </gazebo>
   <xacro:include filename="$(find atlas_description)/urdf/atlas_v4.gazebo" />
   <xacro:include filename="$(find atlas_description)/urdf/atlas_v4.transmission" />
