Commit message: Fix hand placement for sandia and robotiq hands

File: atlas_description/robots/atlas_v5_robotiq_hands.urdf.xacro (robot description, xacro)
@@ -5,5 +5,5 @@
   to mach the values in your actual robot. -->
   <xacro:robotiq_hand prefix="l_" parent="l_hand" reflect="-1">
-    <origin rpy="3.14159 3.14159 3.14159" xyz="-0.00125 0.17 0.01"/>
+    <origin rpy="3.14159 3.14159 0" xyz="-0.00125 -0.17 0.01"/>
   </xacro:robotiq_hand>
   <xacro:robotiq_hand prefix="r_" parent="r_hand" reflect="1">

File: atlas_description/robots/atlas_v5_sandia_hands.urdf.xacro (robot description, xacro)
@@ -6,5 +6,5 @@
   </xacro:sandia_hand>
   <xacro:sandia_hand side="left" parent="l_hand" reflect="-1" joint_type="revolute" thumb_angle="0">
-    <origin xyz="0.00179  0.13516 0.01176" rpy="0 0  1.57079"/>
+    <origin xyz="0.00179  -0.13516 0.01176" rpy="0 0  -1.57079"/>
   </xacro:sandia_hand>
   <xacro:include filename="$(find atlas_description)/urdf/atlas_v5.gazebo" />
