Commit message: Merge adjustments to small masses of sensor frame links

File: multisense_sl_description/urdf/multisense.urdf (robot description, URDF)
Before this commit: robot multisense, 26 links, 25 joints
Links:
- link center_bottom_led_frame: mass 0.1 -> 1e-5
- link center_top_led_frame: mass 0.1 -> 1e-5
- link head_hokuyo_frame: mass 0.01 -> 1e-5
- link left_camera_frame: mass 0.1 -> 1e-5
- link left_led_frame: mass 0.1 -> 1e-5
- link right_camera_frame: mass 0.1 -> 1e-5
- link right_led_frame: mass 0.1 -> 1e-5
