Commit message: added fixed links for accels in the fingers

File: irobot_hand_description/urdf/irobot_hand.urdf.xacro (robot description, xacro)
@@ -264,4 +264,10 @@
     </visual>
   </link>
+  <link name="${side}_finger[0]/proximal_accelerometer" />
+  <joint name="${side}_finger[0]/proximal_link_to_accelerometer" type="fixed">
+    <parent link="${side}_finger[0]/proximal_link"/>
+    <child link="${side}_finger[0]/proximal_accelerometer"/>
+    <origin rpy="${pi/2} 0 0" xyz="0 0 0.05" />
+  </joint>
   <link name="${side}_finger[0]/distal_link">
       <inertial>
@@ -286,4 +292,10 @@
     </visual>
   </link>
+  <link name="${side}_finger[0]/distal_accelerometer" />
+  <joint name="${side}_finger[0]/distal_link_to_accelerometer" type="fixed">
+    <parent link="${side}_finger[0]/distal_link"/>
+    <child link="${side}_finger[0]/distal_accelerometer"/>
+    <origin rpy="${pi/2} 0 0" xyz="0 0 0.02" />
+  </joint>
   <link name="${side}_finger[1]/base_rotation_link">
       <inertial>
@@ -330,4 +342,10 @@
     </visual>
   </link>
+  <link name="${side}_finger[1]/proximal_accelerometer" />
+  <joint name="${side}_finger[1]/proximal_link_to_accelerometer" type="fixed">
+    <parent link="${side}_finger[1]/proximal_link"/>
+    <child link="${side}_finger[1]/proximal_accelerometer"/>
+    <origin rpy="${pi/2} 0 0" xyz="0 0 0.05" />
+  </joint>
   <link name="${side}_finger[1]/distal_link">
       <inertial>
@@ -352,4 +370,10 @@
     </visual>
   </link>
+  <link name="${side}_finger[1]/distal_accelerometer" />
+  <joint name="${side}_finger[1]/distal_link_to_accelerometer" type="fixed">
+    <parent link="${side}_finger[1]/distal_link"/>
+    <child link="${side}_finger[1]/distal_accelerometer"/>
+    <origin rpy="${pi/2} 0 0" xyz="0 0 0.02" />
+  </joint>
   <link name="${side}_finger[2]/proximal_link">
       <inertial>
@@ -374,4 +398,10 @@
     </visual>
   </link>
+  <link name="${side}_finger[2]/proximal_accelerometer" />
+  <joint name="${side}_finger[2]/proximal_link_to_accelerometer" type="fixed">
+    <parent link="${side}_finger[2]/proximal_link"/>
+    <child link="${side}_finger[2]/proximal_accelerometer"/>
+    <origin rpy="${pi/2} 0 0" xyz="0 0 0.05" />
+  </joint>
   <link name="${side}_finger[2]/distal_link">
       <inertial>
@@ -396,4 +426,10 @@
     </visual>
   </link>
+  <link name="${side}_finger[2]/distal_accelerometer" />
+  <joint name="${side}_finger[2]/distal_link_to_accelerometer" type="fixed">
+    <parent link="${side}_finger[2]/distal_link"/>
+    <child link="${side}_finger[2]/distal_accelerometer"/>
+    <origin rpy="${pi/2} 0 0" xyz="0 0 0.02" />
+  </joint>
   <joint name="${side}_finger[0]/joint_base_rotation" type="revolute">
     <parent link="${side}_base_link"/>

Commit message: Substituted simple collision shapes for meshes by grabbing stuff from gazebo_models/irobot_hand and converting it from sdf to urdf.xacro.

File: irobot_hand_description/urdf/irobot_hand.urdf.xacro (robot description, xacro)
@@ -136,4 +136,61 @@
     <limit effort="1000.0" lower="0.0" upper="${pi/2}" velocity="0.5"/>
   </joint>
+</xacro:macro>
+<!-- Simplified collisions for the base_rotation_links on fingers 0 and 1 -->
+<xacro:macro name="base_rotation_link_collisions">
+      <collision name='collision_1'>
+        <origin xyz="0 0 -.0025" rpy="0 0 0"/>
+        <geometry>
+          <cylinder length="0.0145" radius="0.025"/>
+        </geometry>
+      </collision>
+      <collision name='collision_2'>
+        <origin xyz="0 0 -.0104" rpy="0 0 0"/>
+        <geometry>
+          <cylinder length="0.0145" radius="0.0165"/>
+        </geometry>
+      </collision>
+      <collision name='collision_3'>
+        <origin xyz="0 0 .0135" rpy="1.5707 0 1.5707"/>
+        <geometry>
+          <cylinder length="0.02" radius="0.002"/>
+        </geometry>
+      </collision>
+      <collision name='collision_4'>
+        <origin xyz="0.013 0 .0135" rpy="1.5707 0 1.5707"/>
+        <geometry>
+          <cylinder length="0.008" radius="0.009"/>
+        </geometry>
+      </collision>
+      <collision name='collision_5'>
+        <origin xyz="-0.013 0 .0135" rpy="1.5707 0 1.5707"/>
+        <geometry>
+          <cylinder length="0.008" radius="0.009"/>
+        </geometry>
+      </collision>
+</xacro:macro>
+<!-- Simplified collisions for the proximal_link on all fingers -->
+<xacro:macro name="proximal_link_collisions">
+      <collision name='collision1'>
+        <origin xyz="0 0.0028 0.033" rpy="0 0 0"/>
+        <geometry>
+          <box size="0.018 0.019 0.055"/>
+        </geometry>
+      </collision>
+      <collision name='collision2'>
+        <origin xyz="0 0 0" rpy="0 1.5707 0"/>
+        <geometry>
+          <cylinder radius="0.009" length="0.018"/>
+        </geometry>
+      </collision>
+</xacro:macro>
+<!-- Simplified collisions for the distal_link on all fingers -->
+<xacro:macro name="distal_link_collisions">
+      <collision name='collision'>
+        <origin xyz="0 0.0025 0.019" rpy="3.141590 0.001593 3.141590"/>
+        <geometry>
+          <box size="0.0175 0.02023 0.04043"/>
+        </geometry>
+      </collision>
 </xacro:macro>
 <xacro:macro name="irobot_hand" params="side parent reflect *origin">
@@ -204,9 +261,15 @@
         <inertia ixx="0.001" ixy="0.0" ixz="0.0" iyy="0.001" iyz="0.0" izz="0.001"/>
       </inertial>
-    <collision>
-      <geometry>
-        <mesh filename="package://irobot_hand_description/meshes/palm.stl"/>
-      </geometry>
-      <origin rpy="0 0 0" xyz="0 -0.038 -0.023"/>
+    <collision name='collision1'>
+      <origin xyz="0 0.02 0.045" rpy="0 0 0"/>
+      <geometry>
+        <box size="0.114 0.1 0.075"/>
+      </geometry>
+    </collision>
+    <collision name='collision2'>
+      <origin xyz="0 -0.02 0.045" rpy="0 0 0"/>
+      <geometry>
+        <cylinder radius="0.0448" length="0.075"/>
+      </geometry>
     </collision>
     <visual>
@@ -226,10 +289,5 @@
         <inertia ixx="0.001" ixy="0.0" ixz="0.0" iyy="0.001" iyz="0.0" izz="0.001"/>
       </inertial>
-    <collision>
-      <geometry>
-        <mesh filename="package://irobot_hand_description/meshes/finger_base.stl"/>
-      </geometry>
-      <origin rpy="${pi/2} 0 0" xyz="0 0 0"/>
-    </collision>
+    <xacro:base_rotation_link_collisions/>
     <visual>
       <geometry>
@@ -248,10 +306,5 @@
         <inertia ixx="0.001" ixy="0.0" ixz="0.0" iyy="0.001" iyz="0.0" izz="0.001"/>
       </inertial>
-    <collision>
-      <geometry>
-        <mesh filename="package://irobot_hand_description/meshes/finger_proximal.stl"/>
-      </geometry>
-      <origin rpy="${pi/2} -${pi/2} 0" xyz="0 0 0"/>
-    </collision>
+    <xacro:proximal_link_collisions/>
     <visual>
       <geometry>
@@ -276,10 +329,5 @@
         <inertia ixx="0.001" ixy="0.0" ixz="0.0" iyy="0.001" iyz="0.0" izz="0.001"/>
       </inertial>
-    <collision>
-      <geometry>
-        <mesh filename="package://irobot_hand_description/meshes/finger_distal.stl"/>
-      </geometry>
-      <origin rpy="0 ${pi} 0" xyz="0 0 0"/>
-    </collision>
+    <xacro:distal_link_collisions/>
     <visual>
       <geometry>
@@ -304,10 +352,5 @@
         <inertia ixx="0.001" ixy="0.0" ixz="0.0" iyy="0.001" iyz="0.0" izz="0.001"/>
       </inertial>
-    <collision>
-      <geometry>
-        <mesh filename="package://irobot_hand_description/meshes/finger_base.stl"/>
-      </geometry>
-      <origin rpy="${pi/2} 0 0" xyz="0 0 0"/>
-    </collision>
+    <xacro:base_rotation_link_collisions/>
     <visual>
       <geometry>
@@ -326,10 +369,5 @@
         <inertia ixx="0.001" ixy="0.0" ixz="0.0" iyy="0.001" iyz="0.0" izz="0.001"/>
       </inertial>
-    <collision>
-      <geometry>
-        <mesh filename="package://irobot_hand_description/meshes/finger_proximal.stl"/>
-      </geometry>
-      <origin rpy="${pi/2} -${pi/2} 0" xyz="0 0 0"/>
-    </collision>
+    <xacro:proximal_link_collisions/>
     <visual>
       <geometry>
@@ -354,10 +392,5 @@
         <inertia ixx="0.001" ixy="0.0" ixz="0.0" iyy="0.001" iyz="0.0" izz="0.001"/>
       </inertial>
-    <collision>
-      <geometry>
-        <mesh filename="package://irobot_hand_description/meshes/finger_distal.stl"/>
-      </geometry>
-      <origin rpy="0 ${pi} 0" xyz="0 0 0"/>
-    </collision>
+    <xacro:distal_link_collisions/>
     <visual>
       <geometry>
@@ -382,10 +415,5 @@
         <inertia ixx="0.001" ixy="0.0" ixz="0.0" iyy="0.001" iyz="0.0" izz="0.001"/>
       </inertial>
-    <collision>
-      <geometry>
-        <mesh filename="package://irobot_hand_description/meshes/finger_proximal.stl"/>
-      </geometry>
-      <origin rpy="${pi/2} -${pi/2} 0" xyz="0 0 0"/>
-    </collision>
+    <xacro:proximal_link_collisions/>
     <visual>
       <geometry>
@@ -410,10 +438,5 @@
         <inertia ixx="0.001" ixy="0.0" ixz="0.0" iyy="0.001" iyz="0.0" izz="0.001"/>
       </inertial>
-    <collision>
-      <geometry>
-        <mesh filename="package://irobot_hand_description/meshes/finger_distal.stl"/>
-      </geometry>
-      <origin rpy="0 ${pi} 0" xyz="0 0 0"/>
-    </collision>
+    <xacro:distal_link_collisions/>
     <visual>
       <geometry>

Commit message: Worked with John to guess order-of-magnitude values for masses, inertias, and cfm and erp values.  Behavior looks reasonable.

File: irobot_hand_description/urdf/irobot_hand.urdf.xacro (robot description, xacro)
@@ -11,7 +11,7 @@
   <link name="${side}_finger[${finger_id}]/flexible_link_${link_id}">
     <inertial>
-      <mass value="0.1"/>
+      <mass value="0.001"/>
       <origin xyz="0 0 0"/>
-      <inertia ixx="0.001" ixy="0.0" ixz="0.0" iyy="0.001" iyz="0.0" izz="0.001"/>
+      <inertia ixx="0.000001" ixy="0.0" ixz="0.0" iyy="0.000001" iyz="0.0" izz="0.000001"/>
     </inertial>
     <collision>
@@ -42,7 +42,7 @@
   <link name="${side}_finger[${finger_id}]/flexible_link_hidden_between_${link_from}_and_${link_to}">
     <inertial>
-      <mass value="0.1"/>
+      <mass value="0.001"/>
       <origin xyz="0 0 0"/>
-      <inertia ixx="0.001" ixy="0.0" ixz="0.0" iyy="0.001" iyz="0.0" izz="0.001"/>
+      <inertia ixx="0.000001" ixy="0.0" ixz="0.0" iyy="0.000001" iyz="0.0" izz="0.000001"/>
     </inertial>
     <collision>
@@ -78,7 +78,7 @@
   <link name="${side}_finger[${finger_id}]/flexible_link_hidden_between_proximal_link_and_1">
     <inertial>
-      <mass value="0.1"/>
+      <mass value="0.001"/>
       <origin xyz="0 0 0"/>
-      <inertia ixx="0.001" ixy="0.0" ixz="0.0" iyy="0.001" iyz="0.0" izz="0.001"/>
+      <inertia ixx="0.000001" ixy="0.0" ixz="0.0" iyy="0.000001" iyz="0.0" izz="0.000001"/>
     </inertial>
     <collision>
@@ -112,7 +112,7 @@
   <link name="${side}_finger[${finger_id}]/flexible_link_hidden_between_9_and_distal_link">
     <inertial>
-      <mass value="0.1"/>
+      <mass value="0.001"/>
       <origin xyz="0 0 0"/>
-      <inertia ixx="0.001" ixy="0.0" ixz="0.0" iyy="0.001" iyz="0.0" izz="0.001"/>
+      <inertia ixx="0.000001" ixy="0.0" ixz="0.0" iyy="0.000001" iyz="0.0" izz="0.000001"/>
     </inertial>
     <collision>
@@ -257,7 +257,7 @@
   <link name="${side}_base_link">
       <inertial>
-        <mass value="0.1"/>
-        <origin xyz="0 0 0"/>
-        <inertia ixx="0.001" ixy="0.0" ixz="0.0" iyy="0.001" iyz="0.0" izz="0.001"/>
+        <mass value="1.0"/>
+        <origin xyz="0 0 0"/>
+        <inertia ixx="0.00125" ixy="0.0" ixz="0.0" iyy="0.00125" iyz="0.0" izz="0.0002"/>
       </inertial>
     <collision name='collision1'>
@@ -285,7 +285,7 @@
   <link name="${side}_finger[0]/base_rotation_link">
       <inertial>
-        <mass value="0.1"/>
-        <origin xyz="0 0 0"/>
-        <inertia ixx="0.001" ixy="0.0" ixz="0.0" iyy="0.001" iyz="0.0" izz="0.001"/>
+        <mass value="0.05"/>
+        <origin xyz="0 0 0"/>
+        <inertia ixx="0.0000125" ixy="0.0" ixz="0.0" iyy="0.0000125" iyz="0.0" izz="0.000002"/>
       </inertial>
     <xacro:base_rotation_link_collisions/>
@@ -304,5 +304,5 @@
         <mass value="0.1"/>
         <origin xyz="0 0 0"/>
-        <inertia ixx="0.001" ixy="0.0" ixz="0.0" iyy="0.001" iyz="0.0" izz="0.001"/>
+        <inertia ixx="3.78125e-05" ixy="0.0" ixz="0.0" iyy="3.78125e-05" iyz="0.0" izz="6.30208e-06"/>
       </inertial>
     <xacro:proximal_link_collisions/>
@@ -327,5 +327,5 @@
         <mass value="0.1"/>
         <origin xyz="0 0 0"/>
-        <inertia ixx="0.001" ixy="0.0" ixz="0.0" iyy="0.001" iyz="0.0" izz="0.001"/>
+        <inertia ixx="3.78125e-05" ixy="0.0" ixz="0.0" iyy="3.78125e-05" iyz="0.0" izz="6.30208e-06"/>
       </inertial>
     <xacro:distal_link_collisions/>
@@ -348,7 +348,7 @@
   <link name="${side}_finger[1]/base_rotation_link">
       <inertial>
-        <mass value="0.1"/>
-        <origin xyz="0 0 0"/>
-        <inertia ixx="0.001" ixy="0.0" ixz="0.0" iyy="0.001" iyz="0.0" izz="0.001"/>
+        <mass value="0.05"/>
+        <origin xyz="0 0 0"/>
+        <inertia ixx="0.0000125" ixy="0.0" ixz="0.0" iyy="0.0000125" iyz="0.0" izz="0.000002"/>
       </inertial>
     <xacro:base_rotation_link_collisions/>
@@ -367,5 +367,5 @@
         <mass value="0.1"/>
         <origin xyz="0 0 0"/>
-        <inertia ixx="0.001" ixy="0.0" ixz="0.0" iyy="0.001" iyz="0.0" izz="0.001"/>
+        <inertia ixx="3.78125e-05" ixy="0.0" ixz="0.0" iyy="3.78125e-05" iyz="0.0" izz="6.30208e-06"/>
       </inertial>
     <xacro:proximal_link_collisions/>
@@ -390,5 +390,5 @@
         <mass value="0.1"/>
         <origin xyz="0 0 0"/>
-        <inertia ixx="0.001" ixy="0.0" ixz="0.0" iyy="0.001" iyz="0.0" izz="0.001"/>
+        <inertia ixx="3.78125e-05" ixy="0.0" ixz="0.0" iyy="3.78125e-05" iyz="0.0" izz="6.30208e-06"/>
       </inertial>
     <xacro:distal_link_collisions/>
@@ -413,5 +413,5 @@
         <mass value="0.1"/>
         <origin xyz="0 0 0"/>
-        <inertia ixx="0.001" ixy="0.0" ixz="0.0" iyy="0.001" iyz="0.0" izz="0.001"/>
+        <inertia ixx="3.78125e-05" ixy="0.0" ixz="0.0" iyy="3.78125e-05" iyz="0.0" izz="6.30208e-06"/>
       </inertial>
     <xacro:proximal_link_collisions/>
@@ -436,5 +436,5 @@
         <mass value="0.1"/>
         <origin xyz="0 0 0"/>
-        <inertia ixx="0.001" ixy="0.0" ixz="0.0" iyy="0.001" iyz="0.0" izz="0.001"/>
+        <inertia ixx="3.78125e-05" ixy="0.0" ixz="0.0" iyy="3.78125e-05" iyz="0.0" izz="6.30208e-06"/>
       </inertial>
     <xacro:distal_link_collisions/>

Commit message: first shot at putting in the right inertia for finger links (excluding base_link and base_rotation_link for now).

File: irobot_hand_description/urdf/irobot_hand.urdf.xacro (robot description, xacro)
@@ -11,7 +11,12 @@
   <link name="${side}_finger[${finger_id}]/flexible_link_${link_id}">
     <inertial>
-      <mass value="0.001"/>
-      <origin xyz="0 0 0"/>
-      <inertia ixx="0.000001" ixy="0.0" ixz="0.0" iyy="0.000001" iyz="0.0" izz="0.000001"/>
+      <mass value="${0.0029 / 19}"/>
+      <!-- gazebo -> cad mapping
+           x -> y
+           y -> z
+           z -> x
+      -->
+      <origin xyz="0 0 0" rpy="${-pi/2} ${-pi/2} 0"/>
+      <inertia ixx="8.8101e-8" ixy="0" ixz="0.0" iyy="${2.04906e-7 / 19}" iyz="0.0" izz="${2.65921e-7 / 19}"/>
     </inertial>
     <collision>
@@ -42,7 +47,12 @@
   <link name="${side}_finger[${finger_id}]/flexible_link_hidden_between_${link_from}_and_${link_to}">
     <inertial>
-      <mass value="0.001"/>
-      <origin xyz="0 0 0"/>
-      <inertia ixx="0.000001" ixy="0.0" ixz="0.0" iyy="0.000001" iyz="0.0" izz="0.000001"/>
+      <mass value="${0.0029 / 19}"/>
+      <!-- gazebo -> cad mapping
+           x -> y
+           y -> z
+           z -> x
+      -->
+      <origin xyz="0 0 0" rpy="${-pi/2} ${-pi/2} 0"/>
+      <inertia ixx="8.8101e-8" ixy="0" ixz="0.0" iyy="${2.04906e-7 / 19}" iyz="0.0" izz="${2.65921e-7 / 19}"/>
     </inertial>
     <collision>
@@ -78,7 +88,12 @@
   <link name="${side}_finger[${finger_id}]/flexible_link_hidden_between_proximal_link_and_1">
     <inertial>
-      <mass value="0.001"/>
-      <origin xyz="0 0 0"/>
-      <inertia ixx="0.000001" ixy="0.0" ixz="0.0" iyy="0.000001" iyz="0.0" izz="0.000001"/>
+      <mass value="${0.0029 / 19}"/>
+      <!-- gazebo -> cad mapping
+           x -> y
+           y -> z
+           z -> x
+      -->
+      <origin xyz="0 0 0" rpy="${-pi/2} ${-pi/2} 0"/>
+      <inertia ixx="8.8101e-8" ixy="0" ixz="0.0" iyy="${2.04906e-7 / 19}" iyz="0.0" izz="${2.65921e-7 / 19}"/>
     </inertial>
     <collision>
@@ -112,7 +127,12 @@
   <link name="${side}_finger[${finger_id}]/flexible_link_hidden_between_9_and_distal_link">
     <inertial>
-      <mass value="0.001"/>
-      <origin xyz="0 0 0"/>
-      <inertia ixx="0.000001" ixy="0.0" ixz="0.0" iyy="0.000001" iyz="0.0" izz="0.000001"/>
+      <mass value="${0.0029 / 19}"/>
+      <!-- gazebo -> cad mapping
+           x -> y
+           y -> z
+           z -> x
+      -->
+      <origin xyz="0 0 0" rpy="${-pi/2} ${-pi/2} 0"/>
+      <inertia ixx="8.8101e-8" ixy="0" ixz="0.0" iyy="${2.04906e-7 / 19}" iyz="0.0" izz="${2.65921e-7 / 19}"/>
     </inertial>
     <collision>
@@ -257,4 +277,5 @@
   <link name="${side}_base_link">
       <inertial>
+        <!-- needs update -->
         <mass value="1.0"/>
         <origin xyz="0 0 0"/>
@@ -285,4 +306,5 @@
   <link name="${side}_finger[0]/base_rotation_link">
       <inertial>
+        <!-- needs update -->
         <mass value="0.05"/>
         <origin xyz="0 0 0"/>
@@ -302,7 +324,12 @@
   <link name="${side}_finger[0]/proximal_link">
       <inertial>
-        <mass value="0.1"/>
-        <origin xyz="0 0 0"/>
-        <inertia ixx="3.78125e-05" ixy="0.0" ixz="0.0" iyy="3.78125e-05" iyz="0.0" izz="6.30208e-06"/>
+        <mass value="0.0288"/>
+        <!-- gazebo -> cad coordinate mapping
+             x -> -y
+             y -> -z
+             z -> x
+        -->
+        <origin xyz="-0.002630 0.002396 0.021770" rpy="${pi/2} -${pi/2} 0"/>
+        <inertia ixx="2.420689e-6" ixy="-1.449042e-6" ixz="-7.74579e-7" iyy="1.196202e-6" iyz="1.90704e-7" izz="1.2736461e-6"/>
       </inertial>
     <xacro:proximal_link_collisions/>
@@ -325,7 +352,12 @@
   <link name="${side}_finger[0]/distal_link">
       <inertial>
-        <mass value="0.1"/>
-        <origin xyz="0 0 0"/>
-        <inertia ixx="3.78125e-05" ixy="0.0" ixz="0.0" iyy="3.78125e-05" iyz="0.0" izz="6.30208e-06"/>
+        <mass value="0.0133"/>
+        <!-- gazebo -> cad mapping
+             x -> -x
+             y -> y
+             z -> -z
+        -->
+        <origin xyz="-0.000066 -0.003142 0.016633" rpy="0 ${pi} 0" />
+        <inertia ixx="1.624140e-6" ixy="5.60e-10" ixz="1.33e-10" iyy="1.717885e-6" iyz="-1.19970e-7" izz="5.60221e-7"/>
       </inertial>
     <xacro:distal_link_collisions/>
@@ -365,7 +397,12 @@
   <link name="${side}_finger[1]/proximal_link">
       <inertial>
-        <mass value="0.1"/>
-        <origin xyz="0 0 0"/>
-        <inertia ixx="3.78125e-05" ixy="0.0" ixz="0.0" iyy="3.78125e-05" iyz="0.0" izz="6.30208e-06"/>
+        <mass value="0.0288"/>
+        <!-- gazebo -> cad coordinate mapping
+             x -> -y
+             y -> -z
+             z -> x
+        -->
+        <origin xyz="-0.002630 0.002396 0.021770" rpy="${pi/2} -${pi/2} 0"/>
+        <inertia ixx="2.420689e-6" ixy="-1.449042e-6" ixz="-7.74579e-7" iyy="1.196202e-6" iyz="1.90704e-7" izz="1.2736461e-6"/>
       </inertial>
     <xacro:proximal_link_collisions/>
@@ -388,7 +425,12 @@
   <link name="${side}_finger[1]/distal_link">
       <inertial>
-        <mass value="0.1"/>
-        <origin xyz="0 0 0"/>
-        <inertia ixx="3.78125e-05" ixy="0.0" ixz="0.0" iyy="3.78125e-05" iyz="0.0" izz="6.30208e-06"/>
+        <mass value="0.0133"/>
+        <!-- gazebo -> cad mapping
+             x -> -x
+             y -> y
+             z -> -z
+        -->
+        <origin xyz="-0.000066 -0.003142 0.016633" rpy="0 ${pi} 0" />
+        <inertia ixx="1.624140e-6" ixy="5.60e-10" ixz="1.33e-10" iyy="1.717885e-6" iyz="-1.19970e-7" izz="5.60221e-7"/>
       </inertial>
     <xacro:distal_link_collisions/>
@@ -411,7 +453,12 @@
   <link name="${side}_finger[2]/proximal_link">
       <inertial>
-        <mass value="0.1"/>
-        <origin xyz="0 0 0"/>
-        <inertia ixx="3.78125e-05" ixy="0.0" ixz="0.0" iyy="3.78125e-05" iyz="0.0" izz="6.30208e-06"/>
+        <mass value="0.0288"/>
+        <!-- gazebo -> cad coordinate mapping
+             x -> -y
+             y -> -z
+             z -> x
+        -->
+        <origin xyz="-0.002630 0.002396 0.021770" rpy="${pi/2} -${pi/2} 0"/>
+        <inertia ixx="2.420689e-6" ixy="-1.449042e-6" ixz="-7.74579e-7" iyy="1.196202e-6" iyz="1.90704e-7" izz="1.2736461e-6"/>
       </inertial>
     <xacro:proximal_link_collisions/>
@@ -434,7 +481,12 @@
   <link name="${side}_finger[2]/distal_link">
       <inertial>
-        <mass value="0.1"/>
-        <origin xyz="0 0 0"/>
-        <inertia ixx="3.78125e-05" ixy="0.0" ixz="0.0" iyy="3.78125e-05" iyz="0.0" izz="6.30208e-06"/>
+        <mass value="0.0133"/>
+        <!-- gazebo -> cad mapping
+             x -> -x
+             y -> y
+             z -> -z
+        -->
+        <origin xyz="-0.000066 -0.003142 0.016633" rpy="0 ${pi} 0" />
+        <inertia ixx="1.624140e-6" ixy="5.60e-10" ixz="1.33e-10" iyy="1.717885e-6" iyz="-1.19970e-7" izz="5.60221e-7"/>
       </inertial>
     <xacro:distal_link_collisions/>

Commit message: add gearbox to enforce spread symmetry.  testing controller.

File: irobot_hand_description/urdf/irobot_hand.urdf.xacro (robot description, xacro)
@@ -555,4 +555,26 @@
     <limit effort="1000.0" lower="0.0" upper="${pi/2}" velocity="0.5"/>
   </joint>
+  <gazebo>
+    <joint name="${side}_spread_gearbox" type="gearbox">
+      <parent>${side}_finger[0]/base_rotation_link</parent>
+      <child>${side}_finger[1]/base_rotation_link</child>
+      <!-- ${side}_base_link got lumped into ${parent},
+           so we need to fix parser_urdf.cc to propagate name
+           changes into this extension before switching this
+           to use ${side_base_link}. -->
+      <gearbox_reference_body>${parent}</gearbox_reference_body>
+      <gearbox_ratio>1.0</gearbox_ratio>
+      <axis>
+        <!-- yikes, what coordinate frame is this specified in?
+             0 0 1 causes NaNs. 0 1 0 works, but unsure why yet.-->
+        <xyz>0 1 0</xyz>
+      </axis>
+      <axis2>
+        <!-- yikes, what coordinate frame is this specified in?
+             0 0 1 causes NaNs. 0 1 0 works, but unsure why yet.-->
+        <xyz>0 1 0</xyz>
+      </axis2>
+    </joint>
+  </gazebo>
   <gazebo reference="${side}_finger[1]/joint_base">
     <cfmDamping>1</cfmDamping>
