Commit message: testing control modes. switch to 2 intermediate links for flexure

File: irobot_hand_description/urdf/irobot_hand.urdf.xacro (robot description, xacro)
@@ -5,5 +5,5 @@
 <!-- tip: use measurements from solid to find the origins and length -->
 <xacro:property name="flex_joint_length" value=".016" />
-<xacro:property name="flex_joint_steps" value="9" />
+<xacro:property name="flex_joint_steps" value="3" />
 <xacro:property name="proximal_link_length" value=".062" />
 <xacro:property name="pi" value="3.14" />
@@ -11,5 +11,5 @@
   <link name="${side}_finger[${finger_id}]/flexible_link_${link_id}">
     <inertial>
-      <mass value="${0.0029 / 19}"/>
+      <mass value="${0.0029 / (2 * flex_joint_steps + 1)}"/>
       <!-- gazebo -> cad mapping
            x -> y
@@ -18,5 +18,7 @@
       -->
       <origin xyz="0 0 0" rpy="${-pi/2} ${-pi/2} 0"/>
-      <inertia ixx="8.8101e-8" ixy="0" ixz="0.0" iyy="${2.04906e-7 / 19}" iyz="0.0" izz="${2.65921e-7 / 19}"/>
+      <inertia ixx="8.8101e-8" ixy="0" ixz="0.0"
+               iyy="${2.04906e-7 / (2 * flex_joint_steps + 1)}" iyz="0.0"
+               izz="${2.65921e-7 / (2 * flex_joint_steps + 1)}"/>
     </inertial>
     <collision>
@@ -50,5 +52,5 @@
   <link name="${side}_finger[${finger_id}]/flexible_link_hidden_between_${link_from}_and_${link_to}">
     <inertial>
-      <mass value="${0.0029 / 19}"/>
+      <mass value="${0.0029 / (2 * flex_joint_steps + 1)}"/>
       <!-- gazebo -> cad mapping
            x -> y
@@ -57,5 +59,7 @@
       -->
       <origin xyz="0 0 0" rpy="${-pi/2} ${-pi/2} 0"/>
-      <inertia ixx="8.8101e-8" ixy="0" ixz="0.0" iyy="${2.04906e-7 / 19}" iyz="0.0" izz="${2.65921e-7 / 19}"/>
+      <inertia ixx="8.8101e-8" ixy="0" ixz="0.0"
+               iyy="${2.04906e-7 / (2 * flex_joint_steps + 1)}" iyz="0.0"
+               izz="${2.65921e-7 / (2 * flex_joint_steps + 1)}"/>
     </inertial>
     <collision>
@@ -97,5 +101,6 @@
   <link name="${side}_finger[${finger_id}]/flexible_link_hidden_between_proximal_link_and_1">
     <inertial>
-      <mass value="${0.0029 / 19}"/>
+      <!-- <mass value="${0.0029 / 19}"/> -->
+      <mass value="${0.0029 / (2 * flex_joint_steps + 1)}"/>
       <!-- gazebo -> cad mapping
            x -> y
@@ -104,5 +109,7 @@
       -->
       <origin xyz="0 0 0" rpy="${-pi/2} ${-pi/2} 0"/>
-      <inertia ixx="8.8101e-8" ixy="0" ixz="0.0" iyy="${2.04906e-7 / 19}" iyz="0.0" izz="${2.65921e-7 / 19}"/>
+      <inertia ixx="8.8101e-8" ixy="0" ixz="0.0"
+               iyy="${2.04906e-7 / (2 * flex_joint_steps + 1)}" iyz="0.0"
+               izz="${2.65921e-7 / (2 * flex_joint_steps + 1)}"/>
     </inertial>
     <collision>
@@ -130,17 +137,17 @@
   </joint>
   <!-- make a connection between flexible to distal-->
-  <gazebo reference="${side}_finger[${finger_id}]/flexible_joint_flex_from_9_to_distal">
-    <cfmDamping>1</cfmDamping>
-  </gazebo>
-  <joint name="${side}_finger[${finger_id}]/flexible_joint_flex_from_9_to_distal" type="revolute">
-    <parent link="${side}_finger[${finger_id}]/flexible_link_9"/>
-    <child link="${side}_finger[${finger_id}]/flexible_link_hidden_between_9_and_distal_link"/>
+  <gazebo reference="${side}_finger[${finger_id}]/flexible_joint_flex_from_${flex_joint_steps}_to_distal">
+    <cfmDamping>1</cfmDamping>
+  </gazebo>
+  <joint name="${side}_finger[${finger_id}]/flexible_joint_flex_from_${flex_joint_steps}_to_distal" type="revolute">
+    <parent link="${side}_finger[${finger_id}]/flexible_link_${flex_joint_steps}"/>
+    <child link="${side}_finger[${finger_id}]/flexible_link_hidden_between_${flex_joint_steps}_and_distal_link"/>
     <origin xyz="0 0 ${flex_joint_length/flex_joint_steps}" />
     <axis xyz="-1 0 0"/>
     <limit effort="1000.0" lower="0.0" upper="${pi/2}" velocity="0.5"/>
   </joint>
-  <link name="${side}_finger[${finger_id}]/flexible_link_hidden_between_9_and_distal_link">
+  <link name="${side}_finger[${finger_id}]/flexible_link_hidden_between_${flex_joint_steps}_and_distal_link">
     <inertial>
-      <mass value="${0.0029 / 19}"/>
+      <mass value="${0.0029 / (2 * flex_joint_steps + 1)}"/>
       <!-- gazebo -> cad mapping
            x -> y
@@ -149,5 +156,7 @@
       -->
       <origin xyz="0 0 0" rpy="${-pi/2} ${-pi/2} 0"/>
-      <inertia ixx="8.8101e-8" ixy="0" ixz="0.0" iyy="${2.04906e-7 / 19}" iyz="0.0" izz="${2.65921e-7 / 19}"/>
+      <inertia ixx="8.8101e-8" ixy="0" ixz="0.0"
+               iyy="${2.04906e-7 / (2 * flex_joint_steps + 1)}" iyz="0.0"
+               izz="${2.65921e-7 / (2 * flex_joint_steps + 1)}"/>
     </inertial>
     <collision>
@@ -164,9 +173,9 @@
     </visual>
   </link>
-  <gazebo reference="${side}_finger[${finger_id}]/flexible_joint_twist_from_9_to_distal">
-    <cfmDamping>1</cfmDamping>
-  </gazebo>
-  <joint name="${side}_finger[${finger_id}]/flexible_joint_twist_from_9_to_distal" type="revolute">
-    <parent link="${side}_finger[${finger_id}]/flexible_link_hidden_between_9_and_distal_link"/>
+  <gazebo reference="${side}_finger[${finger_id}]/flexible_joint_twist_from_${flex_joint_steps}_to_distal">
+    <cfmDamping>1</cfmDamping>
+  </gazebo>
+  <joint name="${side}_finger[${finger_id}]/flexible_joint_twist_from_${flex_joint_steps}_to_distal" type="revolute">
+    <parent link="${side}_finger[${finger_id}]/flexible_link_hidden_between_${flex_joint_steps}_and_distal_link"/>
     <child link="${side}_finger[${finger_id}]/distal_link"/>
     <origin xyz="0 0 0" />
@@ -235,4 +244,5 @@
   <xacro:flex_link side="${side}" finger_id="0" link_id="1"/>
   <xacro:flex_link side="${side}" finger_id="0" link_id="2"/>
+  <!-- only up to flex_joint_steps
   <xacro:flex_link side="${side}" finger_id="0" link_id="3"/>
   <xacro:flex_link side="${side}" finger_id="0" link_id="4"/>
@@ -242,5 +252,7 @@
   <xacro:flex_link side="${side}" finger_id="0" link_id="8"/>
   <xacro:flex_link side="${side}" finger_id="0" link_id="9"/>
+  -->
   <xacro:flex_joint side="${side}" finger_id="0" link_from="1" link_to="2"/>
+  <!-- only up to flex_joint_steps
   <xacro:flex_joint side="${side}" finger_id="0" link_from="2" link_to="3"/>
   <xacro:flex_joint side="${side}" finger_id="0" link_from="3" link_to="4"/>
@@ -250,7 +262,9 @@
   <xacro:flex_joint side="${side}" finger_id="0" link_from="7" link_to="8"/>
   <xacro:flex_joint side="${side}" finger_id="0" link_from="8" link_to="9"/>
-  <xacro:flex_joint_connector side="${side}" finger_id="0"/>
+  -->
+  <xacro:flex_joint_connector side="${side}" finger_id="0" />
   <xacro:flex_link side="${side}" finger_id="1" link_id="1"/>
   <xacro:flex_link side="${side}" finger_id="1" link_id="2"/>
+  <!-- only up to flex_joint_steps
   <xacro:flex_link side="${side}" finger_id="1" link_id="3"/>
   <xacro:flex_link side="${side}" finger_id="1" link_id="4"/>
@@ -260,5 +274,7 @@
   <xacro:flex_link side="${side}" finger_id="1" link_id="8"/>
   <xacro:flex_link side="${side}" finger_id="1" link_id="9"/>
+  -->
   <xacro:flex_joint side="${side}" finger_id="1" link_from="1" link_to="2"/>
+  <!-- only up to flex_joint_steps
   <xacro:flex_joint side="${side}" finger_id="1" link_from="2" link_to="3"/>
   <xacro:flex_joint side="${side}" finger_id="1" link_from="3" link_to="4"/>
@@ -268,7 +284,9 @@
   <xacro:flex_joint side="${side}" finger_id="1" link_from="7" link_to="8"/>
   <xacro:flex_joint side="${side}" finger_id="1" link_from="8" link_to="9"/>
-  <xacro:flex_joint_connector side="${side}" finger_id="1"/>
+  -->
+  <xacro:flex_joint_connector side="${side}" finger_id="1" />
   <xacro:flex_link side="${side}" finger_id="2" link_id="1"/>
   <xacro:flex_link side="${side}" finger_id="2" link_id="2"/>
+  <!-- only up to flex_joint_steps
   <xacro:flex_link side="${side}" finger_id="2" link_id="3"/>
   <xacro:flex_link side="${side}" finger_id="2" link_id="4"/>
@@ -278,5 +296,7 @@
   <xacro:flex_link side="${side}" finger_id="2" link_id="8"/>
   <xacro:flex_link side="${side}" finger_id="2" link_id="9"/>
+  -->
   <xacro:flex_joint side="${side}" finger_id="2" link_from="1" link_to="2"/>
+  <!-- only up to flex_joint_steps
   <xacro:flex_joint side="${side}" finger_id="2" link_from="2" link_to="3"/>
   <xacro:flex_joint side="${side}" finger_id="2" link_from="3" link_to="4"/>
@@ -286,5 +306,6 @@
   <xacro:flex_joint side="${side}" finger_id="2" link_from="7" link_to="8"/>
   <xacro:flex_joint side="${side}" finger_id="2" link_from="8" link_to="9"/>
-  <xacro:flex_joint_connector side="${side}" finger_id="2"/>
+  -->
+  <xacro:flex_joint_connector side="${side}" finger_id="2" />
   <!-- joint to irobot hand -->
   <joint name="${side}_irobot_hand_joint" type="fixed">

Commit message: fix urdf

File: irobot_hand_description/urdf/irobot_hand.urdf.xacro (robot description, xacro)
@@ -5,5 +5,5 @@
 <!-- tip: use measurements from solid to find the origins and length -->
 <xacro:property name="flex_joint_length" value=".016" />
-<xacro:property name="flex_joint_steps" value="3" />
+<xacro:property name="flex_joint_steps" value="2" />
 <xacro:property name="proximal_link_length" value=".062" />
 <xacro:property name="pi" value="3.14" />

Commit message: fix flex offset

File: irobot_hand_description/urdf/irobot_hand.urdf.xacro (robot description, xacro)
@@ -8,4 +8,5 @@
 <xacro:property name="proximal_link_length" value=".062" />
 <xacro:property name="pi" value="3.14" />
+<xacro:property name="flex_offset" value="0.003"/> <!--${0.5*flex_joint_length/flex_joint_steps}-->
 <xacro:macro name="flex_link" params="side finger_id link_id">
   <link name="${side}_finger[${finger_id}]/flexible_link_${link_id}">
@@ -95,5 +96,5 @@
     <parent link="${side}_finger[${finger_id}]/proximal_link"/>
     <child link="${side}_finger[${finger_id}]/flexible_link_hidden_between_proximal_link_and_1"/>
-    <origin xyz="0 0 ${proximal_link_length}" />
+    <origin xyz="0 0 ${proximal_link_length + flex_offset}" />
     <axis xyz="-1 0 0"/>
     <limit effort="1000.0" lower="0.0" upper="${pi/2}" velocity="0.5"/>
@@ -143,5 +144,5 @@
     <parent link="${side}_finger[${finger_id}]/flexible_link_${flex_joint_steps}"/>
     <child link="${side}_finger[${finger_id}]/flexible_link_hidden_between_${flex_joint_steps}_and_distal_link"/>
-    <origin xyz="0 0 ${flex_joint_length/flex_joint_steps}" />
+    <origin xyz="0 0 ${flex_joint_length/flex_joint_steps - flex_offset}" />
     <axis xyz="-1 0 0"/>
     <limit effort="1000.0" lower="0.0" upper="${pi/2}" velocity="0.5"/>

Commit message: Added better collision models to finger tip

File: irobot_hand_description/urdf/irobot_hand.urdf.xacro (robot description, xacro)
@@ -236,7 +236,20 @@
 <xacro:macro name="distal_link_collisions">
       <collision name='collision'>
-        <origin xyz="0 0.0025 0.019" rpy="3.141590 0.001593 3.141590"/>
-        <geometry>
-          <box size="0.0175 0.02023 0.04043"/>
+        <origin xyz="0 0.0024 0.01476" rpy="3.141590 0.001593
+             3.141590"/>
+        <geometry>
+          <box size="0.0175 0.02011 0.03195"/>
+        </geometry>
+      </collision>
+      <collision name='collision_tip'>
+        <origin xyz="0 0.004 0.03" rpy="1.57078 0.001593 1.57078"/>
+        <geometry>
+          <cylinder radius="0.00848" length="0.0175"/>
+        </geometry>
+      </collision>
+      <collision name='collision_nail'>
+        <origin xyz="0 -0.00529 0.032" rpy="1.57078 0.001593 0"/>
+        <geometry>
+          <cylinder radius="0.00750" length="0.00159"/>
         </geometry>
       </collision>

Commit message: fix issue #106 for irobot hand mass discrepancy.

File: irobot_hand_description/urdf/irobot_hand.urdf.xacro (robot description, xacro)
@@ -331,5 +331,5 @@
       <inertial>
         <!-- needs update -->
-        <mass value="1.0"/>
+        <mass value="1.305"/>
         <origin xyz="0 0 0"/>
         <inertia ixx="0.00125" ixy="0.0" ixz="0.0" iyy="0.00125" iyz="0.0" izz="0.0002"/>

Commit message: Reduce joint limits for irobot fingers, based on patch from @nmertins, per #402

File: irobot_hand_description/urdf/irobot_hand.urdf.xacro (robot description, xacro)
@@ -578,5 +578,5 @@
     <origin xyz="0 0 0.0135" rpy="${pi/2} 0 -${pi}" />
     <axis xyz="-1 0 0"/>
-    <limit effort="1000.0" lower="0.0" upper="${pi/2}" velocity="0.5"/>
+    <limit effort="1000.0" lower="0.0" upper="${7*pi/8}" velocity="0.5"/>
   </joint>
   <gazebo reference="${side}_finger[1]/joint_base_rotation">
@@ -620,5 +620,5 @@
     <origin xyz="0 0 0.0135" rpy="${pi/2} 0 -${pi}" />
     <axis xyz="-1 0 0"/>
-    <limit effort="1000.0" lower="0.0" upper="${pi/2}" velocity="0.5"/>
+    <limit effort="1000.0" lower="0.0" upper="${7*pi/8}" velocity="0.5"/>
   </joint>
   <gazebo reference="${side}_finger[2]/joint_base">
@@ -630,5 +630,5 @@
     <origin xyz="0 -0.038 0.082755" rpy="${pi/2} 0 0" />
     <axis xyz="-1 0 0"/>
-    <limit effort="1000.0" lower="0.0" upper="${pi/2}" velocity="0.5"/>
+    <limit effort="1000.0" lower="0.0" upper="${7*pi/8}" velocity="0.5"/>
   </joint>
 </xacro:macro>
