Commit message: syncing v3 to fixed in v1 and vice versa

File: atlas_description/urdf/atlas_original_inertia.urdf (robot description, URDF)
Before this commit: robot drc_skeleton, 28 links, 28 joints
Links:
- link l_lleg: geometry collision mesh filename=package://atlas_description/meshes/l_lleg.stl scale=1 1 1; visual mesh filename=package://atlas_description/meshes/l_lleg.dae scale=1 1 1
- link l_uleg: geometry collision mesh filename=package://atlas_description/meshes/l_uleg.stl scale=1 1 1; visual mesh filename=package://atlas_description/meshes/l_uleg.dae scale=1 1 1
- link pelvis: geometry collision mesh filename=package://atlas_description/meshes/pelvis.stl scale=1 1 1; visual mesh filename=package://atlas_description/meshes/pelvis.dae scale=1 1 1
- link r_larm: geometry collision mesh filename=package://atlas_description/meshes/r_larm.stl scale=1 1 1; visual mesh filename=package://atlas_description/meshes/r_larm.dae scale=1 1 1
- link r_lglut: geometry collision mesh filename=package://atlas_description/meshes/r_lglut.stl scale=1 1 1; visual mesh filename=package://atlas_description/meshes/r_lglut.dae scale=1 1 1
- link r_lleg: geometry collision mesh filename=package://atlas_description/meshes/r_lleg.stl scale=1 1 1; visual mesh filename=package://atlas_description/meshes/r_lleg.dae scale=1 1 1
- link r_uarm: geometry collision mesh filename=package://atlas_description/meshes/r_uarm.stl scale=1 1 1; visual mesh filename=package://atlas_description/meshes/r_uarm.dae scale=1 1 1
- link r_uglut: geometry collision mesh filename=package://atlas_description/meshes/r_uglut.stl scale=1 1 1; visual mesh filename=package://atlas_description/meshes/r_uglut.dae scale=1 1 1
- link r_uleg: geometry collision mesh filename=package://atlas_description/meshes/r_uleg.stl scale=1 1 1; visual mesh filename=package://atlas_description/meshes/r_uleg.dae scale=1 1 1
Joints:
- joint l_leg_kny: limit lower=0 upper=2.45 effort=400 velocity=12 -> lower=0 upper=2.45 effort=220 velocity=12
- joint l_leg_uay: limit lower=-0.9 upper=0.698 effort=220 velocity=12 -> lower=-0.698 upper=0.698 effort=220 velocity=12
- joint neck_ay: origin xyz=0.21672 0 0.53796 rpy=0 -0 0 -> xyz=0.16555 0 0.50823 rpy=0 -0 0
- joint r_leg_kny: limit lower=0 upper=2.45 effort=400 velocity=12 -> lower=0 upper=2.45 effort=220 velocity=12
- joint r_leg_uay: limit lower=-0.9 upper=0.698 effort=220 velocity=12 -> lower=-0.698 upper=0.698 effort=220 velocity=12
