Commit message: adding atlas_v3.urdf and corresponding DAE files

File: atlas_description/urdf/atlas_v3.urdf (robot description, URDF)
Before this commit: robot drc_skeleton, 29 links, 28 joints
Links:
- removed link head

Commit message: update mesh file names

File: atlas_description/urdf/atlas_v3.urdf (robot description, URDF)
Before this commit: robot drc_skeleton, 28 links, 28 joints
Links:
- added link head, mass 3.751; collision mesh filename=package://atlas/meshes_v3/head.DAE scale=1 1 1; visual mesh filename=package://atlas/meshes_v3/head.DAE scale=1 1 1
- link l_clav: geometry collision mesh filename=package://atlas/meshes_v3/l_clav.DAE scale=1 1 1; visual mesh filename=package://atlas/meshes_v3/l_clav.DAE scale=1 1 1
- link l_farm: geometry collision mesh filename=package://atlas/meshes_v3/l_farm.DAE scale=1 1 1; visual mesh filename=package://atlas/meshes_v3/l_farm.DAE scale=1 1 1
- link l_foot: geometry collision mesh filename=package://atlas/meshes_v3/l_foot.DAE scale=1 1 1; visual mesh filename=package://atlas/meshes_v3/l_foot.DAE scale=1 1 1
- link l_hand: geometry collision mesh filename=package://atlas/meshes_v3/l_hand.DAE scale=1 1 1; visual mesh filename=package://atlas/meshes_v3/l_hand.DAE scale=1 1 1
- link l_larm: geometry collision mesh filename=package://atlas/meshes_v3/l_larm.DAE scale=1 1 1; visual mesh filename=package://atlas/meshes_v3/l_larm.DAE scale=1 1 1
- link l_lglut: geometry collision mesh filename=package://atlas/meshes_v3/l_lglut.DAE scale=1 1 1; visual mesh filename=package://atlas/meshes_v3/l_lglut.DAE scale=1 1 1
- link l_lleg: geometry collision mesh filename=package://atlas/meshes_v3/l_lleg.DAE scale=1 1 1; visual mesh filename=package://atlas/meshes_v3/l_lleg.DAE scale=1 1 1
- link l_scap: geometry collision mesh filename=package://atlas/meshes_v3/l_scap.DAE scale=1 1 1; visual mesh filename=package://atlas/meshes_v3/l_scap.DAE scale=1 1 1
- link l_talus: geometry collision mesh filename=package://atlas/meshes_v3/l_talus.DAE scale=1 1 1; visual mesh filename=package://atlas/meshes_v3/l_talus.DAE scale=1 1 1
- link l_uarm: geometry collision mesh filename=package://atlas/meshes_v3/l_uarm.DAE scale=1 1 1; visual mesh filename=package://atlas/meshes_v3/l_uarm.DAE scale=1 1 1
- link l_uglut: geometry collision mesh filename=package://atlas/meshes_v3/l_uglut.DAE scale=1 1 1; visual mesh filename=package://atlas/meshes_v3/l_uglut.DAE scale=1 1 1
- link l_uleg: geometry collision mesh filename=package://atlas/meshes_v3/l_uleg.DAE scale=1 1 1; visual mesh filename=package://atlas/meshes_v3/l_uleg.DAE scale=1 1 1
- link ltorso: geometry collision mesh filename=package://atlas/meshes_v3/ltorso.DAE scale=1 1 1; visual mesh filename=package://atlas/meshes_v3/ltorso.DAE scale=1 1 1
- link mtorso: geometry collision mesh filename=package://atlas/meshes_v3/mtorso.DAE scale=1 1 1; visual mesh filename=package://atlas/meshes_v3/mtorso.DAE scale=1 1 1
- link pelvis: geometry collision mesh filename=package://atlas/meshes_v3/pelvis.DAE scale=1 1 1; visual mesh filename=package://atlas/meshes_v3/pelvis.DAE scale=1 1 1
- link r_clav: geometry collision mesh filename=package://atlas/meshes_v3/r_clav.DAE scale=1 1 1; visual mesh filename=package://atlas/meshes_v3/r_clav.DAE scale=1 1 1
- link r_farm: geometry collision mesh filename=package://atlas/meshes_v3/r_farm.DAE scale=1 1 1; visual mesh filename=package://atlas/meshes_v3/r_farm.DAE scale=1 1 1
- link r_foot: geometry collision mesh filename=package://atlas/meshes_v3/r_foot.DAE scale=1 1 1; visual mesh filename=package://atlas/meshes_v3/r_foot.DAE scale=1 1 1
- link r_hand: geometry collision mesh filename=package://atlas/meshes_v3/r_hand.DAE scale=1 1 1; visual mesh filename=package://atlas/meshes_v3/r_hand.DAE scale=1 1 1
- link r_larm: geometry collision mesh filename=package://atlas/meshes_v3/r_larm.DAE scale=1 1 1; visual mesh filename=package://atlas/meshes_v3/r_larm.DAE scale=1 1 1
- link r_lglut: geometry collision mesh filename=package://atlas/meshes_v3/r_lglut.DAE scale=1 1 1; visual mesh filename=package://atlas/meshes_v3/r_lglut.DAE scale=1 1 1
- link r_lleg: geometry collision mesh filename=package://atlas/meshes_v3/r_lleg.DAE scale=1 1 1; visual mesh filename=package://atlas/meshes_v3/r_lleg.DAE scale=1 1 1
- link r_scap: geometry collision mesh filename=package://atlas/meshes_v3/r_scap.DAE scale=1 1 1; visual mesh filename=package://atlas/meshes_v3/r_scap.DAE scale=1 1 1
- link r_talus: geometry collision mesh filename=package://atlas/meshes_v3/r_talus.DAE scale=1 1 1; visual mesh filename=package://atlas/meshes_v3/r_talus.DAE scale=1 1 1
- link r_uarm: geometry collision mesh filename=package://atlas/meshes_v3/r_uarm.DAE scale=1 1 1; visual mesh filename=package://atlas/meshes_v3/r_uarm.DAE scale=1 1 1
- link r_uglut: geometry collision mesh filename=package://atlas/meshes_v3/r_uglut.DAE scale=1 1 1; visual mesh filename=package://atlas/meshes_v3/r_uglut.DAE scale=1 1 1
- link r_uleg: geometry collision mesh filename=package://atlas/meshes_v3/r_uleg.DAE scale=1 1 1; visual mesh filename=package://atlas/meshes_v3/r_uleg.DAE scale=1 1 1
- link utorso: geometry collision mesh filename=package://atlas/meshes_v3/utorso.DAE scale=1 1 1; visual mesh filename=package://atlas/meshes_v3/utorso.DAE scale=1 1 1

Commit message: update mesh names to match new meshes_v3

File: atlas_description/urdf/atlas_v3.urdf (robot description, URDF)
Before this commit: robot drc_skeleton, 28 links, 28 joints
Links:
- link l_clav: geometry collision mesh filename=package://atlas_description/meshes_v3/l_clav.DAE scale=1 1 1; visual mesh filename=package://atlas_description/meshes_v3/l_clav.DAE scale=1 1 1
- link l_farm: geometry collision mesh filename=package://atlas_description/meshes_v3/l_farm.DAE scale=1 1 1; visual mesh filename=package://atlas_description/meshes_v3/l_farm.DAE scale=1 1 1
- link l_foot: geometry collision mesh filename=package://atlas_description/meshes_v3/l_foot.DAE scale=1 1 1; visual mesh filename=package://atlas_description/meshes_v3/l_foot.DAE scale=1 1 1
- link l_hand: geometry collision mesh filename=package://atlas_description/meshes_v3/l_hand.DAE scale=1 1 1; visual mesh filename=package://atlas_description/meshes_v3/l_hand.DAE scale=1 1 1
- link l_larm: geometry collision mesh filename=package://atlas_description/meshes_v3/l_elbow_rx.DAE scale=1 1 1; visual mesh filename=package://atlas_description/meshes_v3/l_elbow_rx.DAE scale=1 1 1
- link l_lglut: geometry collision mesh filename=package://atlas_description/meshes_v3/l_lglut.DAE scale=1 1 1; visual mesh filename=package://atlas_description/meshes_v3/l_lglut.DAE scale=1 1 1
- link l_lleg: geometry collision mesh filename=package://atlas_description/meshes_v3/l_lleg.DAE scale=1 1 1; visual mesh filename=package://atlas_description/meshes_v3/l_lleg.DAE scale=1 1 1
- link l_scap: geometry collision mesh filename=package://atlas_description/meshes_v3/l_sh_rx.DAE scale=1 1 1; visual mesh filename=package://atlas_description/meshes_v3/l_sh_rx.DAE scale=1 1 1
- link l_talus: geometry collision mesh filename=package://atlas_description/meshes_v3/l_talus.DAE scale=1 1 1; visual mesh filename=package://atlas_description/meshes_v3/l_talus.DAE scale=1 1 1
- link l_uarm: geometry collision mesh filename=package://atlas_description/meshes_v3/l_elbow_ry.DAE scale=1 1 1; visual mesh filename=package://atlas_description/meshes_v3/l_elbow_ry.DAE scale=1 1 1
- link l_uglut: geometry collision mesh filename=package://atlas_description/meshes_v3/l_uglut.DAE scale=1 1 1; visual mesh filename=package://atlas_description/meshes_v3/l_uglut.DAE scale=1 1 1
- link l_uleg: geometry collision mesh filename=package://atlas_description/meshes_v3/l_uleg.DAE scale=1 1 1; visual mesh filename=package://atlas_description/meshes_v3/l_uleg.DAE scale=1 1 1
- link ltorso: geometry collision mesh filename=package://atlas_description/meshes_v3/ltorso.DAE scale=1 1 1; visual mesh filename=package://atlas_description/meshes_v3/ltorso.DAE scale=1 1 1
- link mtorso: geometry collision mesh filename=package://atlas_description/meshes_v3/mtorso.DAE scale=1 1 1; visual mesh filename=package://atlas_description/meshes_v3/mtorso.DAE scale=1 1 1
- link pelvis: geometry collision mesh filename=package://atlas_description/meshes_v3/pelvis.DAE scale=1 1 1; visual mesh filename=package://atlas_description/meshes_v3/pelvis.DAE scale=1 1 1
- link r_clav: geometry collision mesh filename=package://atlas_description/meshes_v3/r_clav.DAE scale=1 1 1; visual mesh filename=package://atlas_description/meshes_v3/r_clav.DAE scale=1 1 1
- link r_farm: geometry collision mesh filename=package://atlas_description/meshes_v3/r_farm.DAE scale=1 1 1; visual mesh filename=package://atlas_description/meshes_v3/r_farm.DAE scale=1 1 1
- link r_foot: geometry collision mesh filename=package://atlas_description/meshes_v3/r_foot.DAE scale=1 1 1; visual mesh filename=package://atlas_description/meshes_v3/r_foot.DAE scale=1 1 1
- link r_hand: geometry collision mesh filename=package://atlas_description/meshes_v3/r_hand.DAE scale=1 1 1; visual mesh filename=package://atlas_description/meshes_v3/r_hand.DAE scale=1 1 1
- link r_larm: geometry collision mesh filename=package://atlas_description/meshes_v3/r_elbow_rx.DAE scale=1 1 1; visual mesh filename=package://atlas_description/meshes_v3/r_elbow_rx.DAE scale=1 1 1
- link r_lglut: geometry collision mesh filename=package://atlas_description/meshes_v3/r_lglut.DAE scale=1 1 1; visual mesh filename=package://atlas_description/meshes_v3/r_lglut.DAE scale=1 1 1
- link r_lleg: geometry collision mesh filename=package://atlas_description/meshes_v3/r_lleg.DAE scale=1 1 1; visual mesh filename=package://atlas_description/meshes_v3/r_lleg.DAE scale=1 1 1
- link r_scap: geometry collision mesh filename=package://atlas_description/meshes_v3/r_sh_rx.DAE scale=1 1 1; visual mesh filename=package://atlas_description/meshes_v3/r_sh_rx.DAE scale=1 1 1
- link r_talus: geometry collision mesh filename=package://atlas_description/meshes_v3/r_talus.DAE scale=1 1 1; visual mesh filename=package://atlas_description/meshes_v3/r_talus.DAE scale=1 1 1
- link r_uarm: geometry collision mesh filename=package://atlas_description/meshes_v3/r_elbow_ry.DAE scale=1 1 1; visual mesh filename=package://atlas_description/meshes_v3/r_elbow_ry.DAE scale=1 1 1
- link r_uglut: geometry collision mesh filename=package://atlas_description/meshes_v3/r_uglut.DAE scale=1 1 1; visual mesh filename=package://atlas_description/meshes_v3/r_uglut.DAE scale=1 1 1
- link r_uleg: geometry collision mesh filename=package://atlas_description/meshes_v3/r_uleg.DAE scale=1 1 1; visual mesh filename=package://atlas_description/meshes_v3/r_uleg.DAE scale=1 1 1
- link utorso: geometry collision mesh filename=package://atlas_description/meshes_v3/utorso.DAE scale=1 1 1; visual mesh filename=package://atlas_description/meshes_v3/utorso.DAE scale=1 1 1

Commit message: fix wrx offset (didn't pass through parse from raw cfg file for some reason, similar to shy offset).  add inertia without backpack.  add utorso mesh with backpack.

File: atlas_description/urdf/atlas_v3.urdf (robot description, URDF)
Before this commit: robot drc_skeleton, 28 links, 28 joints
Links:
- link utorso: geometry collision mesh filename=package://atlas_description/meshes_v3/utorso.DAE scale=1 1 1; collision mesh filename=package://atlas_description/meshes_v3/utorso_pack.DAE scale=1 1 1
Joints:
- joint l_arm_shx: origin xyz=0 0 0 rpy=0 -0 0 -> xyz=0 0.14035 0.19609 rpy=0 -0 0
- joint l_arm_wrx: origin xyz=0 0 0 rpy=0 -0 0 -> xyz=0 0.119 0.00921 rpy=0 -0 0
- joint r_arm_shx: origin xyz=0 0 0 rpy=0 -0 0 -> xyz=0 -0.14035 0.19609 rpy=0 -0 0
- joint r_arm_wrx: origin xyz=0 0 0 rpy=0 -0 0 -> xyz=0 -0.119 0.00921 rpy=0 -0 0

Commit message: merge from default

File: atlas_description/urdf/atlas_v3.urdf (robot description, URDF)
Before this commit: robot drc_skeleton, 32 links, 32 joints
Links:
- added link rear_situational_awareness_camera_link, mass 0.1; visual box size=0.01 0.01 0.01
- added link rear_situational_awareness_camera_optical_frame
Joints:
- added joint rear_situational_awareness_camera_joint: type fixed, parent utorso, child rear_situational_awareness_camera_link, origin xyz=-0.0026 0.0264 0.6649 rpy=0 0 3.14159
- added joint rear_situational_awareness_camera_optical_frame_joint: type fixed, parent rear_situational_awareness_camera_link, child rear_situational_awareness_camera_optical_frame, origin xyz=0 0 0 rpy=-1.5708 0.0 -1.5708

Commit message: merging from default

File: atlas_description/urdf/atlas_v3.urdf (robot description, URDF)
Before this commit: robot drc_skeleton, 32 links, 32 joints
Links:
- added link rear_situational_awareness_camera_link, mass 0.1; visual box size=0.01 0.01 0.01
- added link rear_situational_awareness_camera_optical_frame
- link l_clav: geometry collision mesh filename=package://atlas_description/meshes_v3/l_clav.stl scale=1 1 1; visual mesh filename=package://atlas_description/meshes_v3/l_clav.DAE scale=1 1 1
- link l_farm: geometry collision mesh filename=package://atlas_description/meshes_v3/l_farm.stl scale=1 1 1; visual mesh filename=package://atlas_description/meshes_v3/l_farm.DAE scale=1 1 1
- link l_foot: geometry collision mesh filename=package://atlas_description/meshes_v3/l_foot.stl scale=1 1 1; visual mesh filename=package://atlas_description/meshes_v3/l_foot.DAE scale=1 1 1
- link l_hand: geometry collision mesh filename=package://atlas_description/meshes_v3/l_hand.stl scale=1 1 1; visual mesh filename=package://atlas_description/meshes_v3/l_hand.DAE scale=1 1 1
- link l_larm: geometry collision mesh filename=package://atlas_description/meshes_v3/l_elbow_rx.stl scale=1 1 1; visual mesh filename=package://atlas_description/meshes_v3/l_elbow_rx.DAE scale=1 1 1
- link l_lglut: geometry collision mesh filename=package://atlas_description/meshes_v3/l_lglut.stl scale=1 1 1; visual mesh filename=package://atlas_description/meshes_v3/l_lglut.DAE scale=1 1 1
- link l_lleg: geometry collision mesh filename=package://atlas_description/meshes_v3/l_lleg.stl scale=1 1 1; visual mesh filename=package://atlas_description/meshes_v3/l_lleg.DAE scale=1 1 1
- link l_scap: geometry collision mesh filename=package://atlas_description/meshes_v3/l_sh_rx.stl scale=1 1 1; visual mesh filename=package://atlas_description/meshes_v3/l_sh_rx.DAE scale=1 1 1
- link l_talus: geometry collision mesh filename=package://atlas_description/meshes_v3/l_talus.stl scale=1 1 1; visual mesh filename=package://atlas_description/meshes_v3/l_talus.DAE scale=1 1 1
- link l_uarm: geometry collision mesh filename=package://atlas_description/meshes_v3/l_elbow_ry.stl scale=1 1 1; visual mesh filename=package://atlas_description/meshes_v3/l_elbow_ry.DAE scale=1 1 1
- link l_uglut: geometry collision mesh filename=package://atlas_description/meshes_v3/l_uglut.stl scale=1 1 1; visual mesh filename=package://atlas_description/meshes_v3/l_uglut.DAE scale=1 1 1
- link l_uleg: geometry collision mesh filename=package://atlas_description/meshes_v3/l_uleg.stl scale=1 1 1; visual mesh filename=package://atlas_description/meshes_v3/l_uleg.DAE scale=1 1 1
- link ltorso: geometry collision mesh filename=package://atlas_description/meshes_v3/ltorso.stl scale=1 1 1; visual mesh filename=package://atlas_description/meshes_v3/ltorso.DAE scale=1 1 1
- link mtorso: geometry collision mesh filename=package://atlas_description/meshes_v3/mtorso.stl scale=1 1 1; visual mesh filename=package://atlas_description/meshes_v3/mtorso.DAE scale=1 1 1
- link pelvis: geometry collision mesh filename=package://atlas_description/meshes_v3/pelvis.stl scale=1 1 1; visual mesh filename=package://atlas_description/meshes_v3/pelvis.DAE scale=1 1 1
- link r_clav: geometry collision mesh filename=package://atlas_description/meshes_v3/r_clav.stl scale=1 1 1; visual mesh filename=package://atlas_description/meshes_v3/r_clav.DAE scale=1 1 1
- link r_farm: geometry collision mesh filename=package://atlas_description/meshes_v3/r_farm.stl scale=1 1 1; visual mesh filename=package://atlas_description/meshes_v3/r_farm.DAE scale=1 1 1
- link r_foot: geometry collision mesh filename=package://atlas_description/meshes_v3/r_foot.stl scale=1 1 1; visual mesh filename=package://atlas_description/meshes_v3/r_foot.DAE scale=1 1 1
- link r_hand: geometry collision mesh filename=package://atlas_description/meshes_v3/r_hand.stl scale=1 1 1; visual mesh filename=package://atlas_description/meshes_v3/r_hand.DAE scale=1 1 1
- link r_larm: geometry collision mesh filename=package://atlas_description/meshes_v3/r_elbow_rx.stl scale=1 1 1; visual mesh filename=package://atlas_description/meshes_v3/r_elbow_rx.DAE scale=1 1 1
- link r_lglut: geometry collision mesh filename=package://atlas_description/meshes_v3/r_lglut.stl scale=1 1 1; visual mesh filename=package://atlas_description/meshes_v3/r_lglut.DAE scale=1 1 1
- link r_lleg: geometry collision mesh filename=package://atlas_description/meshes_v3/r_lleg.stl scale=1 1 1; visual mesh filename=package://atlas_description/meshes_v3/r_lleg.DAE scale=1 1 1
- link r_scap: geometry collision mesh filename=package://atlas_description/meshes_v3/r_sh_rx.stl scale=1 1 1; visual mesh filename=package://atlas_description/meshes_v3/r_sh_rx.DAE scale=1 1 1
- link r_talus: geometry collision mesh filename=package://atlas_description/meshes_v3/r_talus.stl scale=1 1 1; visual mesh filename=package://atlas_description/meshes_v3/r_talus.DAE scale=1 1 1
- link r_uarm: geometry collision mesh filename=package://atlas_description/meshes_v3/r_elbow_ry.stl scale=1 1 1; visual mesh filename=package://atlas_description/meshes_v3/r_elbow_ry.DAE scale=1 1 1
- link r_uglut: geometry collision mesh filename=package://atlas_description/meshes_v3/r_uglut.stl scale=1 1 1; visual mesh filename=package://atlas_description/meshes_v3/r_uglut.DAE scale=1 1 1
- link r_uleg: geometry collision mesh filename=package://atlas_description/meshes_v3/r_uleg.stl scale=1 1 1; visual mesh filename=package://atlas_description/meshes_v3/r_uleg.DAE scale=1 1 1
- link utorso: geometry collision mesh filename=package://atlas_description/meshes_v3/utorso.stl scale=1 1 1; collision mesh filename=package://atlas_description/meshes_v3/utorso_pack.stl scale=1 1 1
Joints:
- added joint rear_situational_awareness_camera_joint: type fixed, parent utorso, child rear_situational_awareness_camera_link, origin xyz=-0.0026 0.0264 0.6649 rpy=0 0 3.14159
- added joint rear_situational_awareness_camera_optical_frame_joint: type fixed, parent rear_situational_awareness_camera_link, child rear_situational_awareness_camera_optical_frame, origin xyz=0 0 0 rpy=-1.5708 0.0 -1.5708
