Commit message: merging from default

File: atlas_description/urdf/atlas_v3.urdf (robot description, URDF)
Before this commit: robot drc_skeleton, 32 links, 32 joints
Links:
- added link rear_situational_awareness_camera_link, mass 0.1; visual box size=0.01 0.01 0.01
- added link rear_situational_awareness_camera_optical_frame
- link l_clav: geometry collision mesh filename=package://atlas_description/meshes_v3/l_clav.stl scale=1 1 1; visual mesh filename=package://atlas_description/meshes_v3/l_clav.dae scale=1 1 1
- link l_farm: geometry collision mesh filename=package://atlas_description/meshes_v3/l_farm.stl scale=1 1 1; visual mesh filename=package://atlas_description/meshes_v3/l_farm.dae scale=1 1 1
- link l_foot: geometry collision mesh filename=package://atlas_description/meshes_v3/l_foot.stl scale=1 1 1; visual mesh filename=package://atlas_description/meshes_v3/l_foot.dae scale=1 1 1
- link l_hand: geometry collision mesh filename=package://atlas_description/meshes_v3/l_hand.stl scale=1 1 1; visual mesh filename=package://atlas_description/meshes_v3/l_hand.dae scale=1 1 1
- link l_larm: geometry collision mesh filename=package://atlas_description/meshes_v3/l_larm.stl scale=1 1 1; visual mesh filename=package://atlas_description/meshes_v3/l_larm.dae scale=1 1 1
- link l_lglut: geometry collision mesh filename=package://atlas_description/meshes_v3/l_lglut.stl scale=1 1 1; visual mesh filename=package://atlas_description/meshes_v3/l_lglut.dae scale=1 1 1
- link l_lleg: geometry collision mesh filename=package://atlas_description/meshes_v3/l_lleg.stl scale=1 1 1; visual mesh filename=package://atlas_description/meshes_v3/l_lleg.dae scale=1 1 1
- link l_scap: geometry collision mesh filename=package://atlas_description/meshes_v3/l_scap.stl scale=1 1 1; visual mesh filename=package://atlas_description/meshes_v3/l_scap.dae scale=1 1 1
- link l_talus: geometry collision mesh filename=package://atlas_description/meshes_v3/l_talus.stl scale=1 1 1; visual mesh filename=package://atlas_description/meshes_v3/l_talus.dae scale=1 1 1
- link l_uarm: geometry collision mesh filename=package://atlas_description/meshes_v3/l_uarm.stl scale=1 1 1; visual mesh filename=package://atlas_description/meshes_v3/l_uarm.dae scale=1 1 1
- link l_uglut: geometry collision mesh filename=package://atlas_description/meshes_v3/l_uglut.stl scale=1 1 1; visual mesh filename=package://atlas_description/meshes_v3/l_uglut.dae scale=1 1 1
- link l_uleg: geometry collision mesh filename=package://atlas_description/meshes_v3/l_uleg.stl scale=1 1 1; visual mesh filename=package://atlas_description/meshes_v3/l_uleg.dae scale=1 1 1
- link ltorso: geometry collision mesh filename=package://atlas_description/meshes_v3/ltorso.stl scale=1 1 1; visual mesh filename=package://atlas_description/meshes_v3/ltorso.dae scale=1 1 1
- link mtorso: geometry collision mesh filename=package://atlas_description/meshes_v3/mtorso.stl scale=1 1 1; visual mesh filename=package://atlas_description/meshes_v3/mtorso.dae scale=1 1 1
- link pelvis: geometry collision mesh filename=package://atlas_description/meshes_v3/pelvis.stl scale=1 1 1; visual mesh filename=package://atlas_description/meshes_v3/pelvis.dae scale=1 1 1
- link r_clav: geometry collision mesh filename=package://atlas_description/meshes_v3/r_clav.stl scale=1 1 1; visual mesh filename=package://atlas_description/meshes_v3/r_clav.dae scale=1 1 1
- link r_farm: geometry collision mesh filename=package://atlas_description/meshes_v3/r_farm.stl scale=1 1 1; visual mesh filename=package://atlas_description/meshes_v3/r_farm.dae scale=1 1 1
- link r_foot: geometry collision mesh filename=package://atlas_description/meshes_v3/r_foot.stl scale=1 1 1; visual mesh filename=package://atlas_description/meshes_v3/r_foot.dae scale=1 1 1
- link r_hand: geometry collision mesh filename=package://atlas_description/meshes_v3/r_hand.stl scale=1 1 1; visual mesh filename=package://atlas_description/meshes_v3/r_hand.dae scale=1 1 1
- link r_larm: geometry collision mesh filename=package://atlas_description/meshes_v3/r_larm.stl scale=1 1 1; visual mesh filename=package://atlas_description/meshes_v3/r_larm.dae scale=1 1 1
- link r_lglut: geometry collision mesh filename=package://atlas_description/meshes_v3/r_lglut.stl scale=1 1 1; visual mesh filename=package://atlas_description/meshes_v3/r_lglut.dae scale=1 1 1
- link r_lleg: geometry collision mesh filename=package://atlas_description/meshes_v3/r_lleg.stl scale=1 1 1; visual mesh filename=package://atlas_description/meshes_v3/r_lleg.dae scale=1 1 1
- link r_scap: geometry collision mesh filename=package://atlas_description/meshes_v3/r_scap.stl scale=1 1 1; visual mesh filename=package://atlas_description/meshes_v3/r_scap.dae scale=1 1 1
- link r_talus: geometry collision mesh filename=package://atlas_description/meshes_v3/r_talus.stl scale=1 1 1; visual mesh filename=package://atlas_description/meshes_v3/r_talus.dae scale=1 1 1
- link r_uarm: geometry collision mesh filename=package://atlas_description/meshes_v3/r_uarm.stl scale=1 1 1; visual mesh filename=package://atlas_description/meshes_v3/r_uarm.dae scale=1 1 1
- link r_uglut: geometry collision mesh filename=package://atlas_description/meshes_v3/r_uglut.stl scale=1 1 1; visual mesh filename=package://atlas_description/meshes_v3/r_uglut.dae scale=1 1 1
- link r_uleg: geometry collision mesh filename=package://atlas_description/meshes_v3/r_uleg.stl scale=1 1 1; visual mesh filename=package://atlas_description/meshes_v3/r_uleg.dae scale=1 1 1
- link utorso: geometry collision mesh filename=package://atlas_description/meshes_v3/utorso.stl scale=1 1 1; collision mesh filename=package://atlas_description/meshes_v3/utorso_pack.stl scale=1 1 1
Joints:
- added joint rear_situational_awareness_camera_joint: type fixed, parent utorso, child rear_situational_awareness_camera_link, origin xyz=-0.0026 0.0264 0.6649 rpy=0 0 3.14159
- added joint rear_situational_awareness_camera_optical_frame_joint: type fixed, parent rear_situational_awareness_camera_link, child rear_situational_awareness_camera_optical_frame, origin xyz=0 0 0 rpy=-1.5708 0.0 -1.5708

File: irobot_hand_description/urdf/irobot_hand.urdf.xacro (robot description, xacro)
@@ -331,5 +331,5 @@
       <inertial>
         <!-- needs update -->
-        <mass value="1.0"/>
+        <mass value="1.305"/>
         <origin xyz="0 0 0"/>
         <inertia ixx="0.00125" ixy="0.0" ixz="0.0" iyy="0.00125" iyz="0.0" izz="0.0002"/>
@@ -578,5 +578,5 @@
     <origin xyz="0 0 0.0135" rpy="${pi/2} 0 -${pi}" />
     <axis xyz="-1 0 0"/>
-    <limit effort="1000.0" lower="0.0" upper="${pi/2}" velocity="0.5"/>
+    <limit effort="1000.0" lower="0.0" upper="${7*pi/8}" velocity="0.5"/>
   </joint>
   <gazebo reference="${side}_finger[1]/joint_base_rotation">
@@ -620,5 +620,5 @@
     <origin xyz="0 0 0.0135" rpy="${pi/2} 0 -${pi}" />
     <axis xyz="-1 0 0"/>
-    <limit effort="1000.0" lower="0.0" upper="${pi/2}" velocity="0.5"/>
+    <limit effort="1000.0" lower="0.0" upper="${7*pi/8}" velocity="0.5"/>
   </joint>
   <gazebo reference="${side}_finger[2]/joint_base">
@@ -630,5 +630,5 @@
     <origin xyz="0 -0.038 0.082755" rpy="${pi/2} 0 0" />
     <axis xyz="-1 0 0"/>
-    <limit effort="1000.0" lower="0.0" upper="${pi/2}" velocity="0.5"/>
+    <limit effort="1000.0" lower="0.0" upper="${7*pi/8}" velocity="0.5"/>
   </joint>
 </xacro:macro>
