Commit message: fix startup sequence

File: atlas_description/urdf/atlas_simple_shapes.urdf (robot description, URDF)
Before this commit: robot drc_skeleton, 28 links, 28 joints
Links:
- link l_clav: geometry collision box size=0.13 0.15 0.05; collision cylinder length=0.1525 radius=0.045
- link l_farm: geometry collision box size=0.135 0.1 0.045; collision cylinder length=0.125 radius=0.045
- link l_foot: geometry collision box size=0.26 0.124887 0.05; visual mesh filename=package://atlas_description/meshes/l_foot.dae scale=1 1 1
- link l_hand: geometry collision box size=0.13 0.09 0.07; collision cylinder length=0.05 radius=0.03
- link l_larm: geometry collision box size=0.135 0.15 0.06; collision cylinder length=0.125 radius=0.045
- link l_lglut: geometry collision cylinder length=0.060306 radius=0.02009687; collision cylinder length=0.12 radius=0.02
- link l_lleg: geometry collision cylinder length=0.40 radius=0.07; visual mesh filename=package://atlas_description/meshes/l_lleg.dae scale=1.0 1.0 1.0
- link l_scap: geometry collision box size=0.15 0.15 0.06; collision cylinder length=0.125 radius=0.045
- link l_talus: geometry collision cylinder length=0.010059 radius=0.010348; collision cylinder length=0.029542 radius=0.010181
- link l_uarm: geometry collision box size=0.04 0.07 0.13; collision cylinder length=0.125 radius=0.045
- link l_uglut: geometry collision cylinder length=0.078396 radius=0.019096; collision cylinder length=0.080842 radius=0.019841
- link l_uleg: geometry collision cylinder length=0.10 radius=0.1; collision cylinder length=0.15 radius=0.07
- link ltorso: geometry visual mesh filename=package://atlas_description/meshes/ltorso.dae scale=1 1 1
- link mtorso: geometry collision cylinder length=0.02 radius=0.015; collision cylinder length=0.02 radius=0.015
- link pelvis: geometry collision box size=0.1 0.15 0.2; collision cylinder length=0.05 radius=0.16
- link r_clav: geometry collision box size=0.13 0.15 0.05; collision cylinder length=0.1525 radius=0.045
- link r_farm: geometry collision box size=0.135 0.1 0.045; collision cylinder length=0.125 radius=0.045
- link r_foot: geometry collision box size=0.26 0.124887 0.05; visual mesh filename=package://atlas_description/meshes/r_foot.dae scale=1 1 1
- link r_hand: geometry collision box size=0.13 0.09 0.07; collision cylinder length=0.05 radius=0.03
- link r_larm: geometry collision box size=0.135 0.15 0.06; collision cylinder length=0.125 radius=0.045
- link r_lglut: geometry collision cylinder length=0.060306 radius=0.02009687; collision cylinder length=0.12 radius=0.02
- link r_lleg: geometry collision cylinder length=0.40 radius=0.07; visual mesh filename=package://atlas_description/meshes/r_lleg.dae scale=1.0 1.0 1.0
- link r_scap: geometry collision box size=0.15 0.15 0.06; collision cylinder length=0.125 radius=0.045
- link r_talus: geometry collision cylinder length=0.010059 radius=0.010348; collision cylinder length=0.029542 radius=0.010181
- link r_uarm: geometry collision box size=0.04 0.07 0.13; collision cylinder length=0.125 radius=0.045
- link r_uglut: geometry collision cylinder length=0.078396 radius=0.019096; collision cylinder length=0.080842 radius=0.019841
- link r_uleg: geometry collision cylinder length=0.10 radius=0.1; collision cylinder length=0.15 radius=0.07
- link utorso: geometry collision box size=0.3188 0.24 0.3162; collision cylinder length=0.22375 radius=0.0363

Commit message: syncing and reverting inertia tweaks for atlas_simple_shapes.urdf

File: atlas_description/urdf/atlas_simple_shapes.urdf (robot description, URDF)
Before this commit: robot drc_skeleton, 28 links, 28 joints
Links:
- link l_foot: mass 0.867 -> 1.634
- link l_lglut: mass 0.803 -> 0.69
- link l_talus: mass 0.867 -> 0.1
- link l_uglut: mass 1.51622 -> 0.5166
- link l_uleg: mass 7.227 -> 7.34
- link ltorso: mass 1.62729 -> 1.92
- link mtorso: mass 3.8068 -> 0.55
- link pelvis: mass 12.54638 -> 14.2529
- link r_foot: mass 0.867 -> 1.634
- link r_lglut: mass 0.803 -> 0.69
- link r_talus: mass 0.867 -> 0.1
- link r_uglut: mass 1.51622 -> 0.5166
- link r_uleg: mass 7.227 -> 7.34
- link utorso: mass 15.2272 -> 18.484

Commit message: testing dart softbody codes

File: atlas_description/urdf/atlas_simple_shapes.urdf (robot description, URDF)
Before this commit: robot drc_skeleton, 28 links, 28 joints
Links:
- link l_foot: geometry collision box ; collision box size=0.26 0.124887 0.05
- link r_foot: geometry collision box ; collision box size=0.26 0.124887 0.05

Commit message: add soft feet <soft_contact> tags.

File: atlas_description/urdf/atlas_simple_shapes.urdf (robot description, URDF)
Before this commit: robot drc_skeleton, 28 links, 28 joints
Links:
- link l_foot: geometry collision box size=0.26 0.124887 0.05; collision box size=0.4 0.175 0.125
- link r_foot: geometry collision box size=0.26 0.124887 0.05; collision box size=0.4 0.175 0.125
