Commit message: [atlas_v3_simple_shapes.urdf] Replacing arm meshes by simple geometries.

File: atlas_description/urdf/atlas_v3_simple_shapes.urdf (robot description, URDF)
Before this commit: robot drc_skeleton, 34 links, 34 joints
Links:
- link l_clav: geometry collision box size=0.045 0.03 0.04; collision box size=0.13 0.15 0.05
- link l_farm: geometry collision box size=0.135 0.1 0.045; collision cylinder length=0.125 radius=0.045
- link l_hand: geometry collision box size=0.13 0.09 0.07; collision cylinder length=0.05 radius=0.03
- link l_larm: geometry collision box size=0.135 0.15 0.06; collision cylinder length=0.125 radius=0.045
- link l_scap: geometry collision box size=0.15 0.15 0.06; collision cylinder length=0.125 radius=0.045
- link l_uarm: geometry collision box size=0.04 0.07 0.13; collision cylinder length=0.125 radius=0.045
- link r_clav: geometry collision box size=0.045 0.03 0.04; collision box size=0.13 0.15 0.05
- link r_farm: geometry collision box size=0.135 0.1 0.045; collision cylinder length=0.125 radius=0.045
- link r_hand: geometry collision box size=0.13 0.09 0.07; collision cylinder length=0.05 radius=0.03
- link r_larm: geometry collision box size=0.135 0.15 0.06; collision cylinder length=0.125 radius=0.045
- link r_scap: geometry collision box size=0.15 0.15 0.06; collision cylinder length=0.125 radius=0.045
- link r_uarm: geometry collision box size=0.04 0.07 0.13; collision cylinder length=0.125 radius=0.045

Commit message: updating leg simple shape collision geometries

File: atlas_description/urdf/atlas_v3_simple_shapes.urdf (robot description, URDF)
Before this commit: robot drc_skeleton, 34 links, 34 joints
Links:
- link l_foot: geometry collision box size=0.26 0.124887 0.05; visual mesh filename=package://atlas_description/meshes_v3/l_foot.dae scale=1 1 1
- link l_lglut: geometry collision cylinder length=0.060306 radius=0.02009687; collision cylinder length=0.12 radius=0.02
- link l_lleg: geometry collision cylinder length=0.40 radius=0.07; visual mesh filename=package://atlas_description/meshes_v3/l_lleg.dae scale=1 1 1
- link l_talus: geometry collision cylinder length=0.010059 radius=0.010348; collision cylinder length=0.029542 radius=0.010181
- link l_uglut: geometry collision cylinder length=0.078396 radius=0.019096; collision cylinder length=0.080842 radius=0.019841
- link l_uleg: geometry collision cylinder length=0.10 radius=0.1; collision cylinder length=0.15 radius=0.07
- link r_foot: geometry collision box size=0.26 0.124887 0.05; visual mesh filename=package://atlas_description/meshes_v3/r_foot.dae scale=1 1 1
- link r_lglut: geometry collision cylinder length=0.060306 radius=0.02009687; collision cylinder length=0.12 radius=0.02
- link r_lleg: geometry collision cylinder length=0.40 radius=0.07; visual mesh filename=package://atlas_description/meshes_v3/r_lleg.dae scale=1 1 1
- link r_talus: geometry collision cylinder length=0.010059 radius=0.010348; collision cylinder length=0.029542 radius=0.010181
- link r_uglut: geometry collision cylinder length=0.078396 radius=0.019096; collision cylinder length=0.080842 radius=0.019841
- link r_uleg: geometry collision cylinder length=0.10 radius=0.1; collision cylinder length=0.15 radius=0.07

Commit message: updating leg simple shape collision geometries

File: atlas_description/urdf/atlas_v3_simple_shapes.urdf (robot description, URDF)
Before this commit: robot drc_skeleton, 34 links, 34 joints
Links:
- link l_lglut: geometry collision cylinder length=0.060306 radius=0.02009687; collision cylinder length=0.144 radius=0.02
- link l_uleg: geometry collision box size=0.07 0.016 0.15; collision box size=0.07 0.038 0.15
- link r_lglut: geometry collision cylinder length=0.060306 radius=0.02009687; collision cylinder length=0.142 radius=0.02
- link r_uleg: geometry collision box size=0.07 0.016 0.15; collision box size=0.07 0.038 0.15

Commit message: torso collision shapes

File: atlas_description/urdf/atlas_v3_simple_shapes.urdf (robot description, URDF)
Before this commit: robot drc_skeleton, 34 links, 34 joints
Links:
- link ltorso: geometry visual mesh filename=package://atlas_description/meshes_v3/ltorso.dae scale=1 1 1
- link mtorso: geometry collision cylinder length=0.06 radius=0.017; collision cylinder length=0.08 radius=0.02
- link pelvis: geometry collision box size=0.1 0.15 0.2; collision cylinder length=0.05 radius=0.16
- link utorso: geometry collision box size=0.266306 0.223 0.091; collision box size=0.266306 0.381719 0.18
