Commit message: shy is now shz in v4

File: atlas_description/urdf/atlas_v4.urdf (robot description, URDF)
Before this commit: robot drc_skeleton, 34 links, 34 joints
Joints:
- removed joint l_arm_shy
- removed joint r_arm_shy
- added joint l_arm_shz: type revolute, parent utorso, child l_clav, origin xyz=0.1406 0.2036 0.4776 rpy=0 -0 0, axis 0 0 1, limit lower=-1.5708 upper=0.785398 effort=198 velocity=12
- added joint r_arm_shz: type revolute, parent utorso, child r_clav, origin xyz=0.1406 -0.2036 0.4776 rpy=0 -0 0, axis 0 0 1, limit lower=-0.785398 upper=1.5708 effort=198 velocity=12

Commit message: update atlas v4 and atlas v4 simple shape joint torques per BDI instruction.

File: atlas_description/urdf/atlas_v4.urdf (robot description, URDF)
Before this commit: robot drc_skeleton, 34 links, 34 joints
Joints:
- joint back_bkx: limit lower=-0.523599 upper=0.523599 effort=163 velocity=12 -> lower=-0.523599 upper=0.523599 effort=300 velocity=12
- joint back_bky: limit lower=-0.219388 upper=0.538783 effort=245 velocity=9 -> lower=-0.219388 upper=0.538783 effort=445 velocity=9
- joint back_bkz: limit lower=-0.663225 upper=0.663225 effort=62 velocity=12 -> lower=-0.663225 upper=0.663225 effort=106 velocity=12
- joint l_arm_elx: limit lower=0 upper=2.35619 effort=159 velocity=12 -> lower=0 upper=2.35619 effort=112 velocity=12
- joint l_arm_ely: limit lower=0 upper=3.14159 effort=106 velocity=12 -> lower=0 upper=3.14159 effort=63 velocity=12
- joint l_arm_shx: limit lower=-1.5708 upper=1.5708 effort=159 velocity=12 -> lower=-1.5708 upper=1.5708 effort=99 velocity=12
- joint l_arm_shz: limit lower=-1.5708 upper=0.785398 effort=198 velocity=12 -> lower=-1.5708 upper=0.785398 effort=87 velocity=12
- joint l_arm_wrx: limit lower=-1.1781 upper=1.1781 effort=56 velocity=12 -> lower=-1.1781 upper=1.1781 effort=25 velocity=12
- joint l_arm_wry: limit lower=0 upper=3.14159 effort=106 velocity=12 -> lower=0 upper=3.14159 effort=25 velocity=12
- joint l_leg_akx: limit lower=-0.8 upper=0.8 effort=45 velocity=12 -> lower=-0.8 upper=0.8 effort=360 velocity=12
- joint l_leg_aky: limit lower=-1 upper=0.7 effort=350 velocity=12 -> lower=-1 upper=0.7 effort=740 velocity=12
- joint l_leg_hpx: limit lower=-0.523599 upper=0.523599 effort=257 velocity=12 -> lower=-0.523599 upper=0.523599 effort=530 velocity=12
- joint l_leg_hpy: limit lower=-1.61234 upper=0.65764 effort=400 velocity=12 -> lower=-1.61234 upper=0.65764 effort=840 velocity=12
- joint l_leg_hpz: limit lower=-0.174358 upper=0.786794 effort=150 velocity=12 -> lower=-0.174358 upper=0.786794 effort=275 velocity=12
- joint l_leg_kny: limit lower=0 upper=2.35637 effort=246 velocity=12 -> lower=0 upper=2.35637 effort=890 velocity=12
- joint r_arm_elx: limit lower=-2.35619 upper=0 effort=159 velocity=12 -> lower=-2.35619 upper=0 effort=112 velocity=12
- joint r_arm_ely: limit lower=0 upper=3.14159 effort=106 velocity=12 -> lower=0 upper=3.14159 effort=63 velocity=12
- joint r_arm_shx: limit lower=-1.5708 upper=1.5708 effort=159 velocity=12 -> lower=-1.5708 upper=1.5708 effort=99 velocity=12
- joint r_arm_shz: limit lower=-0.785398 upper=1.5708 effort=198 velocity=12 -> lower=-0.785398 upper=1.5708 effort=87 velocity=12
- joint r_arm_wrx: limit lower=-1.1781 upper=1.1781 effort=56 velocity=12 -> lower=-1.1781 upper=1.1781 effort=25 velocity=12
- joint r_arm_wry: limit lower=0 upper=3.14159 effort=106 velocity=12 -> lower=0 upper=3.14159 effort=25 velocity=12
- joint r_leg_akx: limit lower=-0.8 upper=0.8 effort=45 velocity=12 -> lower=-0.8 upper=0.8 effort=360 velocity=12
- joint r_leg_aky: limit lower=-1 upper=0.7 effort=350 velocity=12 -> lower=-1 upper=0.7 effort=740 velocity=12
- joint r_leg_hpx: limit lower=-0.523599 upper=0.523599 effort=257 velocity=12 -> lower=-0.523599 upper=0.523599 effort=530 velocity=12
- joint r_leg_hpy: limit lower=-1.61234 upper=0.65764 effort=400 velocity=12 -> lower=-1.61234 upper=0.65764 effort=840 velocity=12
- joint r_leg_hpz: limit lower=-0.786794 upper=0.174358 effort=150 velocity=12 -> lower=-0.786794 upper=0.174358 effort=275 velocity=12
- joint r_leg_kny: limit lower=0 upper=2.35637 effort=246 velocity=12 -> lower=0 upper=2.35637 effort=890 velocity=12

Commit message: update atlas_v4 to use meshes_v4

File: atlas_description/urdf/atlas_v4.urdf (robot description, URDF)
Before this commit: robot drc_skeleton, 34 links, 34 joints
Links:
- link l_clav: geometry collision mesh filename=package://atlas_description/meshes_v4/l_clav.dae scale=1 1 1; visual mesh filename=package://atlas_description/meshes_v4/l_clav.dae scale=1 1 1
- link l_farm: geometry collision mesh filename=package://atlas_description/meshes_v4/l_farm.dae scale=1 1 1; visual mesh filename=package://atlas_description/meshes_v4/l_farm.dae scale=1 1 1
- link l_foot: geometry collision mesh filename=package://atlas_description/meshes_v4/l_foot.dae scale=1 1 1; visual mesh filename=package://atlas_description/meshes_v4/l_foot.dae scale=1 1 1
- link l_hand: geometry collision mesh filename=package://atlas_description/meshes_v4/l_hand.dae scale=1 1 1; visual mesh filename=package://atlas_description/meshes_v4/l_hand.dae scale=1 1 1
- link l_larm: geometry collision mesh filename=package://atlas_description/meshes_v4/l_larm.dae scale=1 1 1; visual mesh filename=package://atlas_description/meshes_v4/l_larm.dae scale=1 1 1
- link l_lglut: geometry collision mesh filename=package://atlas_description/meshes_v4/l_lglut.dae scale=1 1 1; visual mesh filename=package://atlas_description/meshes_v4/l_lglut.dae scale=1 1 1
- link l_lleg: geometry collision mesh filename=package://atlas_description/meshes_v4/l_lleg.dae scale=1 1 1; visual mesh filename=package://atlas_description/meshes_v4/l_lleg.dae scale=1 1 1
- link l_scap: geometry collision mesh filename=package://atlas_description/meshes_v4/l_scap.dae scale=1 1 1; visual mesh filename=package://atlas_description/meshes_v4/l_scap.dae scale=1 1 1
- link l_talus: geometry collision mesh filename=package://atlas_description/meshes_v4/l_talus.dae scale=1 1 1; visual mesh filename=package://atlas_description/meshes_v4/l_talus.dae scale=1 1 1
- link l_uarm: geometry collision mesh filename=package://atlas_description/meshes_v4/l_uarm.dae scale=1 1 1; visual mesh filename=package://atlas_description/meshes_v4/l_uarm.dae scale=1 1 1
- link l_uglut: geometry collision mesh filename=package://atlas_description/meshes_v4/l_uglut.dae scale=1 1 1; visual mesh filename=package://atlas_description/meshes_v4/l_uglut.dae scale=1 1 1
- link l_uleg: geometry collision mesh filename=package://atlas_description/meshes_v4/l_uleg.dae scale=1 1 1; visual mesh filename=package://atlas_description/meshes_v4/l_uleg.dae scale=1 1 1
- link ltorso: geometry collision mesh filename=package://atlas_description/meshes_v4/ltorso.dae scale=1 1 1; visual mesh filename=package://atlas_description/meshes_v4/ltorso.dae scale=1 1 1
- link mtorso: geometry collision mesh filename=package://atlas_description/meshes_v4/mtorso.dae scale=1 1 1; visual mesh filename=package://atlas_description/meshes_v4/mtorso.dae scale=1 1 1
- link pelvis: geometry collision mesh filename=package://atlas_description/meshes_v4/pelvis.dae scale=1 1 1; visual mesh filename=package://atlas_description/meshes_v4/pelvis.dae scale=1 1 1
- link r_clav: geometry collision mesh filename=package://atlas_description/meshes_v4/r_clav.dae scale=1 1 1; visual mesh filename=package://atlas_description/meshes_v4/r_clav.dae scale=1 1 1
- link r_farm: geometry collision mesh filename=package://atlas_description/meshes_v4/r_farm.dae scale=1 1 1; visual mesh filename=package://atlas_description/meshes_v4/r_farm.dae scale=1 1 1
- link r_foot: geometry collision mesh filename=package://atlas_description/meshes_v4/r_foot.dae scale=1 1 1; visual mesh filename=package://atlas_description/meshes_v4/r_foot.dae scale=1 1 1
- link r_hand: geometry collision mesh filename=package://atlas_description/meshes_v4/r_hand.dae scale=1 1 1; visual mesh filename=package://atlas_description/meshes_v4/r_hand.dae scale=1 1 1
- link r_lglut: geometry collision mesh filename=package://atlas_description/meshes_v4/r_lglut.dae scale=1 1 1; visual mesh filename=package://atlas_description/meshes_v4/r_lglut.dae scale=1 1 1
- link r_lleg: geometry collision mesh filename=package://atlas_description/meshes_v4/r_lleg.dae scale=1 1 1; visual mesh filename=package://atlas_description/meshes_v4/r_lleg.dae scale=1 1 1
- link r_scap: geometry collision mesh filename=package://atlas_description/meshes_v4/r_scap.dae scale=1 1 1; visual mesh filename=package://atlas_description/meshes_v4/r_scap.dae scale=1 1 1
- link r_talus: geometry collision mesh filename=package://atlas_description/meshes_v4/r_talus.dae scale=1 1 1; visual mesh filename=package://atlas_description/meshes_v4/r_talus.dae scale=1 1 1
- link r_uarm: geometry collision mesh filename=package://atlas_description/meshes_v4/r_uarm.dae scale=1 1 1; visual mesh filename=package://atlas_description/meshes_v4/r_uarm.dae scale=1 1 1
- link r_uglut: geometry collision mesh filename=package://atlas_description/meshes_v4/r_uglut.dae scale=1 1 1; visual mesh filename=package://atlas_description/meshes_v4/r_uglut.dae scale=1 1 1
- link r_uleg: geometry collision mesh filename=package://atlas_description/meshes_v4/r_uleg.dae scale=1 1 1; visual mesh filename=package://atlas_description/meshes_v4/r_uleg.dae scale=1 1 1
- link utorso: geometry collision mesh filename=package://atlas_description/meshes_v4/utorso.dae scale=1 1 1; visual mesh filename=package://atlas_description/meshes_v4/utorso.dae scale=1 1 1

File: atlas_description/urdf/atlas_v4_simple_shapes.urdf (robot description, URDF)
Before this commit: robot drc_skeleton, 34 links, 34 joints
Joints:
- joint back_bkx: limit lower=-0.523599 upper=0.523599 effort=163 velocity=12 -> lower=-0.523599 upper=0.523599 effort=300 velocity=12
- joint back_bky: limit lower=-0.219388 upper=0.538783 effort=245 velocity=9 -> lower=-0.219388 upper=0.538783 effort=445 velocity=9
- joint back_bkz: limit lower=-0.663225 upper=0.663225 effort=62 velocity=12 -> lower=-0.663225 upper=0.663225 effort=106 velocity=12
- joint l_arm_elx: limit lower=0 upper=2.35619 effort=159 velocity=12 -> lower=0 upper=2.35619 effort=112 velocity=12
- joint l_arm_ely: limit lower=0 upper=3.14159 effort=106 velocity=12 -> lower=0 upper=3.14159 effort=63 velocity=12
- joint l_arm_shx: limit lower=-1.5708 upper=1.5708 effort=159 velocity=12 -> lower=-1.5708 upper=1.5708 effort=99 velocity=12
- joint l_arm_shz: limit lower=-1.5708 upper=0.785398 effort=198 velocity=12 -> lower=-1.5708 upper=0.785398 effort=87 velocity=12
- joint l_arm_wrx: limit lower=-1.1781 upper=1.1781 effort=56 velocity=12 -> lower=-1.1781 upper=1.1781 effort=25 velocity=12
- joint l_arm_wry: limit lower=0 upper=3.14159 effort=106 velocity=12 -> lower=0 upper=3.14159 effort=25 velocity=12
- joint l_leg_akx: limit lower=-0.8 upper=0.8 effort=45 velocity=12 -> lower=-0.8 upper=0.8 effort=360 velocity=12
- joint l_leg_aky: limit lower=-1 upper=0.7 effort=350 velocity=12 -> lower=-1 upper=0.7 effort=740 velocity=12
- joint l_leg_hpx: limit lower=-0.523599 upper=0.523599 effort=257 velocity=12 -> lower=-0.523599 upper=0.523599 effort=530 velocity=12
- joint l_leg_hpy: limit lower=-1.61234 upper=0.65764 effort=400 velocity=12 -> lower=-1.61234 upper=0.65764 effort=840 velocity=12
- joint l_leg_hpz: limit lower=-0.174358 upper=0.786794 effort=150 velocity=12 -> lower=-0.174358 upper=0.786794 effort=275 velocity=12
- joint l_leg_kny: limit lower=0 upper=2.35637 effort=246 velocity=12 -> lower=0 upper=2.35637 effort=890 velocity=12
- joint neck_ry: limit lower=-0.602139 upper=1.14319 effort=5 velocity=6.28 -> lower=-0.602139 upper=1.14319 effort=25 velocity=6.28; origin xyz=${0.2546+0.04} 0 ${0.6215-0.045} rpy=0 -0 0 -> xyz=0.2546 0 0.6215 rpy=0 -0 0
- joint r_arm_elx: limit lower=-2.35619 upper=0 effort=159 velocity=12 -> lower=-2.35619 upper=0 effort=112 velocity=12
- joint r_arm_ely: limit lower=0 upper=3.14159 effort=106 velocity=12 -> lower=0 upper=3.14159 effort=63 velocity=12
- joint r_arm_shx: limit lower=-1.5708 upper=1.5708 effort=159 velocity=12 -> lower=-1.5708 upper=1.5708 effort=99 velocity=12
- joint r_arm_shz: limit lower=-0.785398 upper=1.5708 effort=198 velocity=12 -> lower=-0.785398 upper=1.5708 effort=87 velocity=12
- joint r_arm_wrx: limit lower=-1.1781 upper=1.1781 effort=56 velocity=12 -> lower=-1.1781 upper=1.1781 effort=25 velocity=12
- joint r_arm_wry: limit lower=0 upper=3.14159 effort=106 velocity=12 -> lower=0 upper=3.14159 effort=25 velocity=12
- joint r_leg_akx: limit lower=-0.8 upper=0.8 effort=45 velocity=12 -> lower=-0.8 upper=0.8 effort=360 velocity=12
- joint r_leg_aky: limit lower=-1 upper=0.7 effort=350 velocity=12 -> lower=-1 upper=0.7 effort=740 velocity=12
- joint r_leg_hpx: limit lower=-0.523599 upper=0.523599 effort=257 velocity=12 -> lower=-0.523599 upper=0.523599 effort=530 velocity=12
- joint r_leg_hpy: limit lower=-1.61234 upper=0.65764 effort=400 velocity=12 -> lower=-1.61234 upper=0.65764 effort=840 velocity=12
- joint r_leg_hpz: limit lower=-0.786794 upper=0.174358 effort=150 velocity=12 -> lower=-0.786794 upper=0.174358 effort=275 velocity=12
- joint r_leg_kny: limit lower=0 upper=2.35637 effort=246 velocity=12 -> lower=0 upper=2.35637 effort=890 velocity=12

Commit message: new update from bdi, atlas_v4.urdf arm ely shift in z is reversed.

File: atlas_description/urdf/atlas_v4.urdf (robot description, URDF)
Before this commit: robot drc_skeleton, 34 links, 34 joints
Joints:
- joint l_arm_ely: origin xyz=0 0.187 0.016 rpy=0 -0 0 -> xyz=0 0.187 -0.016 rpy=0 -0 0
- joint r_arm_ely: origin xyz=0 -0.187 0.016 rpy=0 -0 0 -> xyz=0 -0.187 -0.016 rpy=0 -0 0
