Commit message: Modifying the mesh directories

File: atlas_description/urdf/atlas_v4.urdf (robot description, URDF)
Before this commit: robot drc_skeleton, 34 links, 34 joints
Links:
- removed link l_farm
- removed link r_farm
- added link l_lfarm, mass 2.65; collision cylinder length=0.05 radius=0.03
- added link l_ufarm, mass 2.12; collision cylinder length=0.1 radius=0.05; visual mesh filename=package://atlas_description/meshes_v3/l_farm.dae scale=1 1 1
- added link r_lfarm, mass 2.65; collision cylinder length=0.05 radius=0.03
- added link r_ufarm, mass 2.12; collision cylinder length=0.1 radius=0.05; visual mesh filename=package://atlas_description/meshes_v3/r_farm.dae scale=1 1 1
- link l_clav: geometry collision mesh filename=package://atlas_description/meshes_unplugged/l_clav.dae scale=1 1 1; visual mesh filename=package://atlas_description/meshes_unplugged/l_clav.dae scale=1 1 1
- link l_foot: geometry collision mesh filename=package://atlas_description/meshes_unplugged/l_foot.dae scale=1 1 1; visual mesh filename=package://atlas_description/meshes_unplugged/l_foot.dae scale=1 1 1
- link l_hand: mass 2.509 -> 0.53; geometry collision mesh filename=package://atlas_description/meshes_v3/l_hand.dae scale=1 1 1; visual mesh filename=package://atlas_description/meshes_v3/l_hand.dae scale=1 1 1
- link l_larm: geometry collision mesh filename=package://atlas_description/meshes_unplugged/l_larm.dae scale=1 1 1; visual mesh filename=package://atlas_description/meshes_unplugged/l_larm.dae
- link l_lglut: geometry collision mesh filename=package://atlas_description/meshes_unplugged/l_lglut.dae scale=1 1 1; visual mesh filename=package://atlas_description/meshes_unplugged/l_lglut.dae scale=1 1 1
- link l_lleg: geometry collision mesh filename=package://atlas_description/meshes_unplugged/l_lleg.dae scale=1 1 1; visual mesh filename=package://atlas_description/meshes_unplugged/l_lleg.dae scale=1 1 1
- link l_scap: geometry collision mesh filename=package://atlas_description/meshes_unplugged/l_scap.dae scale=1 1 1; visual mesh filename=package://atlas_description/meshes_unplugged/l_scap.dae scale=1 1 1
- link l_talus: geometry collision mesh filename=package://atlas_description/meshes_unplugged/l_talus.dae scale=1 1 1; visual mesh filename=package://atlas_description/meshes_unplugged/l_talus.dae scale=1 1 1
- link l_uarm: geometry collision mesh filename=package://atlas_description/meshes_unplugged/l_uarm.dae scale=1 1 1; visual mesh filename=package://atlas_description/meshes_unplugged/l_uarm.dae scale=1 1 1
- link l_uglut: geometry collision mesh filename=package://atlas_description/meshes_unplugged/l_uglut.dae scale=1 1 1; visual mesh filename=package://atlas_description/meshes_unplugged/l_uglut.dae scale=1 1 1
- link l_uleg: geometry collision mesh filename=package://atlas_description/meshes_unplugged/l_uleg.dae scale=1 1 1; visual mesh filename=package://atlas_description/meshes_unplugged/l_uleg.dae scale=1 1 1
- link ltorso: geometry collision mesh filename=package://atlas_description/meshes_unplugged/ltorso.dae scale=1 1 1; visual mesh filename=package://atlas_description/meshes_unplugged/ltorso.dae scale=1 1 1
- link mtorso: geometry collision mesh filename=package://atlas_description/meshes_unplugged/mtorso.dae scale=1 1 1; visual mesh filename=package://atlas_description/meshes_unplugged/mtorso.dae scale=1 1 1
- link pelvis: geometry collision mesh filename=package://atlas_description/meshes_unplugged/pelvis.dae scale=1 1 1; visual mesh filename=package://atlas_description/meshes_unplugged/pelvis.dae scale=1 1 1
- link r_clav: geometry collision mesh filename=package://atlas_description/meshes_unplugged/r_clav.dae scale=1 1 1; visual mesh filename=package://atlas_description/meshes_unplugged/r_clav.dae scale=1 1 1
- link r_foot: geometry collision mesh filename=package://atlas_description/meshes_unplugged/r_foot.dae scale=1 1 1; visual mesh filename=package://atlas_description/meshes_unplugged/r_foot.dae scale=1 1 1
- link r_hand: mass 2.509 -> 0.53; geometry collision mesh filename=package://atlas_description/meshes_v3/r_hand.dae scale=1 1 1; visual mesh filename=package://atlas_description/meshes_v3/r_hand.dae scale=1 1 1
- link r_larm: geometry collision mesh filename=package://atlas_description/meshes_unplugged/r_larm.dae scale=1 1 1; visual mesh filename=package://atlas_description/meshes_unplugged/r_larm.dae
- link r_lglut: geometry collision mesh filename=package://atlas_description/meshes_unplugged/r_lglut.dae scale=1 1 1; visual mesh filename=package://atlas_description/meshes_unplugged/r_lglut.dae scale=1 1 1
- link r_lleg: geometry collision mesh filename=package://atlas_description/meshes_unplugged/r_lleg.dae scale=1 1 1; visual mesh filename=package://atlas_description/meshes_unplugged/r_lleg.dae scale=1 1 1
- link r_scap: geometry collision mesh filename=package://atlas_description/meshes_unplugged/r_scap.dae scale=1 1 1; visual mesh filename=package://atlas_description/meshes_unplugged/r_scap.dae scale=1 1 1
- link r_talus: geometry collision mesh filename=package://atlas_description/meshes_unplugged/r_talus.dae scale=1 1 1; visual mesh filename=package://atlas_description/meshes_unplugged/r_talus.dae scale=1 1 1
- link r_uarm: geometry collision mesh filename=package://atlas_description/meshes_unplugged/r_uarm.dae scale=1 1 1; visual mesh filename=package://atlas_description/meshes_unplugged/r_uarm.dae scale=1 1 1
- link r_uglut: geometry collision mesh filename=package://atlas_description/meshes_unplugged/r_uglut.dae scale=1 1 1; visual mesh filename=package://atlas_description/meshes_unplugged/r_uglut.dae scale=1 1 1
- link r_uleg: geometry collision mesh filename=package://atlas_description/meshes_unplugged/r_uleg.dae scale=1 1 1; visual mesh filename=package://atlas_description/meshes_unplugged/r_uleg.dae scale=1 1 1
- link utorso: geometry collision mesh filename=package://atlas_description/meshes_unplugged/utorso.dae scale=1 1 1; visual mesh filename=package://atlas_description/meshes_unplugged/utorso.dae scale=1 1 1
Joints:
- added joint l_arm_wry2: type revolute, parent l_lfarm, child l_hand, origin xyz=0 0 0 rpy=0 -0 0, axis 0 1 0, limit lower=-2.9671 upper=2.9671 effort=25 velocity=10
- added joint r_arm_wry2: type revolute, parent r_lfarm, child r_hand, origin xyz=0 0 0 rpy=0 -0 0, axis 0 1 0, limit lower=-2.9671 upper=2.9671 effort=25 velocity=10
- joint l_arm_ely: origin xyz=0 0.187 0.016 rpy=0 -0 0 -> xyz=0 0.187 -0.016 rpy=0 -0 0
- joint l_arm_shx: origin xyz=0 0.0981 -0.2511 rpy=0 -0 0 -> xyz=0 0.11 -0.245 rpy=0 -0 0
- joint l_arm_shz: origin xyz=0.1406 0.2036 0.4776 rpy=0 -0 0 -> xyz=0.1406 0.2256 0.4776 rpy=0 -0 0
- joint l_arm_wrx: child l_hand -> l_lfarm; limit lower=-1.1781 upper=1.1781 effort=25 velocity=12 -> lower=-1.7628 upper=1.7628 effort=25 velocity=10; origin xyz=0 0.119 0.0092 rpy=0 -0 0 -> xyz=0 0 0 rpy=0 -0 0; parent l_farm -> l_ufarm
- joint l_arm_wry: child l_farm -> l_ufarm; limit lower=0 upper=3.14159 effort=25 velocity=12 -> lower=-3.011 upper=3.011 effort=25 velocity=10; origin xyz=0 0.187 -0.0092 rpy=0 -0 0 -> xyz=0 0.29955 -0.0092 rpy=0 -0 0
- joint neck_ry: origin xyz=0.2546 0 0.6215 rpy=0 -0 0 -> xyz=${0.2546+0.04} 0 ${0.6215-0.045} rpy=0 -0 0
- joint r_arm_ely: origin xyz=0 -0.187 0.016 rpy=0 -0 0 -> xyz=0 -0.187 -0.016 rpy=0 -0 0
- joint r_arm_shx: origin xyz=0 -0.0981 -0.2511 rpy=0 -0 0 -> xyz=0 -0.11 -0.245 rpy=0 -0 0
- joint r_arm_shz: origin xyz=0.1406 -0.2036 0.4776 rpy=0 -0 0 -> xyz=0.1406 -0.2256 0.4776 rpy=0 -0 0
- joint r_arm_wrx: child r_hand -> r_lfarm; limit lower=-1.1781 upper=1.1781 effort=25 velocity=12 -> lower=-1.7628 upper=1.7628 effort=25 velocity=10; origin xyz=0 -0.119 0.0092 rpy=0 -0 0 -> xyz=0 0 0 rpy=0 -0 0; parent r_farm -> r_ufarm
- joint r_arm_wry: child r_farm -> r_ufarm; limit lower=0 upper=3.14159 effort=25 velocity=12 -> lower=-3.011 upper=3.011 effort=25 velocity=10; origin xyz=0 -0.187 -0.0092 rpy=0 -0 0 -> xyz=0 -0.29955 -0.00921 rpy=0 -0 0

File: atlas_description/urdf/atlas_v4_simple_shapes.urdf (robot description, URDF)
Before this commit: robot drc_skeleton, 34 links, 34 joints
Links:
- removed link l_farm
- removed link r_farm
- added link l_lfarm, mass 2.65; collision cylinder length=0.05 radius=0.03
- added link l_ufarm, mass 2.12; collision cylinder length=0.1 radius=0.05; visual mesh filename=package://atlas_description/meshes_v3/l_farm.dae scale=1 1 1
- added link r_lfarm, mass 2.65; collision cylinder length=0.05 radius=0.03
- added link r_ufarm, mass 2.12; collision cylinder length=0.1 radius=0.05; visual mesh filename=package://atlas_description/meshes_v3/r_farm.dae scale=1 1 1
- link l_clav: geometry collision box size=0.02 0.029 0.015; collision box size=0.02 0.19 0.072
- link l_foot: geometry collision box size=${0.26-0.0005} ${0.124887+0.009} 0.05; visual mesh filename=package://atlas_description/meshes_unplugged/l_foot.dae scale=1 1 1
- link l_hand: mass 2.509 -> 0.53; geometry collision box size=0.14 0.09 0.06; collision cylinder length=0.03 radius=0.031
- link l_larm: geometry collision box size=0.025 0.125 0.075; collision cylinder length=0.04 radius=0.041
- link l_lglut: geometry collision box size=0.0975 0.069 0.103; collision cylinder length=0.060306 radius=0.02009687
- link l_lleg: geometry collision cylinder length=0.40 radius=0.07; visual mesh filename=package://atlas_description/meshes_unplugged/l_lleg.dae scale=1 1 1
- link l_scap: geometry collision box size=0.15 0.15 0.06; collision cylinder length=0.05 radius=0.04
- link l_talus: geometry collision cylinder length=0.010059 radius=0.010348; collision cylinder length=0.029542 radius=0.010181
- link l_uarm: geometry collision box size=0.05 0.07 0.15; collision cylinder length=0.11 radius=0.065
- link l_uglut: geometry collision cylinder length=0.078396 radius=0.019096; collision cylinder length=0.080842 radius=0.019841
- link l_uleg: geometry collision box size=0.07 0.038 0.14; collision box size=0.07 0.038 0.15
- link ltorso: geometry visual mesh filename=package://atlas_description/meshes_unplugged/ltorso.dae scale=1 1 1
- link mtorso: geometry collision cylinder length=0.15 radius=0.02; visual mesh filename=package://atlas_description/meshes_unplugged/mtorso.dae scale=1 1 1
- link pelvis: geometry collision box size=0.1 0.15 0.2; collision cylinder length=0.05 radius=0.16
- link r_clav: geometry collision box size=0.02 0.029 0.015; collision box size=0.02 0.19 0.072
- link r_foot: geometry collision box size=${0.26-0.0005} ${0.124887+0.009} 0.05; visual mesh filename=package://atlas_description/meshes_unplugged/r_foot.dae scale=1 1 1
- link r_hand: mass 2.509 -> 0.53; geometry collision box size=0.14 0.09 0.06; collision cylinder length=0.03 radius=0.031
- link r_larm: geometry collision box size=0.025 0.125 0.075; collision cylinder length=0.04 radius=0.041
- link r_lglut: geometry collision box size=0.0975 0.069 0.103; collision cylinder length=0.060306 radius=0.02009687
- link r_lleg: geometry collision cylinder length=0.40 radius=0.07; visual mesh filename=package://atlas_description/meshes_unplugged/r_lleg.dae scale=1 1 1
- link r_scap: geometry collision box size=0.15 0.15 0.06; collision cylinder length=0.05 radius=0.04
- link r_talus: geometry collision cylinder length=0.010059 radius=0.010348; collision cylinder length=0.029542 radius=0.010181
- link r_uarm: geometry collision box size=0.05 0.07 0.15; collision cylinder length=0.11 radius=0.065
- link r_uglut: geometry collision cylinder length=0.078396 radius=0.019096; collision cylinder length=0.080842 radius=0.019841
- link r_uleg: geometry collision box size=0.07 0.038 0.14; collision box size=0.07 0.038 0.15
- link utorso: geometry collision box size=0.2 0.25 0.01; collision box size=0.456306 0.341719 0.12
Joints:
- added joint l_arm_wry2: type revolute, parent l_lfarm, child l_hand, origin xyz=0 0 0 rpy=0 -0 0, axis 0 1 0, limit lower=-2.9671 upper=2.9671 effort=25 velocity=10
- added joint r_arm_wry2: type revolute, parent r_lfarm, child r_hand, origin xyz=0 0 0 rpy=0 -0 0, axis 0 1 0, limit lower=-2.9671 upper=2.9671 effort=25 velocity=10
- joint l_arm_ely: origin xyz=0 0.187 0.016 rpy=0 -0 0 -> xyz=0 0.187 -0.016 rpy=0 -0 0
- joint l_arm_shx: origin xyz=0 0.0981 -0.2511 rpy=0 -0 0 -> xyz=0 0.11 -0.245 rpy=0 -0 0
- joint l_arm_shz: origin xyz=0.1406 0.2036 0.4776 rpy=0 -0 0 -> xyz=0.1406 0.2256 0.4776 rpy=0 -0 0
- joint l_arm_wrx: child l_hand -> l_lfarm; limit lower=-1.1781 upper=1.1781 effort=25 velocity=12 -> lower=-1.7628 upper=1.7628 effort=25 velocity=10; origin xyz=0 0.119 0.0092 rpy=0 -0 0 -> xyz=0 0 0 rpy=0 -0 0; parent l_farm -> l_ufarm
- joint l_arm_wry: child l_farm -> l_ufarm; limit lower=0 upper=3.14159 effort=25 velocity=12 -> lower=-3.011 upper=3.011 effort=25 velocity=10; origin xyz=0 0.187 -0.0092 rpy=0 -0 0 -> xyz=0 0.29955 -0.00921 rpy=0 -0 0
- joint neck_ry: origin xyz=0.2546 0 0.6215 rpy=0 -0 0 -> xyz=${0.2546+0.04} 0 ${0.6215-0.045} rpy=0 -0 0
- joint r_arm_ely: origin xyz=0 -0.187 0.016 rpy=0 -0 0 -> xyz=0 -0.187 -0.016 rpy=0 -0 0
- joint r_arm_shx: origin xyz=0 -0.0981 -0.2511 rpy=0 -0 0 -> xyz=0 -0.11 -0.245 rpy=0 -0 0
- joint r_arm_shz: origin xyz=0.1406 -0.2036 0.4776 rpy=0 -0 0 -> xyz=0.1406 -0.2256 0.4776 rpy=0 -0 0
- joint r_arm_wrx: child r_hand -> r_lfarm; limit lower=-1.1781 upper=1.1781 effort=25 velocity=12 -> lower=-1.7628 upper=1.7628 effort=25 velocity=10; origin xyz=0 -0.119 0.0092 rpy=0 -0 0 -> xyz=0 0 0 rpy=0 -0 0; parent r_farm -> r_ufarm
- joint r_arm_wry: child r_farm -> r_ufarm; limit lower=0 upper=3.14159 effort=25 velocity=12 -> lower=-3.011 upper=3.011 effort=25 velocity=10; origin xyz=0 -0.187 -0.0092 rpy=0 -0 0 -> xyz=0 -0.29955 -0.00921 rpy=0 -0 0

File: atlas_description/urdf/atlas_v5.urdf (robot description, URDF)
Before this commit: robot drc_skeleton, 36 links, 36 joints
Links:
- link l_clav: geometry collision mesh filename=package://atlas_description/meshes_unplugged/l_clav.dae scale=1 1 1; visual mesh filename=package://atlas_description/meshes_unplugged/l_clav.dae scale=1 1 1
- link l_foot: geometry collision mesh filename=package://atlas_description/meshes_unplugged/l_foot.dae scale=1 1 1; visual mesh filename=package://atlas_description/meshes_unplugged/l_foot.dae scale=1 1 1
- link l_hand: geometry collision mesh filename=package://atlas_description/meshes_unplugged/l_hand.dae scale=1 1 1; visual mesh filename=package://atlas_description/meshes_unplugged/l_hand.dae scale=1 1 1
- link l_larm: geometry collision mesh filename=package://atlas_description/meshes_unplugged/l_larm.dae scale=1 1 1; visual mesh filename=package://atlas_description/meshes_unplugged/l_larm.dae
- link l_lglut: geometry collision mesh filename=package://atlas_description/meshes_unplugged/l_lglut.dae scale=1 1 1; visual mesh filename=package://atlas_description/meshes_unplugged/l_lglut.dae scale=1 1 1
- link l_lleg: geometry collision mesh filename=package://atlas_description/meshes_unplugged/l_lleg.dae scale=1 1 1; visual mesh filename=package://atlas_description/meshes_unplugged/l_lleg.dae scale=1 1 1
- link l_scap: geometry collision mesh filename=package://atlas_description/meshes_unplugged/l_scap.dae scale=1 1 1; visual mesh filename=package://atlas_description/meshes_unplugged/l_scap.dae scale=1 1 1
- link l_talus: geometry collision mesh filename=package://atlas_description/meshes_unplugged/l_talus.dae scale=1 1 1; visual mesh filename=package://atlas_description/meshes_unplugged/l_talus.dae scale=1 1 1
- link l_uarm: geometry collision mesh filename=package://atlas_description/meshes_unplugged/l_uarm.dae scale=1 1 1; visual mesh filename=package://atlas_description/meshes_unplugged/l_uarm.dae scale=1 1 1
- link l_ufarm: geometry collision cylinder length=0.1 radius=0.05; visual mesh filename=package://atlas_description/meshes_unplugged/l_farm.dae scale=1 1 1
- link l_uglut: geometry collision mesh filename=package://atlas_description/meshes_unplugged/l_uglut.dae scale=1 1 1; visual mesh filename=package://atlas_description/meshes_unplugged/l_uglut.dae scale=1 1 1
- link l_uleg: geometry collision mesh filename=package://atlas_description/meshes_unplugged/l_uleg.dae scale=1 1 1; visual mesh filename=package://atlas_description/meshes_unplugged/l_uleg.dae scale=1 1 1
- link ltorso: geometry collision mesh filename=package://atlas_description/meshes_unplugged/ltorso.dae scale=1 1 1; visual mesh filename=package://atlas_description/meshes_unplugged/ltorso.dae scale=1 1 1
- link mtorso: geometry collision mesh filename=package://atlas_description/meshes_unplugged/mtorso.dae scale=1 1 1; visual mesh filename=package://atlas_description/meshes_unplugged/mtorso.dae scale=1 1 1
- link pelvis: geometry collision mesh filename=package://atlas_description/meshes_unplugged/pelvis.dae scale=1 1 1; visual mesh filename=package://atlas_description/meshes_unplugged/pelvis.dae scale=1 1 1
- link r_clav: geometry collision mesh filename=package://atlas_description/meshes_unplugged/r_clav.dae scale=1 1 1; visual mesh filename=package://atlas_description/meshes_unplugged/r_clav.dae scale=1 1 1
- link r_foot: geometry collision mesh filename=package://atlas_description/meshes_unplugged/r_foot.dae scale=1 1 1; visual mesh filename=package://atlas_description/meshes_unplugged/r_foot.dae scale=1 1 1
- link r_hand: geometry collision mesh filename=package://atlas_description/meshes_unplugged/r_hand.dae scale=1 1 1; visual mesh filename=package://atlas_description/meshes_unplugged/r_hand.dae scale=1 1 1
- link r_larm: geometry collision mesh filename=package://atlas_description/meshes_unplugged/r_larm.dae scale=1 1 1; visual mesh filename=package://atlas_description/meshes_unplugged/r_larm.dae
- link r_lglut: geometry collision mesh filename=package://atlas_description/meshes_unplugged/r_lglut.dae scale=1 1 1; visual mesh filename=package://atlas_description/meshes_unplugged/r_lglut.dae scale=1 1 1
- link r_lleg: geometry collision mesh filename=package://atlas_description/meshes_unplugged/r_lleg.dae scale=1 1 1; visual mesh filename=package://atlas_description/meshes_unplugged/r_lleg.dae scale=1 1 1
- link r_scap: geometry collision mesh filename=package://atlas_description/meshes_unplugged/r_scap.dae scale=1 1 1; visual mesh filename=package://atlas_description/meshes_unplugged/r_scap.dae scale=1 1 1
- link r_talus: geometry collision mesh filename=package://atlas_description/meshes_unplugged/r_talus.dae scale=1 1 1; visual mesh filename=package://atlas_description/meshes_unplugged/r_talus.dae scale=1 1 1
- link r_uarm: geometry collision mesh filename=package://atlas_description/meshes_unplugged/r_uarm.dae scale=1 1 1; visual mesh filename=package://atlas_description/meshes_unplugged/r_uarm.dae scale=1 1 1
- link r_ufarm: geometry collision cylinder length=0.1 radius=0.05; visual mesh filename=package://atlas_description/meshes_unplugged/r_farm.dae scale=1 1 1
- link r_uglut: geometry collision mesh filename=package://atlas_description/meshes_unplugged/r_uglut.dae scale=1 1 1; visual mesh filename=package://atlas_description/meshes_unplugged/r_uglut.dae scale=1 1 1
- link r_uleg: geometry collision mesh filename=package://atlas_description/meshes_unplugged/r_uleg.dae scale=1 1 1; visual mesh filename=package://atlas_description/meshes_unplugged/r_uleg.dae scale=1 1 1
- link utorso: geometry collision mesh filename=package://atlas_description/meshes_unplugged/utorso.dae scale=1 1 1; visual mesh filename=package://atlas_description/meshes_unplugged/utorso.dae scale=1 1 1

File: atlas_description/urdf/atlas_v5_simple_shapes.urdf (robot description, URDF)
Before this commit: robot drc_skeleton, 36 links, 36 joints
Links:
- link l_clav: geometry collision box size=0.02 0.029 0.015; collision box size=0.02 0.19 0.072
- link l_foot: geometry collision box size=${0.26-0.0005} ${0.124887+0.009} 0.05; visual mesh filename=package://atlas_description/meshes_unplugged/l_foot.dae scale=1 1 1
- link l_hand: geometry collision box size=0.14 0.09 0.06; collision cylinder length=0.03 radius=0.031
- link l_larm: geometry collision box size=0.025 0.125 0.075; collision cylinder length=0.04 radius=0.041
- link l_lglut: geometry collision box size=0.0975 0.069 0.103; collision cylinder length=0.060306 radius=0.02009687
- link l_lleg: geometry collision cylinder length=0.40 radius=0.07; visual mesh filename=package://atlas_description/meshes_unplugged/l_lleg.dae scale=1 1 1
- link l_scap: geometry collision box size=0.15 0.15 0.06; collision cylinder length=0.05 radius=0.04
- link l_talus: geometry collision cylinder length=0.010059 radius=0.010348; collision cylinder length=0.029542 radius=0.010181
- link l_uarm: geometry collision box size=0.05 0.07 0.15; collision cylinder length=0.11 radius=0.065
- link l_ufarm: geometry collision cylinder length=0.1 radius=0.05; visual mesh filename=package://atlas_description/meshes_unplugged/l_farm.dae scale=1 1 1
- link l_uglut: geometry collision cylinder length=0.078396 radius=0.019096; collision cylinder length=0.080842 radius=0.019841
- link l_uleg: geometry collision box size=0.07 0.038 0.14; collision box size=0.07 0.038 0.15
- link ltorso: geometry visual mesh filename=package://atlas_description/meshes_unplugged/ltorso.dae scale=1 1 1
- link mtorso: geometry collision cylinder length=0.15 radius=0.02; visual mesh filename=package://atlas_description/meshes_unplugged/mtorso.dae scale=1 1 1
- link pelvis: geometry collision box size=0.1 0.15 0.2; collision cylinder length=0.05 radius=0.16
- link r_clav: geometry collision box size=0.02 0.029 0.015; collision box size=0.02 0.19 0.072
- link r_foot: geometry collision box size=${0.26-0.0005} ${0.124887+0.009} 0.05; visual mesh filename=package://atlas_description/meshes_unplugged/r_foot.dae scale=1 1 1
- link r_hand: geometry collision box size=0.14 0.09 0.06; collision cylinder length=0.03 radius=0.031
- link r_larm: geometry collision box size=0.025 0.125 0.075; collision cylinder length=0.04 radius=0.041
- link r_lglut: geometry collision box size=0.0975 0.069 0.103; collision cylinder length=0.060306 radius=0.02009687
- link r_lleg: geometry collision cylinder length=0.40 radius=0.07; visual mesh filename=package://atlas_description/meshes_unplugged/r_lleg.dae scale=1 1 1
- link r_scap: geometry collision box size=0.15 0.15 0.06; collision cylinder length=0.05 radius=0.04
- link r_talus: geometry collision cylinder length=0.010059 radius=0.010348; collision cylinder length=0.029542 radius=0.010181
- link r_uarm: geometry collision box size=0.05 0.07 0.15; collision cylinder length=0.11 radius=0.065
- link r_ufarm: geometry collision cylinder length=0.1 radius=0.05; visual mesh filename=package://atlas_description/meshes_unplugged/r_farm.dae scale=1 1 1
- link r_uglut: geometry collision cylinder length=0.078396 radius=0.019096; collision cylinder length=0.080842 radius=0.019841
- link r_uleg: geometry collision box size=0.07 0.038 0.14; collision box size=0.07 0.038 0.15
- link utorso: geometry collision box size=0.2 0.25 0.01; collision box size=0.456306 0.341719 0.12
