Commit message: update atlas v5 with visuals and collisions from v3

File: atlas_description/urdf/atlas_v5.urdf (robot description, URDF)
Before this commit: robot drc_skeleton, 31 links, 30 joints
Links:
- removed link head
- added link l_situational_awareness_camera_link, mass 0.1; visual box size=0.01 0.01 0.01
- added link l_situational_awareness_camera_optical_frame
- added link r_situational_awareness_camera_link, mass 0.1; visual box size=0.01 0.01 0.01
- added link r_situational_awareness_camera_optical_frame
- added link rear_situational_awareness_camera_link, mass 0.1; visual box size=0.01 0.01 0.01
- added link rear_situational_awareness_camera_optical_frame
- link l_clav: geometry collision mesh filename=package://atlas_description/meshes_v3/l_clav.stl scale=1 1 1; visual mesh filename=package://atlas_description/meshes_v3/l_clav.dae scale=1 1 1
- link l_foot: geometry collision mesh filename=package://atlas_description/meshes_v3/l_foot.stl scale=1 1 1; visual mesh filename=package://atlas_description/meshes_v3/l_foot.dae scale=1 1 1
- link l_hand: geometry collision mesh filename=package://atlas_description/meshes_v3/l_hand.stl scale=1 1 1; visual mesh filename=package://atlas_description/meshes_v3/l_hand.dae scale=1 1 1
- link l_larm: geometry collision mesh filename=package://atlas_description/meshes_v3/l_larm.stl scale=1 1 1; visual mesh filename=package://atlas_description/meshes_v3/l_larm.dae scale=1 1 1
- link l_lfarm: geometry collision mesh filename=package://atlas_description/meshes_v3/l_farm.stl scale=1 1 1; visual mesh filename=package://atlas_description/meshes_v3/l_farm.dae scale=1 1 1
- link l_lglut: geometry collision mesh filename=package://atlas_description/meshes_v3/l_lglut.stl scale=1 1 1; visual mesh filename=package://atlas_description/meshes_v3/l_lglut.dae scale=1 1 1
- link l_lleg: geometry collision mesh filename=package://atlas_description/meshes_v3/l_lleg.stl scale=1 1 1; visual mesh filename=package://atlas_description/meshes_v3/l_lleg.dae scale=1 1 1
- link l_scap: geometry collision mesh filename=package://atlas_description/meshes_v3/l_scap.stl scale=1 1 1; visual mesh filename=package://atlas_description/meshes_v3/l_scap.dae scale=1 1 1
- link l_talus: geometry collision mesh filename=package://atlas_description/meshes_v3/l_talus.stl scale=1 1 1; visual mesh filename=package://atlas_description/meshes_v3/l_talus.dae scale=1 1 1
- link l_uarm: geometry collision mesh filename=package://atlas_description/meshes_v3/l_uarm.stl scale=1 1 1; visual mesh filename=package://atlas_description/meshes_v3/l_uarm.dae scale=1 1 1
- link l_ufarm: geometry collision mesh filename=package://atlas_description/meshes_v3/l_farm.stl scale=1 1 1; visual mesh filename=package://atlas_description/meshes_v3/l_farm.dae scale=1 1 1
- link l_uglut: geometry collision mesh filename=package://atlas_description/meshes_v3/l_uglut.stl scale=1 1 1; visual mesh filename=package://atlas_description/meshes_v3/l_uglut.dae scale=1 1 1
- link l_uleg: geometry collision mesh filename=package://atlas_description/meshes_v3/l_uleg.stl scale=1 1 1; visual mesh filename=package://atlas_description/meshes_v3/l_uleg.dae scale=1 1 1
- link ltorso: geometry collision mesh filename=package://atlas_description/meshes_v3/ltorso.stl scale=1 1 1; visual mesh filename=package://atlas_description/meshes_v3/ltorso.dae scale=1 1 1
- link mtorso: geometry collision mesh filename=package://atlas_description/meshes_v3/mtorso.stl scale=1 1 1; visual mesh filename=package://atlas_description/meshes_v3/mtorso.dae scale=1 1 1
- link pelvis: geometry collision mesh filename=package://atlas_description/meshes_v3/pelvis.stl scale=1 1 1; visual mesh filename=package://atlas_description/meshes_v3/pelvis.dae scale=1 1 1
- link r_clav: geometry collision mesh filename=package://atlas_description/meshes_v3/r_clav.stl scale=1 1 1; visual mesh filename=package://atlas_description/meshes_v3/r_clav.dae scale=1 1 1
- link r_foot: geometry collision mesh filename=package://atlas_description/meshes_v3/r_foot.stl scale=1 1 1; visual mesh filename=package://atlas_description/meshes_v3/r_foot.dae scale=1 1 1
- link r_hand: geometry collision mesh filename=package://atlas_description/meshes_v3/r_hand.stl scale=1 1 1; visual mesh filename=package://atlas_description/meshes_v3/r_hand.dae scale=1 1 1
- link r_larm: geometry collision mesh filename=package://atlas_description/meshes_v3/r_larm.stl scale=1 1 1; visual mesh filename=package://atlas_description/meshes_v3/r_larm.dae scale=1 1 1
- link r_lfarm: geometry collision mesh filename=package://atlas_description/meshes_v3/r_farm.stl scale=1 1 1; visual mesh filename=package://atlas_description/meshes_v3/r_farm.dae scale=1 1 1
- link r_lglut: geometry collision mesh filename=package://atlas_description/meshes_v3/r_lglut.stl scale=1 1 1; visual mesh filename=package://atlas_description/meshes_v3/r_lglut.dae scale=1 1 1
- link r_lleg: geometry collision mesh filename=package://atlas_description/meshes_v3/r_lleg.stl scale=1 1 1; visual mesh filename=package://atlas_description/meshes_v3/r_lleg.dae scale=1 1 1
- link r_scap: geometry collision mesh filename=package://atlas_description/meshes_v3/r_scap.stl scale=1 1 1; visual mesh filename=package://atlas_description/meshes_v3/r_scap.dae scale=1 1 1
- link r_talus: geometry collision mesh filename=package://atlas_description/meshes_v3/r_talus.stl scale=1 1 1; visual mesh filename=package://atlas_description/meshes_v3/r_talus.dae scale=1 1 1
- link r_uarm: geometry collision mesh filename=package://atlas_description/meshes_v3/r_uarm.stl scale=1 1 1; visual mesh filename=package://atlas_description/meshes_v3/r_uarm.dae scale=1 1 1
- link r_ufarm: geometry collision mesh filename=package://atlas_description/meshes_v3/r_farm.stl scale=1 1 1; visual mesh filename=package://atlas_description/meshes_v3/r_farm.dae scale=1 1 1
- link r_uglut: geometry collision mesh filename=package://atlas_description/meshes_v3/r_uglut.stl scale=1 1 1; visual mesh filename=package://atlas_description/meshes_v3/r_uglut.dae scale=1 1 1
- link r_uleg: geometry collision mesh filename=package://atlas_description/meshes_v3/r_uleg.stl scale=1 1 1; visual mesh filename=package://atlas_description/meshes_v3/r_uleg.dae scale=1 1 1
- link utorso: geometry collision mesh filename=package://atlas_description/meshes_v3/utorso.stl scale=1 1 1; collision mesh filename=package://atlas_description/meshes_v3/utorso_pack.stl scale=1 1 1
Joints:
- added joint l_situational_awareness_camera_joint: type fixed, parent utorso, child l_situational_awareness_camera_link, origin xyz=0.216409 0.121799 0.406759 rpy=-1.57079633 0 1.30899694
- added joint l_situational_awareness_camera_optical_frame_joint: type fixed, parent l_situational_awareness_camera_link, child l_situational_awareness_camera_optical_frame, origin xyz=0 0 0 rpy=-1.5708 0.0 -1.5708
- added joint r_situational_awareness_camera_joint: type fixed, parent utorso, child r_situational_awareness_camera_link, origin xyz=0.216409 -0.121799 0.406759 rpy=1.57079633 0 -1.30899694
- added joint r_situational_awareness_camera_optical_frame_joint: type fixed, parent r_situational_awareness_camera_link, child r_situational_awareness_camera_optical_frame, origin xyz=0 0 0 rpy=-1.5708 0.0 -1.5708
- added joint rear_situational_awareness_camera_joint: type fixed, parent utorso, child rear_situational_awareness_camera_link, origin xyz=-0.0026 0.0264 0.6649 rpy=0 0 3.14159
- added joint rear_situational_awareness_camera_optical_frame_joint: type fixed, parent rear_situational_awareness_camera_link, child rear_situational_awareness_camera_optical_frame, origin xyz=0 0 0 rpy=-1.5708 0.0 -1.5708

Commit message: testing ufarm and lfarm links

File: atlas_description/urdf/atlas_v5.urdf (robot description, URDF)
Before this commit: robot drc_skeleton, 36 links, 36 joints
Links:
- link l_lfarm: geometry collision cylinder length=0.05 radius=0.03; visual cylinder length=0.05 radius=0.03
- link l_ufarm: geometry collision cylinder length=0.1 radius=0.05; visual cylinder length=0.1 radius=0.05
- link r_lfarm: geometry collision cylinder length=0.05 radius=0.03; visual cylinder length=0.05 radius=0.03
- link r_ufarm: geometry collision cylinder length=0.1 radius=0.05; visual cylinder length=0.1 radius=0.05
Joints:
- joint l_arm_wry: origin xyz=0 -0.29955 -0.00921 rpy=0 -0 0 -> xyz=0 0.29955 -0.00921 rpy=0 -0 0
- joint r_arm_wry: origin xyz=0 0.29955 -0.00921 rpy=0 -0 0 -> xyz=0 -0.29955 -0.00921 rpy=0 -0 0

Commit message: fix visual and collision meshes_v4 shifts for atlas_v5

File: atlas_description/urdf/atlas_v5.urdf (robot description, URDF)
Before this commit: robot drc_skeleton, 36 links, 36 joints
Links:
- link l_foot: geometry collision mesh filename=package://atlas_description/meshes_v4/l_foot.dae scale=1 1 1; visual mesh filename=package://atlas_description/meshes_v4/l_foot.dae scale=1 1 1
- link l_lglut: geometry collision mesh filename=package://atlas_description/meshes_v4/l_lglut.dae scale=1 1 1; visual mesh filename=package://atlas_description/meshes_v4/l_lglut.dae scale=1 1 1
- link l_talus: geometry collision mesh filename=package://atlas_description/meshes_v4/l_talus.dae scale=1 1 1; visual mesh filename=package://atlas_description/meshes_v4/l_talus.dae scale=1 1 1
- link l_uleg: geometry collision mesh filename=package://atlas_description/meshes_v4/l_uleg.dae scale=1 1 1; visual mesh filename=package://atlas_description/meshes_v4/l_uleg.dae scale=1 1 1
- link r_foot: geometry collision mesh filename=package://atlas_description/meshes_v4/r_foot.dae scale=1 1 1; visual mesh filename=package://atlas_description/meshes_v4/r_foot.dae scale=1 1 1
- link r_lglut: geometry collision mesh filename=package://atlas_description/meshes_v4/r_lglut.dae scale=1 1 1; visual mesh filename=package://atlas_description/meshes_v4/r_lglut.dae scale=1 1 1
- link r_talus: geometry collision mesh filename=package://atlas_description/meshes_v4/r_talus.dae scale=1 1 1; visual mesh filename=package://atlas_description/meshes_v4/r_talus.dae scale=1 1 1
- link r_uleg: geometry collision mesh filename=package://atlas_description/meshes_v4/r_uleg.dae scale=1 1 1; visual mesh filename=package://atlas_description/meshes_v4/r_uleg.dae scale=1 1 1

Commit message: adjust clav shape location

File: atlas_description/urdf/atlas_v5.urdf (robot description, URDF)
Before this commit: robot drc_skeleton, 36 links, 36 joints
Links:
- link l_clav: geometry collision mesh filename=package://atlas_description/meshes_v4/l_clav.dae scale=1 1 1; visual mesh filename=package://atlas_description/meshes_v4/l_clav.dae scale=1 1 1
- link r_clav: geometry collision mesh filename=package://atlas_description/meshes_v4/r_clav.dae scale=1 1 1; visual mesh filename=package://atlas_description/meshes_v4/r_clav.dae scale=1 1 1

Commit message: fix neck / head alignment for v5

File: atlas_description/urdf/atlas_v5.urdf (robot description, URDF)
Before this commit: robot drc_skeleton, 36 links, 36 joints
Joints:
- joint neck_ry: origin xyz=0.2546 0 0.6215 rpy=0 -0 0 -> xyz=${0.2546+0.04} 0 ${0.6215-0.045} rpy=0 -0 0

Commit message: sync atlas_v5.urdf and atlas_v5_simple_shapes.urdf

File: atlas_description/urdf/atlas_v5.urdf (robot description, URDF)
Before this commit: robot drc_skeleton, 36 links, 36 joints
Links:
- link l_hand: geometry collision mesh filename=package://atlas_description/meshes_v4/l_hand.dae scale=1 1 1; visual mesh filename=package://atlas_description/meshes_v4/l_hand.dae scale=1 1 1
- link l_larm: geometry collision mesh filename=package://atlas_description/meshes_v4/l_larm.dae scale=1 1 1; visual mesh filename=package://atlas_description/meshes_v4/l_larm.dae scale=1 1 1
- link l_lleg: geometry collision mesh filename=package://atlas_description/meshes_v4/l_lleg.dae scale=1 1 1; visual mesh filename=package://atlas_description/meshes_v4/l_lleg.dae scale=1 1 1
- link l_scap: geometry collision mesh filename=package://atlas_description/meshes_v4/l_scap.dae scale=1 1 1; visual mesh filename=package://atlas_description/meshes_v4/l_scap.dae scale=1 1 1
- link l_uarm: geometry collision mesh filename=package://atlas_description/meshes_v4/l_uarm.dae scale=1 1 1; visual mesh filename=package://atlas_description/meshes_v4/l_uarm.dae scale=1 1 1
- link l_uglut: geometry collision mesh filename=package://atlas_description/meshes_v4/l_uglut.dae scale=1 1 1; visual mesh filename=package://atlas_description/meshes_v4/l_uglut.dae scale=1 1 1
- link ltorso: geometry collision mesh filename=package://atlas_description/meshes_v4/ltorso.dae scale=1 1 1; visual mesh filename=package://atlas_description/meshes_v4/ltorso.dae scale=1 1 1
- link mtorso: geometry collision mesh filename=package://atlas_description/meshes_v4/mtorso.dae scale=1 1 1; visual mesh filename=package://atlas_description/meshes_v4/mtorso.dae scale=1 1 1
- link pelvis: geometry collision mesh filename=package://atlas_description/meshes_v4/pelvis.dae scale=1 1 1; visual mesh filename=package://atlas_description/meshes_v4/pelvis.dae scale=1 1 1
- link r_hand: geometry collision mesh filename=package://atlas_description/meshes_v4/r_hand.dae scale=1 1 1; visual mesh filename=package://atlas_description/meshes_v4/r_hand.dae scale=1 1 1
- link r_lleg: geometry collision mesh filename=package://atlas_description/meshes_v4/r_lleg.dae scale=1 1 1; visual mesh filename=package://atlas_description/meshes_v4/r_lleg.dae scale=1 1 1
- link r_scap: geometry collision mesh filename=package://atlas_description/meshes_v4/r_scap.dae scale=1 1 1; visual mesh filename=package://atlas_description/meshes_v4/r_scap.dae scale=1 1 1
- link r_uarm: geometry collision mesh filename=package://atlas_description/meshes_v4/r_uarm.dae scale=1 1 1; visual mesh filename=package://atlas_description/meshes_v4/r_uarm.dae scale=1 1 1
- link r_uglut: geometry collision mesh filename=package://atlas_description/meshes_v4/r_uglut.dae scale=1 1 1; visual mesh filename=package://atlas_description/meshes_v4/r_uglut.dae scale=1 1 1
- link utorso: geometry collision mesh filename=package://atlas_description/meshes_v4/utorso.dae scale=1 1 1; visual mesh filename=package://atlas_description/meshes_v4/utorso.dae scale=1 1 1
Joints:
- joint l_arm_ely: origin xyz=0 0.187 0.016 rpy=0 -0 0 -> xyz=0 0.187 -0.016 rpy=0 -0 0
- joint r_arm_ely: origin xyz=0 -0.187 0.016 rpy=0 -0 0 -> xyz=0 -0.187 -0.016 rpy=0 -0 0

File: atlas_description/urdf/atlas_v5_simple_shapes.urdf (robot description, URDF)
Before this commit: robot drc_skeleton, 36 links, 36 joints
Joints:
- joint l_arm_ely: origin xyz=0 0.187 0.016 rpy=0 -0 0 -> xyz=0 0.187 -0.016 rpy=0 -0 0
- joint r_arm_ely: origin xyz=0 -0.187 0.016 rpy=0 -0 0 -> xyz=0 -0.187 -0.016 rpy=0 -0 0

Commit message: latest file from Bill

File: atlas_description/urdf/atlas_v5.urdf (robot description, URDF)
Before this commit: robot drc_skeleton, 36 links, 36 joints
Links:
- link l_lfarm: geometry collision cylinder length=0.05 radius=0.03
- link l_ufarm: geometry collision cylinder length=0.1 radius=0.05; visual mesh filename=package://atlas_description/meshes_v4/l_farm.dae scale=1 1 1
- link r_larm: geometry collision mesh filename=package://atlas_description/meshes_v3/r_larm.stl scale=1 1 1; visual mesh filename=package://atlas_description/meshes_v4/r_larm.dae scale=1 1 1
- link r_lfarm: geometry collision cylinder length=0.05 radius=0.03
- link r_ufarm: geometry collision cylinder length=0.1 radius=0.05; visual mesh filename=package://atlas_description/meshes_v4/r_farm.dae scale=1 1 1
- link utorso: geometry collision mesh filename=package://atlas_description/meshes_v3/utorso.stl scale=1 1 1; visual mesh filename=package://atlas_description/meshes_v4/utorso.dae scale=1 1 1
Joints:
- joint l_arm_ely: origin xyz=0 0.187 0.016 rpy=0 -0 0 -> xyz=0 0.187 -0.016 rpy=0 -0 0
- joint l_arm_shx: origin xyz=0 0.0981 -0.2511 rpy=0 -0 0 -> xyz=0 0.11 -0.245 rpy=0 -0 0
- joint l_arm_shz: origin xyz=0.1406 0.2036 0.4776 rpy=0 -0 0 -> xyz=0.1406 0.2256 0.4776 rpy=0 -0 0
- joint l_arm_wry: origin xyz=0 0.29955 -0.00921 rpy=0 -0 0 -> xyz=0 0.29955 -0.0092 rpy=0 -0 0
- joint r_arm_ely: origin xyz=0 -0.187 0.016 rpy=0 -0 0 -> xyz=0 -0.187 -0.016 rpy=0 -0 0
- joint r_arm_shx: origin xyz=0 -0.0981 -0.2511 rpy=0 -0 0 -> xyz=0 -0.11 -0.245 rpy=0 -0 0
- joint r_arm_shz: origin xyz=0.1406 -0.2036 0.4776 rpy=0 -0 0 -> xyz=0.1406 -0.2256 0.4776 rpy=0 -0 0

File: atlas_description/urdf/atlas_v5_simple_shapes.urdf (robot description, URDF)
Before this commit: robot drc_skeleton, 36 links, 36 joints
Links:
- link l_lfarm: geometry collision cylinder length=0.05 radius=0.03
- link l_ufarm: geometry collision cylinder length=0.1 radius=0.05; visual mesh filename=package://atlas_description/meshes_v4/l_farm.dae scale=1 1 1
- link r_larm: geometry collision mesh filename=package://atlas_description/meshes_v3/r_larm.stl scale=1 1 1; visual mesh filename=package://atlas_description/meshes_v4/r_larm.dae scale=1 1 1
- link r_lfarm: geometry collision cylinder length=0.05 radius=0.03
- link r_ufarm: geometry collision cylinder length=0.1 radius=0.05; visual mesh filename=package://atlas_description/meshes_v4/r_farm.dae scale=1 1 1
Joints:
- joint l_arm_ely: origin xyz=0 0.187 0.016 rpy=0 -0 0 -> xyz=0 0.187 -0.016 rpy=0 -0 0
- joint l_arm_shx: origin xyz=0 0.0981 -0.2511 rpy=0 -0 0 -> xyz=0 0.11 -0.245 rpy=0 -0 0
- joint l_arm_shz: origin xyz=0.1406 0.2036 0.4776 rpy=0 -0 0 -> xyz=0.1406 0.2256 0.4776 rpy=0 -0 0
- joint r_arm_ely: origin xyz=0 -0.187 0.016 rpy=0 -0 0 -> xyz=0 -0.187 -0.016 rpy=0 -0 0
- joint r_arm_shx: origin xyz=0 -0.0981 -0.2511 rpy=0 -0 0 -> xyz=0 -0.11 -0.245 rpy=0 -0 0
- joint r_arm_shz: origin xyz=0.1406 -0.2036 0.4776 rpy=0 -0 0 -> xyz=0.1406 -0.2256 0.4776 rpy=0 -0 0

Commit message: Minor tweaks to urdf to make the shoulders correct

File: atlas_description/urdf/atlas_v5.urdf (robot description, URDF)
Before this commit: robot drc_skeleton, 36 links, 36 joints
Links:
- link l_larm: geometry collision mesh filename=package://atlas_description/meshes_v4/l_larm.dae scale=1 1 1; visual mesh filename=package://atlas_description/meshes_v4/l_larm.dae
- link r_larm: geometry collision mesh filename=package://atlas_description/meshes_v3/r_larm.stl scale=1 1 1; visual mesh filename=package://atlas_description/meshes_v3/r_larm.dae

File: atlas_description/urdf/atlas_v5_simple_shapes.urdf (robot description, URDF)
Before this commit: robot drc_skeleton, 36 links, 36 joints
Links:
- link r_larm: geometry collision mesh filename=package://atlas_description/meshes_v3/r_larm.stl scale=1 1 1; visual mesh filename=package://atlas_description/meshes_v3/r_larm.dae scale=1 1 1
