Commit message: Added new atlas_v5 meshes and materials

File: atlas_description/urdf/atlas_v5.urdf (robot description, URDF)
Before this commit: robot drc_skeleton, 36 links, 36 joints
Links:
- link l_clav: geometry collision mesh filename=package://atlas_description/meshes_v5/l_clav.dae scale=1 1 1; visual mesh filename=package://atlas_description/meshes_v5/l_clav.dae scale=1 1 1
- link l_foot: geometry collision mesh filename=package://atlas_description/meshes_v5/l_foot.dae scale=1 1 1; visual mesh filename=package://atlas_description/meshes_v5/l_foot.dae scale=1 1 1
- link l_hand: geometry collision mesh filename=package://atlas_description/meshes_v5/l_hand.dae scale=1 1 1; visual mesh filename=package://atlas_description/meshes_v5/l_hand.dae scale=1 1 1
- link l_larm: geometry collision mesh filename=package://atlas_description/meshes_v5/l_larm.dae scale=1 1 1; visual mesh filename=package://atlas_description/meshes_v5/l_larm.dae
- link l_lglut: geometry collision mesh filename=package://atlas_description/meshes_v5/l_lglut.dae scale=1 1 1; visual mesh filename=package://atlas_description/meshes_v5/l_lglut.dae scale=1 1 1
- link l_lleg: geometry collision mesh filename=package://atlas_description/meshes_v5/l_lleg.dae scale=1 1 1; visual mesh filename=package://atlas_description/meshes_v5/l_lleg.dae scale=1 1 1
- link l_scap: geometry collision mesh filename=package://atlas_description/meshes_v5/l_scap.dae scale=1 1 1; visual mesh filename=package://atlas_description/meshes_v5/l_scap.dae scale=1 1 1
- link l_talus: geometry collision mesh filename=package://atlas_description/meshes_v5/l_talus.dae scale=1 1 1; visual mesh filename=package://atlas_description/meshes_v5/l_talus.dae scale=1 1 1
- link l_uarm: geometry collision mesh filename=package://atlas_description/meshes_v5/l_uarm.dae scale=1 1 1; visual mesh filename=package://atlas_description/meshes_v5/l_uarm.dae scale=1 1 1
- link l_ufarm: geometry collision cylinder length=0.1 radius=0.05; visual mesh filename=package://atlas_description/meshes_v5/l_farm.dae scale=1 1 1
- link l_uglut: geometry collision mesh filename=package://atlas_description/meshes_v5/l_uglut.dae scale=1 1 1; visual mesh filename=package://atlas_description/meshes_v5/l_uglut.dae scale=1 1 1
- link l_uleg: geometry collision mesh filename=package://atlas_description/meshes_v5/l_uleg.dae scale=1 1 1; visual mesh filename=package://atlas_description/meshes_v5/l_uleg.dae scale=1 1 1
- link ltorso: geometry collision mesh filename=package://atlas_description/meshes_v5/ltorso.dae scale=1 1 1; visual mesh filename=package://atlas_description/meshes_v5/ltorso.dae scale=1 1 1
- link mtorso: geometry collision mesh filename=package://atlas_description/meshes_v5/mtorso.dae scale=1 1 1; visual mesh filename=package://atlas_description/meshes_v5/mtorso.dae scale=1 1 1
- link pelvis: geometry collision mesh filename=package://atlas_description/meshes_v5/pelvis.dae scale=1 1 1; visual mesh filename=package://atlas_description/meshes_v5/pelvis.dae scale=1 1 1
- link r_clav: geometry collision mesh filename=package://atlas_description/meshes_v5/r_clav.dae scale=1 1 1; visual mesh filename=package://atlas_description/meshes_v5/r_clav.dae scale=1 1 1
- link r_foot: geometry collision mesh filename=package://atlas_description/meshes_v5/r_foot.dae scale=1 1 1; visual mesh filename=package://atlas_description/meshes_v5/r_foot.dae scale=1 1 1
- link r_hand: geometry collision mesh filename=package://atlas_description/meshes_v5/r_hand.dae scale=1 1 1; visual mesh filename=package://atlas_description/meshes_v5/r_hand.dae scale=1 1 1
- link r_larm: geometry collision mesh filename=package://atlas_description/meshes_v5/r_larm.dae scale=1 1 1; visual mesh filename=package://atlas_description/meshes_v5/r_larm.dae
- link r_lglut: geometry collision mesh filename=package://atlas_description/meshes_v5/r_lglut.dae scale=1 1 1; visual mesh filename=package://atlas_description/meshes_v5/r_lglut.dae scale=1 1 1
- link r_lleg: geometry collision mesh filename=package://atlas_description/meshes_v5/r_lleg.dae scale=1 1 1; visual mesh filename=package://atlas_description/meshes_v5/r_lleg.dae scale=1 1 1
- link r_scap: geometry collision mesh filename=package://atlas_description/meshes_v5/r_scap.dae scale=1 1 1; visual mesh filename=package://atlas_description/meshes_v5/r_scap.dae scale=1 1 1
- link r_talus: geometry collision mesh filename=package://atlas_description/meshes_v5/r_talus.dae scale=1 1 1; visual mesh filename=package://atlas_description/meshes_v5/r_talus.dae scale=1 1 1
- link r_uarm: geometry collision mesh filename=package://atlas_description/meshes_v5/r_uarm.dae scale=1 1 1; visual mesh filename=package://atlas_description/meshes_v5/r_uarm.dae scale=1 1 1
- link r_ufarm: geometry collision cylinder length=0.1 radius=0.05; visual mesh filename=package://atlas_description/meshes_v5/r_farm.dae scale=1 1 1
- link r_uglut: geometry collision mesh filename=package://atlas_description/meshes_v5/r_uglut.dae scale=1 1 1; visual mesh filename=package://atlas_description/meshes_v5/r_uglut.dae scale=1 1 1
- link r_uleg: geometry collision mesh filename=package://atlas_description/meshes_v5/r_uleg.dae scale=1 1 1; visual mesh filename=package://atlas_description/meshes_v5/r_uleg.dae scale=1 1 1
- link utorso: geometry collision mesh filename=package://atlas_description/meshes_v5/utorso.dae scale=1 1 1; visual mesh filename=package://atlas_description/meshes_v5/utorso.dae scale=1 1 1

File: atlas_description/urdf/atlas_v5_simple_shapes.urdf (robot description, URDF)
Before this commit: robot drc_skeleton, 36 links, 36 joints
Links:
- link l_clav: geometry collision box size=0.02 0.029 0.015; collision box size=0.02 0.19 0.072
- link l_foot: geometry collision box size=${0.26-0.0005} ${0.124887+0.009} 0.05; visual mesh filename=package://atlas_description/meshes_v5/l_foot.dae scale=1 1 1
- link l_hand: geometry collision box size=0.14 0.09 0.06; collision cylinder length=0.012 radius=0.048
- link l_larm: geometry collision box size=0.025 0.125 0.075; collision cylinder length=0.04 radius=0.041
- link l_lglut: geometry collision cylinder length=0.060306 radius=0.02009687; collision cylinder length=0.144 radius=0.02
- link l_lleg: geometry collision cylinder length=0.40 radius=0.07; visual mesh filename=package://atlas_description/meshes_v5/l_lleg.dae scale=1 1 1
- link l_scap: geometry collision box size=0.15 0.15 0.06; collision cylinder length=0.05 radius=0.04
- link l_talus: geometry collision cylinder length=0.010059 radius=0.010348; collision cylinder length=0.029542 radius=0.010181
- link l_uarm: geometry collision box size=0.05 0.07 0.15; collision cylinder length=0.11 radius=0.065
- link l_ufarm: geometry collision cylinder length=0.1 radius=0.05; visual mesh filename=package://atlas_description/meshes_v5/l_farm.dae scale=1 1 1
- link l_uglut: geometry collision cylinder length=0.078396 radius=0.019096; collision cylinder length=0.080842 radius=0.019841
- link l_uleg: geometry collision box size=0.07 0.038 0.14; collision box size=0.07 0.038 0.15
- link ltorso: geometry visual mesh filename=package://atlas_description/meshes_v5/ltorso.dae scale=1 1 1
- link mtorso: geometry collision cylinder length=0.15 radius=0.02; visual mesh filename=package://atlas_description/meshes_v5/mtorso.dae scale=1 1 1
- link pelvis: geometry collision box size=0.1 0.15 0.2; collision cylinder length=0.05 radius=0.16
- link r_clav: geometry collision box size=0.02 0.029 0.015; collision box size=0.02 0.19 0.072
- link r_foot: geometry collision box size=${0.26-0.0005} ${0.124887+0.009} 0.05; visual mesh filename=package://atlas_description/meshes_v5/r_foot.dae scale=1 1 1
- link r_hand: geometry collision box size=0.14 0.09 0.06; collision cylinder length=0.012 radius=0.048
- link r_larm: geometry collision box size=0.025 0.125 0.075; collision cylinder length=0.04 radius=0.041
- link r_lglut: geometry collision cylinder length=0.060306 radius=0.02009687; collision cylinder length=0.142 radius=0.02
- link r_lleg: geometry collision cylinder length=0.40 radius=0.07; visual mesh filename=package://atlas_description/meshes_v5/r_lleg.dae scale=1 1 1
- link r_scap: geometry collision box size=0.15 0.15 0.06; collision cylinder length=0.05 radius=0.04
- link r_talus: geometry collision cylinder length=0.010059 radius=0.010348; collision cylinder length=0.029542 radius=0.010181
- link r_uarm: geometry collision box size=0.05 0.07 0.15; collision cylinder length=0.11 radius=0.065
- link r_ufarm: geometry collision cylinder length=0.1 radius=0.05; visual mesh filename=package://atlas_description/meshes_v5/r_farm.dae scale=1 1 1
- link r_uglut: geometry collision cylinder length=0.078396 radius=0.019096; collision cylinder length=0.080842 radius=0.019841
- link r_uleg: geometry collision box size=0.07 0.038 0.14; collision box size=0.07 0.038 0.15
- link utorso: geometry collision box size=0.2 0.25 0.01; collision box size=0.266306 0.341719 0.18
