Commit message: Atlas v5 urdf and media

File: atlas_description/urdf/atlas_v5.urdf (robot description, URDF)
Before this commit: robot drc_skeleton, 36 links, 36 joints
Links:
- link l_clav: geometry collision mesh filename=package://atlas_description/meshes_unplugged/l_clav.dae; visual mesh filename=package://atlas_description/meshes_unplugged/l_clav.dae
- link l_foot: geometry collision mesh filename=package://atlas_description/meshes_unplugged/l_foot.dae; visual mesh filename=package://atlas_description/meshes_unplugged/l_foot.dae
- link l_hand: geometry 
- link l_larm: geometry collision mesh filename=package://atlas_description/meshes_unplugged/l_larm.dae; visual mesh filename=package://atlas_description/meshes_unplugged/l_larm.dae
- link l_lfarm: geometry collision mesh filename=package://atlas_description/meshes_unplugged/l_hand.dae; visual mesh filename=package://atlas_description/meshes_unplugged/l_hand.dae
- link l_lglut: geometry collision mesh filename=package://atlas_description/meshes_unplugged/l_lglut.dae; visual mesh filename=package://atlas_description/meshes_unplugged/l_lglut.dae
- link l_lleg: geometry collision mesh filename=package://atlas_description/meshes_unplugged/l_lleg.dae; visual mesh filename=package://atlas_description/meshes_unplugged/l_lleg.dae
- link l_scap: geometry collision mesh filename=package://atlas_description/meshes_unplugged/l_scap.dae; visual mesh filename=package://atlas_description/meshes_unplugged/l_scap.dae
- link l_talus: geometry collision mesh filename=package://atlas_description/meshes_unplugged/l_talus.dae; visual mesh filename=package://atlas_description/meshes_unplugged/l_talus.dae
- link l_uarm: geometry collision mesh filename=package://atlas_description/meshes_unplugged/l_uarm.dae; visual mesh filename=package://atlas_description/meshes_unplugged/l_uarm.dae
- link l_ufarm: geometry collision mesh filename=package://atlas_description/meshes_unplugged/l_farm.dae; visual mesh filename=package://atlas_description/meshes_unplugged/l_farm.dae
- link l_uglut: geometry collision mesh filename=package://atlas_description/meshes_unplugged/l_uglut.dae; visual mesh filename=package://atlas_description/meshes_unplugged/l_uglut.dae
- link l_uleg: geometry collision mesh filename=package://atlas_description/meshes_unplugged/l_uleg.dae; visual mesh filename=package://atlas_description/meshes_unplugged/l_uleg.dae
- link ltorso: geometry collision mesh filename=package://atlas_description/meshes_unplugged/ltorso.dae; visual mesh filename=package://atlas_description/meshes_unplugged/ltorso.dae
- link mtorso: geometry collision mesh filename=package://atlas_description/meshes_unplugged/mtorso.dae; visual mesh filename=package://atlas_description/meshes_unplugged/mtorso.dae
- link pelvis: geometry collision mesh filename=package://atlas_description/meshes_unplugged/pelvis.dae; visual mesh filename=package://atlas_description/meshes_unplugged/pelvis.dae
- link r_clav: geometry collision mesh filename=package://atlas_description/meshes_unplugged/r_clav.dae; visual mesh filename=package://atlas_description/meshes_unplugged/r_clav.dae
- link r_foot: geometry collision mesh filename=package://atlas_description/meshes_unplugged/r_foot.dae; visual mesh filename=package://atlas_description/meshes_unplugged/r_foot.dae
- link r_hand: geometry 
- link r_larm: geometry collision mesh filename=package://atlas_description/meshes_unplugged/r_larm.dae; visual mesh filename=package://atlas_description/meshes_unplugged/r_larm.dae
- link r_lfarm: geometry collision mesh filename=package://atlas_description/meshes_unplugged/r_hand.dae; visual mesh filename=package://atlas_description/meshes_unplugged/r_hand.dae
- link r_lglut: geometry collision mesh filename=package://atlas_description/meshes_unplugged/r_lglut.dae; visual mesh filename=package://atlas_description/meshes_unplugged/r_lglut.dae
- link r_lleg: geometry collision mesh filename=package://atlas_description/meshes_unplugged/r_lleg.dae; visual mesh filename=package://atlas_description/meshes_unplugged/r_lleg.dae
- link r_scap: geometry collision mesh filename=package://atlas_description/meshes_unplugged/r_scap.dae; visual mesh filename=package://atlas_description/meshes_unplugged/r_scap.dae
- link r_talus: geometry collision mesh filename=package://atlas_description/meshes_unplugged/r_talus.dae; visual mesh filename=package://atlas_description/meshes_unplugged/r_talus.dae
- link r_uarm: geometry collision mesh filename=package://atlas_description/meshes_unplugged/r_uarm.dae; visual mesh filename=package://atlas_description/meshes_unplugged/r_uarm.dae
- link r_ufarm: geometry collision mesh filename=package://atlas_description/meshes_unplugged/r_farm.dae; visual mesh filename=package://atlas_description/meshes_unplugged/r_farm.dae
- link r_uglut: geometry collision mesh filename=package://atlas_description/meshes_unplugged/r_uglut.dae; visual mesh filename=package://atlas_description/meshes_unplugged/r_uglut.dae
- link r_uleg: geometry collision mesh filename=package://atlas_description/meshes_unplugged/r_uleg.dae; visual mesh filename=package://atlas_description/meshes_unplugged/r_uleg.dae
- link utorso: geometry collision mesh filename=package://atlas_description/meshes_unplugged/utorso.dae; visual mesh filename=package://atlas_description/meshes_unplugged/utorso.dae
Joints:
- joint back_bkx: origin xyz=0 0 0.05 rpy=0 -0 0 -> xyz=0 0 0.05 rpy=0 0 0
- joint back_bky: origin xyz=0 0 0.162 rpy=0 -0 0 -> xyz=0 0 0.162 rpy=0 0 0
- joint back_bkz: origin xyz=-0.0125 0 0 rpy=0 -0 0 -> xyz=-0.0125 0 0 rpy=0 0 0
- joint l_arm_elx: origin xyz=0 0.119 0.0092 rpy=0 -0 0 -> xyz=0 0.119 0.0092 rpy=0 0 0
- joint l_arm_ely: origin xyz=0 0.187 -0.016 rpy=0 -0 0 -> xyz=0 0.187 -0.016 rpy=0 0 0
- joint l_arm_shx: origin xyz=0 0.11 -0.245 rpy=0 -0 0 -> xyz=0 0.11 -0.245 rpy=0 0 0
- joint l_arm_shz: origin xyz=0.1406 0.2256 0.4776 rpy=0 -0 0 -> xyz=0.1406 0.2256 0.4776 rpy=0 0 0
- joint l_arm_wrx: origin xyz=0 0 0 rpy=0 -0 0 -> xyz=0 0 0 rpy=0 0 0
- joint l_arm_wry: origin xyz=0 0.29955 -0.0092 rpy=0 -0 0 -> xyz=0 0.29955 -0.00921 rpy=0 0 0
- joint l_arm_wry2: origin xyz=0 0 0 rpy=0 -0 0 -> xyz=0 0 0 rpy=0 0 0
- joint l_leg_akx: origin xyz=0 0 0 rpy=0 -0 0 -> xyz=0 0 0 rpy=0 0 0
- joint l_leg_aky: origin xyz=0 0 -0.422 rpy=0 -0 0 -> xyz=0 0 -0.422 rpy=0 0 0
- joint l_leg_hpx: origin xyz=0 0 0 rpy=0 -0 0 -> xyz=0 0 0 rpy=0 0 0
- joint l_leg_hpy: origin xyz=0.05 0.0225 -0.066 rpy=0 -0 0 -> xyz=0.05 0.0225 -0.066 rpy=0 0 0
- joint l_leg_hpz: origin xyz=0 0.089 0 rpy=0 -0 0 -> xyz=0 0.089 0 rpy=0 0 0
- joint l_leg_kny: origin xyz=-0.05 0 -0.374 rpy=0 -0 0 -> xyz=-0.05 0 -0.374 rpy=0 0 0
- joint neck_ry: origin xyz=${0.2546+0.04} 0 ${0.6215-0.045} rpy=0 -0 0 -> xyz=${0.2546+0.04} 0 ${0.6215-0.045} rpy=0 0 0
- joint r_arm_elx: origin xyz=0 -0.119 0.0092 rpy=0 -0 0 -> xyz=0 -0.119 0.0092 rpy=0 0 0
- joint r_arm_ely: origin xyz=0 -0.187 -0.016 rpy=0 -0 0 -> xyz=0 -0.187 -0.016 rpy=0 0 0
- joint r_arm_shx: origin xyz=0 -0.11 -0.245 rpy=0 -0 0 -> xyz=0 -0.11 -0.245 rpy=0 0 0
- joint r_arm_shz: origin xyz=0.1406 -0.2256 0.4776 rpy=0 -0 0 -> xyz=0.1406 -0.2256 0.4776 rpy=0 0 0
- joint r_arm_wrx: origin xyz=0 0 0 rpy=0 -0 0 -> xyz=0 0 0 rpy=0 0 0
- joint r_arm_wry: origin xyz=0 -0.29955 -0.00921 rpy=0 -0 0 -> xyz=0 -0.29955 -0.00921 rpy=0 0 0
- joint r_arm_wry2: origin xyz=0 0 0 rpy=0 -0 0 -> xyz=0 0 0 rpy=0 0 0
- joint r_leg_akx: origin xyz=0 0 0 rpy=0 -0 0 -> xyz=0 0 0 rpy=0 0 0
- joint r_leg_aky: origin xyz=0 0 -0.422 rpy=0 -0 0 -> xyz=0 0 -0.422 rpy=0 0 0
- joint r_leg_hpx: origin xyz=0 0 0 rpy=0 -0 0 -> xyz=0 0 0 rpy=0 0 0
- joint r_leg_hpy: origin xyz=0.05 -0.0225 -0.066 rpy=0 -0 0 -> xyz=0.05 -0.0225 -0.066 rpy=0 0 0
- joint r_leg_hpz: origin xyz=0 -0.089 0 rpy=0 -0 0 -> xyz=0 -0.089 0 rpy=0 0 0
- joint r_leg_kny: origin xyz=-0.05 0 -0.374 rpy=0 -0 0 -> xyz=-0.05 0 -0.374 rpy=0 0 0

File: atlas_description/urdf/atlas_v5_simple_shapes.urdf (robot description, URDF)
Before this commit: robot drc_skeleton, 36 links, 36 joints
Links:
- link l_clav: geometry collision mesh filename=package://atlas_description/meshes_unplugged/l_clav.dae; visual mesh filename=package://atlas_description/meshes_unplugged/l_clav.dae
- link l_foot: geometry collision mesh filename=package://atlas_description/meshes_unplugged/l_foot.dae; visual mesh filename=package://atlas_description/meshes_unplugged/l_foot.dae
- link l_hand: geometry 
- link l_larm: geometry collision mesh filename=package://atlas_description/meshes_unplugged/l_larm.dae; visual mesh filename=package://atlas_description/meshes_unplugged/l_larm.dae
- link l_lfarm: geometry collision mesh filename=package://atlas_description/meshes_unplugged/l_hand.dae; visual mesh filename=package://atlas_description/meshes_unplugged/l_hand.dae
- link l_lglut: geometry collision mesh filename=package://atlas_description/meshes_unplugged/l_lglut.dae; visual mesh filename=package://atlas_description/meshes_unplugged/l_lglut.dae
- link l_lleg: geometry collision mesh filename=package://atlas_description/meshes_unplugged/l_lleg.dae; visual mesh filename=package://atlas_description/meshes_unplugged/l_lleg.dae
- link l_scap: geometry collision mesh filename=package://atlas_description/meshes_unplugged/l_scap.dae; visual mesh filename=package://atlas_description/meshes_unplugged/l_scap.dae
- link l_talus: geometry collision mesh filename=package://atlas_description/meshes_unplugged/l_talus.dae; visual mesh filename=package://atlas_description/meshes_unplugged/l_talus.dae
- link l_uarm: geometry collision mesh filename=package://atlas_description/meshes_unplugged/l_uarm.dae; visual mesh filename=package://atlas_description/meshes_unplugged/l_uarm.dae
- link l_ufarm: geometry collision mesh filename=package://atlas_description/meshes_unplugged/l_farm.dae; visual mesh filename=package://atlas_description/meshes_unplugged/l_farm.dae
- link l_uglut: geometry collision mesh filename=package://atlas_description/meshes_unplugged/l_uglut.dae; visual mesh filename=package://atlas_description/meshes_unplugged/l_uglut.dae
- link l_uleg: geometry collision mesh filename=package://atlas_description/meshes_unplugged/l_uleg.dae; visual mesh filename=package://atlas_description/meshes_unplugged/l_uleg.dae
- link ltorso: geometry collision mesh filename=package://atlas_description/meshes_unplugged/ltorso.dae; visual mesh filename=package://atlas_description/meshes_unplugged/ltorso.dae
- link mtorso: geometry collision mesh filename=package://atlas_description/meshes_unplugged/mtorso.dae; visual mesh filename=package://atlas_description/meshes_unplugged/mtorso.dae
- link pelvis: geometry collision mesh filename=package://atlas_description/meshes_unplugged/pelvis.dae; visual mesh filename=package://atlas_description/meshes_unplugged/pelvis.dae
- link r_clav: geometry collision mesh filename=package://atlas_description/meshes_unplugged/r_clav.dae; visual mesh filename=package://atlas_description/meshes_unplugged/r_clav.dae
- link r_foot: geometry collision mesh filename=package://atlas_description/meshes_unplugged/r_foot.dae; visual mesh filename=package://atlas_description/meshes_unplugged/r_foot.dae
- link r_hand: geometry 
- link r_larm: geometry collision mesh filename=package://atlas_description/meshes_unplugged/r_larm.dae; visual mesh filename=package://atlas_description/meshes_unplugged/r_larm.dae
- link r_lfarm: geometry collision mesh filename=package://atlas_description/meshes_unplugged/r_hand.dae; visual mesh filename=package://atlas_description/meshes_unplugged/r_hand.dae
- link r_lglut: geometry collision mesh filename=package://atlas_description/meshes_unplugged/r_lglut.dae; visual mesh filename=package://atlas_description/meshes_unplugged/r_lglut.dae
- link r_lleg: geometry collision mesh filename=package://atlas_description/meshes_unplugged/r_lleg.dae; visual mesh filename=package://atlas_description/meshes_unplugged/r_lleg.dae
- link r_scap: geometry collision mesh filename=package://atlas_description/meshes_unplugged/r_scap.dae; visual mesh filename=package://atlas_description/meshes_unplugged/r_scap.dae
- link r_talus: geometry collision mesh filename=package://atlas_description/meshes_unplugged/r_talus.dae; visual mesh filename=package://atlas_description/meshes_unplugged/r_talus.dae
- link r_uarm: geometry collision mesh filename=package://atlas_description/meshes_unplugged/r_uarm.dae; visual mesh filename=package://atlas_description/meshes_unplugged/r_uarm.dae
- link r_ufarm: geometry collision mesh filename=package://atlas_description/meshes_unplugged/r_farm.dae; visual mesh filename=package://atlas_description/meshes_unplugged/r_farm.dae
- link r_uglut: geometry collision mesh filename=package://atlas_description/meshes_unplugged/r_uglut.dae; visual mesh filename=package://atlas_description/meshes_unplugged/r_uglut.dae
- link r_uleg: geometry collision mesh filename=package://atlas_description/meshes_unplugged/r_uleg.dae; visual mesh filename=package://atlas_description/meshes_unplugged/r_uleg.dae
- link utorso: geometry collision mesh filename=package://atlas_description/meshes_unplugged/utorso.dae; visual mesh filename=package://atlas_description/meshes_unplugged/utorso.dae
Joints:
- joint back_bkx: origin xyz=0 0 0.05 rpy=0 -0 0 -> xyz=0 0 0.05 rpy=0 0 0
- joint back_bky: origin xyz=0 0 0.162 rpy=0 -0 0 -> xyz=0 0 0.162 rpy=0 0 0
- joint back_bkz: origin xyz=-0.0125 0 0 rpy=0 -0 0 -> xyz=-0.0125 0 0 rpy=0 0 0
- joint l_arm_elx: origin xyz=0 0.119 0.0092 rpy=0 -0 0 -> xyz=0 0.119 0.0092 rpy=0 0 0
- joint l_arm_ely: origin xyz=0 0.187 -0.016 rpy=0 -0 0 -> xyz=0 0.187 -0.016 rpy=0 0 0
- joint l_arm_shx: origin xyz=0 0.11 -0.245 rpy=0 -0 0 -> xyz=0 0.11 -0.245 rpy=0 0 0
- joint l_arm_shz: origin xyz=0.1406 0.2256 0.4776 rpy=0 -0 0 -> xyz=0.1406 0.2256 0.4776 rpy=0 0 0
- joint l_arm_wrx: origin xyz=0 0 0 rpy=0 -0 0 -> xyz=0 0 0 rpy=0 0 0
- joint l_arm_wry: origin xyz=0 0.29955 -0.00921 rpy=0 -0 0 -> xyz=0 0.29955 -0.00921 rpy=0 0 0
- joint l_arm_wry2: origin xyz=0 0 0 rpy=0 -0 0 -> xyz=0 0 0 rpy=0 0 0
- joint l_leg_akx: origin xyz=0 0 0 rpy=0 -0 0 -> xyz=0 0 0 rpy=0 0 0
- joint l_leg_aky: origin xyz=0 0 -0.422 rpy=0 -0 0 -> xyz=0 0 -0.422 rpy=0 0 0
- joint l_leg_hpx: origin xyz=0 0 0 rpy=0 -0 0 -> xyz=0 0 0 rpy=0 0 0
- joint l_leg_hpy: origin xyz=0.05 0.0225 -0.066 rpy=0 -0 0 -> xyz=0.05 0.0225 -0.066 rpy=0 0 0
- joint l_leg_hpz: origin xyz=0 0.089 0 rpy=0 -0 0 -> xyz=0 0.089 0 rpy=0 0 0
- joint l_leg_kny: origin xyz=-0.05 0 -0.374 rpy=0 -0 0 -> xyz=-0.05 0 -0.374 rpy=0 0 0
- joint neck_ry: origin xyz=${0.2546+0.04} 0 ${0.6215-0.045} rpy=0 -0 0 -> xyz=${0.2546+0.04} 0 ${0.6215-0.045} rpy=0 0 0
- joint r_arm_elx: origin xyz=0 -0.119 0.0092 rpy=0 -0 0 -> xyz=0 -0.119 0.0092 rpy=0 0 0
- joint r_arm_ely: origin xyz=0 -0.187 -0.016 rpy=0 -0 0 -> xyz=0 -0.187 -0.016 rpy=0 0 0
- joint r_arm_shx: origin xyz=0 -0.11 -0.245 rpy=0 -0 0 -> xyz=0 -0.11 -0.245 rpy=0 0 0
- joint r_arm_shz: origin xyz=0.1406 -0.2256 0.4776 rpy=0 -0 0 -> xyz=0.1406 -0.2256 0.4776 rpy=0 0 0
- joint r_arm_wrx: origin xyz=0 0 0 rpy=0 -0 0 -> xyz=0 0 0 rpy=0 0 0
- joint r_arm_wry: origin xyz=0 -0.29955 -0.00921 rpy=0 -0 0 -> xyz=0 -0.29955 -0.00921 rpy=0 0 0
- joint r_arm_wry2: origin xyz=0 0 0 rpy=0 -0 0 -> xyz=0 0 0 rpy=0 0 0
- joint r_leg_akx: origin xyz=0 0 0 rpy=0 -0 0 -> xyz=0 0 0 rpy=0 0 0
- joint r_leg_aky: origin xyz=0 0 -0.422 rpy=0 -0 0 -> xyz=0 0 -0.422 rpy=0 0 0
- joint r_leg_hpx: origin xyz=0 0 0 rpy=0 -0 0 -> xyz=0 0 0 rpy=0 0 0
- joint r_leg_hpy: origin xyz=0.05 -0.0225 -0.066 rpy=0 -0 0 -> xyz=0.05 -0.0225 -0.066 rpy=0 0 0
- joint r_leg_hpz: origin xyz=0 -0.089 0 rpy=0 -0 0 -> xyz=0 -0.089 0 rpy=0 0 0
- joint r_leg_kny: origin xyz=-0.05 0 -0.374 rpy=0 -0 0 -> xyz=-0.05 0 -0.374 rpy=0 0 0

Commit message: Fix multisense offsets

File: atlas_description/urdf/atlas_v5.urdf (robot description, URDF)
Before this commit: robot drc_skeleton, 36 links, 36 joints
Joints:
- joint neck_ry: origin xyz=${0.2546+0.04} 0 ${0.6215-0.045} rpy=0 0 0 -> xyz=0.2546 0 0.6215 rpy=0 0 0

File: atlas_description/urdf/atlas_v5_simple_shapes.urdf (robot description, URDF)
Before this commit: robot drc_skeleton, 34 links, 34 joints
Joints:
- joint neck_ry: origin xyz=${0.2546+0.04} 0 ${0.6215-0.045} rpy=0 0 0 -> xyz=0.2546 0 0.6215 rpy=0 0 0
