Commit message: Updated v4_no_wry2

File: atlas_description/urdf/atlas_v4_no_wry2_simple_shapes.urdf (robot description, URDF)
Before this commit: robot drc_skeleton, 34 links, 34 joints
Links:
- link utorso: geometry collision box size=0.2 0.25 0.01; collision box size=0.500175 0.35 0.5

Commit message: Update v4 utorse com, update mass in v4_no_wry2

File: atlas_description/urdf/atlas_v4_no_wry2_simple_shapes.urdf (robot description, URDF)
Before this commit: robot drc_skeleton, 34 links, 34 joints
Links:
- removed link rear_situational_awareness_camera_link
- removed link rear_situational_awareness_camera_optical_frame
- link l_clav: mass 3.45 -> 4.466
- link l_foot: mass 2.05 -> 2.41
- link l_larm: mass 2.509 -> 3.248
- link l_lglut: mass 0.866 -> 0.898
- link l_lleg: mass 5.479 -> 4.515
- link l_scap: mass 3.012 -> 3.899
- link l_uarm: mass 3.388 -> 4.386
- link l_ufarm: mass 3.388 -> 4.386
- link l_uglut: mass 0.648 -> 1.959
- link l_uleg: mass 9.209 -> 8.204
- link ltorso: mass 2.409 -> 2.270
- link mtorso: mass 0.69 -> 0.799
- link pelvis: mass 17.882 -> 9.509
- link r_clav: mass 3.45 -> 4.466
- link r_foot: mass 2.05 -> 2.41
- link r_larm: mass 2.509 -> 3.248
- link r_lglut: mass 0.866 -> 0.898
- link r_lleg: mass 5.479 -> 4.515
- link r_scap: mass 3.012 -> 3.899
- link r_uarm: mass 3.388 -> 4.386
- link r_ufarm: mass 3.388 -> 4.386
- link r_uglut: mass 0.648 -> 1.959
- link r_uleg: mass 9.209 -> 8.204
- link utorso: mass 63.73 -> 84.409
Joints:
- removed joint rear_situational_awareness_camera_joint
- removed joint rear_situational_awareness_camera_optical_frame_joint
- joint l_situational_awareness_camera_joint: origin xyz=0.216409 0.121799 0.406759 rpy=-1.57079633 0 1.30899694 -> xyz=0.155 0.121 0.785 rpy=0 0 1.309
- joint r_situational_awareness_camera_joint: origin xyz=0.216409 -0.121799 0.406759 rpy=1.57079633 0 -1.30899694 -> xyz=0.155 -0.121 0.785 rpy=0 0 -1.309

Commit message: Improve atlas simple shapes

File: atlas_description/urdf/atlas_v4_no_wry2_simple_shapes.urdf (robot description, URDF)
Before this commit: robot drc_skeleton, 34 links, 34 joints
Links:
- link l_lglut: geometry collision box size=0.125 0.05 0.08; collision cylinder length=0.060306 radius=0.02009687
- link l_uglut: geometry collision box size=0.05 0.1 0.1; collision cylinder length=0.080842 radius=0.019841
- link r_lglut: geometry collision box size=0.125 0.05 0.08; collision cylinder length=0.060306 radius=0.02009687
- link r_uglut: geometry collision box size=0.05 0.1 0.1; collision cylinder length=0.080842 radius=0.019841
- link utorso: geometry collision box size=0.13 0.50 0.10; collision box size=0.2 0.18 0.10

File: atlas_description/urdf/atlas_v4_simple_shapes.urdf (robot description, URDF)
Before this commit: robot drc_skeleton, 34 links, 34 joints
Links:
- link l_lglut: geometry collision box size=0.125 0.05 0.08; collision cylinder length=0.060306 radius=0.02009687
- link l_uglut: geometry collision box size=0.05 0.1 0.1; collision cylinder length=0.080842 radius=0.019841
- link r_lglut: geometry collision box size=0.125 0.05 0.08; collision cylinder length=0.060306 radius=0.02009687
- link r_uglut: geometry collision box size=0.05 0.1 0.1; collision cylinder length=0.080842 radius=0.019841
- link utorso: geometry collision box size=0.13 0.50 0.10; collision box size=0.2 0.18 0.10

File: atlas_description/urdf/atlas_v5_simple_shapes.urdf (robot description, URDF)
Before this commit: robot drc_skeleton, 34 links, 34 joints
Links:
- link l_lglut: geometry collision box size=0.0975 0.069 0.103; collision box size=0.125 0.05 0.08
- link l_uglut: geometry collision box size=0.05 0.1 0.1; collision cylinder length=0.080842 radius=0.019841
- link r_lglut: geometry collision box size=0.0975 0.069 0.103; collision box size=0.125 0.05 0.08
- link r_uglut: geometry collision box size=0.05 0.1 0.1; collision cylinder length=0.080842 radius=0.019841
- link utorso: geometry collision box size=0.13 0.50 0.10; collision box size=0.2 0.18 0.10

Commit message: merge drcsim_4.2

File: atlas_description/urdf/atlas_v4_no_wry2_simple_shapes.urdf (robot description, URDF)
Before this commit: robot drc_skeleton, 34 links, 34 joints
Links:
- removed link rear_situational_awareness_camera_link
- removed link rear_situational_awareness_camera_optical_frame
- link l_clav: mass 3.45 -> 4.466
- link l_foot: mass 2.05 -> 2.41
- link l_larm: mass 2.509 -> 3.248
- link l_lglut: mass 0.866 -> 0.898
- link l_lleg: mass 5.479 -> 4.515
- link l_scap: mass 3.012 -> 3.899
- link l_uarm: mass 3.388 -> 4.386
- link l_ufarm: mass 3.388 -> 4.386
- link l_uglut: mass 0.648 -> 1.959
- link l_uleg: mass 9.209 -> 8.204
- link ltorso: mass 2.409 -> 2.270
- link mtorso: mass 0.69 -> 0.799
- link pelvis: mass 17.882 -> 9.509
- link r_clav: mass 3.45 -> 4.466
- link r_foot: mass 2.05 -> 2.41
- link r_larm: mass 2.509 -> 3.248
- link r_lglut: mass 0.866 -> 0.898
- link r_lleg: mass 5.479 -> 4.515
- link r_scap: mass 3.012 -> 3.899
- link r_uarm: mass 3.388 -> 4.386
- link r_ufarm: mass 3.388 -> 4.386
- link r_uglut: mass 0.648 -> 1.959
- link r_uleg: mass 9.209 -> 8.204
- link utorso: mass 63.73 -> 84.409
Joints:
- removed joint rear_situational_awareness_camera_joint
- removed joint rear_situational_awareness_camera_optical_frame_joint
- joint l_situational_awareness_camera_joint: origin xyz=0.216409 0.121799 0.406759 rpy=-1.57079633 0 1.30899694 -> xyz=0.155 0.121 0.785 rpy=0 0 1.309
- joint r_situational_awareness_camera_joint: origin xyz=0.216409 -0.121799 0.406759 rpy=1.57079633 0 -1.30899694 -> xyz=0.155 -0.121 0.785 rpy=0 0 -1.309

File: atlas_description/urdf/atlas_v4_simple_shapes.urdf (robot description, URDF)
Before this commit: robot drc_skeleton, 34 links, 34 joints
Links:
- link l_clav: mass 3.45 -> 4.466
- link l_foot: mass 2.05 -> 2.41
- link l_larm: mass 2.509 -> 3.248
- link l_lglut: mass 0.866 -> 0.898
- link l_lleg: mass 5.479 -> 4.515
- link l_scap: mass 3.012 -> 3.899
- link l_uarm: mass 3.388 -> 4.386
- link l_ufarm: mass 3.388 -> 4.386
- link l_uglut: mass 0.648 -> 1.959
- link l_uleg: mass 9.209 -> 8.204
- link ltorso: mass 2.409 -> 2.270
- link mtorso: mass 0.69 -> 0.799
- link pelvis: mass 17.882 -> 9.509
- link r_clav: mass 3.45 -> 4.466
- link r_foot: mass 2.05 -> 2.41
- link r_larm: mass 2.509 -> 3.248
- link r_lglut: mass 0.866 -> 0.898
- link r_lleg: mass 5.479 -> 4.515
- link r_scap: mass 3.012 -> 3.899
- link r_uarm: mass 3.388 -> 4.386
- link r_ufarm: mass 3.388 -> 4.386
- link r_uglut: mass 0.648 -> 1.959
- link r_uleg: mass 9.209 -> 8.204
- link utorso: mass 63.73 -> 84.409

File: atlas_description/urdf/atlas_v5_simple_shapes.urdf (robot description, URDF)
Before this commit: robot drc_skeleton, 34 links, 34 joints
Links:
- link l_clav: mass 3.45 -> 4.466
- link l_foot: mass 2.05 -> 2.410
- link l_larm: mass 2.509 -> 3.248
- link l_lglut: mass 0.866 -> 0.898
- link l_lleg: mass 5.479 -> 4.515
- link l_scap: mass 3.012 -> 3.899
- link l_uarm: mass 3.388 -> 4.386
- link l_uglut: mass 0.648 -> 1.959
- link l_uleg: mass 9.209 -> 8.204
- link ltorso: mass 2.409 -> 2.270
- link mtorso: mass 0.69 -> 0.799
- link pelvis: mass 17.882 -> 9.509
- link r_clav: mass 3.45 -> 4.466
- link r_foot: mass 2.05 -> 2.41
- link r_larm: mass 2.509 -> 3.248
- link r_lglut: mass 0.866 -> 0.898
- link r_lleg: mass 5.479 -> 4.515
- link r_scap: mass 3.012 -> 3.899
- link r_uarm: mass 3.388 -> 4.386
- link r_uglut: mass 0.648 -> 1.959
- link r_uleg: mass 9.209 -> 8.204
- link utorso: mass 63.73 -> 84.409

Commit message: xacro'ize atlas_v4_no_wry2_simple_shapes.urdf

File: atlas_description/urdf/atlas_v4_no_wry2_simple_shapes.urdf (robot description, URDF)
Before this commit: robot drc_skeleton, 32 links, 32 joints
Links:
- link l_foot: geometry collision box size=0.1 0.08 0.02; collision box size=0.227 0.133887 0.05
- link r_foot: geometry collision box size=0.1 0.08 0.02; collision box size=0.227 0.133887 0.05

Commit message: Apply patch by Twan Koolen to fix left arm kinematics

File: atlas_description/urdf/atlas_v4_no_wry2_simple_shapes.urdf (robot description, URDF)
Before this commit: robot drc_skeleton, 32 links, 32 joints
Links:
- link l_clav: geometry collision box size=0.1 0.07 0.072; collision cylinder length=0.1525 radius=0.0555
- link l_hand: geometry collision box size=0.13 0.09 0.07; collision cylinder length=0.05 radius=0.03
- link l_larm: geometry collision box size=0.135 0.15 0.06; collision cylinder length=0.125 radius=0.045
- link l_scap: geometry collision box size=0.02 0.029 0.018; collision box size=0.028 0.090 0.05
- link l_uarm: geometry collision box size=0.05 0.07 0.15; collision cylinder length=0.11 radius=0.065
- link l_ufarm: geometry collision box size=0.135 0.1 0.045; collision cylinder length=0.125 radius=0.045
Joints:
- joint l_arm_elx: axis 1 0 0 -> -1.0 -0.0 -0.0; origin xyz=0 0.119 0.0092 rpy=0 -0 0 -> xyz=0 -0.119 0.0092 rpy=0 -0 0
- joint l_arm_ely: axis 0 1 0 -> -0.0 -1.0 -0.0; origin xyz=0 0.187 -0.016 rpy=0 -0 0 -> xyz=0 -0.187 -0.016 rpy=0 -0 0
- joint l_arm_shx: axis 1 0 0 -> -1.0 -0.0 -0.0; origin xyz=0 0.11 -0.245 rpy=0 -0 0 -> xyz=0 -0.11 -0.245 rpy=0 -0 0
- joint l_arm_shz: origin xyz=0.1406 0.2256 0.4776 rpy=0 -0 0 -> xyz=0.1406 0.2256 0.4776 rpy=0 0 3.14159265359
- joint l_arm_wrx: origin xyz=0 0.119 0.0092 rpy=0 -0 0 -> xyz=0 -0.119 0.0092 rpy=0 -0 0
- joint l_arm_wry: axis 0 1 0 -> -0.0 -1.0 -0.0; origin xyz=0 0.187 -0.0092 rpy=0 -0 0 -> xyz=0 -0.187 -0.0092 rpy=0 3.14159265359 0
