Commit message: try to use meshes_v4

File: atlas_description/urdf/atlas_v5_simple_shapes.urdf (robot description, URDF)
Before this commit: robot drc_skeleton, 36 links, 36 joints
Links:
- link l_clav: geometry collision mesh filename=package://atlas_description/meshes_v3/l_clav.stl scale=1 1 1; visual mesh filename=package://atlas_description/meshes_v4/l_clav.dae scale=1 1 1
- link l_foot: geometry collision mesh filename=package://atlas_description/meshes_v3/l_foot.stl scale=1 1 1; visual mesh filename=package://atlas_description/meshes_v4/l_foot.dae scale=1 1 1
- link l_hand: geometry collision mesh filename=package://atlas_description/meshes_v3/l_hand.stl scale=1 1 1; visual mesh filename=package://atlas_description/meshes_v4/l_hand.dae scale=1 1 1
- link l_larm: geometry collision mesh filename=package://atlas_description/meshes_v3/l_larm.stl scale=1 1 1; visual mesh filename=package://atlas_description/meshes_v4/l_larm.dae scale=1 1 1
- link l_lglut: geometry collision mesh filename=package://atlas_description/meshes_v3/l_lglut.stl scale=1 1 1; visual mesh filename=package://atlas_description/meshes_v4/l_lglut.dae scale=1 1 1
- link l_lleg: geometry collision mesh filename=package://atlas_description/meshes_v3/l_lleg.stl scale=1 1 1; visual mesh filename=package://atlas_description/meshes_v4/l_lleg.dae scale=1 1 1
- link l_scap: geometry collision mesh filename=package://atlas_description/meshes_v3/l_scap.stl scale=1 1 1; visual mesh filename=package://atlas_description/meshes_v4/l_scap.dae scale=1 1 1
- link l_talus: geometry collision mesh filename=package://atlas_description/meshes_v3/l_talus.stl scale=1 1 1; visual mesh filename=package://atlas_description/meshes_v4/l_talus.dae scale=1 1 1
- link l_uarm: geometry collision mesh filename=package://atlas_description/meshes_v3/l_uarm.stl scale=1 1 1; visual mesh filename=package://atlas_description/meshes_v4/l_uarm.dae scale=1 1 1
- link l_uglut: geometry collision mesh filename=package://atlas_description/meshes_v3/l_uglut.stl scale=1 1 1; visual mesh filename=package://atlas_description/meshes_v4/l_uglut.dae scale=1 1 1
- link l_uleg: geometry collision mesh filename=package://atlas_description/meshes_v3/l_uleg.stl scale=1 1 1; visual mesh filename=package://atlas_description/meshes_v4/l_uleg.dae scale=1 1 1
- link ltorso: geometry collision mesh filename=package://atlas_description/meshes_v3/ltorso.stl scale=1 1 1; visual mesh filename=package://atlas_description/meshes_v4/ltorso.dae scale=1 1 1
- link mtorso: geometry collision mesh filename=package://atlas_description/meshes_v3/mtorso.stl scale=1 1 1; visual mesh filename=package://atlas_description/meshes_v4/mtorso.dae scale=1 1 1
- link pelvis: geometry collision mesh filename=package://atlas_description/meshes_v3/pelvis.stl scale=1 1 1; visual mesh filename=package://atlas_description/meshes_v4/pelvis.dae scale=1 1 1
- link r_clav: geometry collision mesh filename=package://atlas_description/meshes_v3/r_clav.stl scale=1 1 1; visual mesh filename=package://atlas_description/meshes_v4/r_clav.dae scale=1 1 1
- link r_foot: geometry collision mesh filename=package://atlas_description/meshes_v3/r_foot.stl scale=1 1 1; visual mesh filename=package://atlas_description/meshes_v4/r_foot.dae scale=1 1 1
- link r_hand: geometry collision mesh filename=package://atlas_description/meshes_v3/r_hand.stl scale=1 1 1; visual mesh filename=package://atlas_description/meshes_v4/r_hand.dae scale=1 1 1
- link r_lglut: geometry collision mesh filename=package://atlas_description/meshes_v3/r_lglut.stl scale=1 1 1; visual mesh filename=package://atlas_description/meshes_v4/r_lglut.dae scale=1 1 1
- link r_lleg: geometry collision mesh filename=package://atlas_description/meshes_v3/r_lleg.stl scale=1 1 1; visual mesh filename=package://atlas_description/meshes_v4/r_lleg.dae scale=1 1 1
- link r_scap: geometry collision mesh filename=package://atlas_description/meshes_v3/r_scap.stl scale=1 1 1; visual mesh filename=package://atlas_description/meshes_v4/r_scap.dae scale=1 1 1
- link r_talus: geometry collision mesh filename=package://atlas_description/meshes_v3/r_talus.stl scale=1 1 1; visual mesh filename=package://atlas_description/meshes_v4/r_talus.dae scale=1 1 1
- link r_uarm: geometry collision mesh filename=package://atlas_description/meshes_v3/r_uarm.stl scale=1 1 1; visual mesh filename=package://atlas_description/meshes_v4/r_uarm.dae scale=1 1 1
- link r_uglut: geometry collision mesh filename=package://atlas_description/meshes_v3/r_uglut.stl scale=1 1 1; visual mesh filename=package://atlas_description/meshes_v4/r_uglut.dae scale=1 1 1
- link r_uleg: geometry collision mesh filename=package://atlas_description/meshes_v3/r_uleg.stl scale=1 1 1; visual mesh filename=package://atlas_description/meshes_v4/r_uleg.dae scale=1 1 1
- link utorso: geometry collision mesh filename=package://atlas_description/meshes_v3/utorso.stl scale=1 1 1; collision mesh filename=package://atlas_description/meshes_v3/utorso_pack.stl scale=1 1 1

Commit message: Start working on the new arm collisions.

File: atlas_description/urdf/atlas_v5_simple_shapes.urdf (robot description, URDF)
Before this commit: robot drc_skeleton, 36 links, 36 joints
Links:
- link r_hand: geometry collision cylinder length=0.02 radius=0.031; collision cylinder length=0.03 radius=0.048

Commit message: updated torso

File: atlas_description/urdf/atlas_v5_simple_shapes.urdf (robot description, URDF)
Before this commit: robot drc_skeleton, 36 links, 36 joints
Links:
- link utorso: geometry collision box size=0.2 0.25 0.01; collision box size=0.456306 0.341719 0.12

Commit message: Removed connecter shapes

File: atlas_description/urdf/atlas_v5_simple_shapes.urdf (robot description, URDF)
Before this commit: robot drc_skeleton, 36 links, 36 joints
Links:
- link l_hand: geometry collision box size=0.14 0.09 0.06; collision cylinder length=0.03 radius=0.031
- link r_hand: geometry collision box size=0.14 0.09 0.06; collision cylinder length=0.03 radius=0.031

Commit message: Added missing collision shapes for glut

File: atlas_description/urdf/atlas_v5_simple_shapes.urdf (robot description, URDF)
Before this commit: robot drc_skeleton, 36 links, 36 joints
Links:
- link l_lglut: geometry collision box size=0.0975 0.069 0.103; collision cylinder length=0.060306 radius=0.02009687
- link r_lglut: geometry collision box size=0.0975 0.069 0.103; collision cylinder length=0.060306 radius=0.02009687

Commit message: New collission shapes for Atlas V5.

File: atlas_description/urdf/atlas_v5_simple_shapes.urdf (robot description, URDF)
Before this commit: robot drc_skeleton, 36 links, 36 joints
Links:
- link l_clav: geometry collision box size=0.02 0.029 0.015; collision box size=0.028 0.090 0.05
- link l_hand: geometry collision cylinder length=0.015 radius=0.045; collision cylinder length=0.015 radius=0.052
- link l_larm: geometry collision box size=0.025 0.06 0.06; collision box size=0.025 0.155 0.07
- link l_lfarm: geometry 
- link l_scap: geometry collision box size=0.16 0.17 0.08; collision cylinder length=0.105 radius=0.057
- link l_uarm: geometry collision box size=0.05 0.07 0.15; collision cylinder length=0.11 radius=0.065
- link l_ufarm: geometry collision box size=0.08 0.09 0.11; collision cylinder length=0.1 radius=0.053
- link r_clav: geometry collision box size=0.02 0.029 0.015; collision box size=0.028 0.090 0.05
- link r_hand: geometry collision cylinder length=0.015 radius=0.045; collision cylinder length=0.015 radius=0.052
- link r_larm: geometry collision box size=0.025 0.06 0.06; collision box size=0.025 0.155 0.07
- link r_lfarm: geometry 
- link r_scap: geometry collision box size=0.16 0.17 0.08; collision cylinder length=0.105 radius=0.057
- link r_uarm: geometry collision box size=0.05 0.07 0.15; collision cylinder length=0.11 radius=0.065
- link r_ufarm: geometry collision box size=0.08 0.09 0.11; collision cylinder length=0.1 radius=0.053

Commit message: Fix collision shape.

File: atlas_description/urdf/atlas_v5_simple_shapes.urdf (robot description, URDF)
Before this commit: robot drc_skeleton, 36 links, 36 joints
Links:
- link r_clav: geometry collision box size=0.028 0.090 0.05; collision box size=0.1 0.07 0.072
- link r_scap: geometry collision box size=0.02 0.029 0.018; collision box size=0.16 0.17 0.08

Commit message: Fix left arm collision shape.

File: atlas_description/urdf/atlas_v5_simple_shapes.urdf (robot description, URDF)
Before this commit: robot drc_skeleton, 36 links, 36 joints
Links:
- link l_clav: geometry collision box size=0.028 0.090 0.05; collision box size=0.1 0.07 0.072
- link l_scap: geometry collision box size=0.02 0.029 0.018; collision box size=0.16 0.17 0.08

Commit message: Tweaking arm collision shapes.

File: atlas_description/urdf/atlas_v5_simple_shapes.urdf (robot description, URDF)
Before this commit: robot drc_skeleton, 36 links, 36 joints
Links:
- link l_clav: geometry collision box size=0.1 0.07 0.072; collision cylinder length=0.1525 radius=0.0555
- link l_scap: geometry collision box size=0.02 0.029 0.018; collision box size=0.028 0.090 0.05
- link r_clav: geometry collision box size=0.1 0.07 0.072; collision cylinder length=0.1525 radius=0.0555
- link r_scap: geometry collision box size=0.02 0.029 0.018; collision box size=0.028 0.090 0.05

Commit message: Atlas v5 simple shapes

File: atlas_description/urdf/atlas_v5_simple_shapes.urdf (robot description, URDF)
Before this commit: robot drc_skeleton, 36 links, 36 joints
Links:
- link l_clav: geometry collision box size=0.1 0.07 0.072; collision cylinder length=0.1525 radius=0.0555
- link l_foot: geometry collision box size=${0.26-0.0005} ${0.124887+0.009} 0.05; visual mesh filename=package://atlas_description/meshes_unplugged/l_foot.dae
- link l_larm: geometry collision box size=0.025 0.06 0.06; collision box size=0.025 0.155 0.07
- link l_lfarm: geometry collision cylinder length=0.015 radius=0.045; collision cylinder length=0.015 radius=0.052
- link l_lglut: geometry collision box size=0.0975 0.069 0.103; collision cylinder length=0.060306 radius=0.02009687
- link l_lleg: geometry collision cylinder length=0.40 radius=0.07; visual mesh filename=package://atlas_description/meshes_unplugged/l_lleg.dae
- link l_scap: geometry collision box size=0.02 0.029 0.018; collision box size=0.028 0.090 0.05
- link l_talus: geometry collision cylinder length=0.010059 radius=0.010348; collision cylinder length=0.029542 radius=0.010181
- link l_uarm: geometry collision box size=0.05 0.07 0.15; collision cylinder length=0.11 radius=0.065
- link l_ufarm: geometry collision box size=0.08 0.09 0.11; collision cylinder length=0.1 radius=0.053
- link l_uglut: geometry collision cylinder length=0.078396 radius=0.019096; collision cylinder length=0.080842 radius=0.019841
- link l_uleg: geometry collision box size=0.07 0.038 0.14; collision box size=0.07 0.038 0.15
- link ltorso: geometry visual mesh filename=package://atlas_description/meshes_unplugged/ltorso.dae
- link mtorso: geometry collision cylinder length=0.15 radius=0.02; visual mesh filename=package://atlas_description/meshes_unplugged/mtorso.dae
- link pelvis: geometry collision box size=0.1 0.15 0.2; collision cylinder length=0.05 radius=0.16
- link r_clav: geometry collision box size=0.1 0.07 0.072; collision cylinder length=0.1525 radius=0.0555
- link r_foot: geometry collision box size=${0.26-0.0005} ${0.124887+0.009} 0.05; visual mesh filename=package://atlas_description/meshes_unplugged/r_foot.dae
- link r_larm: geometry collision box size=0.025 0.06 0.06; collision box size=0.025 0.155 0.07
- link r_lfarm: geometry collision cylinder length=0.015 radius=0.045; collision cylinder length=0.015 radius=0.052
- link r_lglut: geometry collision box size=0.0975 0.069 0.103; collision cylinder length=0.060306 radius=0.02009687
- link r_lleg: geometry collision cylinder length=0.40 radius=0.07; visual mesh filename=package://atlas_description/meshes_unplugged/r_lleg.dae
- link r_scap: geometry collision box size=0.02 0.029 0.018; collision box size=0.028 0.090 0.05
- link r_talus: geometry collision cylinder length=0.010059 radius=0.010348; collision cylinder length=0.029542 radius=0.010181
- link r_uarm: geometry collision box size=0.05 0.07 0.15; collision cylinder length=0.11 radius=0.065
- link r_ufarm: geometry collision box size=0.08 0.09 0.11; collision cylinder length=0.1 radius=0.053
- link r_uglut: geometry collision cylinder length=0.078396 radius=0.019096; collision cylinder length=0.080842 radius=0.019841
- link r_uleg: geometry collision box size=0.07 0.038 0.14; collision box size=0.07 0.038 0.15
- link utorso: geometry collision box size=0.2 0.25 0.01; collision box size=0.456306 0.341719 0.12

Commit message: Potential Atlas V5 URDF fixes .

File: atlas_description/urdf/atlas_v5_simple_shapes.urdf (robot description, URDF)
Before this commit: robot drc_skeleton, 36 links, 36 joints
Joints:
- joint l_arm_elx: limit lower=0 upper=2.35619 effort=112 velocity=12 -> lower=-2.35619 upper=0 effort=112 velocity=12
- joint r_arm_shz: limit lower=-0.785398 upper=1.5708 effort=87 velocity=12 -> lower=-1.5708 upper=0.785398 effort=87 velocity=12

Commit message: Attempt at fix for atlas_v5_simple_shapes

File: atlas_description/urdf/atlas_v5_simple_shapes.urdf (robot description, URDF)
Before this commit: robot drc_skeleton, 34 links, 34 joints
Links:
- link l_clav: geometry collision box size=0.1 0.07 0.072; collision cylinder length=0.1525 radius=0.0555
- link l_larm: geometry collision box size=0.025 0.06 0.06; collision box size=0.025 0.155 0.07
- link l_scap: geometry collision box size=0.02 0.029 0.018; collision box size=0.028 0.090 0.05
- link l_uarm: geometry collision box size=0.05 0.07 0.15; collision cylinder length=0.11 radius=0.065
Joints:
- joint l_arm_elx: axis 1 0 0 -> -1.0 -0.0 -0.0; origin xyz=0 0.119 0.0092 rpy=0 0 0 -> xyz=0 -0.119 0.0092 rpy=0 0 0
- joint l_arm_ely: axis 0 1 0 -> -0.0 -1.0 -0.0; origin xyz=0 0.187 -0.016 rpy=0 0 0 -> xyz=0 -0.187 -0.016 rpy=0 0 0
- joint l_arm_shx: axis 1 0 0 -> -1 0 0; origin xyz=0 0.11 -0.245 rpy=0 0 0 -> xyz=0 -0.11 -0.245 rpy=0 0 0
- joint l_arm_shz: origin xyz=0.1406 0.2256 0.4776 rpy=0 0 0 -> xyz=0.1406 0.2256 0.4776 rpy=0 0 3.14159265359

Commit message: apply patch from tkoolen that works better than mine

File: atlas_description/urdf/atlas_v5_simple_shapes.urdf (robot description, URDF)
Before this commit: robot drc_skeleton, 34 links, 34 joints
Links:
- link l_clav: geometry collision box size=0.1 0.07 0.072; collision cylinder length=0.1525 radius=0.0555
- link l_larm: geometry collision box size=0.025 0.06 0.06; collision box size=0.025 0.155 0.07
- link l_lfarm: geometry collision cylinder length=0.015 radius=0.045; collision cylinder length=0.015 radius=0.052
- link l_scap: geometry collision box size=0.02 0.029 0.018; collision box size=0.028 0.090 0.05
- link l_uarm: geometry collision box size=0.05 0.07 0.15; collision cylinder length=0.11 radius=0.065
- link l_ufarm: geometry collision box size=0.08 0.09 0.11; collision cylinder length=0.1 radius=0.053
Joints:
- joint l_arm_elx: axis 1 0 0 -> -1.0 -0.0 -0.0; origin xyz=0 0.119 0.0092 rpy=0 0 0 -> xyz=0 -0.119 0.0092 rpy=0 0 0
- joint l_arm_ely: axis 0 1 0 -> -0.0 -1.0 -0.0; origin xyz=0 0.187 -0.016 rpy=0 0 0 -> xyz=0 -0.187 -0.016 rpy=0 0 0
- joint l_arm_shx: axis 1 0 0 -> -1.0 -0.0 -0.0; origin xyz=0 0.11 -0.245 rpy=0 0 0 -> xyz=0 -0.11 -0.245 rpy=0 0 0
- joint l_arm_shz: origin xyz=0.1406 0.2256 0.4776 rpy=0 0 0 -> xyz=0.1406 0.2256 0.4776 rpy=0 0 3.14159265359
- joint l_arm_wry: axis 0 1 0 -> -0.0 -1.0 -0.0; origin xyz=0 0.29955 -0.00921 rpy=0 0 0 -> xyz=0 -0.29955 -0.00921 rpy=0 3.14159265359 0
- joint l_arm_wry2: origin xyz=0 0 0 rpy=0 0 0 -> xyz=0 0 0 rpy=0 3.14159265359 0

Commit message: Update joint limits based on data from Doug Stephen posted in #493

File: atlas_description/urdf/atlas_v5_simple_shapes.urdf (robot description, URDF)
Before this commit: robot drc_skeleton, 34 links, 34 joints
Joints:
- joint l_arm_wrx: limit lower=-1.7628 upper=1.7628 effort=25 velocity=10 -> lower=-1.746 upper=1.767 effort=25 velocity=10
- joint l_arm_wry: limit lower=-3.011 upper=3.011 effort=25 velocity=10 -> lower=-2.999 upper=2.990 effort=25 velocity=10
- joint l_arm_wry2: limit lower=-2.9671 upper=2.9671 effort=25 velocity=10 -> lower=-2.903 upper=2.900 effort=25 velocity=10
- joint r_arm_wrx: limit lower=-1.7628 upper=1.7628 effort=25 velocity=10 -> lower=-1.765 upper=1.762 effort=25 velocity=10
- joint r_arm_wry: limit lower=-3.011 upper=3.011 effort=25 velocity=10 -> lower=-2.979 upper=2.982 effort=25 velocity=10
- joint r_arm_wry2: limit lower=-2.9671 upper=2.9671 effort=25 velocity=10 -> lower=-2.885 upper=2.881 effort=25 velocity=10
