Commit message: Update to simple shapes of atlas v4

File: atlas_description/urdf/atlas_v4_simple_shapes.urdf (robot description, URDF)
Before this commit: robot drc_skeleton, 34 links, 34 joints
Links:
- link l_clav: geometry collision box size=0.045 0.03 0.04; collision box size=0.13 0.15 0.05
- link r_clav: geometry collision box size=0.045 0.03 0.04; collision box size=0.13 0.15 0.05

Commit message: adjust geometry origins

File: atlas_description/urdf/atlas_v4_simple_shapes.urdf (robot description, URDF)
Before this commit: robot drc_skeleton, 34 links, 34 joints
Links:
- link l_clav: geometry collision box size=0.045 0.03 0.04; collision box size=0.13 0.15 0.05
- link l_farm: geometry collision box size=0.135 0.1 0.045; collision cylinder length=0.125 radius=0.045
- link l_foot: geometry collision box size=${0.26-0.0005} ${0.124887+0.009} 0.05; visual mesh filename=package://atlas_description/meshes_v4/l_foot.dae scale=1 1 1
- link l_hand: geometry collision box size=0.13 0.09 0.07; collision cylinder length=0.05 radius=0.03
- link l_larm: geometry collision box size=0.135 0.15 0.06; collision cylinder length=0.125 radius=0.045
- link l_lglut: geometry collision cylinder length=0.060306 radius=0.02009687; collision cylinder length=0.144 radius=0.02
- link l_lleg: geometry collision cylinder length=0.40 radius=0.07; visual mesh filename=package://atlas_description/meshes_v4/l_lleg.dae scale=1 1 1
- link l_scap: geometry collision box size=0.15 0.15 0.06; collision cylinder length=0.125 radius=0.045
- link l_talus: geometry collision cylinder length=0.010059 radius=0.010348; collision cylinder length=0.029542 radius=0.010181
- link l_uarm: geometry collision box size=0.04 0.07 0.13; collision cylinder length=0.125 radius=0.045
- link l_uglut: geometry collision cylinder length=0.078396 radius=0.019096; collision cylinder length=0.080842 radius=0.019841
- link l_uleg: geometry collision box size=0.07 0.038 0.14; collision box size=0.07 0.038 0.15
- link ltorso: geometry visual mesh filename=package://atlas_description/meshes_v4/ltorso.dae scale=1 1 1
- link mtorso: geometry collision cylinder length=0.06 radius=0.017; collision cylinder length=0.08 radius=0.02
- link pelvis: geometry collision box size=0.1 0.15 0.2; collision cylinder length=0.05 radius=0.16
- link r_clav: geometry collision box size=0.045 0.03 0.04; collision box size=0.13 0.15 0.05
- link r_farm: geometry collision box size=0.135 0.1 0.045; collision cylinder length=0.125 radius=0.045
- link r_foot: geometry collision box size=${0.26-0.0005} ${0.124887+0.009} 0.05; visual mesh filename=package://atlas_description/meshes_v4/r_foot.dae scale=1 1 1
- link r_hand: geometry collision box size=0.13 0.09 0.07; collision cylinder length=0.05 radius=0.03
- link r_lglut: geometry collision cylinder length=0.060306 radius=0.02009687; collision cylinder length=0.142 radius=0.02
- link r_lleg: geometry collision cylinder length=0.40 radius=0.07; visual mesh filename=package://atlas_description/meshes_v4/r_lleg.dae scale=1 1 1
- link r_scap: geometry collision box size=0.15 0.15 0.06; collision cylinder length=0.125 radius=0.045
- link r_talus: geometry collision cylinder length=0.010059 radius=0.010348; collision cylinder length=0.029542 radius=0.010181
- link r_uarm: geometry collision box size=0.04 0.07 0.13; collision cylinder length=0.125 radius=0.045
- link r_uglut: geometry collision cylinder length=0.078396 radius=0.019096; collision cylinder length=0.080842 radius=0.019841
- link r_uleg: geometry collision box size=0.07 0.038 0.14; collision box size=0.07 0.038 0.15
- link utorso: geometry collision box size=0.266306 0.223 0.091; collision box size=0.266306 0.381719 0.18
Joints:
- joint neck_ry: origin xyz=0.2546 0 0.6215 rpy=0 -0 0 -> xyz=${0.2546+0.04} 0 ${0.6215-0.045} rpy=0 -0 0

File: atlas_description/urdf/atlas_v5_simple_shapes.urdf (robot description, URDF)
Before this commit: robot drc_skeleton, 36 links, 36 joints
Links:
- link l_hand: geometry collision mesh filename=package://atlas_description/meshes_v4/l_hand.dae scale=1 1 1; visual mesh filename=package://atlas_description/meshes_v4/l_hand.dae scale=1 1 1
- link l_larm: geometry collision mesh filename=package://atlas_description/meshes_v4/l_larm.dae scale=1 1 1; visual mesh filename=package://atlas_description/meshes_v4/l_larm.dae scale=1 1 1
- link l_lleg: geometry collision mesh filename=package://atlas_description/meshes_v4/l_lleg.dae scale=1 1 1; visual mesh filename=package://atlas_description/meshes_v4/l_lleg.dae scale=1 1 1
- link l_scap: geometry collision mesh filename=package://atlas_description/meshes_v4/l_scap.dae scale=1 1 1; visual mesh filename=package://atlas_description/meshes_v4/l_scap.dae scale=1 1 1
- link l_uarm: geometry collision mesh filename=package://atlas_description/meshes_v4/l_uarm.dae scale=1 1 1; visual mesh filename=package://atlas_description/meshes_v4/l_uarm.dae scale=1 1 1
- link l_uglut: geometry collision mesh filename=package://atlas_description/meshes_v4/l_uglut.dae scale=1 1 1; visual mesh filename=package://atlas_description/meshes_v4/l_uglut.dae scale=1 1 1
- link ltorso: geometry collision mesh filename=package://atlas_description/meshes_v4/ltorso.dae scale=1 1 1; visual mesh filename=package://atlas_description/meshes_v4/ltorso.dae scale=1 1 1
- link mtorso: geometry collision mesh filename=package://atlas_description/meshes_v4/mtorso.dae scale=1 1 1; visual mesh filename=package://atlas_description/meshes_v4/mtorso.dae scale=1 1 1
- link pelvis: geometry collision mesh filename=package://atlas_description/meshes_v4/pelvis.dae scale=1 1 1; visual mesh filename=package://atlas_description/meshes_v4/pelvis.dae scale=1 1 1
- link r_hand: geometry collision mesh filename=package://atlas_description/meshes_v4/r_hand.dae scale=1 1 1; visual mesh filename=package://atlas_description/meshes_v4/r_hand.dae scale=1 1 1
- link r_lleg: geometry collision mesh filename=package://atlas_description/meshes_v4/r_lleg.dae scale=1 1 1; visual mesh filename=package://atlas_description/meshes_v4/r_lleg.dae scale=1 1 1
- link r_scap: geometry collision mesh filename=package://atlas_description/meshes_v4/r_scap.dae scale=1 1 1; visual mesh filename=package://atlas_description/meshes_v4/r_scap.dae scale=1 1 1
- link r_uarm: geometry collision mesh filename=package://atlas_description/meshes_v4/r_uarm.dae scale=1 1 1; visual mesh filename=package://atlas_description/meshes_v4/r_uarm.dae scale=1 1 1
- link r_uglut: geometry collision mesh filename=package://atlas_description/meshes_v4/r_uglut.dae scale=1 1 1; visual mesh filename=package://atlas_description/meshes_v4/r_uglut.dae scale=1 1 1
- link utorso: geometry collision mesh filename=package://atlas_description/meshes_v4/utorso.dae scale=1 1 1; visual mesh filename=package://atlas_description/meshes_v4/utorso.dae scale=1 1 1

Commit message: Updated torso simple shapes

File: atlas_description/urdf/atlas_v4_simple_shapes.urdf (robot description, URDF)
Before this commit: robot drc_skeleton, 34 links, 34 joints
Links:
- link mtorso: geometry collision cylinder length=0.15 radius=0.02; visual mesh filename=package://atlas_description/meshes_v4/mtorso.dae scale=1 1 1
- link utorso: geometry collision box size=0.2 0.25 0.01; collision box size=0.266306 0.341719 0.18

Commit message: Merged v3_v4_stand and atlas_v5 branches

File: atlas_description/urdf/atlas_v4_simple_shapes.urdf (robot description, URDF)
Before this commit: robot drc_skeleton, 34 links, 34 joints
Links:
- link l_clav: geometry collision box size=0.02 0.029 0.015; collision box size=0.02 0.19 0.072
- link l_farm: geometry collision box size=0.145 0.115 0.12; collision cylinder length=0.145 radius=0.055
- link l_foot: geometry collision box size=${0.26-0.0005} ${0.124887+0.009} 0.05; visual mesh filename=package://atlas_description/meshes_v4/l_foot.dae scale=1 1 1
- link l_hand: geometry collision box size=0.14 0.09 0.06; collision cylinder length=0.012 radius=0.048
- link l_larm: geometry collision box size=0.025 0.125 0.075; collision cylinder length=0.04 radius=0.041
- link l_lglut: geometry collision cylinder length=0.060306 radius=0.02009687; collision cylinder length=0.144 radius=0.02
- link l_lleg: geometry collision cylinder length=0.40 radius=0.07; visual mesh filename=package://atlas_description/meshes_v4/l_lleg.dae scale=1 1 1
- link l_scap: geometry collision box size=0.15 0.15 0.06; collision cylinder length=0.05 radius=0.04
- link l_talus: geometry collision cylinder length=0.010059 radius=0.010348; collision cylinder length=0.029542 radius=0.010181
- link l_uarm: geometry collision box size=0.05 0.07 0.15; collision cylinder length=0.11 radius=0.065
- link l_uglut: geometry collision cylinder length=0.078396 radius=0.019096; collision cylinder length=0.080842 radius=0.019841
- link l_uleg: geometry collision box size=0.07 0.038 0.14; collision box size=0.07 0.038 0.15
- link ltorso: geometry visual mesh filename=package://atlas_description/meshes_v4/ltorso.dae scale=1 1 1
- link mtorso: geometry collision cylinder length=0.15 radius=0.02; visual mesh filename=package://atlas_description/meshes_v4/mtorso.dae scale=1 1 1
- link pelvis: geometry collision box size=0.1 0.15 0.2; collision cylinder length=0.05 radius=0.16
- link r_clav: geometry collision box size=0.02 0.029 0.015; collision box size=0.02 0.19 0.072
- link r_farm: geometry collision box size=0.145 0.115 0.12; collision cylinder length=0.145 radius=0.055
- link r_foot: geometry collision box size=${0.26-0.0005} ${0.124887+0.009} 0.05; visual mesh filename=package://atlas_description/meshes_v4/r_foot.dae scale=1 1 1
- link r_hand: geometry collision box size=0.14 0.09 0.06; collision cylinder length=0.012 radius=0.048
- link r_larm: geometry collision box size=0.025 0.125 0.075; collision cylinder length=0.04 radius=0.041
- link r_lglut: geometry collision cylinder length=0.060306 radius=0.02009687; collision cylinder length=0.142 radius=0.02
- link r_lleg: geometry collision cylinder length=0.40 radius=0.07; visual mesh filename=package://atlas_description/meshes_v4/r_lleg.dae scale=1 1 1
- link r_scap: geometry collision box size=0.15 0.15 0.06; collision cylinder length=0.05 radius=0.04
- link r_talus: geometry collision cylinder length=0.010059 radius=0.010348; collision cylinder length=0.029542 radius=0.010181
- link r_uarm: geometry collision box size=0.05 0.07 0.15; collision cylinder length=0.11 radius=0.065
- link r_uglut: geometry collision cylinder length=0.078396 radius=0.019096; collision cylinder length=0.080842 radius=0.019841
- link r_uleg: geometry collision box size=0.07 0.038 0.14; collision box size=0.07 0.038 0.15
- link utorso: geometry collision box size=0.2 0.25 0.01; collision box size=0.266306 0.341719 0.18

Commit message: Tweaking the collision shapes of Atlas V4.

File: atlas_description/urdf/atlas_v4_simple_shapes.urdf (robot description, URDF)
Before this commit: robot drc_skeleton, 34 links, 34 joints
Links:
- link l_clav: geometry collision box size=0.1 0.07 0.072; collision cylinder length=0.1525 radius=0.045
- link l_scap: geometry collision box size=0.02 0.029 0.015; collision box size=0.02 0.19 0.072
- link r_clav: geometry collision box size=0.1 0.07 0.072; collision cylinder length=0.1525 radius=0.045
- link r_scap: geometry collision box size=0.02 0.029 0.015; collision box size=0.02 0.19 0.072

Commit message: Integrated latest atlast models

File: atlas_description/urdf/atlas_v4_simple_shapes.urdf (robot description, URDF)
Before this commit: robot drc_skeleton, 34 links, 34 joints
Links:
- removed link l_farm
- removed link r_farm
- added link l_lfarm, mass 2.509; collision box size=0.14 0.09 0.06; collision cylinder length=0.012 radius=0.048
- added link l_ufarm, mass 3.388; collision box size=0.145 0.115 0.12; collision cylinder length=0.145 radius=0.055
- added link r_lfarm, mass 2.509; collision box size=0.14 0.09 0.06; collision cylinder length=0.012 radius=0.048
- added link r_ufarm, mass 3.388; collision box size=0.145 0.115 0.12; collision cylinder length=0.145 radius=0.055
- link l_clav: geometry collision box size=0.1 0.07 0.072; collision cylinder length=0.1525 radius=0.045
- link l_foot: geometry collision box size=${0.26-0.0005} ${0.124887+0.009} 0.05; visual mesh filename=package://atlas_description/meshes_unplugged/l_foot.dae scale=1 1 1
- link l_hand: mass 2.509 -> 0.1; geometry 
- link l_larm: geometry collision box size=0.025 0.125 0.075; collision cylinder length=0.04 radius=0.041
- link l_lglut: geometry collision cylinder length=0.060306 radius=0.02009687; collision cylinder length=0.144 radius=0.02
- link l_lleg: geometry collision cylinder length=0.40 radius=0.07; visual mesh filename=package://atlas_description/meshes_unplugged/l_lleg.dae scale=1 1 1
- link l_scap: geometry collision box size=0.02 0.029 0.015; collision box size=0.02 0.19 0.072
- link l_talus: geometry collision cylinder length=0.010059 radius=0.010348; collision cylinder length=0.029542 radius=0.010181
- link l_uarm: geometry collision box size=0.05 0.07 0.15; collision cylinder length=0.11 radius=0.065
- link l_uglut: geometry collision cylinder length=0.078396 radius=0.019096; collision cylinder length=0.080842 radius=0.019841
- link l_uleg: geometry collision box size=0.07 0.038 0.14; collision box size=0.07 0.038 0.15
- link ltorso: geometry visual mesh filename=package://atlas_description/meshes_unplugged/ltorso.dae scale=1 1 1
- link mtorso: geometry collision cylinder length=0.15 radius=0.02; visual mesh filename=package://atlas_description/meshes_unplugged/mtorso.dae scale=1 1 1
- link pelvis: geometry collision box size=0.1 0.15 0.2; collision cylinder length=0.05 radius=0.16
- link r_clav: geometry collision box size=0.1 0.07 0.072; collision cylinder length=0.1525 radius=0.045
- link r_foot: geometry collision box size=${0.26-0.0005} ${0.124887+0.009} 0.05; visual mesh filename=package://atlas_description/meshes_unplugged/r_foot.dae scale=1 1 1
- link r_hand: mass 2.509 -> 0.1; geometry 
- link r_lglut: geometry collision cylinder length=0.060306 radius=0.02009687; collision cylinder length=0.142 radius=0.02
- link r_lleg: geometry collision cylinder length=0.40 radius=0.07; visual mesh filename=package://atlas_description/meshes_unplugged/r_lleg.dae scale=1 1 1
- link r_scap: geometry collision box size=0.02 0.029 0.015; collision box size=0.02 0.19 0.072
- link r_talus: geometry collision cylinder length=0.010059 radius=0.010348; collision cylinder length=0.029542 radius=0.010181
- link r_uarm: geometry collision box size=0.05 0.07 0.15; collision cylinder length=0.11 radius=0.065
- link r_uglut: geometry collision cylinder length=0.078396 radius=0.019096; collision cylinder length=0.080842 radius=0.019841
- link r_uleg: geometry collision box size=0.07 0.038 0.14; collision box size=0.07 0.038 0.15
- link utorso: geometry collision box size=0.2 0.25 0.01; collision box size=0.266306 0.341719 0.18
Joints:
- added joint l_arm_wry2: type revolute, parent l_lfarm, child l_hand, origin xyz=0 0 0 rpy=0 0 0, axis 0 1 0, limit lower=-0.001 upper=0.001 effort=5 velocity=1
- added joint r_arm_wry2: type revolute, parent r_lfarm, child r_hand, origin xyz=0 0 0 rpy=0 0 0, axis 0 1 0, limit lower=-0.001 upper=0.001 effort=5 velocity=1
- joint l_arm_ely: origin xyz=0 0.187 0.016 rpy=0 -0 0 -> xyz=0 0.187 -0.016 rpy=0 -0 0
- joint l_arm_shx: origin xyz=0 0.0981 -0.2511 rpy=0 -0 0 -> xyz=0 0.11 -0.245 rpy=0 -0 0
- joint l_arm_shz: origin xyz=0.1406 0.2036 0.4776 rpy=0 -0 0 -> xyz=0.1406 0.2256 0.4776 rpy=0 -0 0
- joint l_arm_wrx: child l_hand -> l_lfarm; parent l_farm -> l_ufarm
- joint l_arm_wry: child l_farm -> l_ufarm
- joint r_arm_ely: origin xyz=0 -0.187 0.016 rpy=0 -0 0 -> xyz=0 -0.187 -0.016 rpy=0 -0 0
- joint r_arm_shx: origin xyz=0 -0.0981 -0.2511 rpy=0 -0 0 -> xyz=0 -0.11 -0.245 rpy=0 -0 0
- joint r_arm_shz: origin xyz=0.1406 -0.2036 0.4776 rpy=0 -0 0 -> xyz=0.1406 -0.2256 0.4776 rpy=0 -0 0
- joint r_arm_wrx: child r_hand -> r_lfarm; parent r_farm -> r_ufarm
- joint r_arm_wry: child r_farm -> r_ufarm

File: atlas_description/urdf/atlas_v5_simple_shapes.urdf (robot description, URDF)
Before this commit: robot drc_skeleton, 36 links, 36 joints
Links:
- link l_hand: mass 0.53 -> 0.5839
- link l_lfarm: mass 2.65 -> 0.648
- link l_ufarm: mass 2.12 -> 2.4798
- link r_hand: mass 0.53 -> 0.5839
- link r_lfarm: mass 2.65 -> 0.648
- link r_ufarm: mass 2.12 -> 2.4798

Commit message: Update collision shapes

File: atlas_description/urdf/atlas_v4_simple_shapes.urdf (robot description, URDF)
Before this commit: robot drc_skeleton, 36 links, 36 joints
Links:
- link l_scap: geometry collision box size=0.02 0.029 0.018; collision box size=0.028 0.090 0.05
- link r_scap: geometry collision box size=0.02 0.029 0.018; collision box size=0.028 0.090 0.05

Commit message: stable seating pos

File: atlas_description/urdf/atlas_v4_simple_shapes.urdf (robot description, URDF)
Before this commit: robot drc_skeleton, 36 links, 36 joints
Links:
- link l_uleg: geometry collision box size=0.07 0.038 0.14; collision box size=0.07 0.038 0.15
- link r_uleg: geometry collision box size=0.07 0.038 0.14; collision box size=0.07 0.038 0.15

File: atlas_description/urdf/atlas_v5_simple_shapes.urdf (robot description, URDF)
Before this commit: robot drc_skeleton, 36 links, 36 joints
Links:
- link l_uleg: geometry collision box size=0.07 0.038 0.14; collision box size=0.07 0.038 0.15
- link r_uleg: geometry collision box size=0.07 0.038 0.14; collision box size=0.07 0.038 0.15

Commit message: update v4 collisions

File: atlas_description/urdf/atlas_v4_simple_shapes.urdf (robot description, URDF)
Before this commit: robot drc_skeleton, 36 links, 36 joints
Links:
- link l_clav: geometry collision box size=0.1 0.07 0.072; collision cylinder length=0.1525 radius=0.0555
- link l_larm: geometry collision box size=0.135 0.15 0.06; collision cylinder length=0.125 radius=0.045
- link l_lfarm: geometry collision box size=0.13 0.09 0.07; collision cylinder length=0.05 radius=0.03
- link l_ufarm: geometry collision box size=0.135 0.1 0.045; collision cylinder length=0.125 radius=0.045
- link l_uleg: geometry collision box size=0.07 0.038 0.14; collision box size=0.07 0.038 0.15
- link r_clav: geometry collision box size=0.1 0.07 0.072; collision cylinder length=0.1525 radius=0.0555
- link r_larm: geometry collision box size=0.135 0.15 0.06; collision cylinder length=0.125 radius=0.045
- link r_lfarm: geometry collision box size=0.13 0.09 0.07; collision cylinder length=0.05 radius=0.03
- link r_ufarm: geometry collision box size=0.135 0.1 0.045; collision cylinder length=0.125 radius=0.045
- link r_uleg: geometry collision box size=0.07 0.038 0.14; collision box size=0.07 0.038 0.15
- link utorso: geometry collision box size=0.2 0.25 0.01; collision box size=0.456306 0.341719 0.12
