Commit message: 4.2 -> default

File: atlas_description/urdf/atlas_v4_simple_shapes.urdf (robot description, URDF)
Before this commit: robot drc_skeleton, 34 links, 34 joints
Links:
- removed link l_farm
- removed link r_farm
- added link l_lfarm, mass 2.509; collision box size=0.13 0.09 0.07; collision cylinder length=0.05 radius=0.03
- added link l_ufarm, mass 3.388; collision box size=0.135 0.1 0.045; collision cylinder length=0.125 radius=0.045
- added link r_lfarm, mass 2.509; collision box size=0.13 0.09 0.07; collision cylinder length=0.05 radius=0.03
- added link r_ufarm, mass 3.388; collision box size=0.135 0.1 0.045; collision cylinder length=0.125 radius=0.045
- link l_clav: geometry collision box size=0.1 0.07 0.072; collision cylinder length=0.1525 radius=0.0555
- link l_foot: geometry collision box size=${0.26-0.033} ${0.124887+0.009} 0.05; collision box size=0.1 ${0.08} 0.02
- link l_hand: mass 2.509 -> 0.1; geometry 
- link l_lglut: geometry collision cylinder length=0.060306 radius=0.02009687; collision cylinder length=0.144 radius=0.02
- link l_lleg: geometry collision cylinder length=0.40 radius=0.07; visual mesh filename=package://atlas_description/meshes_unplugged/l_lleg.dae scale=1 1 1
- link l_scap: geometry collision box size=0.02 0.029 0.018; collision box size=0.028 0.090 0.05
- link l_talus: geometry collision cylinder length=0.010059 radius=0.010348; collision cylinder length=0.029542 radius=0.010181
- link l_uarm: geometry collision box size=0.05 0.07 0.15; collision cylinder length=0.11 radius=0.065
- link l_uglut: geometry collision cylinder length=0.078396 radius=0.019096; collision cylinder length=0.080842 radius=0.019841
- link l_uleg: geometry collision box size=0.07 0.038 0.14; collision box size=0.07 0.038 0.15
- link ltorso: geometry visual mesh filename=package://atlas_description/meshes_unplugged/ltorso.dae scale=1 1 1
- link mtorso: geometry collision cylinder length=0.15 radius=0.02; visual mesh filename=package://atlas_description/meshes_unplugged/mtorso.dae scale=1 1 1
- link pelvis: geometry collision box size=0.1 0.15 0.2; collision cylinder length=0.05 radius=0.16
- link r_clav: geometry collision box size=0.1 0.07 0.072; collision cylinder length=0.1525 radius=0.0555
- link r_foot: geometry collision box size=${0.26-0.033} ${0.124887+0.009} 0.05; collision box size=0.1 ${0.08} 0.02
- link r_hand: mass 2.509 -> 0.1; geometry 
- link r_lglut: geometry collision cylinder length=0.060306 radius=0.02009687; collision cylinder length=0.142 radius=0.02
- link r_lleg: geometry collision cylinder length=0.40 radius=0.07; visual mesh filename=package://atlas_description/meshes_unplugged/r_lleg.dae scale=1 1 1
- link r_scap: geometry collision box size=0.02 0.029 0.018; collision box size=0.028 0.090 0.05
- link r_talus: geometry collision cylinder length=0.010059 radius=0.010348; collision cylinder length=0.029542 radius=0.010181
- link r_uarm: geometry collision box size=0.05 0.07 0.15; collision cylinder length=0.11 radius=0.065
- link r_uglut: geometry collision cylinder length=0.078396 radius=0.019096; collision cylinder length=0.080842 radius=0.019841
- link r_uleg: geometry collision box size=0.07 0.038 0.14; collision box size=0.07 0.038 0.15
- link utorso: geometry collision box size=0.2 0.25 0.01; collision box size=0.456306 0.341719 0.12
Joints:
- added joint l_arm_wry2: type revolute, parent l_lfarm, child l_hand, origin xyz=0 0 0 rpy=0 0 0, axis 0 1 0, limit lower=-0.001 upper=0.001 effort=5 velocity=1
- added joint r_arm_wry2: type revolute, parent r_lfarm, child r_hand, origin xyz=0 0 0 rpy=0 0 0, axis 0 1 0, limit lower=-0.001 upper=0.001 effort=5 velocity=1
- joint l_arm_ely: origin xyz=0 0.187 0.016 rpy=0 -0 0 -> xyz=0 0.187 -0.016 rpy=0 -0 0
- joint l_arm_shx: origin xyz=0 0.0981 -0.2511 rpy=0 -0 0 -> xyz=0 0.11 -0.245 rpy=0 -0 0
- joint l_arm_shz: origin xyz=0.1406 0.2036 0.4776 rpy=0 -0 0 -> xyz=0.1406 0.2256 0.4776 rpy=0 -0 0
- joint l_arm_wrx: child l_hand -> l_lfarm; parent l_farm -> l_ufarm
- joint l_arm_wry: child l_farm -> l_ufarm
- joint r_arm_ely: origin xyz=0 -0.187 0.016 rpy=0 -0 0 -> xyz=0 -0.187 -0.016 rpy=0 -0 0
- joint r_arm_shx: origin xyz=0 -0.0981 -0.2511 rpy=0 -0 0 -> xyz=0 -0.11 -0.245 rpy=0 -0 0
- joint r_arm_shz: origin xyz=0.1406 -0.2036 0.4776 rpy=0 -0 0 -> xyz=0.1406 -0.2256 0.4776 rpy=0 -0 0
- joint r_arm_wrx: child r_hand -> r_lfarm; parent r_farm -> r_ufarm
- joint r_arm_wry: child r_farm -> r_ufarm

Commit message: updated inertia from issue #487

File: atlas_description/urdf/atlas_v4_simple_shapes.urdf (robot description, URDF)
Before this commit: robot drc_skeleton, 34 links, 34 joints
Links:
- link l_clav: mass 3.45 -> 4.466
- link l_foot: mass 2.05 -> 2.41
- link l_larm: mass 2.509 -> 3.248
- link l_lglut: mass 0.866 -> 0.898
- link l_lleg: mass 5.479 -> 4.515
- link l_scap: mass 3.012 -> 3.899
- link l_uarm: mass 3.388 -> 4.386
- link l_ufarm: mass 3.388 -> 4.386
- link l_uglut: mass 0.648 -> 1.959
- link l_uleg: mass 9.209 -> 8.204
- link ltorso: mass 2.409 -> 2.270
- link mtorso: mass 0.69 -> 0.799
- link pelvis: mass 17.882 -> 9.509
- link r_clav: mass 3.45 -> 4.466
- link r_foot: mass 2.05 -> 2.41
- link r_larm: mass 2.509 -> 3.248
- link r_lglut: mass 0.866 -> 0.898
- link r_lleg: mass 5.479 -> 4.515
- link r_scap: mass 3.012 -> 3.899
- link r_uarm: mass 3.388 -> 4.386
- link r_ufarm: mass 3.388 -> 4.386
- link r_uglut: mass 0.648 -> 1.959
- link r_uleg: mass 9.209 -> 8.204
- link utorso: mass 63.73 -> 84.409

File: atlas_description/urdf/atlas_v5_simple_shapes.urdf (robot description, URDF)
Before this commit: robot drc_skeleton, 34 links, 34 joints
Links:
- link l_clav: mass 3.45 -> 4.466
- link l_foot: mass 2.05 -> 2.410
- link l_larm: mass 2.509 -> 3.248
- link l_lglut: mass 0.866 -> 0.898
- link l_lleg: mass 5.479 -> 4.515
- link l_scap: mass 3.012 -> 3.899
- link l_uarm: mass 3.388 -> 4.386
- link l_uglut: mass 0.648 -> 1.959
- link l_uleg: mass 9.209 -> 8.204
- link ltorso: mass 2.409 -> 2.270
- link mtorso: mass 0.69 -> 0.799
- link pelvis: mass 17.882 -> 9.509
- link r_clav: mass 3.45 -> 4.466
- link r_foot: mass 2.05 -> 2.41
- link r_larm: mass 2.509 -> 3.248
- link r_lglut: mass 0.866 -> 0.898
- link r_lleg: mass 5.479 -> 4.515
- link r_scap: mass 3.012 -> 3.899
- link r_uarm: mass 3.388 -> 4.386
- link r_uglut: mass 0.648 -> 1.959
- link r_uleg: mass 9.209 -> 8.204
- link utorso: mass 63.73 -> 84.409

Commit message: Attempt at applying patch from Twan Koolen to atlas_v4_simple_shapes

File: atlas_description/urdf/atlas_v4_simple_shapes.urdf (robot description, URDF)
Before this commit: robot drc_skeleton, 34 links, 34 joints
Links:
- link l_clav: geometry collision box size=0.1 0.07 0.072; collision cylinder length=0.1525 radius=0.0555
- link l_larm: geometry collision box size=0.135 0.15 0.06; collision cylinder length=0.125 radius=0.045
- link l_lfarm: geometry collision box size=0.13 0.09 0.07; collision cylinder length=0.05 radius=0.03
- link l_scap: geometry collision box size=0.02 0.029 0.018; collision box size=0.028 0.090 0.05
- link l_uarm: geometry collision box size=0.05 0.07 0.15; collision cylinder length=0.11 radius=0.065
- link l_ufarm: geometry collision box size=0.135 0.1 0.045; collision cylinder length=0.125 radius=0.045
Joints:
- joint l_arm_elx: axis 1 0 0 -> -1.0 -0.0 -0.0; origin xyz=0 0.119 0.0092 rpy=0 -0 0 -> xyz=0 -0.119 0.0092 rpy=0 -0 0
- joint l_arm_ely: axis 0 1 0 -> -0.0 -1.0 -0.0; origin xyz=0 0.187 -0.016 rpy=0 -0 0 -> xyz=0 -0.187 -0.016 rpy=0 -0 0
- joint l_arm_shx: axis 1 0 0 -> -1.0 -0.0 -0.0; origin xyz=0 0.11 -0.245 rpy=0 -0 0 -> xyz=0 -0.11 -0.245 rpy=0 -0 0
- joint l_arm_shz: origin xyz=0.1406 0.2256 0.4776 rpy=0 -0 0 -> xyz=0.1406 0.2256 0.4776 rpy=0 0 3.14159265359
- joint l_arm_wrx: origin xyz=0 0.119 0.0092 rpy=0 -0 0 -> xyz=0 -0.119 0.0092 rpy=0 -0 0
- joint l_arm_wry: axis 0 1 0 -> -0.0 -1.0 -0.0; origin xyz=0 0.187 -0.0092 rpy=0 -0 0 -> xyz=0 -0.187 -0.0092 rpy=0 3.14159265359 0
- joint l_arm_wry2: origin xyz=0 0 0 rpy=0 0 0 -> xyz=0 0 0 rpy=0 3.14159265359 0

Commit message: 4.2 -> default

File: atlas_description/urdf/atlas_v4_simple_shapes.urdf (robot description, URDF)
Before this commit: robot drc_skeleton, 34 links, 34 joints
Links:
- link l_clav: geometry collision box size=0.1 0.07 0.072; collision cylinder length=0.1525 radius=0.0555
- link l_foot: geometry collision box size=0.1 0.08 0.02; collision box size=0.227 0.133887 0.05
- link l_larm: geometry collision box size=0.135 0.15 0.06; collision cylinder length=0.125 radius=0.045
- link l_lfarm: geometry collision box size=0.13 0.09 0.07; collision cylinder length=0.05 radius=0.03
- link l_scap: geometry collision box size=0.02 0.029 0.018; collision box size=0.028 0.090 0.05
- link l_uarm: geometry collision box size=0.05 0.07 0.15; collision cylinder length=0.11 radius=0.065
- link l_ufarm: geometry collision box size=0.135 0.1 0.045; collision cylinder length=0.125 radius=0.045
- link r_foot: geometry collision box size=0.1 0.08 0.02; collision box size=0.227 0.133887 0.05
Joints:
- joint l_arm_elx: axis 1 0 0 -> -1.0 -0.0 -0.0; origin xyz=0 0.119 0.0092 rpy=0 -0 0 -> xyz=0 -0.119 0.0092 rpy=0 -0 0
- joint l_arm_ely: axis 0 1 0 -> -0.0 -1.0 -0.0; origin xyz=0 0.187 -0.016 rpy=0 -0 0 -> xyz=0 -0.187 -0.016 rpy=0 -0 0
- joint l_arm_shx: axis 1 0 0 -> -1.0 -0.0 -0.0; origin xyz=0 0.11 -0.245 rpy=0 -0 0 -> xyz=0 -0.11 -0.245 rpy=0 -0 0
- joint l_arm_shz: origin xyz=0.1406 0.2256 0.4776 rpy=0 -0 0 -> xyz=0.1406 0.2256 0.4776 rpy=0 0 3.14159265359
- joint l_arm_wrx: origin xyz=0 0.119 0.0092 rpy=0 -0 0 -> xyz=0 -0.119 0.0092 rpy=0 -0 0
- joint l_arm_wry: axis 0 1 0 -> -0.0 -1.0 -0.0; origin xyz=0 0.187 -0.0092 rpy=0 -0 0 -> xyz=0 -0.187 -0.0092 rpy=0 3.14159265359 0
- joint l_arm_wry2: origin xyz=0 0 0 rpy=0 0 0 -> xyz=0 0 0 rpy=0 3.14159265359 0
