Commit message: Tweaking robotiq joints.

File: robotiq_hand_description/urdf/robotiq_hand.urdf.xacro (robot description, xacro)
@@ -45,7 +45,7 @@
 			</collision>
 			<inertial>
-        <mass value="0.01"/>
-      	<origin xyz="0 0 0"/>
-      	<inertia ixx="0.000018" ixy="0" ixz="0" iyy="0.000018" iyz="0" izz="0.000018"/>
+        <mass value="0.1"/>
+      	<origin xyz="-0.01 0 0"/>
+      	<inertia ixx="0.000018" ixy="0" ixz="0" iyy="0.000025" iyz="0" izz="0.000025"/>
       </inertial>
 		</link>
@@ -132,20 +132,31 @@
         <safety_controller k_position="100" k_velocity="100" soft_lower_limit="-10.6981" soft_upper_limit="10.6981" />
 		</joint>
-		<!-- WARNING: LIMITS NOT CORRECT -->
-		<joint name="${prefix}joint_2" type="fixed">
+		<gazebo reference="${prefix}joint_1">
+		  <implicitSpringDamper>1</implicitSpringDamper>
+		</gazebo>
+		<!-- WARNING: LIMITS NOT CORRECT -->
+		<joint name="${prefix}joint_2" type="revolute">
 			<parent link="${prefix}link_1"/>
 			<child link="${prefix}link_2"/>
+			<dynamics damping="0.1" friction="0" />
 			<axis xyz="0 0 1"/>
 			<origin rpy="0 0 -0.52" xyz="0.050 -.028 0"/>
 			<limit lower="0" upper="3.1416" effort="100" velocity="100"/>
 		</joint>
-		<!-- WARNING: LIMITS NOT CORRECT -->
-		<joint name="${prefix}joint_3" type="fixed">
+		<gazebo reference="${prefix}joint_2">
+		  <implicitSpringDamper>1</implicitSpringDamper>
+		</gazebo>
+		<!-- WARNING: LIMITS NOT CORRECT -->
+		<joint name="${prefix}joint_3" type="revolute">
 			<parent link="${prefix}link_2"/>
 			<child link="${prefix}link_3"/>
+			<dynamics damping="0.1" friction="0" />
 			<axis xyz="0 0 1"/>
 			<origin rpy="0 0 0.52" xyz="0.039 0 0"/>
 			<limit lower="0" upper="3.1416" effort="100" velocity="100"/>
 		</joint>
+		<gazebo reference="${prefix}joint_3">
+		  <implicitSpringDamper>1</implicitSpringDamper>
+		</gazebo>
 		<!-- end of joint list -->
 	</xacro:macro>
@@ -200,5 +211,5 @@
 		<!-- joint list -->
 		<!-- WARNING: LIMITS NOT CORRECT -->
-		<joint name="${prefix}palm_finger_1_joint" type="fixed">
+		<joint name="${prefix}palm_finger_1_joint" type="revolute">
 			<parent link="${prefix}palm"/>
 			<child link="${prefix}finger_1_link_0"/>
@@ -208,5 +219,5 @@
 		</joint>
 		<!-- WARNING: LIMITS NOT CORRECT -->
-		<joint name="${prefix}palm_finger_2_joint" type="fixed">
+		<joint name="${prefix}palm_finger_2_joint" type="revolute">
 			<parent link="${prefix}palm"/>
 			<child link="${prefix}finger_2_link_0"/>
@@ -215,9 +226,10 @@
 			<limit lower="-0.25" upper="0.16" effort="100" velocity="100"/>
 		</joint>
-		<joint name="${prefix}palm_finger_middle_joint" type="fixed">
+		<joint name="${prefix}palm_finger_middle_joint" type="revolute">
 			<parent link="${prefix}palm"/>
 			<child link="${prefix}finger_middle_link_0"/>
-			<axis xyz="0 0 1"/>
+			<axis xyz="0 1 0"/>
 			<origin rpy="0 0 1.57" xyz="0.0455 0.0214 0"/>
+			<limit lower="-0.25" upper="0.16" effort="100" velocity="100"/>
 		</joint>
 		<!-- end of joint list -->

Commit message: Changing joint limits.

File: robotiq_hand_description/urdf/robotiq_hand.urdf.xacro (robot description, xacro)
@@ -122,5 +122,4 @@
 		<!-- end of link list -->
 		<!-- joint list -->
-		<!-- WARNING: LIMITS NOT CORRECT -->
 		<joint name="${prefix}joint_1" type="revolute">
 			<origin rpy="0 0 0" xyz="0 0 0"/>
@@ -129,11 +128,11 @@
 			<child link="${prefix}link_1"/>
       <dynamics damping="1" friction="0" />
-      <limit effort="20" velocity="2" lower="-1.5" upper="1.5" />
-      <safety_controller k_position="100" k_velocity="100" soft_lower_limit="-10.6981" soft_upper_limit="10.6981" />
+      <!-- Limits: [0deg.-70deg.] -->
+      <limit effort="20" velocity="-1" lower="0" upper="1.2217" />
+      <!--<safety_controller k_position="100" k_velocity="100" soft_lower_limit="-10.6981" soft_upper_limit="10.6981" />-->
 		</joint>
 		<gazebo reference="${prefix}joint_1">
 		  <implicitSpringDamper>1</implicitSpringDamper>
 		</gazebo>
-		<!-- WARNING: LIMITS NOT CORRECT -->
 		<joint name="${prefix}joint_2" type="revolute">
 			<parent link="${prefix}link_1"/>
@@ -142,10 +141,10 @@
 			<axis xyz="0 0 1"/>
 			<origin rpy="0 0 -0.52" xyz="0.050 -.028 0"/>
-			<limit lower="0" upper="3.1416" effort="100" velocity="100"/>
+			<!-- Limits: [0deg.,90deg.] -->
+			<limit lower="0" upper="1.5708" effort="20" velocity="-1"/>
 		</joint>
 		<gazebo reference="${prefix}joint_2">
 		  <implicitSpringDamper>1</implicitSpringDamper>
 		</gazebo>
-		<!-- WARNING: LIMITS NOT CORRECT -->
 		<joint name="${prefix}joint_3" type="revolute">
 			<parent link="${prefix}link_2"/>
@@ -153,6 +152,7 @@
 			<dynamics damping="1" friction="0" />
 			<axis xyz="0 0 1"/>
-			<origin rpy="0 0 0.52" xyz="0.039 0 0"/>
-			<limit lower="0" upper="3.1416" effort="100" velocity="100"/>
+  		<origin rpy="0 0 0.52" xyz="0.039 0 0"/>
+	  	<!-- Limits: [-38deg.,60deg.] -->
+			<limit lower="-0.6632" upper="1.0471" effort="20" velocity="-1"/>
 		</joint>
 		<gazebo reference="${prefix}joint_3">
@@ -210,5 +210,4 @@
 		<!-- end of link list -->
 		<!-- joint list -->
-		<!-- WARNING: LIMITS NOT CORRECT -->
 		<joint name="${prefix}palm_finger_1_joint" type="revolute">
 			<parent link="${prefix}palm"/>
@@ -217,10 +216,10 @@
 			<axis xyz="0 1 0"/>
 			<origin rpy="0 3.1416 -1.57" xyz="-0.0455 0.0214 0.036"/>
-			<limit lower="-0.16" upper="0.25" effort="100" velocity="100"/>
+			<!-- Limits: [-17deg.,17deg.] -->
+			<limit lower="-0.2967" upper="0.2967" effort="100" velocity="100"/>
 		</joint>
 		<gazebo reference="${prefix}palm_finger_1_joint">
 		  <implicitSpringDamper>1</implicitSpringDamper>
 		</gazebo>
-		<!-- WARNING: LIMITS NOT CORRECT -->
 		<joint name="${prefix}palm_finger_2_joint" type="revolute">
 			<parent link="${prefix}palm"/>
@@ -229,5 +228,6 @@
 			<axis xyz="0 1 0"/>
 			<origin rpy="0 3.1416 -1.57" xyz="-0.0455 0.0214 -0.036"/>
-			<limit lower="-0.25" upper="0.16" effort="100" velocity="100"/>
+			<!-- Limits: [-17deg.,17deg.] -->
+			<limit lower="-0.2967" upper="0.2967" effort="100" velocity="100"/>
 		</joint>
 		<gazebo reference="${prefix}palm_finger_2_joint">
@@ -240,5 +240,5 @@
 			<axis xyz="0 1 0"/>
 			<origin rpy="0 0 1.57" xyz="0.0455 0.0214 0"/>
-			<limit lower="-0.25" upper="0.16" effort="100" velocity="100"/>
+			<limit lower="0" upper="0" effort="100" velocity="100"/>
 		</joint>
 		<gazebo reference="${prefix}palm_finger_middle_joint">

Commit message: Filling the state fields that show the current joint positions.

File: robotiq_hand_description/urdf/robotiq_hand.urdf.xacro (robot description, xacro)
@@ -217,5 +217,5 @@
 			<origin rpy="0 3.1416 -1.57" xyz="-0.0455 0.0214 0.036"/>
 			<!-- Limits: [-17deg.,17deg.] -->
-			<limit lower="-0.2967" upper="0.2967" effort="100" velocity="100"/>
+			<limit lower="-0.2967" upper="0.2967" effort="100" velocity="-1"/>
 		</joint>
 		<gazebo reference="${prefix}palm_finger_1_joint">
@@ -229,5 +229,5 @@
 			<origin rpy="0 3.1416 -1.57" xyz="-0.0455 0.0214 -0.036"/>
 			<!-- Limits: [-17deg.,17deg.] -->
-			<limit lower="-0.2967" upper="0.2967" effort="100" velocity="100"/>
+			<limit lower="-0.2967" upper="0.2967" effort="100" velocity="-1"/>
 		</joint>
 		<gazebo reference="${prefix}palm_finger_2_joint">
@@ -240,5 +240,5 @@
 			<axis xyz="0 1 0"/>
 			<origin rpy="0 0 1.57" xyz="0.0455 0.0214 0"/>
-			<limit lower="0" upper="0" effort="100" velocity="100"/>
+			<limit lower="0" upper="0" effort="100" velocity="-1"/>
 		</joint>
 		<gazebo reference="${prefix}palm_finger_middle_joint">

Commit message: New Robotiq PID to limit the max velocity of the joints.

File: robotiq_hand_description/urdf/robotiq_hand.urdf.xacro (robot description, xacro)
@@ -129,5 +129,5 @@
       <dynamics damping="1" friction="0" />
       <!-- Limits: [0deg.,70deg.] -->
-      <limit effort="20" velocity="-1" lower="0" upper="1.2217" />
+      <limit effort="60" velocity="-1" lower="0" upper="1.2217" />
     </joint>
     <gazebo reference="${prefix}joint_1">
@@ -142,5 +142,5 @@
       <origin rpy="0 0 -0.52" xyz="0.050 -.028 0"/>
       <!-- Limits: [0deg.,90deg.] -->
-      <limit lower="0" upper="1.5708" effort="20" velocity="-1"/>
+      <limit lower="0" upper="1.5708" effort="60" velocity="-1"/>
     </joint>
     <gazebo reference="${prefix}joint_2">
@@ -155,5 +155,5 @@
       <origin rpy="0 0 0.52" xyz="0.039 0 0"/>
       <!-- Limits: [-38deg.,60deg.] -->
-      <limit lower="-0.6632" upper="1.0471" effort="20" velocity="-1"/>
+      <limit lower="-0.6632" upper="1.0471" effort="60" velocity="-1"/>
     </joint>
     <gazebo reference="${prefix}joint_3">
@@ -223,5 +223,5 @@
       <origin rpy="0 3.1416 -1.57" xyz="-0.0455 0.0214 0.036"/>
       <!-- Limits: [-17deg.,17deg.] -->
-      <limit lower="-0.2967" upper="0.2967" effort="100" velocity="-1"/>
+      <limit lower="-0.2967" upper="0.2967" effort="60" velocity="-1"/>
     </joint>
     <gazebo reference="${prefix}palm_finger_1_joint">
@@ -236,5 +236,5 @@
       <origin rpy="0 3.1416 -1.57" xyz="-0.0455 0.0214 -0.036"/>
       <!-- Limits: [-17deg.,17deg.] -->
-      <limit lower="-0.2967" upper="0.2967" effort="100" velocity="-1"/>
+      <limit lower="-0.2967" upper="0.2967" effort="60" velocity="-1"/>
     </joint>
     <gazebo reference="${prefix}palm_finger_2_joint">
@@ -248,5 +248,5 @@
       <axis xyz="0 1 0"/>
       <origin rpy="0 0 1.57" xyz="0.0455 0.0214 0"/>
-      <limit lower="0" upper="0" effort="100" velocity="-1"/>
+      <limit lower="0" upper="0" effort="60" velocity="-1"/>
     </joint>
     <gazebo reference="${prefix}palm_finger_middle_joint">

Commit message: Tweaking palm collision.

File: robotiq_hand_description/urdf/robotiq_hand.urdf.xacro (robot description, xacro)
@@ -197,5 +197,5 @@
           <origin rpy="0 0 0" xyz="0 0 0"/>
           <geometry>
-            <box size="0.1 0.1 0.08"/>
+            <box size="0.1 0.1 0.1"/>
           </geometry>
           <material name="yellow">

Commit message: adding coupling joints in sdf

File: robotiq_hand_description/urdf/robotiq_hand.urdf.xacro (robot description, xacro)
@@ -570,4 +570,79 @@
     </gazebo>
     <!-- end of joint list -->
+    <!-- coupling joints in sdf -->
+    <gazebo>
+      <joint name="proximal_actuating_hinge_link_1" type="revolute">
+        <parent>${prefix}link_proximal_actuating_hinge</parent>
+        <child>${prefix}link_1</child>
+        <axis>
+          <dynamics>
+            <damping>1</damping>
+            <friction>1</friction>
+          </dynamics>
+          <xyz>0 0 1</xyz>
+          <use_parent_model_frame>true</use_parent_model_frame>
+        </axis>
+      </joint>
+      <joint name="proximal_actuating_bar_median_actuating_hinge" type="revolute">
+        <parent>${prefix}link_proximal_actuating_bar</parent>
+        <child>${prefix}link_median_actuating_hinge</child>
+        <axis>
+          <dynamics>
+            <damping>1</damping>
+            <friction>1</friction>
+          </dynamics>
+          <xyz>0 0 1</xyz>
+          <use_parent_model_frame>true</use_parent_model_frame>
+        </axis>
+      </joint>
+      <joint name="median_bar_paradistal_hinge" type="revolute">
+        <parent>${prefix}link_median_bar</parent>
+        <child>${prefix}link_paradistal_hinge</child>
+        <axis>
+          <dynamics>
+            <damping>1</damping>
+            <friction>1</friction>
+          </dynamics>
+          <xyz>0 0 1</xyz>
+          <use_parent_model_frame>true</use_parent_model_frame>
+        </axis>
+      </joint>
+      <joint name="paraproximal_actuating_hinge_link_1" type="revolute">
+        <parent>${prefix}link_paraproximal_actuating_hinge</parent>
+        <child>${prefix}link_1</child>
+        <axis>
+          <dynamics>
+            <damping>1</damping>
+            <friction>1</friction>
+          </dynamics>
+          <xyz>0 0 1</xyz>
+          <use_parent_model_frame>true</use_parent_model_frame>
+        </axis>
+      </joint>
+      <joint name="paraproximal_bar_paramedian_hinge" type="revolute">
+        <parent>${prefix}link_paraproximal_bar</parent>
+        <child>${prefix}link_paramedian_hinge</child>
+        <axis>
+          <dynamics>
+            <damping>1</damping>
+            <friction>1</friction>
+          </dynamics>
+          <xyz>0 0 1</xyz>
+          <use_parent_model_frame>true</use_parent_model_frame>
+        </axis>
+      </joint>
+      <joint name="median_bar_paradistal_hinge" type="revolute">
+        <parent>${prefix}link_median_bar</parent>
+        <child>${prefix}link_paradistal_hinge</child>
+        <axis>
+          <dynamics>
+            <damping>1</damping>
+            <friction>1</friction>
+          </dynamics>
+          <xyz>0 0 1</xyz>
+          <use_parent_model_frame>true</use_parent_model_frame>
+        </axis>
+      </joint>
+    </gazebo>
   </xacro:macro>
 </robot>

Commit message: fix coupling

File: robotiq_hand_description/urdf/robotiq_hand.urdf.xacro (robot description, xacro)
@@ -477,4 +477,82 @@
     </gazebo>
     <!-- end of joint list -->
+    <!-- coupling joints in sdf -->
+    <gazebo>
+      <joint name="${prefix}link_proximal_actuating_hinge_link_1" type="revolute">
+        <parent>${prefix}link_proximal_actuating_hinge</parent>
+        <child>${prefix}link_1</child>
+        <axis>
+          <dynamics>
+            <damping>1</damping>
+            <friction>0</friction>
+          </dynamics>
+          <xyz>0 0 1</xyz>
+          <use_parent_model_frame>true</use_parent_model_frame>
+        </axis>
+      </joint>
+      <joint name="${prefix}link_proximal_actuating_bar_median_actuating_hinge" type="revolute">
+        <parent>${prefix}link_proximal_actuating_bar</parent>
+        <child>${prefix}link_median_actuating_hinge</child>
+        <axis>
+          <dynamics>
+            <damping>1</damping>
+            <friction>0</friction>
+          </dynamics>
+          <xyz>0 0 1</xyz>
+          <use_parent_model_frame>true</use_parent_model_frame>
+        </axis>
+      </joint>
+      <joint name="${prefix}link_median_bar_paradistal_hinge" type="revolute">
+        <parent>${prefix}link_median_bar</parent>
+        <child>${prefix}link_paradistal_hinge</child>
+        <axis>
+          <dynamics>
+            <damping>1</damping>
+            <friction>0</friction>
+          </dynamics>
+          <xyz>0 0 1</xyz>
+          <use_parent_model_frame>true</use_parent_model_frame>
+        </axis>
+      </joint>
+      <joint name="${prefix}link_paraproximal_actuating_hinge_link_1" type="revolute">
+        <parent>${prefix}link_paraproximal_actuating_hinge</parent>
+        <child>${prefix}link_1</child>
+        <axis>
+          <dynamics>
+            <damping>1</damping>
+            <friction>0</friction>
+          </dynamics>
+          <xyz>0 0 1</xyz>
+          <use_parent_model_frame>true</use_parent_model_frame>
+        </axis>
+      </joint>
+      <joint name="${prefix}link_paraproximal_bar_paramedian_hinge" type="revolute">
+        <parent>${prefix}link_paraproximal_bar</parent>
+        <child>${prefix}link_paramedian_hinge</child>
+        <axis>
+          <dynamics>
+            <damping>1</damping>
+            <friction>0</friction>
+          </dynamics>
+          <xyz>0 0 1</xyz>
+          <use_parent_model_frame>true</use_parent_model_frame>
+        </axis>
+      </joint>
+    </gazebo>
+    <gazebo reference="${prefix}link_proximal_actuating_hinge_link_1">
+      <implicitSpringDamper>1</implicitSpringDamper>
+    </gazebo>
+    <gazebo reference="${prefix}link_proximal_actuating_bar_median_actuating_hinge">
+      <implicitSpringDamper>1</implicitSpringDamper>
+    </gazebo>
+    <gazebo reference="${prefix}link_median_bar_paradistal_hinge">
+      <implicitSpringDamper>1</implicitSpringDamper>
+    </gazebo>
+    <gazebo reference="${prefix}link_paraproximal_actuating_hinge_link_1">
+      <implicitSpringDamper>1</implicitSpringDamper>
+    </gazebo>
+    <gazebo reference="${prefix}link_paraproximal_bar_paramedian_hinge">
+      <implicitSpringDamper>1</implicitSpringDamper>
+    </gazebo>
   </xacro:macro>
   <xacro:macro name="robotiq_hand" params="prefix *origin reflect parent">
@@ -570,79 +648,4 @@
     </gazebo>
     <!-- end of joint list -->
-    <!-- coupling joints in sdf -->
-    <gazebo>
-      <joint name="proximal_actuating_hinge_link_1" type="revolute">
-        <parent>${prefix}link_proximal_actuating_hinge</parent>
-        <child>${prefix}link_1</child>
-        <axis>
-          <dynamics>
-            <damping>1</damping>
-            <friction>1</friction>
-          </dynamics>
-          <xyz>0 0 1</xyz>
-          <use_parent_model_frame>true</use_parent_model_frame>
-        </axis>
-      </joint>
-      <joint name="proximal_actuating_bar_median_actuating_hinge" type="revolute">
-        <parent>${prefix}link_proximal_actuating_bar</parent>
-        <child>${prefix}link_median_actuating_hinge</child>
-        <axis>
-          <dynamics>
-            <damping>1</damping>
-            <friction>1</friction>
-          </dynamics>
-          <xyz>0 0 1</xyz>
-          <use_parent_model_frame>true</use_parent_model_frame>
-        </axis>
-      </joint>
-      <joint name="median_bar_paradistal_hinge" type="revolute">
-        <parent>${prefix}link_median_bar</parent>
-        <child>${prefix}link_paradistal_hinge</child>
-        <axis>
-          <dynamics>
-            <damping>1</damping>
-            <friction>1</friction>
-          </dynamics>
-          <xyz>0 0 1</xyz>
-          <use_parent_model_frame>true</use_parent_model_frame>
-        </axis>
-      </joint>
-      <joint name="paraproximal_actuating_hinge_link_1" type="revolute">
-        <parent>${prefix}link_paraproximal_actuating_hinge</parent>
-        <child>${prefix}link_1</child>
-        <axis>
-          <dynamics>
-            <damping>1</damping>
-            <friction>1</friction>
-          </dynamics>
-          <xyz>0 0 1</xyz>
-          <use_parent_model_frame>true</use_parent_model_frame>
-        </axis>
-      </joint>
-      <joint name="paraproximal_bar_paramedian_hinge" type="revolute">
-        <parent>${prefix}link_paraproximal_bar</parent>
-        <child>${prefix}link_paramedian_hinge</child>
-        <axis>
-          <dynamics>
-            <damping>1</damping>
-            <friction>1</friction>
-          </dynamics>
-          <xyz>0 0 1</xyz>
-          <use_parent_model_frame>true</use_parent_model_frame>
-        </axis>
-      </joint>
-      <joint name="median_bar_paradistal_hinge" type="revolute">
-        <parent>${prefix}link_median_bar</parent>
-        <child>${prefix}link_paradistal_hinge</child>
-        <axis>
-          <dynamics>
-            <damping>1</damping>
-            <friction>1</friction>
-          </dynamics>
-          <xyz>0 0 1</xyz>
-          <use_parent_model_frame>true</use_parent_model_frame>
-        </axis>
-      </joint>
-    </gazebo>
   </xacro:macro>
 </robot>

Commit message: debugging parallel joints without the coupling joints first.

File: robotiq_hand_description/urdf/robotiq_hand.urdf.xacro (robot description, xacro)
@@ -122,5 +122,5 @@
     <link name="${prefix}link_proximal_actuating_hinge">
       <visual>
-        <origin rpy="0 0 0" xyz="0 0 0"/>
+        <origin rpy="0 0 0" xyz="-0.015 0 0"/>
         <geometry>
           <box size="0.03 .0075 .002"/>
@@ -128,5 +128,5 @@
       </visual>
       <collision>
-        <origin rpy="0 0 0" xyz="0 0 0"/>
+        <origin rpy="0 0 0" xyz="-0.015 0 0"/>
          <geometry>
           <box size="0.03 .0075 .002"/>
@@ -134,5 +134,5 @@
       </collision>
       <inertial>
-        <origin rpy="0 0 0" xyz="0 0 0"/>
+        <origin rpy="0 0 0" xyz="-0.015 0 0"/>
         <mass value="0.047"/>
         <inertia ixx="0.00000499332" ixy="0.00000091312" ixz="-0.00000000120" iyy  ="0.00006434531" iyz="-0.00000000007" izz="0.00006061917"/>
@@ -171,5 +171,5 @@
     <link name="${prefix}link_proximal_actuating_bar">
       <visual>
-        <origin rpy="0 0 0" xyz="0 0 0"/>
+        <origin rpy="0 0 0" xyz="0.026789 0 0"/>
         <geometry>
           <box size="0.053578 .0075 .002"/>
@@ -177,5 +177,5 @@
       </visual>
       <collision>
-        <origin rpy="0 0 0" xyz="0 0 0"/>
+        <origin rpy="0 0 0" xyz="0.026789 0 0"/>
          <geometry>
           <box size="0.053578 .0075 .002"/>
@@ -183,5 +183,5 @@
       </collision>
       <inertial>
-        <origin rpy="0 0 0" xyz="0 0 0"/>
+        <origin rpy="0 0 0" xyz="0.026789 0 0"/>
         <mass value="0.047"/>
         <inertia ixx="0.00000499332" ixy="0.00000091312" ixz="-0.00000000120" iyy  ="0.00006434531" iyz="-0.00000000007" izz="0.00006061917"/>
@@ -343,5 +343,5 @@
       <child link="${prefix}link_proximal_actuating_hinge"/>
       <axis xyz="0 0 1"/>
-      <origin rpy="0 0 1.051" xyz="-0.0071 -0.012 0.01"/>
+      <origin rpy="0 0 1.051" xyz="0 0 0.01"/>
       <limit effort="100" lower="0" upper="3.1416" velocity="100"/>
     </joint>
@@ -477,5 +477,5 @@
     </gazebo>
     <!-- end of joint list -->
-    <!-- coupling joints in sdf -->
+    <!-- coupling joints in sdf
     <gazebo>
       <joint name="${prefix}link_proximal_actuating_hinge_link_1" type="revolute">
@@ -555,4 +555,5 @@
       <implicitSpringDamper>1</implicitSpringDamper>
     </gazebo>
+ -->
   </xacro:macro>
   <xacro:macro name="robotiq_hand" params="prefix *origin reflect parent">

Commit message: fixing proximal_actuating_hinge and proximal_actuating_bar joint locations.

File: robotiq_hand_description/urdf/robotiq_hand.urdf.xacro (robot description, xacro)
@@ -147,5 +147,5 @@
     <link name="${prefix}link_paraproximal_actuating_hinge">
       <visual>
-        <origin rpy="0 0 0" xyz="0 0 0"/>
+        <origin rpy="-0.015 0 0" xyz="0 0 0"/>
         <geometry>
           <box size="0.03 .0075 .002"/>
@@ -153,5 +153,5 @@
       </visual>
       <collision>
-        <origin rpy="0 0 0" xyz="0 0 0"/>
+        <origin rpy="-0.015 0 0" xyz="0 0 0"/>
          <geometry>
           <box size="0.03 .0075 .002"/>
@@ -159,5 +159,5 @@
       </collision>
       <inertial>
-        <origin rpy="0 0 0" xyz="0 0 0"/>
+        <origin rpy="-0.015 0 0" xyz="0 0 0"/>
         <mass value="0.047"/>
         <inertia ixx="0.00000499332" ixy="0.00000091312" ixz="-0.00000000120" iyy  ="0.00006434531" iyz="-0.00000000007" izz="0.00006061917"/>
@@ -354,5 +354,5 @@
       <child link="${prefix}link_paraproximal_actuating_hinge"/>
       <axis xyz="0 0 1"/>
-      <origin rpy="0 0 1.051" xyz="-0.0071 -0.012 -0.01"/>
+      <origin rpy="0 0 1.051" xyz="0 0 -0.01"/>
       <limit effort="100" lower="0" upper="3.1416" velocity="100"/>
     </joint>
@@ -365,5 +365,5 @@
       <child link="${prefix}link_proximal_actuating_bar"/>
       <axis xyz="0 0 1"/>
-      <origin rpy="0 0 -1.28" xyz="-0.0067 -0.0257 0"/>
+      <origin rpy="0 0 -1.28" xyz="0 -0.02858 0"/>
       <limit effort="100" lower="0" upper="3.1416" velocity="100"/>
     </joint>
