Commit message: reorganize link_1, link_2, link_3 orientation to match document provided by RobotiQ

File: robotiq_hand_description/urdf/robotiq_hand.urdf.xacro (robot description, xacro)
@@ -42,5 +42,5 @@
     <link name="${prefix}link_1">
       <visual>
-        <origin rpy="0 0 -0.52" xyz="0.050 -.028 0"/>
+        <origin rpy="0 0 ${3.1416/2}" xyz="0 0.05717 0"/>
         <geometry>
           <mesh filename="package://robotiq_hand_description/meshes/s-model_articulated/visual/link_1.STL" />
@@ -49,5 +49,5 @@
       </visual>
       <collision>
-        <origin rpy="0 0 -0.52" xyz="0.050 -.028 0"/>
+        <origin rpy="0 0 ${3.1416/2}" xyz="0 0.05717 0"/>
         <geometry>
           <mesh filename="package://robotiq_hand_description/meshes/s-model_articulated/collision/link_1.STL"/>
@@ -58,5 +58,5 @@
       </collision>
       <inertial>
-        <origin rpy="0 0 -0.52" xyz="0.0282 -0.0155 0"/>
+        <origin rpy="0 0 ${3.1416/2}" xyz="0 0.05717 0"/>
         <mass value="0.047"/>
         <inertia ixx="0.00000499332" ixy="0.00000091312" ixz="-0.00000000120" iyy="0.00006434531" iyz="-0.00000000007" izz="0.00006061917"/>
@@ -70,5 +70,5 @@
     <link name="${prefix}link_2">
       <visual>
-        <origin xyz="0.039 0 0.0075" rpy="0 0 0"/>
+        <origin rpy="0 0 ${3.1416/2}" xyz="0 0.03810 0"/>
         <geometry>
           <mesh filename="package://robotiq_hand_description/meshes/s-model_articulated/visual/link_2.STL" />
@@ -77,5 +77,5 @@
       </visual>
       <collision>
-        <origin rpy="0 0 0" xyz="0.039 0 0.0075"/>
+        <origin rpy="0 0 ${3.1416/2}" xyz="0 0.03810 0"/>
           <geometry>
             <mesh filename="package://robotiq_hand_description/meshes/s-model_articulated/collision/link_2.STL"/>
@@ -84,5 +84,5 @@
       </collision>
       <inertial>
-        <origin rpy="0 0 0" xyz="0.02167 0.00048 0.00018"/>
+        <origin rpy="0 0 ${3.1416/2}" xyz="0 0.03810 0"/>
         <mass value="0.03284"/>
         <inertia ixx="0.00000348008" ixy="0.00000031940" ixz="0.00000013041" iyy="0.00002248123" iyz="0.00000000291" izz="0.00001986346"/>
@@ -96,5 +96,5 @@
     <link name="${prefix}link_3">
       <visual>
-        <origin xyz="0 0 0" rpy="0 0 0"/>
+        <origin xyz="0 0 0" rpy="0 0 ${3.1416/2}"/>
         <geometry>
           <mesh filename="package://robotiq_hand_description/meshes/s-model_articulated/visual/link_3.STL" />
@@ -103,5 +103,5 @@
       </visual>
       <collision>
-        <origin rpy="0 0 0" xyz="0 0 0"/>
+        <origin xyz="0 0 0" rpy="0 0 ${3.1416/2}"/>
         <geometry>
           <mesh filename="package://robotiq_hand_description/meshes/s-model_articulated/collision/link_3.STL"/>
@@ -110,5 +110,5 @@
       </collision>
       <inertial>
-        <origin rpy="0 0 0" xyz="0.01626 0.00049 0.0002"/>
+        <origin rpy="0 0 ${3.1416/2}" xyz="0.01626 0.00049 0.0002"/>
         <mass value="0.03354"/>
         <inertia ixx="0.00000305151" ixy="0.00000089792" ixz="0.00000000249" iyy="0.00001427978" iyz="-0.00000001191" izz="0.00001264126"/>
@@ -122,5 +122,5 @@
     <link name="${prefix}link_proximal_actuating_hinge">
       <visual>
-        <origin rpy="0 0 0" xyz="-0.015 0 0"/>
+        <origin rpy="0 0 0" xyz="0.015 0 0"/>
         <geometry>
           <box size="0.03 .0075 .002"/>
@@ -128,5 +128,5 @@
       </visual>
       <collision>
-        <origin rpy="0 0 0" xyz="-0.015 0 0"/>
+        <origin rpy="0 0 0" xyz="0.015 0 0"/>
          <geometry>
           <box size="0.03 .0075 .002"/>
@@ -134,5 +134,5 @@
       </collision>
       <inertial>
-        <origin rpy="0 0 0" xyz="-0.015 0 0"/>
+        <origin rpy="0 0 0" xyz="0.015 0 0"/>
         <mass value="0.047"/>
         <inertia ixx="0.00000499332" ixy="0.00000091312" ixz="-0.00000000120" iyy  ="0.00006434531" iyz="-0.00000000007" izz="0.00006061917"/>
@@ -173,5 +173,5 @@
         <origin rpy="0 0 0" xyz="0.026789 0 0"/>
         <geometry>
-          <box size="0.053578 .0075 .002"/>
+          <box size="0.05398 .0075 .002"/>
         </geometry>
       </visual>
@@ -179,9 +179,9 @@
         <origin rpy="0 0 0" xyz="0.026789 0 0"/>
          <geometry>
-          <box size="0.053578 .0075 .002"/>
-        </geometry>
-      </collision>
-      <inertial>
-        <origin rpy="0 0 0" xyz="0.026789 0 0"/>
+          <box size="0.05398 .0075 .002"/>
+        </geometry>
+      </collision>
+      <inertial>
+        <origin rpy="0.5398 0 0" xyz="0.026789 0 0"/>
         <mass value="0.047"/>
         <inertia ixx="0.00000499332" ixy="0.00000091312" ixz="-0.00000000120" iyy  ="0.00006434531" iyz="-0.00000000007" izz="0.00006061917"/>
@@ -343,5 +343,5 @@
       <child link="${prefix}link_proximal_actuating_hinge"/>
       <axis xyz="0 0 1"/>
-      <origin rpy="0 0 1.051" xyz="0 0 0.01"/>
+      <origin rpy="0 0 -2.0906" xyz="0 0 0.01"/>
       <limit effort="100" lower="0" upper="3.1416" velocity="100"/>
     </joint>
@@ -365,5 +365,5 @@
       <child link="${prefix}link_proximal_actuating_bar"/>
       <axis xyz="0 0 1"/>
-      <origin rpy="0 0 -1.28" xyz="0 -0.02858 0"/>
+      <origin rpy="0 0 1.8616" xyz="0.02858 0 0"/>
       <limit effort="100" lower="0" upper="3.1416" velocity="100"/>
     </joint>
@@ -387,5 +387,6 @@
       <child link="${prefix}link_median_actuating_hinge"/>
       <axis xyz="0 0 1"/>
-      <origin rpy="0 0 -0.52" xyz="0.050 -.028 0.01"/>
+      <!--<origin rpy="0 0 -0.52" xyz="0.050 -.028 0.01"/>-->
+      <origin rpy="0 0 ${-0.29-3.14159/2}" xyz="0 0.05715 0.01"/>
       <limit effort="100" lower="0" upper="3.1416" velocity="100"/>
     </joint>
@@ -398,5 +399,5 @@
       <child link="${prefix}link_paramedian_hinge"/>
       <axis xyz="0 0 1"/>
-      <origin rpy="0 0 -0.52" xyz="0.050 -.028 -0.01"/>
+      <origin rpy="0 0 -0.52" xyz="0 0.05715 -0.01"/>
       <limit effort="100" lower="0" upper="3.1416" velocity="100"/>
     </joint>
@@ -420,5 +421,5 @@
       <child link="${prefix}link_paradistal_hinge"/>
       <axis xyz="0 0 1"/>
-      <origin rpy="0 0 0" xyz="0.039 0 0.01"/>
+      <origin rpy="0 0 0" xyz="0 0.039 0.01"/>
       <limit effort="100" lower="0" upper="3.1416" velocity="100"/>
     </joint>
@@ -439,5 +440,5 @@
     <!-- Joint 1 -->
     <joint name="${prefix}joint_1" type="revolute">
-      <origin rpy="0 0 0" xyz="0 0 0"/>
+      <origin rpy="0 0 -2.0906" xyz="0 0 0"/>
       <axis xyz="0 0 1" />
       <parent link="${prefix}link_0"/>
@@ -456,5 +457,5 @@
       <dynamics damping="1" friction="0" />
       <axis xyz="0 0 1"/>
-      <origin rpy="0 0 -0.52" xyz="0.050 -.028 0"/>
+      <origin rpy="0 0 0" xyz="0 0.05715 0"/>
       <!-- Limits: [0deg.,90deg.] -->
       <limit lower="0" upper="1.5708" effort="60" velocity="-1"/>
@@ -469,5 +470,5 @@
       <dynamics damping="1" friction="0" />
       <axis xyz="0 0 1"/>
-      <origin rpy="0 0 0.52" xyz="0.039 0 0"/>
+      <origin rpy="0 0 0.5198" xyz="0 0.039 0"/>
       <!-- Limits: [-38deg.,60deg.] -->
       <limit lower="-0.6632" upper="1.0471" effort="60" velocity="-1"/>
@@ -491,7 +492,14 @@
         </axis>
       </joint>
+    </gazebo>
+    <gazebo reference="${prefix}link_proximal_actuating_hinge_link_1">
+      <implicitSpringDamper>1</implicitSpringDamper>
+    </gazebo>
+    -->
+    <gazebo>
       <joint name="${prefix}link_proximal_actuating_bar_median_actuating_hinge" type="revolute">
-        <parent>${prefix}link_proximal_actuating_bar</parent>
-        <child>${prefix}link_median_actuating_hinge</child>
+        <parent>${prefix}link_median_actuating_hinge</parent>
+        <child>${prefix}link_proximal_actuating_bar</child>
+        <pose>0.05398 0 0 0 0 0</pose>
         <axis>
           <dynamics>
@@ -500,7 +508,13 @@
           </dynamics>
           <xyz>0 0 1</xyz>
-          <use_parent_model_frame>true</use_parent_model_frame>
+          <use_parent_model_frame>false</use_parent_model_frame>
         </axis>
       </joint>
+    </gazebo>
+    <gazebo reference="${prefix}link_proximal_actuating_bar_median_actuating_hinge">
+      <implicitSpringDamper>1</implicitSpringDamper>
+    </gazebo>
+    <!--
+    <gazebo>
       <joint name="${prefix}link_median_bar_paradistal_hinge" type="revolute">
         <parent>${prefix}link_median_bar</parent>
@@ -515,4 +529,9 @@
         </axis>
       </joint>
+    </gazebo>
+    <gazebo reference="${prefix}link_median_bar_paradistal_hinge">
+      <implicitSpringDamper>1</implicitSpringDamper>
+    </gazebo>
+    <gazebo>
       <joint name="${prefix}link_paraproximal_actuating_hinge_link_1" type="revolute">
         <parent>${prefix}link_paraproximal_actuating_hinge</parent>
@@ -527,4 +546,9 @@
         </axis>
       </joint>
+    </gazebo>
+    <gazebo reference="${prefix}link_paraproximal_actuating_hinge_link_1">
+      <implicitSpringDamper>1</implicitSpringDamper>
+    </gazebo>
+    <gazebo>
       <joint name="${prefix}link_paraproximal_bar_paramedian_hinge" type="revolute">
         <parent>${prefix}link_paraproximal_bar</parent>
@@ -539,16 +563,4 @@
         </axis>
       </joint>
-    </gazebo>
-    <gazebo reference="${prefix}link_proximal_actuating_hinge_link_1">
-      <implicitSpringDamper>1</implicitSpringDamper>
-    </gazebo>
-    <gazebo reference="${prefix}link_proximal_actuating_bar_median_actuating_hinge">
-      <implicitSpringDamper>1</implicitSpringDamper>
-    </gazebo>
-    <gazebo reference="${prefix}link_median_bar_paradistal_hinge">
-      <implicitSpringDamper>1</implicitSpringDamper>
-    </gazebo>
-    <gazebo reference="${prefix}link_paraproximal_actuating_hinge_link_1">
-      <implicitSpringDamper>1</implicitSpringDamper>
     </gazebo>
     <gazebo reference="${prefix}link_paraproximal_bar_paramedian_hinge">

Commit message: fixed link_1, link_2, link_3 frames and top bars

File: robotiq_hand_description/urdf/robotiq_hand.urdf.xacro (robot description, xacro)
@@ -70,5 +70,5 @@
     <link name="${prefix}link_2">
       <visual>
-        <origin rpy="0 0 ${3.1416/2}" xyz="0 0.03810 0"/>
+        <origin rpy="0 0 ${3.1416/2}" xyz="0 0.03810 0.0075"/>
         <geometry>
           <mesh filename="package://robotiq_hand_description/meshes/s-model_articulated/visual/link_2.STL" />
@@ -77,5 +77,5 @@
       </visual>
       <collision>
-        <origin rpy="0 0 ${3.1416/2}" xyz="0 0.03810 0"/>
+        <origin rpy="0 0 ${3.1416/2}" xyz="0 0.03810 0.0075"/>
           <geometry>
             <mesh filename="package://robotiq_hand_description/meshes/s-model_articulated/collision/link_2.STL"/>
@@ -84,5 +84,5 @@
       </collision>
       <inertial>
-        <origin rpy="0 0 ${3.1416/2}" xyz="0 0.03810 0"/>
+        <origin rpy="0 0 ${3.1416/2}" xyz="0 0.03810 0.0075"/>
         <mass value="0.03284"/>
         <inertia ixx="0.00000348008" ixy="0.00000031940" ixz="0.00000013041" iyy="0.00002248123" iyz="0.00000000291" izz="0.00001986346"/>
@@ -96,5 +96,5 @@
     <link name="${prefix}link_3">
       <visual>
-        <origin xyz="0 0 0" rpy="0 0 ${3.1416/2}"/>
+        <origin xyz="0 0 0" rpy="0 0 0"/>
         <geometry>
           <mesh filename="package://robotiq_hand_description/meshes/s-model_articulated/visual/link_3.STL" />
@@ -103,5 +103,5 @@
       </visual>
       <collision>
-        <origin xyz="0 0 0" rpy="0 0 ${3.1416/2}"/>
+        <origin xyz="0 0 0" rpy="0 0 0"/>
         <geometry>
           <mesh filename="package://robotiq_hand_description/meshes/s-model_articulated/collision/link_3.STL"/>
@@ -110,5 +110,5 @@
       </collision>
       <inertial>
-        <origin rpy="0 0 ${3.1416/2}" xyz="0.01626 0.00049 0.0002"/>
+        <origin rpy="0 0 0" xyz="0.01626 0.00049 0.0002"/>
         <mass value="0.03354"/>
         <inertia ixx="0.00000305151" ixy="0.00000089792" ixz="0.00000000249" iyy="0.00001427978" iyz="-0.00000001191" izz="0.00001264126"/>
@@ -243,5 +243,5 @@
     <link name="${prefix}link_median_bar">
       <visual>
-        <origin rpy="0 0 0" xyz="0 0 0"/>
+        <origin rpy="0 0 0" xyz="0.01905 0 0"/>
         <geometry>
           <box size="0.0381 .0075 .002"/>
@@ -249,5 +249,5 @@
       </visual>
       <collision>
-        <origin rpy="0 0 0" xyz="0 0 0"/>
+        <origin rpy="0 0 0" xyz="0.01905 0 0"/>
          <geometry>
           <box size="0.0381 .0075 .002"/>
@@ -255,5 +255,5 @@
       </collision>
       <inertial>
-        <origin rpy="0 0 0" xyz="0 0 0"/>
+        <origin rpy="0 0 0" xyz="0.01905 0 0"/>
         <mass value="0.047"/>
         <inertia ixx="0.00000499332" ixy="0.00000091312" ixz="-0.00000000120" iyy  ="0.00006434531" iyz="-0.00000000007" izz="0.00006061917"/>
@@ -387,6 +387,6 @@
       <child link="${prefix}link_median_actuating_hinge"/>
       <axis xyz="0 0 1"/>
-      <!--<origin rpy="0 0 -0.52" xyz="0.050 -.028 0.01"/>-->
-      <origin rpy="0 0 ${-0.29-3.14159/2}" xyz="0 0.05715 0.01"/>
+      <!-- \TODO: -0.37 is hand picked, double check -->
+      <origin rpy="0 0 ${-0.37}" xyz="0 0.05715 0.01"/>
       <limit effort="100" lower="0" upper="3.1416" velocity="100"/>
     </joint>
@@ -399,5 +399,7 @@
       <child link="${prefix}link_paramedian_hinge"/>
       <axis xyz="0 0 1"/>
-      <origin rpy="0 0 -0.52" xyz="0 0.05715 -0.01"/>
+      <!-- \TODO: -0.37 is hand picked, 0.9719 is hand calculated from atan(0.02381/0.01625), double check -->
+      <origin rpy="0 0 ${-0.37+0.9719}" xyz="0 0.05715 -0.01"/>
+      <origin rpy="0 0 0.29" xyz="0.01625 0.02381 0"/>
       <limit effort="100" lower="0" upper="3.1416" velocity="100"/>
     </joint>
@@ -410,5 +412,6 @@
       <child link="${prefix}link_median_bar"/>
       <axis xyz="0 0 1"/>
-      <origin rpy="0 0 0.29" xyz="0.019 -0.02381 0"/>
+      <!-- \TODO: hand calc 90 deg + atan(0.01516/0.01625) -->
+      <origin rpy="0 0 ${3.1416/2 + 0.7507}" xyz="0.01625 0.01516 0"/>
       <limit effort="100" lower="0" upper="3.1416" velocity="100"/>
     </joint>
@@ -421,5 +424,5 @@
       <child link="${prefix}link_paradistal_hinge"/>
       <axis xyz="0 0 1"/>
-      <origin rpy="0 0 0" xyz="0 0.039 0.01"/>
+      <origin rpy="0 0 0" xyz="0 0.039 -0.01"/>
       <limit effort="100" lower="0" upper="3.1416" velocity="100"/>
     </joint>
@@ -470,5 +473,5 @@
       <dynamics damping="1" friction="0" />
       <axis xyz="0 0 1"/>
-      <origin rpy="0 0 0.5198" xyz="0 0.039 0"/>
+      <origin rpy="0 0 ${3.1416/2 + 0.5198}" xyz="0 0.039 0"/>
       <!-- Limits: [-38deg.,60deg.] -->
       <limit lower="-0.6632" upper="1.0471" effort="60" velocity="-1"/>
@@ -515,9 +518,9 @@
       <implicitSpringDamper>1</implicitSpringDamper>
     </gazebo>
-    <!--
     <gazebo>
-      <joint name="${prefix}link_median_bar_paradistal_hinge" type="revolute">
-        <parent>${prefix}link_median_bar</parent>
-        <child>${prefix}link_paradistal_hinge</child>
+      <joint name="${prefix}link_median_bar_link_3" type="revolute">
+        <parent>${prefix}link_3</parent>
+        <child>${prefix}link_median_bar</child>
+        <pose>0.0381 0 0 0 0 0</pose>
         <axis>
           <dynamics>
@@ -526,5 +529,5 @@
           </dynamics>
           <xyz>0 0 1</xyz>
-          <use_parent_model_frame>true</use_parent_model_frame>
+          <use_parent_model_frame>false</use_parent_model_frame>
         </axis>
       </joint>
@@ -533,4 +536,5 @@
       <implicitSpringDamper>1</implicitSpringDamper>
     </gazebo>
+    <!--
     <gazebo>
       <joint name="${prefix}link_paraproximal_actuating_hinge_link_1" type="revolute">

Commit message: fix inertia for proximal_actuating_hinge

File: robotiq_hand_description/urdf/robotiq_hand.urdf.xacro (robot description, xacro)
@@ -58,7 +58,12 @@
       </collision>
       <inertial>
-        <origin rpy="0 0 ${3.1416/2}" xyz="0 0.05717 0"/>
-        <mass value="0.047"/>
-        <inertia ixx="0.00000499332" ixy="0.00000091312" ixz="-0.00000000120" iyy="0.00006434531" iyz="-0.00000000007" izz="0.00006061917"/>
+        <origin rpy="0 0 0" xyz="0 0.05717 0"/>
+        <mass value="0.047"/>
+        <inertia ixx= "0.00000499332"
+                 ixy= "0.00000091312"
+                 ixz="-0.00000000120"
+                 iyy= "0.00006434531"
+                 iyz="-0.00000000007"
+                 izz= "0.00006061917"/>
       </inertial>
     </link>
@@ -84,5 +89,5 @@
       </collision>
       <inertial>
-        <origin rpy="0 0 ${3.1416/2}" xyz="0 0.03810 0.0075"/>
+        <origin rpy="0 0 0" xyz="0 0.03810 0.0075"/>
         <mass value="0.03284"/>
         <inertia ixx="0.00000348008" ixy="0.00000031940" ixz="0.00000013041" iyy="0.00002248123" iyz="0.00000000291" izz="0.00001986346"/>
@@ -135,6 +140,11 @@
       <inertial>
         <origin rpy="0 0 0" xyz="0.015 0 0"/>
-        <mass value="0.047"/>
-        <inertia ixx="0.00000499332" ixy="0.00000091312" ixz="-0.00000000120" iyy  ="0.00006434531" iyz="-0.00000000007" izz="0.00006061917"/>
+        <mass value="0.02647"/>
+        <inertia ixx= "0.00000156447"
+                 ixy= "0.000000236226"
+                 ixz="-0.00000014862"
+                 iyy= "0.00000221068"
+                 iyz="-0.00000014369"
+                 izz= "0.00000323175"/>
       </inertial>
     </link>
