Commit message: fix link_1 link_2 link_3 inertias

File: robotiq_hand_description/urdf/robotiq_hand.urdf.xacro (robot description, xacro)
@@ -58,5 +58,6 @@
       </collision>
       <inertial>
-        <origin rpy="0 0 0" xyz="0 0.05717 0"/>
+        <!-- link_1 inertia visually incorrect, please double check values -->
+        <origin rpy="0 0 ${3.1416/2}" xyz="0.00053 0.03218 0"/>
         <mass value="0.047"/>
         <inertia ixx= "0.00000499332"
@@ -89,7 +90,13 @@
       </collision>
       <inertial>
-        <origin rpy="0 0 0" xyz="0 0.03810 0.0075"/>
+        <!-- link_2 inertia visually incorrect, please double check values -->
+        <origin rpy="0 0 ${3.1416/2}" xyz="0.00048 0.02167 0.00018"/>
         <mass value="0.03284"/>
-        <inertia ixx="0.00000348008" ixy="0.00000031940" ixz="0.00000013041" iyy="0.00002248123" iyz="0.00000000291" izz="0.00001986346"/>
+        <inertia ixx="0.00000348008"
+                 ixy="0.00000031940"
+                 ixz="0.00000013041"
+                 iyy="0.00002248123"
+                 iyz="0.00000000291"
+                 izz="0.00001986346"/>
       </inertial>
     </link>
@@ -117,5 +124,10 @@
         <origin rpy="0 0 0" xyz="0.01626 0.00049 0.0002"/>
         <mass value="0.03354"/>
-        <inertia ixx="0.00000305151" ixy="0.00000089792" ixz="0.00000000249" iyy="0.00001427978" iyz="-0.00000001191" izz="0.00001264126"/>
+        <inertia ixx="0.00000305151"
+                 ixy="0.00000089792"
+                 ixz="0.00000000249"
+                 iyy="0.00001427978"
+                 iyz="-0.00000001191"
+                 izz="0.00001264126"/>
       </inertial>
     </link>
@@ -170,6 +182,12 @@
       <inertial>
         <origin rpy="-0.015 0 0" xyz="0 0 0"/>
-        <mass value="0.047"/>
-        <inertia ixx="0.00000499332" ixy="0.00000091312" ixz="-0.00000000120" iyy  ="0.00006434531" iyz="-0.00000000007" izz="0.00006061917"/>
+        <!-- copied from proximal_actuating_hinge -->
+        <mass value="0.02647"/>
+        <inertia ixx= "0.00000156447"
+                 ixy= "0.000000236226"
+                 ixz="-0.00000014862"
+                 iyy= "0.00000221068"
+                 iyz="-0.00000014369"
+                 izz= "0.00000323175"/>
       </inertial>
     </link>
@@ -194,6 +212,12 @@
       <inertial>
         <origin rpy="0.5398 0 0" xyz="0.026789 0 0"/>
-        <mass value="0.047"/>
-        <inertia ixx="0.00000499332" ixy="0.00000091312" ixz="-0.00000000120" iyy  ="0.00006434531" iyz="-0.00000000007" izz="0.00006061917"/>
+        <!-- copied from proximal_actuating_hinge -->
+        <mass value="0.02647"/>
+        <inertia ixx= "0.00000156447"
+                 ixy= "0.000000236226"
+                 ixz="-0.00000014862"
+                 iyy= "0.00000221068"
+                 iyz="-0.00000014369"
+                 izz= "0.00000323175"/>
       </inertial>
     </link>
@@ -218,6 +242,12 @@
       <inertial>
         <origin rpy="0 0 0" xyz="0 0 0"/>
-        <mass value="0.047"/>
-        <inertia ixx="0.00000499332" ixy="0.00000091312" ixz="-0.00000000120" iyy  ="0.00006434531" iyz="-0.00000000007" izz="0.00006061917"/>
+        <!-- copied from proximal_actuating_hinge -->
+        <mass value="0.02647"/>
+        <inertia ixx= "0.00000156447"
+                 ixy= "0.000000236226"
+                 ixz="-0.00000014862"
+                 iyy= "0.00000221068"
+                 iyz="-0.00000014369"
+                 izz= "0.00000323175"/>
       </inertial>
     </link>
@@ -242,6 +272,12 @@
       <inertial>
         <origin rpy="0 0 0" xyz="0 0 0"/>
-        <mass value="0.047"/>
-        <inertia ixx="0.00000499332" ixy="0.00000091312" ixz="-0.00000000120" iyy  ="0.00006434531" iyz="-0.00000000007" izz="0.00006061917"/>
+        <!-- copied from proximal_actuating_hinge -->
+        <mass value="0.02647"/>
+        <inertia ixx= "0.00000156447"
+                 ixy= "0.000000236226"
+                 ixz="-0.00000014862"
+                 iyy= "0.00000221068"
+                 iyz="-0.00000014369"
+                 izz= "0.00000323175"/>
       </inertial>
     </link>
@@ -266,6 +302,12 @@
       <inertial>
         <origin rpy="0 0 0" xyz="0.01905 0 0"/>
-        <mass value="0.047"/>
-        <inertia ixx="0.00000499332" ixy="0.00000091312" ixz="-0.00000000120" iyy  ="0.00006434531" iyz="-0.00000000007" izz="0.00006061917"/>
+        <!-- copied from proximal_actuating_hinge -->
+        <mass value="0.02647"/>
+        <inertia ixx= "0.00000156447"
+                 ixy= "0.000000236226"
+                 ixz="-0.00000014862"
+                 iyy= "0.00000221068"
+                 iyz="-0.00000014369"
+                 izz= "0.00000323175"/>
       </inertial>
     </link>
@@ -290,6 +332,12 @@
       <inertial>
         <origin rpy="0 0 0" xyz="0 0 0"/>
-        <mass value="0.047"/>
-        <inertia ixx="0.00000499332" ixy="0.00000091312" ixz="-0.00000000120" iyy  ="0.00006434531" iyz="-0.00000000007" izz="0.00006061917"/>
+        <!-- copied from proximal_actuating_hinge -->
+        <mass value="0.02647"/>
+        <inertia ixx= "0.00000156447"
+                 ixy= "0.000000236226"
+                 ixz="-0.00000014862"
+                 iyy= "0.00000221068"
+                 iyz="-0.00000014369"
+                 izz= "0.00000323175"/>
       </inertial>
     </link>
@@ -314,6 +362,12 @@
       <inertial>
         <origin rpy="0 0 0" xyz="0 0 0"/>
-        <mass value="0.047"/>
-        <inertia ixx="0.00000499332" ixy="0.00000091312" ixz="-0.00000000120" iyy  ="0.00006434531" iyz="-0.00000000007" izz="0.00006061917"/>
+        <!-- copied from proximal_actuating_hinge -->
+        <mass value="0.02647"/>
+        <inertia ixx= "0.00000156447"
+                 ixy= "0.000000236226"
+                 ixz="-0.00000014862"
+                 iyy= "0.00000221068"
+                 iyz="-0.00000014369"
+                 izz= "0.00000323175"/>
       </inertial>
     </link>
@@ -338,6 +392,12 @@
       <inertial>
         <origin rpy="0 0 0" xyz="0 0 0"/>
-        <mass value="0.047"/>
-        <inertia ixx="0.00000499332" ixy="0.00000091312" ixz="-0.00000000120" iyy  ="0.00006434531" iyz="-0.00000000007" izz="0.00006061917"/>
+        <!-- copied from proximal_actuating_hinge -->
+        <mass value="0.02647"/>
+        <inertia ixx= "0.00000156447"
+                 ixy= "0.000000236226"
+                 ixz="-0.00000014862"
+                 iyy= "0.00000221068"
+                 iyz="-0.00000014369"
+                 izz= "0.00000323175"/>
       </inertial>
     </link>
@@ -491,7 +551,8 @@
     </gazebo>
     <!-- end of joint list -->
-    <!-- coupling joints in sdf
+    <!-- coupling joints in sdf -->
+    <!--
     <gazebo>
-      <joint name="${prefix}link_proximal_actuating_hinge_link_1" type="revolute">
+      <joint name="${prefix}link_proximal_actuating_hinge_link_1_couple" type="revolute">
         <parent>${prefix}link_proximal_actuating_hinge</parent>
         <child>${prefix}link_1</child>
@@ -506,10 +567,11 @@
       </joint>
     </gazebo>
-    <gazebo reference="${prefix}link_proximal_actuating_hinge_link_1">
+    <gazebo reference="${prefix}link_proximal_actuating_hinge_link_1_couple">
       <implicitSpringDamper>1</implicitSpringDamper>
     </gazebo>
     -->
+    <!--
     <gazebo>
-      <joint name="${prefix}link_proximal_actuating_bar_median_actuating_hinge" type="revolute">
+      <joint name="${prefix}link_proximal_actuating_bar_median_actuating_hinge_couple" type="revolute">
         <parent>${prefix}link_median_actuating_hinge</parent>
         <child>${prefix}link_proximal_actuating_bar</child>
@@ -525,9 +587,9 @@
       </joint>
     </gazebo>
-    <gazebo reference="${prefix}link_proximal_actuating_bar_median_actuating_hinge">
+    <gazebo reference="${prefix}link_proximal_actuating_bar_median_actuating_hinge_couple">
       <implicitSpringDamper>1</implicitSpringDamper>
     </gazebo>
     <gazebo>
-      <joint name="${prefix}link_median_bar_link_3" type="revolute">
+      <joint name="${prefix}link_median_bar_link_3_couple" type="revolute">
         <parent>${prefix}link_3</parent>
         <child>${prefix}link_median_bar</child>
@@ -543,10 +605,9 @@
       </joint>
     </gazebo>
-    <gazebo reference="${prefix}link_median_bar_paradistal_hinge">
-      <implicitSpringDamper>1</implicitSpringDamper>
-    </gazebo>
-    <!--
+    <gazebo reference="${prefix}link_median_bar_paradistal_hinge_couple">
+      <implicitSpringDamper>1</implicitSpringDamper>
+    </gazebo>
     <gazebo>
-      <joint name="${prefix}link_paraproximal_actuating_hinge_link_1" type="revolute">
+      <joint name="${prefix}link_paraproximal_actuating_hinge_link_1_couple" type="revolute">
         <parent>${prefix}link_paraproximal_actuating_hinge</parent>
         <child>${prefix}link_1</child>
@@ -561,9 +622,9 @@
       </joint>
     </gazebo>
-    <gazebo reference="${prefix}link_paraproximal_actuating_hinge_link_1">
+    <gazebo reference="${prefix}link_paraproximal_actuating_hinge_link_1_couple">
       <implicitSpringDamper>1</implicitSpringDamper>
     </gazebo>
     <gazebo>
-      <joint name="${prefix}link_paraproximal_bar_paramedian_hinge" type="revolute">
+      <joint name="${prefix}link_paraproximal_bar_paramedian_hinge_couple" type="revolute">
         <parent>${prefix}link_paraproximal_bar</parent>
         <child>${prefix}link_paramedian_hinge</child>
@@ -578,5 +639,5 @@
       </joint>
     </gazebo>
-    <gazebo reference="${prefix}link_paraproximal_bar_paramedian_hinge">
+    <gazebo reference="${prefix}link_paraproximal_bar_paramedian_hinge_couple">
       <implicitSpringDamper>1</implicitSpringDamper>
     </gazebo>

Commit message: Adjusting inertias.

File: robotiq_hand_description/urdf/robotiq_hand.urdf.xacro (robot description, xacro)
@@ -151,5 +151,5 @@
       </collision>
       <inertial>
-        <origin rpy="0 0 0" xyz="0.015 0 0"/>
+        <origin rpy="0 0 0" xyz="0.0012 -0.00162 -0.00161"/>
         <mass value="0.02647"/>
         <inertia ixx= "0.00000156447"
@@ -181,13 +181,13 @@
       </collision>
       <inertial>
-        <origin rpy="-0.015 0 0" xyz="0 0 0"/>
+        <origin rpy="-0.015 0 0" xyz="0.0064 0 0"/>
         <!-- copied from proximal_actuating_hinge -->
-        <mass value="0.02647"/>
-        <inertia ixx= "0.00000156447"
-                 ixy= "0.000000236226"
-                 ixz="-0.00000014862"
-                 iyy= "0.00000221068"
-                 iyz="-0.00000014369"
-                 izz= "0.00000323175"/>
+        <mass value="0.00362"/>
+        <inertia ixx= "0.00000012043"
+                 ixy= "0"
+                 ixz= "0"
+                 iyy= "0.00000053588"
+                 iyz= "0"
+                 izz= "0.00000065322"/>
       </inertial>
     </link>
@@ -211,13 +211,12 @@
       </collision>
       <inertial>
-        <origin rpy="0.5398 0 0" xyz="0.026789 0 0"/>
-        <!-- copied from proximal_actuating_hinge -->
-        <mass value="0.02647"/>
-        <inertia ixx= "0.00000156447"
-                 ixy= "0.000000236226"
-                 ixz="-0.00000014862"
-                 iyy= "0.00000221068"
-                 iyz="-0.00000014369"
-                 izz= "0.00000323175"/>
+        <origin rpy="0 0 0" xyz="0.02699 -0.00122 0"/>
+        <mass value="0.00659"/>
+        <inertia ixx= "0.00000008348"
+                 ixy="-0.0000002179"
+                 ixz= "0.00000000134"
+                 iyy= "0.00000719076"
+                 iyz= "0"
+                 izz= "0.00000718272"/>
       </inertial>
     </link>
@@ -241,13 +240,13 @@
       </collision>
       <inertial>
-        <origin rpy="0 0 0" xyz="0 0 0"/>
+        <origin rpy="0 0 0" xyz="0.02858 -0.00129 0"/>
         <!-- copied from proximal_actuating_hinge -->
-        <mass value="0.02647"/>
-        <inertia ixx= "0.00000156447"
-                 ixy= "0.000000236226"
-                 ixz="-0.00000014862"
-                 iyy= "0.00000221068"
-                 iyz="-0.00000014369"
-                 izz= "0.00000323175"/>
+        <mass value="0.00732"/>
+        <inertia ixx= "0.00000009065"
+                 ixy="-0.00000027047"
+                 ixz= "0.00000000142"
+                 iyy= "0.00000878034"
+                 iyz= "0"
+                 izz= "0.00000877558"/>
       </inertial>
     </link>
@@ -271,13 +270,12 @@
       </collision>
       <inertial>
-        <origin rpy="0 0 0" xyz="0 0 0"/>
-        <!-- copied from proximal_actuating_hinge -->
-        <mass value="0.02647"/>
-        <inertia ixx= "0.00000156447"
-                 ixy= "0.000000236226"
-                 ixz="-0.00000014862"
-                 iyy= "0.00000221068"
-                 iyz="-0.00000014369"
-                 izz= "0.00000323175"/>
+        <origin rpy="0 0 0" xyz="0.0092 0.00514 0"/>
+        <mass value="0.00359"/>
+        <inertia ixx= "0.00000024735"
+                 ixy= "0.00000023619"
+                 ixz= "0"
+                 iyy= "0.00000047681"
+                 iyz= "0"
+                 izz= "0.00000071813"/>
       </inertial>
     </link>
@@ -301,13 +299,12 @@
       </collision>
       <inertial>
-        <origin rpy="0 0 0" xyz="0.01905 0 0"/>
-        <!-- copied from proximal_actuating_hinge -->
-        <mass value="0.02647"/>
-        <inertia ixx= "0.00000156447"
-                 ixy= "0.000000236226"
-                 ixz="-0.00000014862"
-                 iyy= "0.00000221068"
-                 iyz="-0.00000014369"
-                 izz= "0.00000323175"/>
+        <origin rpy="0 0 0" xyz="0.01905 -0.00107 0"/>
+        <mass value="0.00538"/>
+        <inertia ixx= "0.00000006639"
+                 ixy="-0.00000010996"
+                 ixz= "0.00000000094"
+                 iyy= "0.00000305318"
+                 iyz= "0"
+                 izz= "0.00000304657"/>
       </inertial>
     </link>
@@ -331,13 +328,12 @@
       </collision>
       <inertial>
-        <origin rpy="0 0 0" xyz="0 0 0"/>
-        <!-- copied from proximal_actuating_hinge -->
-        <mass value="0.02647"/>
-        <inertia ixx= "0.00000156447"
-                 ixy= "0.000000236226"
-                 ixz="-0.00000014862"
-                 iyy= "0.00000221068"
-                 iyz="-0.00000014369"
-                 izz= "0.00000323175"/>
+        <origin rpy="0 0 0" xyz="-0.01025 0.00046 0"/>
+        <mass value="0.00276"/>
+        <inertia ixx= "0.00000004213"
+                 ixy="-0.00000001491"
+                 ixz= "0"
+                 iyy= "0.00000050258"
+                 iyz= "0"
+                 izz= "0.00000054007"/>
       </inertial>
     </link>
@@ -361,13 +357,12 @@
       </collision>
       <inertial>
-        <origin rpy="0 0 0" xyz="0 0 0"/>
-        <!-- copied from proximal_actuating_hinge -->
-        <mass value="0.02647"/>
-        <inertia ixx= "0.00000156447"
-                 ixy= "0.000000236226"
-                 ixz="-0.00000014862"
-                 iyy= "0.00000221068"
-                 iyz="-0.00000014369"
-                 izz= "0.00000323175"/>
+        <origin rpy="0 0 0" xyz="0.01905 -0.00107 0"/>
+        <mass value="0.00538"/>
+        <inertia ixx= "0.00000006639"
+                 ixy="-0.00000010996"
+                 ixz="-0.00000000094"
+                 iyy= "0.00000305318"
+                 iyz= "0"
+                 izz= "0.00000304657"/>
       </inertial>
     </link>
@@ -391,13 +386,12 @@
       </collision>
       <inertial>
-        <origin rpy="0 0 0" xyz="0 0 0"/>
-        <!-- copied from proximal_actuating_hinge -->
-        <mass value="0.02647"/>
-        <inertia ixx= "0.00000156447"
-                 ixy= "0.000000236226"
-                 ixz="-0.00000014862"
-                 iyy= "0.00000221068"
-                 iyz="-0.00000014369"
-                 izz= "0.00000323175"/>
+        <origin rpy="0 0 0" xyz="0.00548 0 0"/>
+        <mass value="0.00158"/>
+        <inertia ixx= "0.00000001907"
+                 ixy= "0"
+                 ixz= "0"
+                 iyy= "0.00000010970"
+                 iyz= "0"
+                 izz= "0.00000012610"/>
       </inertial>
     </link>

Commit message: Fix inertia.

File: robotiq_hand_description/urdf/robotiq_hand.urdf.xacro (robot description, xacro)
@@ -499,5 +499,6 @@
       <child link="${prefix}link_median_bar_underactuated"/>
       <axis xyz="0 0 1"/>
-      <origin rpy="0 0 0" xyz="0.01786 -0.011905 0"/>
+      <!-- \TODO: hand calc 90 deg + atan(0.01227/0.00329) -->
+      <origin rpy="0 0 ${3.1416/2 + 1.30882484}" xyz="0.01227 0.00329 0"/>
       <limit effort="100" lower="0" upper="3.1416" velocity="100"/>
     </joint>

Commit message: relaxing joint limits for coupling joints

File: robotiq_hand_description/urdf/robotiq_hand.urdf.xacro (robot description, xacro)
@@ -430,5 +430,6 @@
       <axis xyz="0 0 1"/>
       <origin rpy="0 0 1.8616" xyz="0.02858 0 0"/>
-      <limit effort="100" lower="0" upper="3.1416" velocity="100"/>
+      <!-- john changed lower from 0 to -3.1416 -->
+      <limit effort="100" lower="-3.1416" upper="3.1416" velocity="100"/>
     </joint>
     <gazebo reference="${prefix}joint_proximal_actuating_bar">
@@ -453,5 +454,6 @@
       <!-- \TODO: -0.37 is hand picked, double check -->
       <origin rpy="0 0 ${-0.37}" xyz="0 0.05715 0.01"/>
-      <limit effort="100" lower="0" upper="3.1416" velocity="100"/>
+      <!-- john changed lower from 0 to -3.1416 -->
+      <limit effort="100" lower="-3.1416" upper="3.1416" velocity="100"/>
     </joint>
     <gazebo reference="${prefix}joint_median_actuating_hinge">
@@ -593,5 +595,5 @@
         <axis>
           <dynamics>
-            <damping>1</damping>
+            <damping>0</damping>
             <friction>0</friction>
           </dynamics>
