Commit message: More improvements.

File: robotiq_hand_description/urdf/robotiq_hand.urdf.xacro (robot description, xacro)
@@ -139,13 +139,13 @@
     <link name="${prefix}link_proximal_actuating_hinge">
       <visual>
-        <origin rpy="0 0 0" xyz="0.015 0 0"/>
-        <geometry>
-          <box size="0.03 .0075 .002"/>
-        </geometry>
-      </visual>
-      <collision>
-        <origin rpy="0 0 0" xyz="0.015 0 0"/>
-         <geometry>
-          <box size="0.03 .0075 .002"/>
+        <origin rpy="0 0 0" xyz="0.01429 0 0"/>
+        <geometry>
+          <box size="0.02858 .0075 .002"/>
+        </geometry>
+      </visual>
+      <collision>
+        <origin rpy="0 0 0" xyz="0.01429 0 0"/>
+         <geometry>
+          <box size="0.02858 .0075 .002"/>
         </geometry>
       </collision>
@@ -169,17 +169,17 @@
     <link name="${prefix}link_paraproximal_actuating_hinge">
       <visual>
-        <origin rpy="-0.015 0 0" xyz="0 0 0"/>
-        <geometry>
-          <box size="0.03 .0075 .002"/>
-        </geometry>
-      </visual>
-      <collision>
-        <origin rpy="-0.015 0 0" xyz="0 0 0"/>
-         <geometry>
-          <box size="0.03 .0075 .002"/>
-        </geometry>
-      </collision>
-      <inertial>
-        <origin rpy="-0.015 0 0" xyz="0.0064 0 0"/>
+        <origin rpy="0 0 0" xyz="0.01143 0 0"/>
+        <geometry>
+          <box size="0.02286 .0075 .002"/>
+        </geometry>
+      </visual>
+      <collision>
+        <origin rpy="0 0 0" xyz="0.01143 0 0"/>
+         <geometry>
+          <box size="0.02286 .0075 .002"/>
+        </geometry>
+      </collision>
+      <inertial>
+        <origin rpy="0 0 0" xyz="0.0064 0 0"/>
         <!-- copied from proximal_actuating_hinge -->
         <mass value="0.00362"/>
@@ -228,13 +228,13 @@
     <link name="${prefix}link_paraproximal_bar">
       <visual>
-        <origin rpy="0 0 0" xyz="0 0 0"/>
-        <geometry>
-          <box size="0.05715 .0075 .002"/>
-        </geometry>
-      </visual>
-      <collision>
-        <origin rpy="0 0 0" xyz="0 0 0"/>
-         <geometry>
-          <box size="0.05715 .0075 .002"/>
+        <origin rpy="0 0 0" xyz="0.02885 0 0"/>
+        <geometry>
+          <box size="0.05770 .0075 .002"/>
+        </geometry>
+      </visual>
+      <collision>
+        <origin rpy="0 0 0" xyz="0.02885 0 0"/>
+         <geometry>
+          <box size="0.05770 .0075 .002"/>
         </geometry>
       </collision>
@@ -266,5 +266,5 @@
         <origin rpy="0 0 0" xyz="0 0 0"/>
          <geometry>
-          <box size=".02 0.2 0.002"/>
+          <box size=".02 .02 .002"/>
         </geometry>
       </collision>
@@ -324,5 +324,5 @@
         <origin rpy="0 0 0" xyz="0 0 0"/>
          <geometry>
-          <box size=".02 0.2 0.002"/>
+          <box size=".02 .02 .002"/>
         </geometry>
       </collision>
@@ -345,5 +345,5 @@
     <link name="${prefix}link_median_bar_underactuated">
       <visual>
-        <origin rpy="0 0 0" xyz="0 0 0"/>
+        <origin rpy="0 0 0" xyz="0.01905 0 0"/>
         <geometry>
           <box size="0.0381 .0075 .002"/>
@@ -351,5 +351,5 @@
       </visual>
       <collision>
-        <origin rpy="0 0 0" xyz="0 0 0"/>
+        <origin rpy="0 0 0" xyz="0.01905 0 0"/>
          <geometry>
           <box size="0.0381 .0075 .002"/>
@@ -382,5 +382,5 @@
         <origin rpy="0 0 0" xyz="0 0 0"/>
          <geometry>
-          <box size=".02 0.2 0.002"/>
+          <box size=".02 0.02 .002"/>
         </geometry>
       </collision>
@@ -418,5 +418,5 @@
       <child link="${prefix}link_paraproximal_actuating_hinge"/>
       <axis xyz="0 0 1"/>
-      <origin rpy="0 0 1.051" xyz="0 0 -0.01"/>
+      <origin rpy="0 0 -2.0906" xyz="0 0 -0.01"/>
       <limit effort="100" lower="0" upper="3.1416" velocity="100"/>
     </joint>
@@ -441,6 +441,7 @@
       <child link="${prefix}link_paraproximal_bar"/>
       <axis xyz="0 0 1"/>
-      <origin rpy="0 0 -1.57" xyz="-0.015 -0.029 0"/>
-      <limit effort="100" lower="0" upper="3.1416" velocity="100"/>
+      <origin rpy="0 0 1.57" xyz="0.02286 0 0"/>
+      <!-- caguero changed lower from 0 to -3.1416 -->
+      <limit effort="100" lower="-3.1416" upper="3.1416" velocity="100"/>
     </joint>
     <gazebo reference="${prefix}joint_paraproximal_bar">
@@ -466,7 +467,9 @@
       <axis xyz="0 0 1"/>
       <!-- \TODO: -0.37 is hand picked, 0.9719 is hand calculated from atan(0.02381/0.01625), double check -->
-      <origin rpy="0 0 ${-0.37+0.9719}" xyz="0 0.05715 -0.01"/>
-      <origin rpy="0 0 0.29" xyz="0.01625 0.02381 0"/>
-      <limit effort="100" lower="0" upper="3.1416" velocity="100"/>
+      <!--<origin rpy="0 0 ${-0.37+0.9719}" xyz="0 0.05715 -0.01"/>-->
+      <origin rpy="0 0 0" xyz="0 0.05715 -0.01"/>
+      <!--<origin rpy="0 0 0.29" xyz="0.01625 0.02381 0"/>-->
+      <!-- caguero changed lower from 0 to -3.1416 -->
+      <limit effort="100" lower="-3.1416" upper="3.1416" velocity="100"/>
     </joint>
     <gazebo reference="${prefix}joint_paramedian_hinge">
@@ -480,5 +483,6 @@
       <!-- \TODO: hand calc 90 deg + atan(0.01516/0.01625) -->
       <origin rpy="0 0 ${3.1416/2 + 0.7507}" xyz="0.01625 0.01516 0"/>
-      <limit effort="100" lower="0" upper="3.1416" velocity="100"/>
+      <!-- caguero changed lower from 0 to -3.1416 -->
+      <limit effort="100" lower="-3.1416" upper="3.1416" velocity="100"/>
     </joint>
     <gazebo reference="${prefix}joint_median_actuating_hinge_median_bar">
@@ -491,5 +495,6 @@
       <axis xyz="0 0 1"/>
       <origin rpy="0 0 0" xyz="0 0.039 -0.01"/>
-      <limit effort="100" lower="0" upper="3.1416" velocity="100"/>
+      <!-- caguero changed lower from 0 to -3.1416 -->
+      <limit effort="100" lower="-3.1416" upper="3.1416" velocity="100"/>
     </joint>
     <gazebo reference="${prefix}joint_paradistal_hinge">
@@ -502,6 +507,7 @@
       <axis xyz="0 0 1"/>
       <!-- \TODO: hand calc 90 deg + atan(0.01227/0.00329) -->
-      <origin rpy="0 0 ${3.1416/2 + 1.30882484}" xyz="0.01227 0.00329 0"/>
-      <limit effort="100" lower="0" upper="3.1416" velocity="100"/>
+      <origin rpy="0 0 ${3.1416/2}" xyz="0.01227 0.00329 0"/>
+      <!-- caguero changed lower from 0 to -3.1416 -->
+      <limit effort="100" lower="-3.1416" upper="3.1416" velocity="100"/>
     </joint>
     <gazebo reference="${prefix}joint_paramedian_hinge_median_bar_underactuated">
@@ -556,9 +562,9 @@
         <axis>
           <dynamics>
-            <damping>1</damping>
+            <damping>0</damping>
             <friction>0</friction>
           </dynamics>
           <xyz>0 0 1</xyz>
-          <use_parent_model_frame>true</use_parent_model_frame>
+          <use_parent_model_frame>false</use_parent_model_frame>
         </axis>
       </joint>
@@ -603,5 +609,23 @@
       </joint>
     </gazebo>
-    <gazebo reference="${prefix}link_median_bar_paradistal_hinge_couple">
+    <gazebo reference="${prefix}link_median_bar_link_3_couple">
+      <implicitSpringDamper>1</implicitSpringDamper>
+    </gazebo>
+    <gazebo>
+      <joint name="${prefix}link_paramedian_bar_paradistal_hinge_couple" type="revolute">
+        <parent>${prefix}link_paradistal_hinge</parent>
+        <child>${prefix}link_median_bar_underactuated</child>
+        <pose>0.0381 0 0 0 0 0</pose>
+        <axis>
+          <dynamics>
+            <damping>0</damping>
+            <friction>0</friction>
+          </dynamics>
+          <xyz>0 0 1</xyz>
+          <use_parent_model_frame>false</use_parent_model_frame>
+        </axis>
+      </joint>
+    </gazebo>
+    <gazebo reference="${prefix}link_median_bar_link_3_couple">
       <implicitSpringDamper>1</implicitSpringDamper>
     </gazebo>
@@ -613,9 +637,9 @@
         <axis>
           <dynamics>
-            <damping>1</damping>
+            <damping>0</damping>
             <friction>0</friction>
           </dynamics>
           <xyz>0 0 1</xyz>
-          <use_parent_model_frame>true</use_parent_model_frame>
+          <use_parent_model_frame>false</use_parent_model_frame>
         </axis>
       </joint>
@@ -623,16 +647,17 @@
     <gazebo reference="${prefix}link_paraproximal_actuating_hinge_link_1_couple">
       <implicitSpringDamper>1</implicitSpringDamper>
-    </gazebo>
+    </gazebo>-->
     <gazebo>
       <joint name="${prefix}link_paraproximal_bar_paramedian_hinge_couple" type="revolute">
-        <parent>${prefix}link_paraproximal_bar</parent>
-        <child>${prefix}link_paramedian_hinge</child>
+        <parent>${prefix}link_paramedian_hinge</parent>
+        <child>${prefix}link_paraproximal_bar</child>
+        <pose>0.05770 0 0 0 0 0</pose>
         <axis>
           <dynamics>
-            <damping>1</damping>
+            <damping>0</damping>
             <friction>0</friction>
           </dynamics>
           <xyz>0 0 1</xyz>
-          <use_parent_model_frame>true</use_parent_model_frame>
+          <use_parent_model_frame>false</use_parent_model_frame>
         </axis>
       </joint>

Commit message: Connecting paradistal with link3.

File: robotiq_hand_description/urdf/robotiq_hand.urdf.xacro (robot description, xacro)
@@ -161,5 +161,4 @@
       </inertial>
     </link>
-    <!-- Link 2 -->
     <gazebo reference="${prefix}link_proximal_actuating_hinge">
       <mu1>1.1</mu1>
@@ -408,5 +407,5 @@
       <axis xyz="0 0 1"/>
       <origin rpy="0 0 -2.0906" xyz="0 0 0.01"/>
-      <limit effort="100" lower="0" upper="3.1416" velocity="100"/>
+      <limit effort="100" lower="-3.1416" upper="3.1416" velocity="100"/>
     </joint>
     <gazebo reference="${prefix}joint_proximal_actuating_hinge">
@@ -419,5 +418,5 @@
       <axis xyz="0 0 1"/>
       <origin rpy="0 0 -2.0906" xyz="0 0 -0.01"/>
-      <limit effort="100" lower="0" upper="3.1416" velocity="100"/>
+      <limit effort="100" lower="-3.1416" upper="3.1416" velocity="100"/>
     </joint>
     <gazebo reference="${prefix}joint_paraproximal_actuating_hinge">
@@ -628,4 +627,22 @@
     </gazebo>
     <gazebo reference="${prefix}link_median_bar_link_3_couple">
+      <implicitSpringDamper>1</implicitSpringDamper>
+    </gazebo>
+    <gazebo>
+      <joint name="${prefix}link_paradistal_hinge_link_3_couple" type="revolute">
+        <parent>${prefix}link_paradistal_hinge</parent>
+        <child>${prefix}link_3</child>
+        <pose>0.0381 0 0 0 0 0</pose>
+        <axis>
+          <dynamics>
+            <damping>0</damping>
+            <friction>0</friction>
+          </dynamics>
+          <xyz>0 0 1</xyz>
+          <use_parent_model_frame>false</use_parent_model_frame>
+        </axis>
+      </joint>
+    </gazebo>
+    <gazebo reference="${prefix}link_paradistal_hinge_link_3_couple">
       <implicitSpringDamper>1</implicitSpringDamper>
     </gazebo>

Commit message: Removing commented code.

File: robotiq_hand_description/urdf/robotiq_hand.urdf.xacro (robot description, xacro)
@@ -58,5 +58,4 @@
       </collision>
       <inertial>
-        <!-- link_1 inertia visually incorrect, please double check values -->
         <origin rpy="0 0 ${3.1416/2}" xyz="0.00053 0.03218 0"/>
         <mass value="0.047"/>
@@ -90,5 +89,4 @@
       </collision>
       <inertial>
-        <!-- link_2 inertia visually incorrect, please double check values -->
         <origin rpy="0 0 ${3.1416/2}" xyz="0.00048 0.02167 0.00018"/>
         <mass value="0.03284"/>
@@ -240,5 +238,4 @@
       <inertial>
         <origin rpy="0 0 0" xyz="0.02858 -0.00129 0"/>
-        <!-- copied from proximal_actuating_hinge -->
         <mass value="0.00732"/>
         <inertia ixx= "0.00000009065"
@@ -429,5 +426,4 @@
       <axis xyz="0 0 1"/>
       <origin rpy="0 0 1.8616" xyz="0.02858 0 0"/>
-      <!-- john changed lower from 0 to -3.1416 -->
       <limit effort="100" lower="-3.1416" upper="3.1416" velocity="100"/>
     </joint>
@@ -441,5 +437,4 @@
       <axis xyz="0 0 1"/>
       <origin rpy="0 0 1.57" xyz="0.02286 0 0"/>
-      <!-- caguero changed lower from 0 to -3.1416 -->
       <limit effort="100" lower="-3.1416" upper="3.1416" velocity="100"/>
     </joint>
@@ -452,7 +447,5 @@
       <child link="${prefix}link_median_actuating_hinge"/>
       <axis xyz="0 0 1"/>
-      <!-- \TODO: -0.37 is hand picked, double check -->
       <origin rpy="0 0 ${-0.37}" xyz="0 0.05715 0.01"/>
-      <!-- john changed lower from 0 to -3.1416 -->
       <limit effort="100" lower="-3.1416" upper="3.1416" velocity="100"/>
     </joint>
@@ -465,9 +458,6 @@
       <child link="${prefix}link_paramedian_hinge"/>
       <axis xyz="0 0 1"/>
-      <!-- \TODO: -0.37 is hand picked, 0.9719 is hand calculated from atan(0.02381/0.01625), double check -->
-      <!--<origin rpy="0 0 ${-0.37+0.9719}" xyz="0 0.05715 -0.01"/>-->
+      <!-- -0.37 is hand picked, 0.9719 is hand calculated from atan(0.02381/0.01625) -->
       <origin rpy="0 0 0" xyz="0 0.05715 -0.01"/>
-      <!--<origin rpy="0 0 0.29" xyz="0.01625 0.02381 0"/>-->
-      <!-- caguero changed lower from 0 to -3.1416 -->
       <limit effort="100" lower="-3.1416" upper="3.1416" velocity="100"/>
     </joint>
@@ -480,7 +470,6 @@
       <child link="${prefix}link_median_bar"/>
       <axis xyz="0 0 1"/>
-      <!-- \TODO: hand calc 90 deg + atan(0.01516/0.01625) -->
+      <!-- hand calc 90 deg + atan(0.01516/0.01625) -->
       <origin rpy="0 0 ${3.1416/2 + 0.7507}" xyz="0.01625 0.01516 0"/>
-      <!-- caguero changed lower from 0 to -3.1416 -->
       <limit effort="100" lower="-3.1416" upper="3.1416" velocity="100"/>
     </joint>
@@ -494,5 +483,4 @@
       <axis xyz="0 0 1"/>
       <origin rpy="0 0 0" xyz="0 0.039 -0.01"/>
-      <!-- caguero changed lower from 0 to -3.1416 -->
       <limit effort="100" lower="-3.1416" upper="3.1416" velocity="100"/>
     </joint>
@@ -505,7 +493,6 @@
       <child link="${prefix}link_median_bar_underactuated"/>
       <axis xyz="0 0 1"/>
-      <!-- \TODO: hand calc 90 deg + atan(0.01227/0.00329) -->
+      <!-- hand calc 90 deg + atan(0.01227/0.00329) -->
       <origin rpy="0 0 ${3.1416/2}" xyz="0.01227 0.00329 0"/>
-      <!-- caguero changed lower from 0 to -3.1416 -->
       <limit effort="100" lower="-3.1416" upper="3.1416" velocity="100"/>
     </joint>
@@ -554,25 +541,4 @@
     <!-- end of joint list -->
     <!-- coupling joints in sdf -->
-    <!--
-    <gazebo>
-      <joint name="${prefix}link_proximal_actuating_hinge_link_1_couple" type="revolute">
-        <parent>${prefix}link_proximal_actuating_hinge</parent>
-        <child>${prefix}link_1</child>
-        <axis>
-          <dynamics>
-            <damping>0</damping>
-            <friction>0</friction>
-          </dynamics>
-          <xyz>0 0 1</xyz>
-          <use_parent_model_frame>false</use_parent_model_frame>
-        </axis>
-      </joint>
-    </gazebo>
-    <gazebo reference="${prefix}link_proximal_actuating_hinge_link_1_couple">
-      <implicitSpringDamper>1</implicitSpringDamper>
-    </gazebo>
-    -->
-    <!--
-    -->
     <gazebo>
       <joint name="${prefix}link_proximal_actuating_bar_median_actuating_hinge_couple" type="revolute">
@@ -647,22 +613,4 @@
       <implicitSpringDamper>1</implicitSpringDamper>
     </gazebo>
-    <!--
-    <gazebo>
-      <joint name="${prefix}link_paraproximal_actuating_hinge_link_1_couple" type="revolute">
-        <parent>${prefix}link_paraproximal_actuating_hinge</parent>
-        <child>${prefix}link_1</child>
-        <axis>
-          <dynamics>
-            <damping>0</damping>
-            <friction>0</friction>
-          </dynamics>
-          <xyz>0 0 1</xyz>
-          <use_parent_model_frame>false</use_parent_model_frame>
-        </axis>
-      </joint>
-    </gazebo>
-    <gazebo reference="${prefix}link_paraproximal_actuating_hinge_link_1_couple">
-      <implicitSpringDamper>1</implicitSpringDamper>
-    </gazebo>-->
     <gazebo>
       <joint name="${prefix}link_paraproximal_bar_paramedian_hinge_couple" type="revolute">
